File: node_pcb/iso_3v3_supply.sch (KiCad schematic (older format))
At the start: 42 parts

Commit message: Resolved stock issues for 3v3 supply components
Parts:
- added Cout2: 180 uF 11 mOhm, symbol Device:CP1
- added Csnub?: 15 nF 1 mOhm, symbol Device:C
- C12: renamed from C?; value C -> 100 nF 64 mOhm
- C13: renamed from C?; value C -> 1 nF
- C21: renamed from C?; value C -> 6.8uF 2 mOhm
- C22: renamed from C?; value C -> 22 pF
- C23: renamed from C?; value C -> 100 nF
- Ccs: renamed from C?; value C -> 470 pF
- Cin: renamed from C?; value C -> 10 uF 1 mOhm
- Cout1: renamed from C?; value CP1 -> 180 uF 11 mOhm
- Cref: renamed from C?; value C -> 100 nF 1 mOhm
- Csnub1: renamed from C?; value C -> 15 nF 1 mOhm
- Ct: renamed from C?; value C -> 1 nF 25 mOhm
- Cvcc: renamed from C?; value CP1 -> 15 uF
- D21: renamed from D?; value D_Schottky -> 470 mV 500 mA
- Daux: renamed from D?; value D_Schottky -> 750 mV 3A
- Dsec, Dsec2: renamed from D?; value D_Schottky -> 750 mV 5 A
- Dsnub: renamed from D?; value D_Schottky -> 800 mV 2 A
- M1: renamed from ?; value CSD19538Q2 -> BSC160N10NS3GATMA1; footprint DQK0006C -> (none); symbol CSD19538Q2:CSD19538Q2 -> Transistor_FET:BSC160N10NS3G
- Qsc: renamed from Q?; value Q_NPN_BCE -> PMBT2222A
- R11, R21, Rt: renamed from R?; value R -> 10k
- R12: renamed from R?; value R -> 2.74k
- R13: renamed from R?; value R -> 4.99k
- R22, Rcs: renamed from R?; value R -> 1k
- Raux: renamed from R?; value R -> 10 Ohm
- Rbias: renamed from R?; value R -> 21k
- Rdrv: renamed from R?; value R -> 12 Ohm
- Rfbb: renamed from R?; value R -> 1.33k
- Rfbt: renamed from R?; value R -> 2.21k
- Rled: renamed from R?; value R -> 1.27k
- Rsc: renamed from R?; value R -> 4.64k
- Rsns: renamed from R?; value R -> 750 mOhm
- Rsnub1, Rsnub2: renamed from R?; value R -> 8.2k
- Rstartup1, Rstartup2: renamed from R?; value R -> 33k
- U?: value TCMT1109 -> TLP385(BLL,E; footprint Package_SO:SOP-4_4.4x2.6mm_P1.27mm -> (none)
- gave numbers to parts that had none: 1
Connections:
- wire segments 148 -> 156
Other:
- moved on the sheet: ?, C12, C13, C21, C22, C23, Ccs, Cin, Cout1, Cref, Csnub1, Ct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

Commit message: Added Yassine's CAN interface schematic
Annotated all components
Added an isolated SPI interface to connect to Jetson/PSU
Updated flash memory's symbol to a custom one
Added ADC inputs as appropriate and broke out DAC/extra GPIOs
Found a cheaper digital isolator series in stock so substituted it in
Parts:
- VR1: renamed from ?; footprint MF05A -> node_pcb:LMV431CM5
- gave numbers to parts that had none: 3
- renumbered Ccs to Ccs1, Cin to Cin1, Cref to Cref1, Ct to Ct1, Cvcc to Cvcc1, Daux to Daux1, Dsec to Dsec1, Dsnub to Dsnub1, Qsc to Qsc1, Raux to Raux1, Rbias to Rbias1, Rcs to Rcs1, Rdrv to Rdrv1, Rfbb to Rfbb1, Rfbt to Rfbt1, Rled to Rled1, Rsc to Rsc1, Rsns to Rsns1, Rt to Rt1
Changed lines of the file:
@@
 $Descr A4 11693 8268
 encoding utf-8
-Sheet 7 7
+Sheet 6 10
 Title ""
 Date ""
 Rev ""
-Comp ""
-Comment1 ""
+Comp "EPFL Xplore"
+Comment1 "Authors: Yassine Bakkali, Paolo Celati"
 Comment2 ""
 Comment3 ""
@@
 $EndDescr
 $Comp
-L avionics_library:UCC2813-3D U?
+L avionics_library:UCC2813-3D U5
 U 1 1 61906C07
 P 3400 2950
-F 0 "U?" H 3400 3415 50  0000 C CNN
+F 0 "U5" H 3400 3415 50  0000 C CNN
 F 1 "UCC2813-3D" H 3400 3324 50  0000 C CNN
 F 2 "" H 3050 2950 50  0001 C CNN
@@
 $EndComp
 $Comp
-L Device:R Rsc
+L Device:R Rsc1
 U 1 1 619079BE
 P 1650 3700
-F 0 "Rsc" H 1720 3746 50  0000 L CNN
+F 0 "Rsc1" H 1720 3746 50  0000 L CNN
 F 1 "4.64k" H 1720 3655 50  0000 L CNN
 F 2 "" V 1580 3700 50  0001 C CNN
@@
 $EndComp
 $Comp
-L Device:R Rt
+L Device:R Rt1
 U 1 1 61907AF0
 P 700 4050
-F 0 "Rt" H 770 4096 50  0000 L CNN
+F 0 "Rt1" H 770 4096 50  0000 L CNN
 F 1 "10k" H 770 4005 50  0000 L CNN
 F 2 "" V 630 4050 50  0001 C CNN
@@
 $EndComp
 $Comp
-L Device:R Raux
+L Device:R Raux1
 U 1 1 619081DA
 P 5550 2100
-F 0 "Raux" V 5343 2100 50  0000 C CNN
+F 0 "Raux1" V 5343 2100 50  0000 C CNN
 F 1 "10 Ohm" V 5434 2100 50  0000 C CNN
 F 2 "" V 5480 2100 50  0001 C CNN
@@
 $EndComp
 $Comp
-L Device:R Rdrv
+L Device:R Rdrv1
 U 1 1 6190838B
 P 5450 2950
-F 0 "Rdrv" V 5243 2950 50  0000 C CNN
+F 0 "Rdrv1" V 5243 2950 50  0000 C CNN
 F 1 "12 Ohm" V 5334 2950 50  0000 C CNN
 F 2 "" V 5380 2950 50  0001 C CNN
@@
 $EndComp
 $Comp
-L Device:R Rcs
+L Device:R Rcs1
 U 1 1 6190854C
 P 5150 3950
-F 0 "Rcs" V 4943 3950 50  0000 C CNN
+F 0 "Rcs1" V 4943 3950 50  0000 C CNN
 F 1 "1k" V 5034 3950 50  0000 C CNN
 F 2 "" V 5080 3950 50  0001 C CNN
@@
 $EndComp
 $Comp
-L Device:R Rsns
+L Device:R Rsns1
 U 1 1 61908728
 P 6250 3750
-F 0 "Rsns" H 6320 3796 50  0000 L CNN
+F 0 "Rsns1" H 6320 3796 50  0000 L CNN
 F 1 "750 mOhm" H 6320 3705 50  0000 L CNN
 F 2 "" V 6180 3750 50  0001 C CNN
@@
 $EndComp
 $Comp
-L Device:R Rled
+L Device:R Rled1
 U 1 1 61908CBD
 P 8000 4100
-F 0 "Rled" H 8070 4146 50  0000 L CNN
+F 0 "Rled1" H 8070 4146 50  0000 L CNN
 F 1 "1.27k" H 8070 4055 50  0000 L CNN
 F 2 "" V 7930 4100 50  0001 C CNN
@@
 $EndComp
 $Comp
-L Device:R Rbias
+L Device:R Rbias1
 U 1 1 61908EAF
 P 8350 4100
-F 0 "Rbias" H 8420 4146 50  0000 L CNN
+F 0 "Rbias1" H 8420 4146 50  0000 L CNN
 F 1 "21k" H 8420 4055 50  0000 L CNN
 F 2 "" V 8280 4100 50  0001 C CNN
@@
 $EndComp
 $Comp
-L Device:R Rfbb
+L Device:R Rfbb1
 U 1 1 61909533
 P 10750 5800
-F 0 "Rfbb" H 10820 5846 50  0000 L CNN
+F 0 "Rfbb1" H 10820 5846 50  0000 L CNN
 F 1 "1.33k" H 10820 5755 50  0000 L CNN
 F 2 "" V 10680 5800 50  0001 C CNN
@@
 $EndComp
 $Comp
-L Device:R Rfbt
+L Device:R Rfbt1
 U 1 1 61909765
 P 10750 2500
-F 0 "Rfbt" H 10820 2546 50  0000 L CNN
+F 0 "Rfbt1" H 10820 2546 50  0000 L CNN
 F 1 "2.21k" H 10820 2455 50  0000 L CNN
 F 2 "" V 10680 2500 50  0001 C CNN
@@
 $EndComp
 $Comp
-L Device:C Cin
+L Device:C Cin1
 U 1 1 6190A41B
 P 2550 1100
-F 0 "Cin" V 2298 1100 50  0000 C CNN
+F 0 "Cin1" V 2298 1100 50  0000 C CNN
 F 1 "10 uF 1 mOhm" V 2389 1100 50  0000 C CNN
 F 2 "" H 2588 950 50  0001 C CNN
@@
 $EndComp
 $Comp
-L Device:C Cref
+L Device:C Cref1
 U 1 1 6190A98B
 P 2000 2150
-F 0 "Cref" V 1748 2150 50  0000 C CNN
+F 0 "Cref1" V 1748 2150 50  0000 C CNN
 F 1 "100 nF 1 mOhm" V 1839 2150 50  0000 C CNN
 F 2 "" H 2038 2000 50  0001 C CNN
@@
 $EndComp
 $Comp
-L Device:C Ct
+L Device:C Ct1
 U 1 1 6190B866
 P 1050 3200
-F 0 "Ct" V 798 3200 50  0000 C CNN
+F 0 "Ct1" V 798 3200 50  0000 C CNN
 F 1 "1 nF 25 mOhm" V 889 3200 50  0000 C CNN
 F 2 "" H 1088 3050 50  0001 C CNN
@@
 $EndComp
 $Comp
-L Device:D_Schottky Dsnub
+L Device:D_Schottky Dsnub1
 U 1 1 6190DD82
 P 6050 1350
-F 0 "Dsnub" H 6050 1567 50  0000 C CNN
+F 0 "Dsnub1" H 6050 1567 50  0000 C CNN
 F 1 "800 mV 2 A" H 6050 1476 50  0000 C CNN
 F 2 "" H 6050 1350 50  0001 C CNN
@@
 $EndComp
 $Comp
-L Device:D_Schottky Daux
+L Device:D_Schottky Daux1
 U 1 1 6190E0A4
 P 6000 2100
-F 0 "Daux" H 6000 2317 50  0000 C CNN
+F 0 "Daux1" H 6000 2317 50  0000 C CNN
 F 1 "750 mV 3A" H 6000 2226 50  0000 C CNN
 F 2 "" H 6000 2100 50  0001 C CNN
@@
 $EndComp
 $Comp
-L Device:D_Schottky Dsec
+L Device:D_Schottky Dsec1
 U 1 1 6190E443
 P 8050 1200
-F 0 "Dsec" H 8050 983 50  0000 C CNN
+F 0 "Dsec1" H 8050 983 50  0000 C CNN
 F 1 "750 mV 5 A" H 8050 1074 50  0000 C CNN
 F 2 "" H 8050 1200 50  0001 C CNN
@@
 $EndComp
 $Comp
-L Device:CP1 Cvcc
+L Device:CP1 Cvcc1
 U 1 1 6190F978
 P 5050 2400
-F 0 "Cvcc" H 5165 2446 50  0000 L CNN
+F 0 "Cvcc1" H 5165 2446 50  0000 L CNN
 F 1 "15 uF" H 5165 2355 50  0000 L CNN
 F 2 "" H 5050 2400 50  0001 C CNN
@@
 	4150 3950 4150 4050
 $Comp
-L Device:C Ccs
+L Device:C Ccs1
 U 1 1 619344F6
 P 4150 4200
-F 0 "Ccs" V 3898 4200 50  0000 C CNN
+F 0 "Ccs1" V 3898 4200 50  0000 C CNN
 F 1 "470 pF" V 3989 4200 50  0000 C CNN
 F 2 "" H 4188 4050 50  0001 C CNN
@@
 $EndComp
 $Comp
-L Isolator:TCMT1109 U?
+L Isolator:TCMT1109 U6
 U 1 1 61A68873
 P 7150 5150
-F 0 "U?" H 7150 4833 50  0000 C CNN
+F 0 "U6" H 7150 4833 50  0000 C CNN
 F 1 "TLP385(BLL,E" H 7150 4924 50  0000 C CNN
 F 2 "" H 7150 4850 50  0001 C CNN
@@
 	700  5050 6850 5050
 $Comp
-L lmv431:LMV431CM5 ?
+L lmv431:LMV431CM5 VR1
 U 1 1 61910CB8
 P 9120 5850
-F 0 "?" H 9115 5403 60  0000 C CNN
+F 0 "VR1" H 9115 5403 60  0000 C CNN
 F 1 "LMV431CM5" H 9115 5509 60  0000 C CNN
-F 2 "MF05A" H 9120 6160 60  0001 C CNN
+F 2 "node_pcb:LMV431CM5" H 9120 6160 60  0001 C CNN
 F 3 "" H 8640 6040 60  0000 C CNN
 	1    9120 5850
@@
 	1650 3550 1650 3400
 $Comp
-L Device:Q_NPN_BCE Qsc
+L Device:Q_NPN_BCE Qsc1
 U 1 1 619E0F0F
 P 1550 3200
-F 0 "Qsc" H 1741 3246 50  0000 L CNN
+F 0 "Qsc1" H 1741 3246 50  0000 L CNN
 F 1 "PMBT2222A" H 1741 3155 50  0000 L CNN
 F 2 "" H 1750 3300 50  0001 C CNN
@@
 	3150 2100 3150 1750
 $Comp
-L Device:C Csnub?
+L Device:C Csnub2
 U 1 1 61988D3A
 P 5700 1000
-F 0 "Csnub?" V 5448 1000 50  0000 C CNN
+F 0 "Csnub2" V 5448 1000 50  0000 C CNN
 F 1 "15 nF 1 mOhm" V 5539 1000 50  0000 C CNN
 F 2 "" H 5738 850 50  0001 C CNN

Commit message: Added test pads+LEDs to generic node and assigned footprints
Changed from 4 independent RJ45s to 1 ganged 4 port for USART
Parts:
- C12, C13, C21, C22, Ccs1, Cref1, Csnub1, Csnub2, Ct1: footprint (none) -> Capacitor_SMD:C_0805_2012Metric_Pad1.18x1.45mm_HandSolder
- C23: footprint (none) -> Capacitor_SMD:C_1206_3216Metric_Pad1.33x1.80mm_HandSolder
- Cin1: footprint (none) -> Capacitor_SMD:C_1210_3225Metric_Pad1.33x2.70mm_HandSolder
- Cout1, Cout2: footprint (none) -> Capacitor_SMD:CP_Elec_6.3x9.9
- Cvcc1: footprint (none) -> Capacitor_SMD:CP_Elec_4x5.8
- D21: footprint (none) -> Diode_SMD:D_SOD-323_HandSoldering
- Daux1, Dsnub1: footprint (none) -> Diode_SMD:D_SMA_Handsoldering
- Dsec1, Dsec2: footprint (none) -> Diode_SMD:D_SMC_Handsoldering
- M1: footprint (none) -> Package_TO_SOT_SMD:TDSON-8-1
- Qsc1: footprint (none) -> Package_TO_SOT_SMD:SOT-23_Handsoldering
- R11, R12, R13, R21, R22, Raux1, Rbias1, Rcs1, Rdrv1, Rfbb1, Rfbt1, Rled1, Rsc1, Rsns1, Rt1: footprint (none) -> Resistor_SMD:R_0805_2012Metric_Pad1.20x1.40mm_HandSolder
- Rsnub1, Rsnub2: footprint (none) -> Resistor_THT:R_Axial_DIN0207_L6.3mm_D2.5mm_P5.08mm_Vertical
- Rstartup1, Rstartup2: footprint (none) -> Resistor_SMD:R_1206_3216Metric_Pad1.30x1.75mm_HandSolder
- T1: footprint (none) -> B65808E1508T001:TDK-B65808E1508T001-MFG
- U5: value UCC2813-3D -> UCC2813-3PW; footprint (none) -> Package_SO:TSSOP-8_4.4x3mm_P0.65mm
- U6: footprint (none) -> Package_SO:SO-4_7.6x3.6mm_P2.54mm

Commit message: Replaced values and names of components. Finished assigning all footprints.
Parts:
- T1: footprint B65808E1508T001:TDK-B65808E1508T001-MFG -> node_pcb:PTS647SM50SMTR2LFS
Changed lines of the file:
@@
 Connection ~ 1300 2850
 $Comp
-L power:GND #PWR?
+L power:GND #PWR0128
 U 1 1 619BEB18
 P 8500 2100
-F 0 "#PWR?" H 8500 1850 50  0001 C CNN
+F 0 "#PWR0128" H 8500 1850 50  0001 C CNN
 F 1 "GND" H 8505 1927 50  0000 C CNN
 F 2 "" H 8500 2100 50  0001 C CNN
@@
 $EndComp
 $Comp
-L power:GND #PWR?
+L power:GND #PWR0129
 U 1 1 619BF807
 P 10750 6250
-F 0 "#PWR?" H 10750 6000 50  0001 C CNN
+F 0 "#PWR0129" H 10750 6000 50  0001 C CNN
 F 1 "GND" H 10755 6077 50  0000 C CNN
 F 2 "" H 10750 6250 50  0001 C CNN
@@
 $EndComp
 $Comp
-L power:GND #PWR?
+L power:GND #PWR0130
 U 1 1 619C2A14
 P 9500 4400
-F 0 "#PWR?" H 9500 4150 50  0001 C CNN
+F 0 "#PWR0130" H 9500 4150 50  0001 C CNN
 F 1 "GND" H 9505 4227 50  0000 C CNN
 F 2 "" H 9500 4400 50  0001 C CNN
@@
 	6500 1500 6500 1650
 $Comp
-L power:GND #PWR?
+L power:GND #PWR0131
 U 1 1 61A66DCF
 P 7350 1750
-F 0 "#PWR?" H 7350 1500 50  0001 C CNN
+F 0 "#PWR0131" H 7350 1500 50  0001 C CNN
 F 1 "GND" H 7355 1577 50  0000 C CNN
 F 2 "" H 7350 1750 50  0001 C CNN
@@
 Connection ~ 6250 3500
 $Comp
-L power:-BATT #PWR?
+L power:-BATT #PWR0132
 U 1 1 6196684A
 P 2550 1500
-F 0 "#PWR?" H 2550 1350 50  0001 C CNN
+F 0 "#PWR0132" H 2550 1350 50  0001 C CNN
 F 1 "-BATT" H 2565 1673 50  0000 C CNN
 F 2 "" H 2550 1500 50  0001 C CNN
@@
 $EndComp
 $Comp
-L power:-BATT #PWR?
+L power:-BATT #PWR0133
 U 1 1 6199DF10
 P 4600 2550
-F 0 "#PWR?" H 4600 2400 50  0001 C CNN
+F 0 "#PWR0133" H 4600 2400 50  0001 C CNN
 F 1 "-BATT" H 4615 2723 50  0000 C CNN
 F 2 "" H 4600 2550 50  0001 C CNN
@@
 $EndComp
 $Comp
-L power:-BATT #PWR?
+L power:-BATT #PWR0134
 U 1 1 619A2DE0
 P 5050 2550
-F 0 "#PWR?" H 5050 2400 50  0001 C CNN
+F 0 "#PWR0134" H 5050 2400 50  0001 C CNN
 F 1 "-BATT" H 5065 2723 50  0000 C CNN
 F 2 "" H 5050 2550 50  0001 C CNN
@@
 $EndComp
 $Comp
-L power:-BATT #PWR?
+L power:-BATT #PWR0135
 U 1 1 619A810C
 P 6500 1650
-F 0 "#PWR?" H 6500 1500 50  0001 C CNN
+F 0 "#PWR0135" H 6500 1500 50  0001 C CNN
 F 1 "-BATT" H 6515 1823 50  0000 C CNN
 F 2 "" H 6500 1650 50  0001 C CNN
@@
 $EndComp
 $Comp
-L power:-BATT #PWR?
+L power:-BATT #PWR0136
 U 1 1 619AD6C0
 P 4150 3350
-F 0 "#PWR?" H 4150 3200 50  0001 C CNN
+F 0 "#PWR0136" H 4150 3200 50  0001 C CNN
 F 1 "-BATT" H 4165 3523 50  0000 C CNN
 F 2 "" H 4150 3350 50  0001 C CNN
@@
 $EndComp
 $Comp
-L power:-BATT #PWR?
+L power:-BATT #PWR0137
 U 1 1 619B23AE
 P 4150 4500
-F 0 "#PWR?" H 4150 4350 50  0001 C CNN
+F 0 "#PWR0137" H 4150 4350 50  0001 C CNN
 F 1 "-BATT" H 4165 4673 50  0000 C CNN
 F 2 "" H 4150 4500 50  0001 C CNN
@@
 $EndComp
 $Comp
-L power:-BATT #PWR?
+L power:-BATT #PWR0138
 U 1 1 619B7021
 P 6250 4250
-F 0 "#PWR?" H 6250 4100 50  0001 C CNN
+F 0 "#PWR0138" H 6250 4100 50  0001 C CNN
 F 1 "-BATT" H 6265 4423 50  0000 C CNN
 F 2 "" H 6250 4250 50  0001 C CNN
@@
 $EndComp
 $Comp
-L power:-BATT #PWR?
+L power:-BATT #PWR0139
 U 1 1 619BBEEE
 P 6600 6100
-F 0 "#PWR?" H 6600 5950 50  0001 C CNN
+F 0 "#PWR0139" H 6600 5950 50  0001 C CNN
 F 1 "-BATT" H 6615 6273 50  0000 C CNN
 F 2 "" H 6600 6100 50  0001 C CNN
@@
 	4300 5500 6600 5500
 $Comp
-L power:-BATT #PWR?
+L power:-BATT #PWR0140
 U 1 1 619C6CCE
 P 2000 2450
-F 0 "#PWR?" H 2000 2300 50  0001 C CNN
+F 0 "#PWR0140" H 2000 2300 50  0001 C CNN
 F 1 "-BATT" H 2015 2623 50  0000 C CNN
 F 2 "" H 2000 2450 50  0001 C CNN
@@
 $EndComp
 $Comp
-L power:-BATT #PWR?
+L power:-BATT #PWR0141
 U 1 1 619D045D
 P 1050 3500
-F 0 "#PWR?" H 1050 3350 50  0001 C CNN
+F 0 "#PWR0141" H 1050 3350 50  0001 C CNN
 F 1 "-BATT" H 1065 3673 50  0000 C CNN
 F 2 "" H 1050 3500 50  0001 C CNN
@@
 F 0 "T1" H 6950 2081 50  0000 C CNN
 F 1 "B65807J0000R049 + B65808E1508T001" H 6950 1990 50  0000 C CNN
-F 2 "B65808E1508T001:TDK-B65808E1508T001-MFG" H 6950 1400 50  0001 C CNN
+F 2 "node_pcb:PTS647SM50SMTR2LFS" H 6950 1400 50  0001 C CNN
 F 3 "https://product.tdk.com/system/files/dam/doc/product/ferrite/ferrite/ferrite-acc/data_sheet/80/db/fer/rm_6.pdf" H 7250 1400 50  0001 C CNN
 	1    6950 1400
@@
 -BATT
 $Comp
-L power:-BATT #PWR?
+L power:-BATT #PWR0142
 U 1 1 61916689
 P 1800 6250
-F 0 "#PWR?" H 1800 6100 50  0001 C CNN
+F 0 "#PWR0142" H 1800 6100 50  0001 C CNN
 F 1 "-BATT" H 1815 6423 50  0000 C CNN
 F 2 "" H 1800 6250 50  0001 C CNN
@@
 	5700 1350 5900 1350
 $Comp
-L power:GND #PWR?
+L power:GND #PWR0143
 U 1 1 619424EA
 P 9400 2100
-F 0 "#PWR?" H 9400 1850 50  0001 C CNN
+F 0 "#PWR0143" H 9400 1850 50  0001 C CNN
 F 1 "GND" H 9405 1927 50  0000 C CNN
 F 2 "" H 9400 2100 50  0001 C CNN
