File: node_pcb/uart_iso_with_bypass.kicad_sch (KiCad schematic)
At the start: 8 parts, among them U3 MAX14850AEE+

Commit message: Finalised R3 node PCB iteration, and cleaned up Kicad v5.1.7 files.
Parts:
- C7, C8: value 100 nF -> (none); footprint Capacitor_SMD:C_0603_1608Metric -> (none)
- C9: value 2.2 uF -> (none); footprint Capacitor_SMD:C_0603_1608Metric -> (none)
- R18, R19, R20, R21: value 0 -> (none); footprint Resistor_SMD:R_0603_1608Metric -> (none)
- U3: value MAX14850AEE+ -> (none); footprint Package_SO:QSOP-16_3.9x4.9mm_P0.635mm -> (none)
Changed lines of the file:
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@@
     (in_bom yes) (on_board yes) (fields_autoplaced)
     (property "Reference" "R21" (id 0) (at 158.1912 71.1032 90))
-    (property "Value" "0" (id 1) (at 158.1912 73.6401 90))
-    (property "Footprint" "Resistor_SMD:R_0603_1608Metric" (id 2) (at 158.1912 75.5396 0)
+    (property "Value" "" (id 1) (at 158.1912 73.6401 90))
+    (property "Footprint" "" (id 2) (at 158.1912 75.5396 0)
       (effects (font (size 1.27 1.27)) hide)
     )
@@
     (in_bom yes) (on_board yes) (fields_autoplaced)
     (property "Reference" "R19" (id 0) (at 158.0896 65.566 90))
-    (property "Value" "0" (id 1) (at 158.0896 68.1029 90))
-    (property "Footprint" "Resistor_SMD:R_0603_1608Metric" (id 2) (at 158.0896 70.0024 0)
+    (property "Value" "" (id 1) (at 158.0896 68.1029 90))
+    (property "Footprint" "" (id 2) (at 158.0896 70.0024 0)
       (effects (font (size 1.27 1.27)) hide)
     )
@@
       (effects (font (size 1.27 1.27)) (justify left))
     )
-    (property "Value" "100 nF" (id 1) (at 196.1769 94.0629 0)
+    (property "Value" "" (id 1) (at 196.1769 94.0629 0)
       (effects (font (size 1.27 1.27)) (justify left))
     )
-    (property "Footprint" "Capacitor_SMD:C_0603_1608Metric" (id 2) (at 193.8528 92.3544 0)
+    (property "Footprint" "" (id 2) (at 193.8528 92.3544 0)
       (effects (font (size 1.27 1.27)) hide)
     )
@@
       (effects (font (size 1.27 1.27)) (justify left))
     )
-    (property "Value" "2.2 uF" (id 1) (at 201.2569 93.4533 0)
+    (property "Value" "" (id 1) (at 201.2569 93.4533 0)
       (effects (font (size 1.27 1.27)) (justify left))
     )
-    (property "Footprint" "Capacitor_SMD:C_0603_1608Metric" (id 2) (at 198.9328 91.7448 0)
+    (property "Footprint" "" (id 2) (at 198.9328 91.7448 0)
       (effects (font (size 1.27 1.27)) hide)
     )
@@
     (in_bom yes) (on_board yes) (fields_autoplaced)
     (property "Reference" "R18" (id 0) (at 158.0896 60.486 90))
-    (property "Value" "0" (id 1) (at 158.0896 63.0229 90))
-    (property "Footprint" "Resistor_SMD:R_0603_1608Metric" (id 2) (at 158.0896 64.9224 0)
+    (property "Value" "" (id 1) (at 158.0896 63.0229 90))
+    (property "Footprint" "" (id 2) (at 158.0896 64.9224 0)
       (effects (font (size 1.27 1.27)) hide)
     )
@@
     (in_bom yes) (on_board yes) (fields_autoplaced)
     (property "Reference" "R20" (id 0) (at 158.1912 55.3044 90))
-    (property "Value" "0" (id 1) (at 158.1912 57.8413 90))
-    (property "Footprint" "Resistor_SMD:R_0603_1608Metric" (id 2) (at 158.1912 59.7408 0)
+    (property "Value" "" (id 1) (at 158.1912 57.8413 90))
+    (property "Footprint" "" (id 2) (at 158.1912 59.7408 0)
       (effects (font (size 1.27 1.27)) hide)
     )
@@
     (in_bom yes) (on_board yes) (fields_autoplaced)
     (property "Reference" "U3" (id 0) (at 158.9024 80.1964 0))
-    (property "Value" "MAX14850AEE+" (id 1) (at 172.2374 77.4192 0))
-    (property "Footprint" "Package_SO:QSOP-16_3.9x4.9mm_P0.635mm" (id 2) (at 158.9024 92.6592 0)
+    (property "Value" "" (id 1) (at 172.2374 77.4192 0))
+    (property "Footprint" "" (id 2) (at 158.9024 92.6592 0)
       (effects (font (size 1.27 1.27)) hide)
     )
@@
       (effects (font (size 1.27 1.27)) (justify left))
     )
-    (property "Value" "100 nF" (id 1) (at 121.2977 93.4025 0)
+    (property "Value" "" (id 1) (at 121.2977 93.4025 0)
       (effects (font (size 1.27 1.27)) (justify left))
     )
-    (property "Footprint" "Capacitor_SMD:C_0603_1608Metric" (id 2) (at 118.9736 91.694 0)
+    (property "Footprint" "" (id 2) (at 118.9736 91.694 0)
       (effects (font (size 1.27 1.27)) hide)
     )
