File: node_pcb/node_pcb.kicad_sch (KiCad schematic)
At the start: 59 parts, among them J1 Screw_Terminal_01x02, J10 CLP-102-02-L-D-BE, J11 CLP-102-02-L-D-BE, J12 CLP-102-02-L-D-BE, J13 CLP-106-02-F-D-BE-A-K-TR, J14 CLP-102-02-L-D-BE, J15 Conn_01x06_Female, J16 Conn_01x06_Female, J17 Conn_01x06_Female, J18 Conn_01x06_Female, J19 Conn_01x04_Female, J2 CLP-102-02-L-D-BE, J22 Conn_01x04_Male, J23 Conn_01x04_Male, J3 CLP-102-02-L-D-BE, J4 CLP-102-02-L-D-BE, J5 CLP-102-02-L-D-BE, J6 CLP-102-02-L-D-BE, J7 CLP-106-02-F-D-BE-A-K-TR, J8 CLP-106-02-F-D-BE-A-K-TR, J9 CLP-106-02-F-D-BE-A-K-TR

Commit message: Finalised R3 node PCB iteration, and cleaned up Kicad v5.1.7 files.
Parts:
- removed J10, J11: CLP-102-02-L-D-BE, node_pcb:SAMTEC-CLP-102-02-X-D-BE, symbol Connector_Generic:Conn_02x02_Odd_Even
- added J10: Conn_01x04_Female, Connector_PinSocket_2.54mm:PinSocket_1x04_P2.54mm_Vertical, symbol Connector:Conn_01x04_Female
- D3, D4: value LED -> (none); footprint LED_SMD:LED_1206_3216Metric_Pad1.42x1.75mm_HandSolder -> (none)
- F1: value 3A -> (none); footprint Fuse:Fuse_0805_2012Metric_Pad1.15x1.40mm_HandSolder -> (none)
- H1, H2, H3, H4, H5, H6, H7, H8, H9: value MountingHole -> (none); footprint MountingHole:MountingHole_2.2mm_M2 -> (none)
- J1: value Screw_Terminal_01x02 -> (none); footprint TerminalBlock:TerminalBlock_Altech_AK300-2_P5.00mm -> (none)
- J12, J14, J2, J3, J4, J5, J6: value CLP-102-02-L-D-BE -> (none); footprint node_pcb:SAMTEC-CLP-102-02-X-D-BE -> (none)
- J13, J7, J8, J9: value CLP-106-02-F-D-BE-A-K-TR -> (none); footprint node_pcb:SAMTEC-CLP-106-02-X-D-BE -> (none)
- J15, J16, J17, J18: value Conn_01x06_Female -> (none); footprint Connector_Molex:Molex_PicoBlade_53047-0610_1x06_P1.25mm_Vertical -> (none)
- J19: value Conn_01x04_Female -> (none); footprint Connector_PinSocket_2.54mm:PinSocket_1x04_P2.54mm_Vertical -> (none)
- J22, J23: value Conn_01x04_Male -> (none); footprint Connector_Molex:Molex_PicoBlade_53047-0410_1x04_P1.25mm_Vertical -> (none)
- R6, R7: value 768 -> (none); footprint Resistor_SMD:R_0805_2012Metric_Pad1.20x1.40mm_HandSolder -> (none)
- TP1, TP10, TP11, TP12, TP13, TP14, TP15, TP16, TP17, TP18, TP19, TP2, TP20, TP21, TP22, TP23, TP24, TP3, TP4, TP5, TP6, TP7, TP8, TP9: value TestPoint -> (none); footprint TestPoint:TestPoint_Pad_D2.5mm -> (none)
Connections:
- net +3V3: now also J10.1 (Pin_1), J10.2 (Pin_2)
- net GND: now also J10.3 (Pin_3), J10.4 (Pin_4)
- no-connect marks 16 -> 14
Other:
- added sheet H_Bridge (H_Bridge.kicad_sch)

Commit message: Had forgotten ADCs need to be switched away from CLP-102s
Parts:
- removed J2, J3, J4, J5, J6: (no value), symbol Connector_Generic:Conn_02x02_Odd_Even
- added J2, J3, J4, J5, J6: Conn_01x04_Male, Connector_Molex:Molex_PicoBlade_53047-0410_1x04_P1.25mm_Vertical, symbol Connector:Conn_01x04_Male
Connections:
- net +3V3: now also J2.2 (Pin_2), J3.2 (Pin_2), J4.2 (Pin_2), J5.2 (Pin_2), J6.2 (Pin_2)
- net ADC_2: now also J4.4 (Pin_4)
- net ADC_3: now also J5.4 (Pin_4)
- net ADC_4: now also J6.4 (Pin_4)
- net ADC_DIFF_0_N: now also J2.4 (Pin_4)
- net ADC_DIFF_0_P: now also J2.3 (Pin_3)
- net ADC_DIFF_1_N: now also J3.4 (Pin_4)
- net ADC_DIFF_1_P: now also J3.3 (Pin_3)
- net GND: now also J2.1 (Pin_1), J3.1 (Pin_1), J4.1 (Pin_1), J5.1 (Pin_1), J6.1 (Pin_1)
