File: breakout_modules/ISOLATED_PWM/ISOLATED_PWM.kicad_pcb (KiCad board)
At the start: 2 copper layers, 29.2 x 24.8 mm, 15 parts, among them J1 01x03 2.54mm Pin headers, J2 Barrel_Jack, J3 SM04B-GHS-TB(LF)(SN), J4 01x03 2.54mm Pin headers, J5 01x03 2.54mm Pin headers, U1 TLP2710(TP4,E, U2 TLP2710(TP4,E

Commit message: Replaced barrel jacks with terminal blocks
Parts:
- removed  : , graphics:xplore_logo_10mm
- J2: value Barrel_Jack -> TB001-500-02BE; footprint Connector_BarrelJack:BarrelJack_CUI_PJ-102AH_Horizontal -> 0_lib_fp:TB001-500-02BE
- moved J2 9.41 mm to (136.0, 79.0)
Routing:
- net VDD: track 62.5 -> 58.6 mm
Other:
- board text added: "Isolated PWM VDD max: 5V"
- board text added: "ROV_5V"
- board text added: "ROV_GND"
- board text removed: "Isolated PWM Power supply: 5V"
