File: breakout_modules/ISOLATED_PWM/ISOLATED_PWM.kicad_sch (KiCad schematic)
At the start: 13 parts, among them J1 TB001-500-02BE, J3 SM04B-GHS-TB(LF)(SN), J4 01x07 2.54mm Pin headers, U1 TLP2710(TP4,E, U2 SI3402-TP

Commit message: Updated isolated PWM and isolated LED with barrel jack, fixed 2x2 to JST adapter board
Parts:
- removed H2: 2.2mm M2, MountingHole:MountingHole_2.2mm_M2_Pad, symbol Mechanical:MountingHole_Pad
- removed J1: TB001-500-02BE, 0_lib_fp:TB001-500-02BE, symbol Connector_Generic:Conn_01x02
- removed R3: 10k, Resistor_SMD:R_0805_2012Metric, symbol Device:R
- removed R4: 4.7k, Resistor_SMD:R_0805_2012Metric, symbol Device:R
- removed U2: SI3402-TP, Package_TO_SOT_SMD:SOT-23, symbol 0_Led_Switch:SI3402-TP
- added C2: 0.1uF, Capacitor_SMD:C_0805_2012Metric, symbol Device:C
- added H2, H3: 2.2mm M2, MountingHole:MountingHole_2.2mm_M2_Pad_Via, symbol Mechanical:MountingHole
- added J1, J5: 01x03 2.54mm Pin headers, Connector_PinHeader_2.54mm:PinHeader_1x03_P2.54mm_Vertical, symbol Connector_Generic:Conn_01x03
- added U2: TLP2710(TP4,E, 0_lib_fp:SO6L(LF4), symbol 0_ISOLATED_PWM:TLP2710(TP4,E
- H1: value 2.2mm M2 -> (none); footprint MountingHole:MountingHole_2.2mm_M2_Pad -> (none); symbol Mechanical:MountingHole_Pad -> Mechanical:MountingHole; now in the parts list
- J2: value (none) -> Barrel_Jack; footprint (none) -> Connector_BarrelJack:BarrelJack_CUI_PJ-102AH_Horizontal
- J4: value 01x07 2.54mm Pin headers -> 01x03 2.54mm Pin headers; footprint Connector_PinHeader_2.54mm:PinHeader_1x07_P2.54mm_Vertical -> Connector_PinHeader_2.54mm:PinHeader_1x03_P2.54mm_Vertical; symbol Connector_Generic:Conn_01x07 -> Connector_Generic:Conn_01x03; now in the parts list
- R1: value 10k -> 680; Manufacturer ref WCR0805-10KFI -> CRCW0805680RFKEAC; Mouser ref 756-WCR0805-10KFI -> 71-CRCW0805680RFKEAC
- U1: symbol 0_Led_Switch:TLP2710(TP4,E -> 0_ISOLATED_PWM:TLP2710(TP4,E
Connections:
- net GND: now also J4.1 (Pin_1), C2.2, J1.1 (Pin_1), U2.4 (GND); no longer H1.1, J4.2 (Pin_2)
- net MCU_GND: now also U1.3 (K), J5.1 (Pin_1), U2.3 (K); no longer J4.7 (Pin_7), R1.2
- net VDD: now also J4.2 (Pin_2), C2.1, J1.2 (Pin_2), U2.6 (VDD); no longer J4.1 (Pin_1), J4.3 (Pin_3)
- net PWM_ISO1: now reaches U1.5 (VO)
- net PWM_ISO1: now also J4.3 (Pin_3)
- net at R2.2: now also U1.1 (A); no longer U1.3 (K)
- net PWM_IN2: now reaches J3.1 (Pin_1)
- net PWM_IN2: now also R1.1, J5.3 (Pin_3)
- net GPIO renamed PWM_IN1
- net PWM_IN1: now also J5.2 (Pin_2); no longer J4.5 (Pin_5), R1.1
- removed net LED_CATHODE-: J4.4 (Pin_4)
- removed net MCU_3V3: J3.3 (Pin_3), J4.6 (Pin_6), U1.1 (A)
- new net: R1.2, U2.1 (A)
- new net PWM_ISO2: J1.3 (Pin_3), U2.5 (VO)
Other:
- note added: "Isolated PWM circuit"
- note added: "Optional 2.54mm pin headers"
- note added: "PWM 2.54mm pin headers"
- note added: "Vf_max = 1.9V If_th_max = 1.0 mA, we choose 2.0 mA V_MCU = 3.3V R = (3.3V-1.9V)/(2mA) = 700 ohms -> 680 ohms"
- note removed: "2.54mm pin headers"
- note removed: "LED strip Terminal block"
- note removed: "Optocoupler + Switch circuit"
- note removed: "Vf_max = 1.9V If_th_max = 1.0 mA, we choose 2.0 mA V_MCU = 3.3V R = (3.3V-1.9V)/(2mA) = 700 ohms -> 680 ohms Pulldown resistor might be optional, to test"
- title: Isolated LED Switch -> Isolated PWM 
- moved on the sheet: C1, J2, J3, R2, U1
Changed lines of the file:
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@@
   (paper "A4")
   (title_block
-    (title "Isolated LED Switch")
+    (title "Isolated PWM ")
+    (date "2022-05-01")
     (rev "2")
     (comment 1 "Power supply: 5V")

Commit message: Replaced barrel jacks with terminal blocks
Parts:
- removed J2: Barrel_Jack, Connector_BarrelJack:BarrelJack_CUI_PJ-102AH_Horizontal, symbol Connector:Barrel_Jack
- added J2: (no value), symbol Connector_Generic:Conn_01x02
- H1: value (none) -> 2.2mm M2; footprint (none) -> MountingHole:MountingHole_2.2mm_M2_Pad_Via
Connections:
- net GND: now also J2.2 (Pin_2)
- net VDD: now also J2.1 (Pin_1)

Commit message: Changed connectors from jst to molex
Parts:
- J2: value (none) -> TB001-500-02BE; footprint (none) -> 0_lib_fp:TB001-500-02BE
- J3: value SM04B-GHS-TB(LF)(SN) -> Molex 0532610471; footprint Connector_JST:JST_GH_SM04B-GHS-TB_1x04-1MP_P1.25mm_Horizontal -> Connector_Molex:Molex_PicoBlade_53261-0471_1x04-1MP_P1.25mm_Horizontal; Comments I think we already have enough stock -> (none); Digikey ref (none) -> WM7622TR-ND; Manufacturer ref (none) -> 0532610471

Commit message: Updated bom
Parts:
- H1, H2, H3: now left out of the parts list

Commit message: Updated bom
Parts:
- J1, J4, J5: now left out of the parts list
