File: adapter_boards/JETSON_INTERFACE_BOARD/JETSON_INTERFACE_BOARD.kicad_pcb (KiCad board)
At the start: 2 copper layers, 23.2 x 52.2 mm, 22 parts, among them J1 Conn_02x20_Odd_Even, J2 Terminal block 01x04, J3 Terminal block 01x05, J4 Terminal block 01x05, U1 SN65HVD232QDR, U2 SN65HVD232QDR

Commit message: Updated references
Parts:
- renumbered C7 to C10, C10 to C3, C12 to C4, C4 to C5, C3 to C6, C8 to C7, C11 to C8, J2 to J1, J3 to J2, J1 to J3, R4 to R1, R3 to R2, R1 to R3, R2 to R4, U2 to U1, U1 to U2
