File: breakout_modules/ADS1113/ADS1113.kicad_sch (KiCad schematic)
At the start: 17 parts, among them J1 TB001-500-02BE, J2 01x07 2.54mm Pin headers, J3 SM04B-GHS-TB(LF)(SN), U1 ADS1113BQDGSRQ1, U2 SMDA03C-4

Commit message: Changed connectors from jst to molex
Parts:
- J3: value SM04B-GHS-TB(LF)(SN) -> (none); footprint Connector_JST:JST_GH_SM04B-GHS-TB_1x04-1MP_P1.25mm_Horizontal -> (none); Comments I think we already have enough stock -> (none); Digikey ref (none) -> WM7622TR-ND; Manufacturer ref (none) -> 0532610471
Changed lines of the file:
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@@
       (effects (font (size 1.27 1.27)) (justify left))
     )
-    (property "Value" "SM04B-GHS-TB(LF)(SN)" (id 1) (at 257.175 89.535 0)
-      (effects (font (size 1.27 1.27)) (justify left))
-    )
-    (property "Footprint" "Connector_JST:JST_GH_SM04B-GHS-TB_1x04-1MP_P1.25mm_Horizontal" (id 2) (at 264.795 79.375 0)
-      (effects (font (size 1.27 1.27)) hide)
-    )
-    (property "Datasheet" "https://www.jst-mfg.com/product/pdf/eng/eGH.pdf" (id 3) (at 264.795 79.375 0)
-      (effects (font (size 1.27 1.27)) hide)
-    )
-    (property "Comments" "I think we already have enough stock" (id 4) (at 264.795 79.375 0)
+    (property "Value" "" (id 1) (at 257.175 89.535 0)
+      (effects (font (size 1.27 1.27)) (justify left))
+    )
+    (property "Footprint" "" (id 2) (at 264.795 79.375 0)
+      (effects (font (size 1.27 1.27)) hide)
+    )
+    (property "Datasheet" "https://www.molex.com/pdm_docs/sd/532610471_sd.pdf" (id 3) (at 264.795 79.375 0)
+      (effects (font (size 1.27 1.27)) hide)
+    )
+    (property "Digikey ref" "WM7622TR-ND" (id 4) (at 264.795 79.375 0)
+      (effects (font (size 1.27 1.27)) hide)
+    )
+    (property "Manufacturer ref" "0532610471" (id 5) (at 264.795 79.375 0)
       (effects (font (size 1.27 1.27)) hide)
     )
@@
     )
     (path "/7b04a873-e176-4092-860a-283aca17f8c1"
-      (reference "J3") (unit 1) (value "SM04B-GHS-TB(LF)(SN)") (footprint "Connector_JST:JST_GH_SM04B-GHS-TB_1x04-1MP_P1.25mm_Horizontal")
+      (reference "J3") (unit 1) (value "Molex 0532610471") (footprint "Connector_Molex:Molex_PicoBlade_53261-0471_1x04-1MP_P1.25mm_Horizontal")
     )
     (path "/2db3c459-1a55-4c59-ba78-36ca3ca31430"

Commit message: Updated bom
Parts:
- J3: value (none) -> Molex 0532610471; footprint (none) -> Connector_Molex:Molex_PicoBlade_53261-0471_1x04-1MP_P1.25mm_Horizontal
Changed lines of the file:
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@@
       (effects (font (size 1.27 1.27)) (justify left))
     )
-    (property "Value" "" (id 1) (at 257.175 89.535 0)
+    (property "Value" "Molex 0532610471" (id 1) (at 257.175 89.535 0)
       (effects (font (size 1.27 1.27)) (justify left))
     )
-    (property "Footprint" "" (id 2) (at 264.795 79.375 0)
+    (property "Footprint" "Connector_Molex:Molex_PicoBlade_53261-0471_1x04-1MP_P1.25mm_Horizontal" (id 2) (at 264.795 79.375 0)
       (effects (font (size 1.27 1.27)) hide)
     )

Commit message: Added offset to voltage divider for reverse polarity
Parts:
- removed R1: 26.7k, Resistor_SMD:R_0805_2012Metric, symbol Device:R_Small
- removed R2: 3.3k, Resistor_SMD:R_0805_2012Metric, symbol Device:R_Small
- added JP1: CONN_TO_VDD, Jumper:SolderJumper-2_P1.3mm_Open_RoundedPad1.0x1.5mm, symbol Jumper:Jumper_2_Open
- added JP2: CONN_TO_GND, Jumper:SolderJumper-2_P1.3mm_Open_RoundedPad1.0x1.5mm, symbol Jumper:Jumper_2_Open
- added R1: 100k, Resistor_SMD:R_0603_1608Metric_Pad0.98x0.95mm_HandSolder, symbol Device:R
- added R2: 11k, Resistor_SMD:R_0603_1608Metric_Pad0.98x0.95mm_HandSolder, symbol Device:R
- added R6: 12.4k, Resistor_SMD:R_0603_1608Metric_Pad0.98x0.95mm_HandSolder, symbol Device:R
- C1, C2: footprint Capacitor_SMD:C_0805_2012Metric -> Capacitor_SMD:C_0603_1608Metric_Pad1.08x0.95mm_HandSolder; Comments We already have some stock -> (none); Manufacturer ref CL21B104KACNNNC -> (none); Mouser ref 187-CL21B104KACNNNC -> (none); Package 0805 (2012 metric) -> (none)
- R3, R4, R5: footprint Resistor_SMD:R_0805_2012Metric -> Resistor_SMD:R_0603_1608Metric_Pad0.98x0.95mm_HandSolder; Manufacturer ref WCR0805-10KFI -> (none); Mouser ref 756-WCR0805-10KFI -> (none); Package 0805 (2012 metric) -> (none)
Connections:
- net GND: now also JP2.2 (B); no longer C3.2, J1.2 (Pin_2), J2.7 (Pin_7), U1.5 (AIN1)
- net VDD: now also JP1.1 (A), R2.2
- net VIN+: now also R1.1
- net VO: now reaches C3.1, U1.4 (AIN0), U2.1
- net VO: now also JP1.2 (B), R1.2, R2.1, R6.2
- new net VIN-: C3.2, J1.2 (Pin_2), J2.7 (Pin_7), JP2.1 (A), R6.1, U1.5 (AIN1)
Other:
- note added: "VDD = 3.3V When VIN+ = 30 V, we want VO = VDD (VIN+ - VO)/R1 = (VO - VIN-)/R6 = VO/R6 -> (30 - 3.3)/R1 = 3.3/R6 When VIN- = -30 V, we want VO = 0 = VIN- -VIN+/R1 = VDD/R2 -> 30/R1 = 3.3/R2 We choose R1 = 100k, which gives us R2 = 3.3/(30/R1) = 11 kOhm R6 = 3.3/(26.7/R1) = 12.36 kOhm Closest 1% resistors R6 = 12.4 kOhm R2 = 11 kOhm R1 = 100 kOhm"
- note removed: "We want to measure voltages between 1-24 VDC with unknown polarity. For this application, we choose VMAX = 30V AIN0/AIN1 must be less than VDD + 0.3V = 3.6V It is then needed to divide input voltage by at least ratio_max = 30/3.3V = 9.09 = (R1+R2)/R1 R1*(9.09 - 1) = 8.09R1 = R2 Pd_max = VMAX^2/(R1+R2) R2 = 3.3k R1 = 26.7k ratio = 9.09 Pd = 30^2/(30k) = 30mW"
- moved on the sheet: C1, C3, U1, U2

Commit message: Corrected comment
Other:
- note added: "VDD = 3.3V When VIN+ = 30 V, we want VO = VDD (VIN+ - VO)/R1 = (VO - VIN-)/R6 = VO/R6 -> (30 - 3.3)/R1 = 3.3/R6 When VIN+ = -30 V, we want VO = 0 = VIN- -VIN+/R1 = VDD/R2 -> 30/R1 = 3.3/R2 We choose R1 = 100k, which gives us R2 = 3.3/(30/R1) = 11 kOhm R6 = 3.3/(26.7/R1) = 12.36 kOhm Closest 1% resistors R6 = 12.4 kOhm R2 = 11 kOhm R1 = 100 kOhm"
- note removed: "VDD = 3.3V When VIN+ = 30 V, we want VO = VDD (VIN+ - VO)/R1 = (VO - VIN-)/R6 = VO/R6 -> (30 - 3.3)/R1 = 3.3/R6 When VIN- = -30 V, we want VO = 0 = VIN- -VIN+/R1 = VDD/R2 -> 30/R1 = 3.3/R2 We choose R1 = 100k, which gives us R2 = 3.3/(30/R1) = 11 kOhm R6 = 3.3/(26.7/R1) = 12.36 kOhm Closest 1% resistors R6 = 12.4 kOhm R2 = 11 kOhm R1 = 100 kOhm"
Changed lines of the file:
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@@
     (stroke (width 0) (type default) (color 0 0 0 0))
   )
-  (text "VDD = 3.3V\nWhen VIN+ = 30 V, we want VO = VDD\n(VIN+ - VO)/R1 = (VO - VIN-)/R6 = VO/R6\n-> (30 - 3.3)/R1 = 3.3/R6\n\nWhen VIN- = -30 V, we want VO = 0 = VIN-\n-VIN+/R1 = VDD/R2 \n-> 30/R1 = 3.3/R2\n\nWe choose R1 = 100k, which gives us\nR2 = 3.3/(30/R1) = 11 kOhm\nR6 = 3.3/(26.7/R1) = 12.36 kOhm\nClosest 1% resistors\nR6 = 12.4 kOhm\nR2 = 11 kOhm\nR1 = 100 kOhm"
+  (text "VDD = 3.3V\nWhen VIN+ = 30 V, we want VO = VDD\n(VIN+ - VO)/R1 = (VO - VIN-)/R6 = VO/R6\n-> (30 - 3.3)/R1 = 3.3/R6\n\nWhen VIN+ = -30 V, we want VO = 0 = VIN-\n-VIN+/R1 = VDD/R2 \n-> 30/R1 = 3.3/R2\n\nWe choose R1 = 100k, which gives us\nR2 = 3.3/(30/R1) = 11 kOhm\nR6 = 3.3/(26.7/R1) = 12.36 kOhm\nClosest 1% resistors\nR6 = 12.4 kOhm\nR2 = 11 kOhm\nR1 = 100 kOhm"
     (at 22.86 125.73 0)
     (effects (font (size 1.27 1.27)) (justify left bottom))
