File: adapter_boards/LIMIT_SWITCHES/LIMIT_SWITCHES.kicad_pcb (KiCad board)
At the start: 2 copper layers, 19 x 23.2 mm, 3 parts, among them J1 Conn_01x06_Female, J2 Conn_02x06_Odd_Even

Commit message: Added 2x6 1.27mm pin header to JST PH with holes, fixed pinout of limit switch board
Connections:
- J2 pad 1: GND -> unconnected-(J2-Pad1)
- J2 pad 11: unconnected-(J2-Pad11) -> +3.3V
- J2 pad 12: +3.3V -> unconnected-(J2-Pad12)
- J2 pad 2: unconnected-(J2-Pad2) -> GND
Routing:
- net GND: track 7.32 -> 9.24 mm
- net +3.3V: track 9.00 -> 7.32 mm
Other:
- board text added: "3.3V"
- board text added: "GND"
- board text added: "SW1"
- board text added: "SW2"
- board text added: "SW3"
- board text added: "SW4"
Changed lines of the file:
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@@
   (net 5 "/GPIO3")
   (net 6 "GND")
-  (net 7 "unconnected-(J2-Pad2)")
-  (net 8 "unconnected-(J2-Pad4)")
-  (net 9 "unconnected-(J2-Pad6)")
-  (net 10 "unconnected-(J2-Pad8)")
-  (net 11 "unconnected-(J2-Pad10)")
-  (net 12 "unconnected-(J2-Pad11)")
+  (net 7 "unconnected-(J2-Pad4)")
+  (net 8 "unconnected-(J2-Pad6)")
+  (net 9 "unconnected-(J2-Pad8)")
+  (net 10 "unconnected-(J2-Pad10)")
+  (net 11 "unconnected-(J2-Pad1)")
+  (net 12 "unconnected-(J2-Pad12)")
   (footprint "MountingHole:MountingHole_2.2mm_M2" (layer "F.Cu")
     (at 121.9 134.5)
@@
     (property "Sheetname" "")
     (attr exclude_from_pos_files)
-    (fp_text reference "H1" (at 0 -3.2) (layer "F.SilkS")
+    (fp_text reference "H1" (at 0 -3.2) (layer "F.SilkS") hide
       (effects (font (size 1 1) (thickness 0.15)))
     )
@@
     (property "Sheetname" "")
     (attr through_hole)
-    (fp_text reference "J2" (at 0.635 -1.695 90) (layer "F.SilkS")
+    (fp_text reference "J2" (at 0.635 -1.695 90) (layer "F.SilkS") hide
       (effects (font (size 1 1) (thickness 0.15)))
     )
@@
     (fp_line (start -1.07 6.985) (end -1.07 0.2175) (layer "F.Fab") (width 0.1))
     (pad "1" thru_hole rect (at 0 0 90) (size 1 1) (drill 0.65) (layers *.Cu *.Mask)
-      (net 6 "GND") (pinfunction "Pin_1") (pintype "passive"))
+      (net 11 "unconnected-(J2-Pad1)") (pinfunction "Pin_1") (pintype "passive+no_connect"))
     (pad "2" thru_hole oval (at 1.27 0 90) (size 1 1) (drill 0.65) (layers *.Cu *.Mask)
-      (net 7 "unconnected-(J2-Pad2)") (pinfunction "Pin_2") (pintype "passive+no_connect"))
+      (net 6 "GND") (pinfunction "Pin_2") (pintype "passive"))
     (pad "3" thru_hole oval (at 0 1.27 90) (size 1 1) (drill 0.65) (layers *.Cu *.Mask)
       (net 5 "/GPIO3") (pinfunction "Pin_3") (pintype "passive"))
     (pad "4" thru_hole oval (at 1.27 1.27 90) (size 1 1) (drill 0.65) (layers *.Cu *.Mask)
-      (net 8 "unconnected-(J2-Pad4)") (pinfunction "Pin_4") (pintype "passive+no_connect"))
+      (net 7 "unconnected-(J2-Pad4)") (pinfunction "Pin_4") (pintype "passive+no_connect"))
     (pad "5" thru_hole oval (at 0 2.54 90) (size 1 1) (drill 0.65) (layers *.Cu *.Mask)
       (net 4 "/GPIO5") (pinfunction "Pin_5") (pintype "passive"))
     (pad "6" thru_hole oval (at 1.27 2.54 90) (size 1 1) (drill 0.65) (layers *.Cu *.Mask)
-      (net 9 "unconnected-(J2-Pad6)") (pinfunction "Pin_6") (pintype "passive+no_connect"))
+      (net 8 "unconnected-(J2-Pad6)") (pinfunction "Pin_6") (pintype "passive+no_connect"))
     (pad "7" thru_hole oval (at 0 3.81 90) (size 1 1) (drill 0.65) (layers *.Cu *.Mask)
       (net 3 "/GPIO7") (pinfunction "Pin_7") (pintype "passive"))
     (pad "8" thru_hole oval (at 1.27 3.81 90) (size 1 1) (drill 0.65) (layers *.Cu *.Mask)
-      (net 10 "unconnected-(J2-Pad8)") (pinfunction "Pin_8") (pintype "passive+no_connect"))
+      (net 9 "unconnected-(J2-Pad8)") (pinfunction "Pin_8") (pintype "passive+no_connect"))
     (pad "9" thru_hole oval (at 0 5.08 90) (size 1 1) (drill 0.65) (layers *.Cu *.Mask)
       (net 2 "/GPIO9") (pinfunction "Pin_9") (pintype "passive"))
     (pad "10" thru_hole oval (at 1.27 5.08 90) (size 1 1) (drill 0.65) (layers *.Cu *.Mask)
-      (net 11 "unconnected-(J2-Pad10)") (pinfunction "Pin_10") (pintype "passive+no_connect"))
+      (net 10 "unconnected-(J2-Pad10)") (pinfunction "Pin_10") (pintype "passive+no_connect"))
     (pad "11" thru_hole oval (at 0 6.35 90) (size 1 1) (drill 0.65) (layers *.Cu *.Mask)
-      (net 12 "unconnected-(J2-Pad11)") (pinfunction "Pin_11") (pintype "passive+no_connect"))
+      (net 1 "+3.3V") (pinfunction "Pin_11") (pintype "passive"))
     (pad "12" thru_hole oval (at 1.27 6.35 90) (size 1 1) (drill 0.65) (layers *.Cu *.Mask)
-      (net 1 "+3.3V") (pinfunction "Pin_12") (pintype "passive"))
+      (net 12 "unconnected-(J2-Pad12)") (pinfunction "Pin_12") (pintype "passive+no_connect"))
     (model "${KICAD6_3DMODEL_DIR}/Connector_PinHeader_1.27mm.3dshapes/PinHeader_2x06_P1.27mm_Vertical.wrl"
       (offset (xyz 0 0 0))
@@
     (property "Sheetname" "")
     (attr through_hole)
-    (fp_text reference "J1" (at -0.685 0.3 180 unlocked) (layer "F.SilkS")
+    (fp_text reference "J1" (at 0 1.618 180 unlocked) (layer "F.SilkS")
       (effects (font (size 1 1) (thickness 0.15)))
     )
@@
       (effects (font (size 1 1) (thickness 0.15)))
     )
-    (fp_text user "${REFERENCE}" (at -0.685 3.3 180 unlocked) (layer "F.Fab")
+    (fp_text user "${REFERENCE}" (at -0.2 1.568 180 unlocked) (layer "F.Fab")
       (effects (font (size 1 1) (thickness 0.15)))
     )
@@
   (gr_line (start 112.4 153.2) (end 112.4 145.8) (layer "Edge.Cuts") (width 0.1))
   (gr_line (start 126.4 134.5) (end 126.4 140.6) (layer "Edge.Cuts") (width 0.1))
-  (segment (start 125.782106 142.248) (end 128.25 144.715894) (width 0.5) (layer "F.Cu") (net 1))
-  (segment (start 125.075 142.248) (end 125.782106 142.248) (width 0.5) (layer "F.Cu") (net 1))
-  (segment (start 128.25 144.715894) (end 128.25 149.518) (width 0.5) (layer "F.Cu") (net 1))
+  (gr_text "GND" (at 115.55 145.018) (layer "B.SilkS")
+    (effects (font (size 1 1) (thickness 0.25)) (justify mirror))
+  )
+  (gr_text "SW1" (at 118.09 148.018 -90) (layer "B.SilkS")
+    (effects (font (size 1 1) (thickness 0.25)) (justify left mirror))
+  )
+  (gr_text "SW4" (at 125.71 148.018 -90) (layer "B.SilkS")
+    (effects (font (size 1 1) (thickness 0.25)) (justify left mirror))
+  )
+  (gr_text "3.3V" (at 128.25 145.018) (layer "B.SilkS")
+    (effects (font (size 1 1) (thickness 0.25)) (justify mirror))
+  )
+  (gr_text "SW2" (at 120.63 148.018 -90) (layer "B.SilkS")
+    (effects (font (size 1 1) (thickness 0.25)) (justify left mirror))
+  )
+  (gr_text "SW3" (at 123.17 148.018 -90) (layer "B.SilkS")
+    (effects (font (size 1 1) (thickness 0.25)) (justify left mirror))
+  )
+  (gr_text "GND" (at 115.55 145.018) (layer "F.SilkS")
+    (effects (font (size 1 1) (thickness 0.25)))
+  )
+  (gr_text "3.3V" (at 128.25 145.018) (layer "F.SilkS")
+    (effects (font (size 1 1) (thickness 0.25)))
+  )
+  (segment (start 128.25 149.518) (end 128.25 146.693) (width 0.5) (layer "F.Cu") (net 1))
+  (segment (start 128.25 146.693) (end 125.075 143.518) (width 0.5) (layer "F.Cu") (net 1))
   (segment (start 123.805 143.518) (end 123.805 147.613) (width 0.5) (layer "F.Cu") (net 2))
   (segment (start 123.805 147.613) (end 125.71 149.518) (width 0.5) (layer "F.Cu") (net 2))
@@
   (segment (start 119.995 143.518) (end 119.995 147.613) (width 0.5) (layer "F.Cu") (net 5))
   (segment (start 119.995 147.613) (end 118.09 149.518) (width 0.5) (layer "F.Cu") (net 5))
-  (segment (start 118.725 146.343) (end 115.55 149.518) (width 0.5) (layer "F.Cu") (net 6))
-  (segment (start 118.725 143.518) (end 118.725 146.343) (width 0.5) (layer "F.Cu") (net 6))
+  (segment (start 117.602 142.248) (end 118.725 142.248) (width 0.5) (layer "F.Cu") (net 6))
+  (segment (start 115.55 149.518) (end 115.55 144.3) (width 0.5) (layer "F.Cu") (net 6))
+  (segment (start 115.55 144.3) (end 117.602 142.248) (width 0.5) (layer "F.Cu") (net 6))
 )

Commit message: moved board outline to avoid collision with molex connector
Parts:
- moved H1 5.04 mm to (116.9, 135.1)
- moved J2 5.04 mm to (113.7, 144.1)
Routing:
- net +3.3V: track 7.32 -> 10.4 mm
- net /GPIO9: track 6.79 -> 9.14 mm
- net /GPIO7: track 6.26 -> 7.87 mm
- net /GPIO5: track 6.26 -> 7.21 mm
- net GND: track 9.24 -> 8.57 mm
Other:
- board size 19 x 23.2 mm -> 19 x 22.6 mm
Changed lines of the file:
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@@
   (net 12 "unconnected-(J2-Pad12)")
   (footprint "MountingHole:MountingHole_2.2mm_M2" (layer "F.Cu")
-    (at 121.9 134.5)
+    (at 116.9 135.1)
     (descr "Mounting Hole 2.2mm, no annular, M2")
     (tags "mounting hole 2.2mm no annular m2")
@@
   )
   (footprint "Connector_PinHeader_1.27mm:PinHeader_2x06_P1.27mm_Vertical" (layer "F.Cu")
-    (at 118.725 143.518 90)
+    (at 113.725 144.118 90)
     (descr "Through hole straight pin header, 2x06, 1.27mm pitch, double rows")
     (tags "Through hole pin header THT 2x06 1.27mm double row")
@@
       (net 6 "GND") (pinfunction "Pin_6") (pintype "passive"))
   )
-  (gr_line (start 131.4 153.2) (end 131.4 145.8) (layer "Edge.Cuts") (width 0.1))
-  (gr_line (start 126.4 140.6) (end 131.4 145.8) (layer "Edge.Cuts") (width 0.1))
-  (gr_arc (start 117.4 134.5) (mid 121.9 130) (end 126.4 134.5) (layer "Edge.Cuts") (width 0.1))
-  (gr_line (start 112.4 145.8) (end 117.4 140.7) (layer "Edge.Cuts") (width 0.1))
-  (gr_line (start 117.4 134.5) (end 117.4 140.7) (layer "Edge.Cuts") (width 0.1))
+  (gr_line (start 131.4 153.2) (end 131.4 146.45) (layer "Edge.Cuts") (width 0.1))
+  (gr_line (start 123.4 144.45) (end 129.4 144.45) (layer "Edge.Cuts") (width 0.1))
+  (gr_arc (start 112.4 135.1) (mid 116.9 130.6) (end 121.4 135.1) (layer "Edge.Cuts") (width 0.1))
+  (gr_arc (start 129.4 144.45) (mid 130.814213 145.035787) (end 131.4 146.45) (layer "Edge.Cuts") (width 0.1))
+  (gr_arc (start 123.4 144.45) (mid 121.985786 143.864213) (end 121.4 142.45) (layer "Edge.Cuts") (width 0.1))
+  (gr_line (start 112.4 135.1) (end 112.4 145.8) (layer "Edge.Cuts") (width 0.1))
   (gr_line (start 112.4 153.2) (end 131.4 153.2) (layer "Edge.Cuts") (width 0.1))
   (gr_line (start 112.4 153.2) (end 112.4 145.8) (layer "Edge.Cuts") (width 0.1))
-  (gr_line (start 126.4 134.5) (end 126.4 140.6) (layer "Edge.Cuts") (width 0.1))
-  (gr_text "GND" (at 115.55 145.018) (layer "B.SilkS")
-    (effects (font (size 1 1) (thickness 0.25)) (justify mirror))
+  (gr_line (start 121.4 135.1) (end 121.4 142.45) (layer "Edge.Cuts") (width 0.1))
+  (gr_text "GND" (at 115.55 148.018 90) (layer "B.SilkS")
+    (effects (font (size 1 1) (thickness 0.25)) (justify right mirror))
   )
   (gr_text "SW1" (at 118.09 148.018 -90) (layer "B.SilkS")
@@
     (effects (font (size 1 1) (thickness 0.25)) (justify left mirror))
   )
-  (gr_text "3.3V" (at 128.25 145.018) (layer "B.SilkS")
-    (effects (font (size 1 1) (thickness 0.25)) (justify mirror))
+  (gr_text "3.3V" (at 128.25 148.018 90) (layer "B.SilkS")
+    (effects (font (size 1 1) (thickness 0.25)) (justify right mirror))
   )
   (gr_text "SW2" (at 120.63 148.018 -90) (layer "B.SilkS")
@@
     (effects (font (size 1 1) (thickness 0.25)) (justify left mirror))
   )
-  (gr_text "GND" (at 115.55 145.018) (layer "F.SilkS")
+  (gr_text "GND" (at 115.55 145.768) (layer "F.SilkS")
+    (effects (font (size 0.8 0.8) (thickness 0.2)))
+  )
+  (gr_text "3.3V" (at 128.25 145.518) (layer "F.SilkS")
     (effects (font (size 1 1) (thickness 0.25)))
   )
-  (gr_text "3.3V" (at 128.25 145.018) (layer "F.SilkS")
-    (effects (font (size 1 1) (thickness 0.25)))
-  )
-  (segment (start 128.25 149.518) (end 128.25 146.693) (width 0.5) (layer "F.Cu") (net 1))
-  (segment (start 128.25 146.693) (end 125.075 143.518) (width 0.5) (layer "F.Cu") (net 1))
-  (segment (start 123.805 143.518) (end 123.805 147.613) (width 0.5) (layer "F.Cu") (net 2))
-  (segment (start 123.805 147.613) (end 125.71 149.518) (width 0.5) (layer "F.Cu") (net 2))
-  (segment (start 122.535 148.883) (end 123.17 149.518) (width 0.5) (layer "F.Cu") (net 3))
-  (segment (start 122.535 143.518) (end 122.535 148.883) (width 0.5) (layer "F.Cu") (net 3))
-  (segment (start 121.265 148.883) (end 120.63 149.518) (width 0.5) (layer "F.Cu") (net 4))
-  (segment (start 121.265 143.518) (end 121.265 148.883) (width 0.5) (layer "F.Cu") (net 4))
-  (segment (start 119.995 143.518) (end 119.995 147.613) (width 0.5) (layer "F.Cu") (net 5))
-  (segment (start 119.995 147.613) (end 118.09 149.518) (width 0.5) (layer "F.Cu") (net 5))
-  (segment (start 117.602 142.248) (end 118.725 142.248) (width 0.5) (layer "F.Cu") (net 6))
-  (segment (start 115.55 149.518) (end 115.55 144.3) (width 0.5) (layer "F.Cu") (net 6))
-  (segment (start 115.55 144.3) (end 117.602 142.248) (width 0.5) (layer "F.Cu") (net 6))
+  (segment (start 125.882 147.15) (end 128.25 149.518) (width 0.35) (layer "F.Cu") (net 1))
+  (segment (start 120.075 144.118) (end 123.107 147.15) (width 0.35) (layer "F.Cu") (net 1))
+  (segment (start 123.107 147.15) (end 125.882 147.15) (width 0.35) (layer "F.Cu") (net 1))
+  (segment (start 122.73 148.043) (end 124.235 148.043) (width 0.35) (layer "F.Cu") (net 2))
+  (segment (start 118.805 144.118) (end 122.73 148.043) (width 0.35) (layer "F.Cu") (net 2))
+  (segment (start 124.235 148.043) (end 125.71 149.518) (width 0.35) (layer "F.Cu") (net 2))
+  (segment (start 122.935 149.518) (end 123.17 149.518) (width 0.35) (layer "F.Cu") (net 3))
+  (segment (start 117.535 144.118) (end 122.935 149.518) (width 0.35) (layer "F.Cu") (net 3))
+  (segment (start 116.265 145.153) (end 120.63 149.518) (width 0.35) (layer "F.Cu") (net 4))
+  (segment (start 116.265 144.118) (end 116.265 145.153) (width 0.35) (layer "F.Cu") (net 4))
+  (segment (start 114.995 146.423) (end 118.09 149.518) (width 0.35) (layer "F.Cu") (net 5))
+  (segment (start 114.995 144.118) (end 114.995 146.423) (width 0.35) (layer "F.Cu") (net 5))
+  (segment (start 112.85 146.818) (end 112.85 143.015894) (width 0.35) (layer "F.Cu") (net 6))
+  (segment (start 112.85 143.015894) (end 113.017894 142.848) (width 0.35) (layer "F.Cu") (net 6))
+  (segment (start 113.017894 142.848) (end 113.725 142.848) (width 0.35) (layer "F.Cu") (net 6))
+  (segment (start 115.55 149.518) (end 112.85 146.818) (width 0.35) (layer "F.Cu") (net 6))
 )
