File: adapter_boards/2X6_1.27MM_TO_JST_PH_I2C_HOLE/2X6_1.27MM_TO_JST_PH_I2C_HOLE.kicad_pcb (KiCad board)
At the start: 2 copper layers, 14 x 25.8 mm, 3 parts, among them J1 1.27mm 2x6-PTH, J2 S4B-PH-SM4-K-TB

Commit message: moved board outline to avoid collision with molex connector
Parts:
- moved J2 1.91 mm to (153.6, 99.3)
Routing:
- net /3V3: track 6.91 -> 5.08 mm
- net /GND: track 7.16 -> 8.71 mm
- net /I2C_SDA: track 12.0 -> 10.7 mm
Other:
- outline, holes or cut-outs redrawn
Changed lines of the file:
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@@
   (net 12 "/GND")
   (footprint "Connector_JST:JST_PH_S4B-PH-SM4-TB_1x04-1MP_P2.00mm_Horizontal" (layer "F.Cu")
-    (at 151.699999 99.303001)
+    (at 153.604999 99.303)
     (descr "JST PH series connector, S4B-PH-SM4-TB (http://www.jst-mfg.com/product/pdf/eng/ePH.pdf), generated with kicad-footprint-generator")
     (tags "connector JST PH top entry")
@@
       (effects (font (size 1 1) (thickness 0.15)))
     )
-    (fp_text value "1.27mm 2x6-PTH" (at -3.175 3.175) (layer "F.Fab")
+    (fp_text value "1.27mm 2x6-PTH" (at -3.174999 5.08) (layer "F.Fab")
       (effects (font (size 1 1) (thickness 0.15)))
     )
@@
   (gr_line (start 146.62 94.096) (end 147.2 89.4) (layer "Edge.Cuts") (width 0.1))
   (gr_arc (start 147.2 83.3) (mid 151.7 78.8) (end 156.2 83.3) (layer "Edge.Cuts") (width 0.1))
-  (gr_line (start 144.715 94.096001) (end 144.7 104.6) (layer "Edge.Cuts") (width 0.1))
-  (gr_line (start 144.7 104.6) (end 158.7 104.6) (layer "Edge.Cuts") (width 0.1))
+  (gr_line (start 146.62 94.096) (end 146.605 104.599999) (layer "Edge.Cuts") (width 0.1))
+  (gr_line (start 146.605 104.599999) (end 160.605 104.599999) (layer "Edge.Cuts") (width 0.1))
   (gr_line (start 156.779998 94.096002) (end 156.2 89.4) (layer "Edge.Cuts") (width 0.1))
-  (gr_line (start 156.779998 94.096002) (end 158.684998 94.096001) (layer "Edge.Cuts") (width 0.1))
+  (gr_line (start 156.779998 94.096002) (end 160.589998 94.096) (layer "Edge.Cuts") (width 0.1))
   (gr_line (start 156.2 83.3) (end 156.2 89.4) (layer "Edge.Cuts") (width 0.1))
   (gr_line (start 147.2 83.3) (end 147.2 89.4) (layer "Edge.Cuts") (width 0.1))
-  (gr_line (start 144.715 94.096001) (end 146.62 94.096) (layer "Edge.Cuts") (width 0.1))
-  (gr_line (start 158.684998 94.096001) (end 158.7 104.6) (layer "Edge.Cuts") (width 0.1))
+  (gr_line (start 160.589998 94.096) (end 160.605 104.599999) (layer "Edge.Cuts") (width 0.1))
   (gr_text "GND" (at 148.525 89.778 90) (layer "B.SilkS")
     (effects (font (size 0.381 0.381) (thickness 0.0762)) (justify mirror))
@@
     (effects (font (size 0.381 0.381) (thickness 0.0762)) (justify mirror))
   )
-  (gr_text "S4B-PH-SM4-TB" (at 146.62 103.748 90) (layer "B.SilkS")
+  (gr_text "S4B-PH-SM4-TB" (at 148.525 103.747999 90) (layer "B.SilkS")
     (effects (font (size 0.508 0.508) (thickness 0.0762)) (justify right mirror))
   )
@@
     (effects (font (size 0.381 0.381) (thickness 0.0762)) (justify mirror))
   )
-  (gr_text "1.27mm 2x6 to" (at 145.604 103.748002 90) (layer "B.SilkS")
+  (gr_text "1.27mm 2x6 to" (at 147.509 103.748001 90) (layer "B.SilkS")
     (effects (font (size 0.508 0.508) (thickness 0.0762)) (justify right mirror))
   )
-  (gr_text "JST-PH" (at 151.7 100.7) (layer "F.SilkS")
+  (gr_text "JST-PH" (at 153.605 100.699999) (layer "F.SilkS")
     (effects (font (size 1.016 1.016) (thickness 0.1778)))
   )
-  (gr_text "I2C" (at 151.7 102.224) (layer "F.SilkS")
+  (gr_text "I2C" (at 153.605 102.223999) (layer "F.SilkS")
     (effects (font (size 1.016 1.016) (thickness 0.1778)))
   )
-  (segment (start 150.699999 94.703001) (end 152.209999 93.193001) (width 0.25) (layer "F.Cu") (net 1))
-  (segment (start 152.209999 93.193001) (end 153.999999 93.193001) (width 0.25) (layer "F.Cu") (net 1))
-  (segment (start 153.999999 93.193001) (end 154.875 92.318) (width 0.25) (layer "F.Cu") (net 1))
-  (segment (start 150.7 96.453) (end 150.699999 94.703001) (width 0.25) (layer "F.Cu") (net 1))
-  (segment (start 152.699999 96.453001) (end 152.699999 94.112001) (width 0.25) (layer "F.Cu") (net 6))
-  (segment (start 152.699999 94.112001) (end 152.716 94.096) (width 0.25) (layer "F.Cu") (net 6))
-  (via (at 152.716 94.096) (size 0.8) (drill 0.4) (layers "F.Cu" "B.Cu") (net 6))
-  (segment (start 154.392001 94.096001) (end 155.750001 92.738001) (width 0.25) (layer "B.Cu") (net 6))
-  (segment (start 155.750001 92.738001) (end 155.750001 90.628) (width 0.25) (layer "B.Cu") (net 6))
-  (segment (start 155.295001 90.172999) (end 153.210002 90.172999) (width 0.25) (layer "B.Cu") (net 6))
-  (segment (start 152.716 94.096) (end 154.392001 94.096001) (width 0.25) (layer "B.Cu") (net 6))
-  (segment (start 153.210002 90.172999) (end 152.335 91.048001) (width 0.25) (layer "B.Cu") (net 6))
-  (segment (start 155.750001 90.628) (end 155.295001 90.172999) (width 0.25) (layer "B.Cu") (net 6))
-  (segment (start 155.750001 93.653) (end 155.750001 90.628) (width 0.25) (layer "F.Cu") (net 8))
-  (segment (start 155.750001 90.628) (end 155.295001 90.172999) (width 0.25) (layer "F.Cu") (net 8))
-  (segment (start 154.7 96.453) (end 154.7 94.703) (width 0.25) (layer "F.Cu") (net 8))
-  (segment (start 151.94 90.173) (end 151.065001 91.048001) (width 0.25) (layer "F.Cu") (net 8))
-  (segment (start 154.7 94.703) (end 155.750001 93.653) (width 0.25) (layer "F.Cu") (net 8))
-  (segment (start 155.295001 90.172999) (end 151.94 90.173) (width 0.25) (layer "F.Cu") (net 8))
-  (segment (start 147.795 91.048) (end 147.5 91.343) (width 0.5) (layer "F.Cu") (net 12))
-  (segment (start 147.5 95.253002) (end 148.699999 96.453001) (width 0.5) (layer "F.Cu") (net 12))
-  (segment (start 147.5 91.343) (end 147.5 95.253002) (width 0.5) (layer "F.Cu") (net 12))
+  (segment (start 152.604999 96.453) (end 152.604999 95.295001) (width 0.5) (layer "F.Cu") (net 1))
+  (segment (start 152.604999 95.295001) (end 154.875 93.025) (width 0.5) (layer "F.Cu") (net 1))
+  (segment (start 154.875 93.025) (end 154.875 92.318) (width 0.5) (layer "F.Cu") (net 1))
+  (segment (start 155.1505 94.3) (end 154.604999 94.845501) (width 0.2) (layer "F.Cu") (net 6))
+  (segment (start 154.604999 94.845501) (end 154.604999 96.453) (width 0.2) (layer "F.Cu") (net 6))
+  (via (at 155.1505 94.3) (size 0.8) (drill 0.4) (layers "F.Cu" "B.Cu") (net 6))
+  (segment (start 155.3 90) (end 155.9 90.6) (width 0.2) (layer "B.Cu") (net 6))
+  (segment (start 155.1 94.2495) (end 155.1505 94.3) (width 0.2) (layer "B.Cu") (net 6))
+  (segment (start 153.383 90) (end 153.7 90) (width 0.2) (layer "B.Cu") (net 6))
+  (segment (start 152.335 91.048) (end 153.383 90) (width 0.2) (layer "B.Cu") (net 6))
+  (segment (start 153.7 90) (end 155.3 90) (width 0.2) (layer "B.Cu") (net 6))
+  (segment (start 155.9 90.6) (end 155.9 92.7) (width 0.2) (layer "B.Cu") (net 6))
+  (segment (start 155.9 92.7) (end 155.1 93.5) (width 0.2) (layer "B.Cu") (net 6))
+  (segment (start 155.1 93.5) (end 155.1 94.2495) (width 0.2) (layer "B.Cu") (net 6))
+  (segment (start 155.9 95.748001) (end 156.604999 96.453) (width 0.2) (layer "F.Cu") (net 8))
+  (segment (start 155.3 90) (end 155.9 90.6) (width 0.2) (layer "F.Cu") (net 8))
+  (segment (start 155.9 90.6) (end 155.9 95.748001) (width 0.2) (layer "F.Cu") (net 8))
+  (segment (start 151.065 91.048) (end 152.113 90) (width 0.2) (layer "F.Cu") (net 8))
+  (segment (start 152.113 90) (end 155.3 90) (width 0.2) (layer "F.Cu") (net 8))
+  (segment (start 147.4 91.443) (end 147.4 94.4) (width 0.5) (layer "F.Cu") (net 12))
+  (segment (start 148.525 91.048) (end 147.795 91.048) (width 0.5) (layer "F.Cu") (net 12))
+  (segment (start 147.4 94.4) (end 149.453 96.453) (width 0.5) (layer "F.Cu") (net 12))
   (segment (start 148.119997 91.048002) (end 148.524998 91.048002) (width 0.25) (layer "F.Cu") (net 12))
-  (segment (start 148.525 91.048) (end 147.795 91.048) (width 0.5) (layer "F.Cu") (net 12))
+  (segment (start 149.453 96.453) (end 150.604999 96.453) (width 0.5) (layer "F.Cu") (net 12))
+  (segment (start 147.795 91.048) (end 147.4 91.443) (width 0.5) (layer "F.Cu") (net 12))
 )

Commit message: simplified board outline
Parts:
- moved J1 0.58 mm to (147.9, 92.3)
- moved H1 0.58 mm to (151.1, 83.3)
Other:
- outline, holes or cut-outs redrawn
Changed lines of the file:
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@@
 (kicad_pcb (version 20211014) (generator pcbnew)
   (general
-    (thickness 1.6002)
+    (thickness 1.6)
   )
   (paper "A4")
@@
   )
   (setup
+    (stackup
+      (layer "F.SilkS" (type "Top Silk Screen"))
+      (layer "F.Paste" (type "Top Solder Paste"))
+      (layer "F.Mask" (type "Top Solder Mask") (thickness 0.01))
+      (layer "F.Cu" (type "copper") (thickness 0.035))
+      (layer "dielectric 1" (type "core") (thickness 1.51) (material "FR4") (epsilon_r 4.5) (loss_tangent 0.02))
+      (layer "B.Cu" (type "copper") (thickness 0.035))
+      (layer "B.Mask" (type "Bottom Solder Mask") (thickness 0.01))
+      (layer "B.Paste" (type "Bottom Solder Paste"))
+      (layer "B.SilkS" (type "Bottom Silk Screen"))
+      (copper_finish "None")
+      (dielectric_constraints no)
+    )
     (pad_to_mask_clearance 0)
     (solder_mask_min_width 0.1)
@@
   )
   (footprint "Connector_PinHeader_1.27mm:PinHeader_2x06_P1.27mm_Vertical" (layer "F.Cu")
-    (at 148.525 92.318 90)
+    (at 147.945 92.318 90)
     (descr "Through hole straight pin header, 2x06, 1.27mm pitch, double rows")
     (tags "Through hole pin header THT 2x06 1.27mm double row")
@@
   )
   (footprint "MountingHole:MountingHole_2.2mm_M2" (layer "F.Cu")
-    (at 151.7 83.3)
+    (at 151.12 83.3)
     (descr "Mounting Hole 2.2mm, no annular, M2")
     (tags "mounting hole 2.2mm no annular m2")
@@
     (pad "" np_thru_hole circle (at 0 0) (size 2.2 2.2) (drill 2.2) (layers *.Cu *.Mask))
   )
-  (gr_line (start 124 93) (end 120 107) (layer "Cmts.User") (width 0.1524))
-  (gr_line (start 100 100) (end 124 93) (layer "Cmts.User") (width 0.1524))
-  (gr_line (start 146.62 94.096) (end 147.2 89.4) (layer "Edge.Cuts") (width 0.1))
-  (gr_arc (start 147.2 83.3) (mid 151.7 78.8) (end 156.2 83.3) (layer "Edge.Cuts") (width 0.1))
-  (gr_line (start 146.62 94.096) (end 146.605 104.599999) (layer "Edge.Cuts") (width 0.1))
-  (gr_line (start 146.605 104.599999) (end 160.605 104.599999) (layer "Edge.Cuts") (width 0.1))
-  (gr_line (start 156.779998 94.096002) (end 156.2 89.4) (layer "Edge.Cuts") (width 0.1))
-  (gr_line (start 156.779998 94.096002) (end 160.589998 94.096) (layer "Edge.Cuts") (width 0.1))
-  (gr_line (start 156.2 83.3) (end 156.2 89.4) (layer "Edge.Cuts") (width 0.1))
-  (gr_line (start 147.2 83.3) (end 147.2 89.4) (layer "Edge.Cuts") (width 0.1))
-  (gr_line (start 160.589998 94.096) (end 160.605 104.599999) (layer "Edge.Cuts") (width 0.1))
-  (gr_text "GND" (at 148.525 89.778 90) (layer "B.SilkS")
-    (effects (font (size 0.381 0.381) (thickness 0.0762)) (justify mirror))
-  )
-  (gr_text "SCL" (at 151.065 89.778001 90) (layer "B.SilkS")
-    (effects (font (size 0.381 0.381) (thickness 0.0762)) (justify mirror))
-  )
-  (gr_text "SDA" (at 152.334999 89.778001 90) (layer "B.SilkS")
+  (gr_arc (start 146.62 83.3) (mid 151.12 78.8) (end 155.62 83.3) (layer "Edge.Cuts") (width 0.1))
+  (gr_arc (start 158.6 94.012) (mid 160.014214 94.597786) (end 160.6 96.012) (layer "Edge.Cuts") (width 0.1))
+  (gr_line (start 146.62 89.4) (end 146.62 104.599999) (layer "Edge.Cuts") (width 0.1))
+  (gr_line (start 146.62 104.599999) (end 160.605 104.599999) (layer "Edge.Cuts") (width 0.1))
+  (gr_arc (start 157.62 94.012) (mid 156.205786 93.426214) (end 155.62 92.012) (layer "Edge.Cuts") (width 0.1))
+  (gr_line (start 158.6 94.012) (end 157.62 94.012) (layer "Edge.Cuts") (width 0.1))
+  (gr_line (start 155.62 83.3) (end 155.62 92.012) (layer "Edge.Cuts") (width 0.1))
+  (gr_line (start 146.62 83.3) (end 146.62 89.4) (layer "Edge.Cuts") (width 0.1))
+  (gr_line (start 160.6 96.012) (end 160.605 104.599999) (layer "Edge.Cuts") (width 0.1))
+  (gr_text "GND" (at 147.945 89.778 90) (layer "B.SilkS")
+    (effects (font (size 0.381 0.381) (thickness 0.0762)) (justify mirror))
+  )
+  (gr_text "SCL" (at 150.485 89.778001 90) (layer "B.SilkS")
+    (effects (font (size 0.381 0.381) (thickness 0.0762)) (justify mirror))
+  )
+  (gr_text "SDA" (at 151.754999 89.778001 90) (layer "B.SilkS")
     (effects (font (size 0.381 0.381) (thickness 0.0762)) (justify mirror))
   )
@@
     (effects (font (size 0.508 0.508) (thickness 0.0762)) (justify right mirror))
   )
-  (gr_text "3V3" (at 154.875 93.588001 90) (layer "B.SilkS")
+  (gr_text "3V3" (at 154.295 93.588001 90) (layer "B.SilkS")
     (effects (font (size 0.381 0.381) (thickness 0.0762)) (justify mirror))
   )
@@
     (effects (font (size 1.016 1.016) (thickness 0.1778)))
   )
-  (segment (start 152.604999 96.453) (end 152.604999 95.295001) (width 0.5) (layer "F.Cu") (net 1))
-  (segment (start 152.604999 95.295001) (end 154.875 93.025) (width 0.5) (layer "F.Cu") (net 1))
-  (segment (start 154.875 93.025) (end 154.875 92.318) (width 0.5) (layer "F.Cu") (net 1))
-  (segment (start 155.1505 94.3) (end 154.604999 94.845501) (width 0.2) (layer "F.Cu") (net 6))
-  (segment (start 154.604999 94.845501) (end 154.604999 96.453) (width 0.2) (layer "F.Cu") (net 6))
-  (via (at 155.1505 94.3) (size 0.8) (drill 0.4) (layers "F.Cu" "B.Cu") (net 6))
-  (segment (start 155.3 90) (end 155.9 90.6) (width 0.2) (layer "B.Cu") (net 6))
-  (segment (start 155.1 94.2495) (end 155.1505 94.3) (width 0.2) (layer "B.Cu") (net 6))
-  (segment (start 153.383 90) (end 153.7 90) (width 0.2) (layer "B.Cu") (net 6))
-  (segment (start 152.335 91.048) (end 153.383 90) (width 0.2) (layer "B.Cu") (net 6))
-  (segment (start 153.7 90) (end 155.3 90) (width 0.2) (layer "B.Cu") (net 6))
-  (segment (start 155.9 90.6) (end 155.9 92.7) (width 0.2) (layer "B.Cu") (net 6))
-  (segment (start 155.9 92.7) (end 155.1 93.5) (width 0.2) (layer "B.Cu") (net 6))
-  (segment (start 155.1 93.5) (end 155.1 94.2495) (width 0.2) (layer "B.Cu") (net 6))
-  (segment (start 155.9 95.748001) (end 156.604999 96.453) (width 0.2) (layer "F.Cu") (net 8))
-  (segment (start 155.3 90) (end 155.9 90.6) (width 0.2) (layer "F.Cu") (net 8))
-  (segment (start 155.9 90.6) (end 155.9 95.748001) (width 0.2) (layer "F.Cu") (net 8))
-  (segment (start 151.065 91.048) (end 152.113 90) (width 0.2) (layer "F.Cu") (net 8))
-  (segment (start 152.113 90) (end 155.3 90) (width 0.2) (layer "F.Cu") (net 8))
-  (segment (start 147.4 91.443) (end 147.4 94.4) (width 0.5) (layer "F.Cu") (net 12))
-  (segment (start 148.525 91.048) (end 147.795 91.048) (width 0.5) (layer "F.Cu") (net 12))
-  (segment (start 147.4 94.4) (end 149.453 96.453) (width 0.5) (layer "F.Cu") (net 12))
-  (segment (start 148.119997 91.048002) (end 148.524998 91.048002) (width 0.25) (layer "F.Cu") (net 12))
-  (segment (start 149.453 96.453) (end 150.604999 96.453) (width 0.5) (layer "F.Cu") (net 12))
-  (segment (start 147.795 91.048) (end 147.4 91.443) (width 0.5) (layer "F.Cu") (net 12))
+  (segment (start 152.604999 95.748406) (end 152.604999 96.453) (width 0.35) (layer "F.Cu") (net 1))
+  (segment (start 154.295 94.058405) (end 152.604999 95.748406) (width 0.35) (layer "F.Cu") (net 1))
+  (segment (start 154.295 92.318) (end 154.295 94.058405) (width 0.35) (layer "F.Cu") (net 1))
+  (segment (start 154.604999 95.195001) (end 154.604999 96.453) (width 0.2) (layer "F.Cu") (net 6))
+  (segment (start 155.220023 94.579977) (end 154.604999 95.195001) (width 0.2) (layer "F.Cu") (net 6))
+  (via (at 155.220023 94.579977) (size 0.8) (drill 0.4) (layers "F.Cu" "B.Cu") (net 6))
+  (segment (start 154.5 90) (end 155.2 90.7) (width 0.2) (layer "B.Cu") (net 6))
+  (segment (start 152.803 90) (end 154.5 90) (width 0.2) (layer "B.Cu") (net 6))
+  (segment (start 151.755 91.048) (end 152.803 90) (width 0.2) (layer "B.Cu") (net 6))
+  (segment (start 155.2 93.1) (end 155.2 94.559954) (width 0.2) (layer "B.Cu") (net 6))
+  (segment (start 155.2 90.7) (end 155.2 93.1) (width 0.2) (layer "B.Cu") (net 6))
+  (segment (start 155.2 94.559954) (end 155.220023 94.579977) (width 0.2) (layer "B.Cu") (net 6))
+  (segment (start 154.5 90) (end 155.145 90.645) (width 0.2) (layer "F.Cu") (net 8))
+  (segment (start 155.145 93.445) (end 156.604999 94.904999) (width 0.2) (layer "F.Cu") (net 8))
+  (segment (start 151.533 90) (end 154.5 90) (width 0.2) (layer "F.Cu") (net 8))
+  (segment (start 150.485 91.048) (end 151.533 90) (width 0.2) (layer "F.Cu") (net 8))
+  (segment (start 155.145 90.645) (end 155.145 93.445) (width 0.2) (layer "F.Cu") (net 8))
+  (segment (start 156.604999 94.904999) (end 156.604999 96.453) (width 0.2) (layer "F.Cu") (net 8))
+  (segment (start 147.02 94.52) (end 148.953 96.453) (width 0.35) (layer "F.Cu") (net 12))
+  (segment (start 147.945 91.048) (end 147.237894 91.048) (width 0.35) (layer "F.Cu") (net 12))
+  (segment (start 147.02 91.265894) (end 147.02 94.52) (width 0.35) (layer "F.Cu") (net 12))
+  (segment (start 148.953 96.453) (end 150.604999 96.453) (width 0.35) (layer "F.Cu") (net 12))
+  (segment (start 147.237894 91.048) (end 147.02 91.265894) (width 0.35) (layer "F.Cu") (net 12))
 )
