File: orion_pcb/NODE_CONNECTORS.kicad_sch (KiCad schematic)
At the start: 50 parts

Commit message: Added dual channel switching regulator. TODO: add reverse polarity protection on voltage input
Other:
- note added: "Maximum speed is 250 kb/s if using RS232 transceiver"
- note added: "To use TTL voltage levels, short ALL of the jumpers for both nodes, for the corresponding UART buses."
- note removed: "Note: Maximum speed is 250 kb/s if using RS232 transceiver"
- note removed: "Note: To use TTL voltage levels, short ALL of the jumpers for both nodes, for the corresponding UART buses."
Changed lines of the file:
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@@
     (effects (font (size 5.08 5.08) (thickness 1.016) bold) (justify left bottom))
   )
-  (text "Note:\nMaximum speed is 250 kb/s if using RS232 transceiver"
+  (text "Maximum speed is 250 kb/s if using RS232 transceiver"
     (at 18.415 246.38 0)
     (effects (font (size 1.27 1.27)) (justify left bottom))
@@
     (effects (font (size 2.54 2.54)) (justify left bottom))
   )
-  (text "Note:\nTo use TTL voltage levels, short ALL of the jumpers\nfor both nodes, for the corresponding UART buses."
+  (text "To use TTL voltage levels, short ALL of the jumpers\nfor both nodes, for the corresponding UART buses."
     (at 201.93 246.38 0)
     (effects (font (size 1.27 1.27)) (justify left bottom))
@@
   (symbol (lib_id "power:GND") (at 149.225 219.075 0) (unit 1)
     (in_bom yes) (on_board yes) (fields_autoplaced)
-    (property "Reference" "#PWR?" (id 0) (at 149.225 225.425 0)
+    (property "Reference" "#PWR0153" (id 0) (at 149.225 225.425 0)
       (effects (font (size 1.27 1.27)) hide)
     )
@@
   (symbol (lib_id "power:GND") (at 388.62 156.21 0) (unit 1)
     (in_bom yes) (on_board yes) (fields_autoplaced)
-    (property "Reference" "#PWR?" (id 0) (at 388.62 162.56 0)
+    (property "Reference" "#PWR0161" (id 0) (at 388.62 162.56 0)
       (effects (font (size 1.27 1.27)) hide)
     )
@@
   (symbol (lib_id "power:+3.3V") (at 361.315 78.105 0) (unit 1)
     (in_bom yes) (on_board yes) (fields_autoplaced)
-    (property "Reference" "#PWR?" (id 0) (at 361.315 81.915 0)
+    (property "Reference" "#PWR0160" (id 0) (at 361.315 81.915 0)
       (effects (font (size 1.27 1.27)) hide)
     )
@@
   (symbol (lib_id "power:+3.3V") (at 53.34 45.72 0) (unit 1)
     (in_bom yes) (on_board yes) (fields_autoplaced)
-    (property "Reference" "#PWR?" (id 0) (at 53.34 49.53 0)
+    (property "Reference" "#PWR0149" (id 0) (at 53.34 49.53 0)
       (effects (font (size 1.27 1.27)) hide)
     )
@@
   (symbol (lib_id "power:GND") (at 149.225 101.6 0) (unit 1)
     (in_bom yes) (on_board yes) (fields_autoplaced)
-    (property "Reference" "#PWR?" (id 0) (at 149.225 107.95 0)
+    (property "Reference" "#PWR0154" (id 0) (at 149.225 107.95 0)
       (effects (font (size 1.27 1.27)) hide)
     )
@@
   (symbol (lib_id "power:+3.3V") (at 361.95 192.405 0) (unit 1)
     (in_bom yes) (on_board yes) (fields_autoplaced)
-    (property "Reference" "#PWR?" (id 0) (at 361.95 196.215 0)
+    (property "Reference" "#PWR0156" (id 0) (at 361.95 196.215 0)
       (effects (font (size 1.27 1.27)) hide)
     )
@@
   (symbol (lib_id "power:+3.3V") (at 361.95 167.005 0) (unit 1)
     (in_bom yes) (on_board yes) (fields_autoplaced)
-    (property "Reference" "#PWR?" (id 0) (at 361.95 170.815 0)
+    (property "Reference" "#PWR0162" (id 0) (at 361.95 170.815 0)
       (effects (font (size 1.27 1.27)) hide)
     )
@@
   (symbol (lib_id "power:GND") (at 53.34 191.77 0) (unit 1)
     (in_bom yes) (on_board yes) (fields_autoplaced)
-    (property "Reference" "#PWR?" (id 0) (at 53.34 198.12 0)
+    (property "Reference" "#PWR0150" (id 0) (at 53.34 198.12 0)
       (effects (font (size 1.27 1.27)) hide)
     )
@@
   (symbol (lib_id "power:+3.3V") (at 361.315 141.605 0) (unit 1)
     (in_bom yes) (on_board yes) (fields_autoplaced)
-    (property "Reference" "#PWR?" (id 0) (at 361.315 145.415 0)
+    (property "Reference" "#PWR0159" (id 0) (at 361.315 145.415 0)
       (effects (font (size 1.27 1.27)) hide)
     )
@@
   (symbol (lib_id "power:+3.3V") (at 360.68 29.845 0) (unit 1)
     (in_bom yes) (on_board yes) (fields_autoplaced)
-    (property "Reference" "#PWR?" (id 0) (at 360.68 33.655 0)
+    (property "Reference" "#PWR0165" (id 0) (at 360.68 33.655 0)
       (effects (font (size 1.27 1.27)) hide)
     )
@@
   (symbol (lib_id "power:GND") (at 387.985 44.45 0) (unit 1)
     (in_bom yes) (on_board yes) (fields_autoplaced)
-    (property "Reference" "#PWR?" (id 0) (at 387.985 50.8 0)
+    (property "Reference" "#PWR0166" (id 0) (at 387.985 50.8 0)
       (effects (font (size 1.27 1.27)) hide)
     )
@@
   (symbol (lib_id "power:+3.3V") (at 361.315 53.975 0) (unit 1)
     (in_bom yes) (on_board yes) (fields_autoplaced)
-    (property "Reference" "#PWR?" (id 0) (at 361.315 57.785 0)
+    (property "Reference" "#PWR0155" (id 0) (at 361.315 57.785 0)
       (effects (font (size 1.27 1.27)) hide)
     )
@@
   (symbol (lib_id "power:+3.3V") (at 361.95 217.805 0) (unit 1)
     (in_bom yes) (on_board yes) (fields_autoplaced)
-    (property "Reference" "#PWR?" (id 0) (at 361.95 221.615 0)
+    (property "Reference" "#PWR0157" (id 0) (at 361.95 221.615 0)
       (effects (font (size 1.27 1.27)) hide)
     )
@@
   (symbol (lib_id "power:+3.3V") (at 388.62 140.97 0) (unit 1)
     (in_bom yes) (on_board yes) (fields_autoplaced)
-    (property "Reference" "#PWR?" (id 0) (at 388.62 144.78 0)
+    (property "Reference" "#PWR0163" (id 0) (at 388.62 144.78 0)
       (effects (font (size 1.27 1.27)) hide)
     )
@@
   (symbol (lib_id "power:GND") (at 104.775 111.76 0) (unit 1)
     (in_bom yes) (on_board yes)
-    (property "Reference" "#PWR?" (id 0) (at 104.775 118.11 0)
+    (property "Reference" "#PWR0148" (id 0) (at 104.775 118.11 0)
       (effects (font (size 1.27 1.27)) hide)
     )
@@
   (symbol (lib_id "power:GND") (at 53.34 74.295 0) (unit 1)
     (in_bom yes) (on_board yes) (fields_autoplaced)
-    (property "Reference" "#PWR?" (id 0) (at 53.34 80.645 0)
+    (property "Reference" "#PWR0147" (id 0) (at 53.34 80.645 0)
       (effects (font (size 1.27 1.27)) hide)
     )
@@
   (symbol (lib_id "power:+3.3V") (at 361.315 102.235 0) (unit 1)
     (in_bom yes) (on_board yes) (fields_autoplaced)
-    (property "Reference" "#PWR?" (id 0) (at 361.315 106.045 0)
+    (property "Reference" "#PWR0158" (id 0) (at 361.315 106.045 0)
       (effects (font (size 1.27 1.27)) hide)
     )
@@
   (symbol (lib_id "power:+3.3V") (at 387.985 29.21 0) (unit 1)
     (in_bom yes) (on_board yes) (fields_autoplaced)
-    (property "Reference" "#PWR?" (id 0) (at 387.985 33.02 0)
+    (property "Reference" "#PWR0164" (id 0) (at 387.985 33.02 0)
       (effects (font (size 1.27 1.27)) hide)
     )
@@
   (symbol (lib_id "power:+3.3V") (at 53.34 163.195 0) (unit 1)
     (in_bom yes) (on_board yes) (fields_autoplaced)
-    (property "Reference" "#PWR?" (id 0) (at 53.34 167.005 0)
+    (property "Reference" "#PWR0151" (id 0) (at 53.34 167.005 0)
       (effects (font (size 1.27 1.27)) hide)
     )
@@
   (symbol (lib_id "power:GND") (at 104.775 229.235 0) (unit 1)
     (in_bom yes) (on_board yes) (fields_autoplaced)
-    (property "Reference" "#PWR?" (id 0) (at 104.775 235.585 0)
-      (effects (font (size 1.27 1.27)) hide)
-    )
+    (property "Reference" "#PWR0152" (id 0) (at 104.775 235.585 0)
+      (effects (font (size 1.27 1.27)) hide)
+    )
