File: node_pcb/orion_pcb/HAT_DELOCALIZED.kicad_sch (KiCad schematic)
At the start: 5 parts

Commit message: Power and ESP32 moved to daugtherboards
Parts:
- gave numbers to parts that had none: 5
Other:
- company: (none) -> EPFL Xplore
- title: (none) -> Delocalized Connector
Changed lines of the file:
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@@
 (kicad_sch (version 20211123) (generator eeschema)
   (paper "A4")
+  (title_block
+    (title "Delocalized Connector")
+    (company "EPFL Xplore")
+    (comment 2 "Author: Vincent Nguyen")
+  )
   (junction (at 160.02 97.79) (diameter 0) (color 0 0 0 0)
   )
@@
     (stroke (width 0) (type default) (color 0 0 0 0))
   )
-  (wire (pts (xy 167.005 45.085) (xy 167.005 49.53))
+  (wire (pts (xy 167.005 42.545) (xy 167.005 49.53))
     (stroke (width 0) (type default) (color 0 0 0 0))
   )
@@
     (stroke (width 0) (type default) (color 0 0 0 0))
   )
-  (wire (pts (xy 131.445 40.005) (xy 131.445 49.53))
+  (wire (pts (xy 131.445 42.545) (xy 131.445 49.53))
     (stroke (width 0) (type default) (color 0 0 0 0))
   )
@@
     (stroke (width 0) (type default) (color 0 0 0 0))
   )
-  (wire (pts (xy 102.87 45.085) (xy 102.87 49.53))
+  (wire (pts (xy 102.87 42.545) (xy 102.87 49.53))
     (stroke (width 0) (type default) (color 0 0 0 0))
   )
@@
   (symbol (lib_id "power:GND") (at 189.865 130.81 0) (unit 1)
     (in_bom yes) (on_board yes) (fields_autoplaced)
-    (property "Reference" "#PWR0203" (id 0) (at 189.865 137.16 0)
+    (property "Reference" "#PWR01208" (id 0) (at 189.865 137.16 0)
       (effects (font (size 1.27 1.27)) hide)
     )
@@
   (symbol (lib_id "power:GND") (at 102.87 65.405 0) (unit 1)
     (in_bom yes) (on_board yes) (fields_autoplaced)
-    (property "Reference" "#PWR0210" (id 0) (at 102.87 71.755 0)
+    (property "Reference" "#PWR01202" (id 0) (at 102.87 71.755 0)
       (effects (font (size 1.27 1.27)) hide)
     )
@@
     (pin "1")
   )
-  (symbol (lib_id "power:+3.3V") (at 102.87 45.085 0) (unit 1)
-    (in_bom yes) (on_board yes) (fields_autoplaced)
-    (property "Reference" "#PWR0209" (id 0) (at 102.87 48.895 0)
-      (effects (font (size 1.27 1.27)) hide)
-    )
-    (property "Value" "+3.3V" (id 1) (at 102.87 40.005 0))
-    (property "Footprint" "" (id 2) (at 102.87 45.085 0)
-      (effects (font (size 1.27 1.27)) hide)
-    )
-    (property "Datasheet" "" (id 3) (at 102.87 45.085 0)
+  (symbol (lib_id "power:+3.3V") (at 102.87 42.545 0) (unit 1)
+    (in_bom yes) (on_board yes) (fields_autoplaced)
+    (property "Reference" "#PWR01201" (id 0) (at 102.87 46.355 0)
+      (effects (font (size 1.27 1.27)) hide)
+    )
+    (property "Value" "+3.3V" (id 1) (at 102.87 37.465 0))
+    (property "Footprint" "" (id 2) (at 102.87 42.545 0)
+      (effects (font (size 1.27 1.27)) hide)
+    )
+    (property "Datasheet" "" (id 3) (at 102.87 42.545 0)
       (effects (font (size 1.27 1.27)) hide)
     )
@@
   (symbol (lib_id "0_power_protection:ESDA6V1U1RL") (at 189.865 121.92 0) (unit 1)
     (in_bom yes) (on_board yes)
-    (property "Reference" "D?" (id 0) (at 199.39 121.285 0)
+    (property "Reference" "D1202" (id 0) (at 199.39 121.285 0)
       (effects (font (size 1.27 1.27)) (justify left))
     )
@@
   (symbol (lib_id "Connector_Generic:Conn_01x06") (at 178.435 57.15 0) (mirror x) (unit 1)
     (in_bom yes) (on_board yes)
-    (property "Reference" "J?" (id 0) (at 178.435 43.18 0))
+    (property "Reference" "J1203" (id 0) (at 178.435 43.18 0))
     (property "Value" "Conn_Picoblade_GPIO" (id 1) (at 178.435 45.72 0))
     (property "Footprint" "Connector_Molex:Molex_PicoBlade_53047-0610_1x06_P1.25mm_Vertical" (id 2) (at 178.435 57.15 0)
@@
   (symbol (lib_id "power:GND") (at 171.45 130.81 0) (unit 1)
     (in_bom yes) (on_board yes) (fields_autoplaced)
-    (property "Reference" "#PWR0204" (id 0) (at 171.45 137.16 0)
+    (property "Reference" "#PWR01207" (id 0) (at 171.45 137.16 0)
       (effects (font (size 1.27 1.27)) hide)
     )
@@
   (symbol (lib_id "0_power_protection:ESDA6V1U1RL") (at 171.45 121.92 0) (unit 1)
     (in_bom yes) (on_board yes)
-    (property "Reference" "D?" (id 0) (at 161.925 121.285 0)
+    (property "Reference" "D1201" (id 0) (at 161.925 121.285 0)
       (effects (font (size 1.27 1.27)) (justify right))
     )
@@
   (symbol (lib_id "Connector_Generic:Conn_01x06") (at 114.3 57.15 0) (mirror x) (unit 1)
     (in_bom yes) (on_board yes)
-    (property "Reference" "J?" (id 0) (at 114.3 43.18 0))
+    (property "Reference" "J1201" (id 0) (at 114.3 43.18 0))
     (property "Value" "Conn_Picoblade_SPI" (id 1) (at 114.3 45.72 0))
     (property "Footprint" "Connector_Molex:Molex_PicoBlade_53047-0610_1x06_P1.25mm_Vertical" (id 2) (at 114.3 57.15 0)
@@
   (symbol (lib_id "Connector_Generic:Conn_01x04") (at 144.145 54.61 0) (mirror x) (unit 1)
     (in_bom yes) (on_board yes) (fields_autoplaced)
-    (property "Reference" "J?" (id 0) (at 144.145 43.18 0))
+    (property "Reference" "J1202" (id 0) (at 144.145 43.18 0))
     (property "Value" "Conn_Picoblade_I2C" (id 1) (at 144.145 45.72 0))
     (property "Footprint" "Connector_Molex:Molex_PicoBlade_53047-0410_1x04_P1.25mm_Vertical" (id 2) (at 144.145 54.61 0)
@@
   (symbol (lib_id "power:GND") (at 131.445 66.04 0) (unit 1)
     (in_bom yes) (on_board yes) (fields_autoplaced)
-    (property "Reference" "#PWR0206" (id 0) (at 131.445 72.39 0)
+    (property "Reference" "#PWR01204" (id 0) (at 131.445 72.39 0)
       (effects (font (size 1.27 1.27)) hide)
     )
@@
     (pin "1")
   )
-  (symbol (lib_id "power:+3.3V") (at 131.445 40.005 0) (unit 1)
-    (in_bom yes) (on_board yes) (fields_autoplaced)
-    (property "Reference" "#PWR0207" (id 0) (at 131.445 43.815 0)
-      (effects (font (size 1.27 1.27)) hide)
-    )
-    (property "Value" "+3.3V" (id 1) (at 131.445 34.925 0))
-    (property "Footprint" "" (id 2) (at 131.445 40.005 0)
-      (effects (font (size 1.27 1.27)) hide)
-    )
-    (property "Datasheet" "" (id 3) (at 131.445 40.005 0)
-      (effects (font (size 1.27 1.27)) hide)
-    )
-    (pin "1")
-  )
-  (symbol (lib_id "power:+3.3V") (at 167.005 45.085 0) (unit 1)
-    (in_bom yes) (on_board yes) (fields_autoplaced)
-    (property "Reference" "#PWR0205" (id 0) (at 167.005 48.895 0)
-      (effects (font (size 1.27 1.27)) hide)
-    )
-    (property "Value" "+3.3V" (id 1) (at 167.005 40.005 0))
-    (property "Footprint" "" (id 2) (at 167.005 45.085 0)
-      (effects (font (size 1.27 1.27)) hide)
-    )
-    (property "Datasheet" "" (id 3) (at 167.005 45.085 0)
+  (symbol (lib_id "power:+3.3V") (at 131.445 42.545 0) (unit 1)
+    (in_bom yes) (on_board yes) (fields_autoplaced)
+    (property "Reference" "#PWR01203" (id 0) (at 131.445 46.355 0)
+      (effects (font (size 1.27 1.27)) hide)
+    )
+    (property "Value" "+3.3V" (id 1) (at 131.445 37.465 0))
+    (property "Footprint" "" (id 2) (at 131.445 42.545 0)
+      (effects (font (size 1.27 1.27)) hide)
+    )
+    (property "Datasheet" "" (id 3) (at 131.445 42.545 0)
+      (effects (font (size 1.27 1.27)) hide)
+    )
+    (pin "1")
+  )
+  (symbol (lib_id "power:+3.3V") (at 167.005 42.545 0) (unit 1)
+    (in_bom yes) (on_board yes) (fields_autoplaced)
+    (property "Reference" "#PWR01205" (id 0) (at 167.005 46.355 0)
+      (effects (font (size 1.27 1.27)) hide)
+    )
+    (property "Value" "+3.3V" (id 1) (at 167.005 37.465 0))
+    (property "Footprint" "" (id 2) (at 167.005 42.545 0)
+      (effects (font (size 1.27 1.27)) hide)
+    )
+    (property "Datasheet" "" (id 3) (at 167.005 42.545 0)
       (effects (font (size 1.27 1.27)) hide)
     )
@@
   (symbol (lib_id "power:GND") (at 167.005 65.405 0) (unit 1)
     (in_bom yes) (on_board yes) (fields_autoplaced)
-    (property "Reference" "#PWR0208" (id 0) (at 167.005 71.755 0)
-      (effects (font (size 1.27 1.27)) hide)
-    )
+    (property "Reference" "#PWR01206" (id 0) (at 167.005 71.755 0)
+      (effects (font (size 1.27 1.27)) hide)
+    )

Commit message: Added titles and plots
Other:
- note added: "Delocalized hat connector"
- note added: "Note: For now only 3.3V is connected for remote sensors to avoid damaging USB's 5V power rail. Use terminal block for 5V and VDD power rails."
- note removed: "Note: For now only 3.3V is connected for remote sensors. Use terminal block for 5V and VDD power rails."
- moved on the sheet: D1201, D1202, J1201, J1202, J1203

Commit message: Partial layout with max3232. To change to max3225
Other:
- note added: "Note: For now only 3.3V is connected for remote sensors to avoid damaging USB's 5V power rail. Use terminal block for 5V and VIN power rails."
- note removed: "Note: For now only 3.3V is connected for remote sensors to avoid damaging USB's 5V power rail. Use terminal block for 5V and VDD power rails."
Changed lines of the file:
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@@
     (effects (font (size 5.08 5.08) bold) (justify left bottom))
   )
-  (text "Note:\nFor now only 3.3V is connected for remote sensors\nto avoid damaging USB's 5V power rail.\nUse terminal block for 5V and VDD power rails."
+  (text "Note:\nFor now only 3.3V is connected for remote sensors\nto avoid damaging USB's 5V power rail.\nUse terminal block for 5V and VIN power rails."
     (at 86.995 131.445 0)
     (effects (font (size 1.27 1.27)) (justify left bottom))
