File: node_pcb/orion_pcb/MECHANICAL_TP.kicad_sch (KiCad schematic)
At the start: 10 parts

Commit message: Added titles and plots
Changed lines of the file:
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@@
     (stroke (width 0) (type default) (color 0 0 0 0))
   )
-  (text "Mounting holes" (at 93.98 21.59 0)
+  (text "Mounting holes" (at 92.075 20.32 0)
     (effects (font (size 2.54 2.54) bold) (justify left bottom))
   )
-  (text "Test points" (at 19.05 21.59 0)
+  (text "Test points" (at 16.51 20.32 0)
     (effects (font (size 2.54 2.54) bold) (justify left bottom))
   )

Commit message: Partial layout with max3232. To change to max3225
Parts:
- added H705, H706, H707, H708: MountingHole, MountingHole:MountingHole_2.2mm_M2, symbol Mechanical:MountingHole
- H701, H702, H703, H704: footprint (none) -> MountingHole:MountingHole_2.2mm_M2
Changed lines of the file:
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@@
       (effects (font (size 1.27 1.27)) (justify left))
     )
-    (property "Footprint" "" (id 2) (at 133.35 54.61 0)
+    (property "Footprint" "MountingHole:MountingHole_2.2mm_M2" (id 2) (at 133.35 54.61 0)
       (effects (font (size 1.27 1.27)) hide)
     )
@@
       (effects (font (size 1.27 1.27)) (justify left))
     )
-    (property "Footprint" "" (id 2) (at 133.35 70.485 0)
+    (property "Footprint" "MountingHole:MountingHole_2.2mm_M2" (id 2) (at 133.35 70.485 0)
       (effects (font (size 1.27 1.27)) hide)
     )
@@
       (effects (font (size 1.27 1.27)) (justify left))
     )
-    (property "Footprint" "" (id 2) (at 133.35 46.355 0)
+    (property "Footprint" "MountingHole:MountingHole_2.2mm_M2" (id 2) (at 133.35 46.355 0)
       (effects (font (size 1.27 1.27)) hide)
     )
@@
     (pin "1")
   )
+  (symbol (lib_id "Mechanical:MountingHole") (at 156.845 54.61 0) (unit 1)
+    (in_bom no) (on_board yes) (fields_autoplaced)
+    (property "Reference" "H706" (id 0) (at 159.385 53.3399 0)
+      (effects (font (size 1.27 1.27)) (justify left))
+    )
+    (property "Value" "MountingHole" (id 1) (at 159.385 55.8799 0)
+      (effects (font (size 1.27 1.27)) (justify left))
+    )
+    (property "Footprint" "MountingHole:MountingHole_2.2mm_M2" (id 2) (at 156.845 54.61 0)
+      (effects (font (size 1.27 1.27)) hide)
+    )
+    (property "Datasheet" "~" (id 3) (at 156.845 54.61 0)
+      (effects (font (size 1.27 1.27)) hide)
+    )
+  )
   (symbol (lib_id "Connector:TestPoint") (at 51.435 88.9 90) (unit 1)
     (in_bom no) (on_board yes)
@@
     (pin "1")
   )
+  (symbol (lib_id "Mechanical:MountingHole") (at 156.845 62.865 0) (unit 1)
+    (in_bom no) (on_board yes) (fields_autoplaced)
+    (property "Reference" "H707" (id 0) (at 159.385 61.5949 0)
+      (effects (font (size 1.27 1.27)) (justify left))
+    )
+    (property "Value" "MountingHole" (id 1) (at 159.385 64.1349 0)
+      (effects (font (size 1.27 1.27)) (justify left))
+    )
+    (property "Footprint" "MountingHole:MountingHole_2.2mm_M2" (id 2) (at 156.845 62.865 0)
+      (effects (font (size 1.27 1.27)) hide)
+    )
+    (property "Datasheet" "~" (id 3) (at 156.845 62.865 0)
+      (effects (font (size 1.27 1.27)) hide)
+    )
+  )
   (symbol (lib_id "Mechanical:MountingHole") (at 133.35 62.865 0) (unit 1)
     (in_bom no) (on_board yes) (fields_autoplaced)
@@
       (effects (font (size 1.27 1.27)) (justify left))
     )
-    (property "Footprint" "" (id 2) (at 133.35 62.865 0)
+    (property "Footprint" "MountingHole:MountingHole_2.2mm_M2" (id 2) (at 133.35 62.865 0)
       (effects (font (size 1.27 1.27)) hide)
     )
@@
     )
   )
+  (symbol (lib_id "Mechanical:MountingHole") (at 156.845 46.355 0) (unit 1)
+    (in_bom no) (on_board yes) (fields_autoplaced)
+    (property "Reference" "H705" (id 0) (at 159.385 45.0849 0)
+      (effects (font (size 1.27 1.27)) (justify left))
+    )
+    (property "Value" "MountingHole" (id 1) (at 159.385 47.6249 0)
+      (effects (font (size 1.27 1.27)) (justify left))
+    )
+    (property "Footprint" "MountingHole:MountingHole_2.2mm_M2" (id 2) (at 156.845 46.355 0)
+      (effects (font (size 1.27 1.27)) hide)
+    )
+    (property "Datasheet" "~" (id 3) (at 156.845 46.355 0)
+      (effects (font (size 1.27 1.27)) hide)
+    )
+  )
   (symbol (lib_id "Connector:TestPoint") (at 51.435 73.66 90) (unit 1)
     (in_bom no) (on_board yes)
@@
     (pin "1")
   )
+  (symbol (lib_id "Mechanical:MountingHole") (at 156.845 70.485 0) (unit 1)
+    (in_bom no) (on_board yes) (fields_autoplaced)
+    (property "Reference" "H708" (id 0) (at 159.385 69.2149 0)
+      (effects (font (size 1.27 1.27)) (justify left))
+    )
+    (property "Value" "MountingHole" (id 1) (at 159.385 71.7549 0)
+      (effects (font (size 1.27 1.27)) (justify left))
+    )
+    (property "Footprint" "MountingHole:MountingHole_2.2mm_M2" (id 2) (at 156.845 70.485 0)
+      (effects (font (size 1.27 1.27)) hide)
+    )
+    (property "Datasheet" "~" (id 3) (at 156.845 70.485 0)
+      (effects (font (size 1.27 1.27)) hide)
+    )
+  )
   (symbol (lib_id "Connector:TestPoint") (at 51.435 66.04 90) (unit 1)

Commit message: updated paths
Parts:
- H705: footprint MountingHole:MountingHole_2.2mm_M2 -> MountingHole:MountingHole_2.2mm_M2_DIN965_Pad
- H706, H707, H708: footprint MountingHole:MountingHole_2.2mm_M2 -> MountingHole:MountingHole_2.2mm_M2_Pad
Changed lines of the file:
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@@
       (effects (font (size 1.27 1.27)) (justify left))
     )
-    (property "Footprint" "MountingHole:MountingHole_2.2mm_M2" (id 2) (at 156.845 54.61 0)
+    (property "Footprint" "MountingHole:MountingHole_2.2mm_M2_Pad" (id 2) (at 156.845 54.61 0)
       (effects (font (size 1.27 1.27)) hide)
     )
@@
       (effects (font (size 1.27 1.27)) (justify left))
     )
-    (property "Footprint" "MountingHole:MountingHole_2.2mm_M2" (id 2) (at 156.845 62.865 0)
+    (property "Footprint" "MountingHole:MountingHole_2.2mm_M2_Pad" (id 2) (at 156.845 62.865 0)
       (effects (font (size 1.27 1.27)) hide)
     )
@@
       (effects (font (size 1.27 1.27)) (justify left))
     )
-    (property "Footprint" "MountingHole:MountingHole_2.2mm_M2" (id 2) (at 156.845 46.355 0)
+    (property "Footprint" "MountingHole:MountingHole_2.2mm_M2_DIN965_Pad" (id 2) (at 156.845 46.355 0)
       (effects (font (size 1.27 1.27)) hide)
     )
@@
       (effects (font (size 1.27 1.27)) (justify left))
     )
-    (property "Footprint" "MountingHole:MountingHole_2.2mm_M2" (id 2) (at 156.845 70.485 0)
+    (property "Footprint" "MountingHole:MountingHole_2.2mm_M2_Pad" (id 2) (at 156.845 70.485 0)
       (effects (font (size 1.27 1.27)) hide)
     )

Commit message: Updated pin type
Changed lines of the file:
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@@
     (comment 2 "Author: Vincent Nguyen")
   )
+  (junction (at 54.61 50.8) (diameter 0) (color 0 0 0 0)
+  )
+  (junction (at 54.61 66.04) (diameter 0) (color 0 0 0 0)
+  )
+  (junction (at 54.61 58.42) (diameter 0) (color 0 0 0 0)
+  )
   (wire (pts (xy 51.435 88.9) (xy 60.325 88.9))
     (stroke (width 0) (type default) (color 0 0 0 0))
@@
     (stroke (width 0) (type default) (color 0 0 0 0))
   )
+  (wire (pts (xy 54.61 50.8) (xy 60.325 50.8))
+    (stroke (width 0) (type default) (color 0 0 0 0))
+  )
   (polyline (pts (xy 90.17 14.605) (xy 194.31 14.605))
     (stroke (width 0) (type default) (color 0 0 0 0))
@@
     (stroke (width 0) (type default) (color 0 0 0 0))
   )
-  (wire (pts (xy 51.435 66.04) (xy 60.325 66.04))
-    (stroke (width 0) (type default) (color 0 0 0 0))
-  )
-  (wire (pts (xy 51.435 50.8) (xy 60.325 50.8))
+  (wire (pts (xy 51.435 66.04) (xy 54.61 66.04))
+    (stroke (width 0) (type default) (color 0 0 0 0))
+  )
+  (wire (pts (xy 54.61 66.04) (xy 60.325 66.04))
+    (stroke (width 0) (type default) (color 0 0 0 0))
+  )
+  (wire (pts (xy 51.435 50.8) (xy 54.61 50.8))
     (stroke (width 0) (type default) (color 0 0 0 0))
   )
@@
     (stroke (width 0) (type default) (color 0 0 0 0))
   )
-  (wire (pts (xy 51.435 58.42) (xy 60.325 58.42))
+  (wire (pts (xy 51.435 58.42) (xy 54.61 58.42))
     (stroke (width 0) (type default) (color 0 0 0 0))
   )
   (polyline (pts (xy 86.36 132.715) (xy 14.605 132.715))
+    (stroke (width 0) (type default) (color 0 0 0 0))
+  )
+  (wire (pts (xy 54.61 58.42) (xy 60.325 58.42))
     (stroke (width 0) (type default) (color 0 0 0 0))
   )
@@
     )
   )
+  (symbol (lib_id "power:PWR_FLAG") (at 54.61 58.42 0) (unit 1)
+    (in_bom yes) (on_board yes) (fields_autoplaced)
+    (property "Reference" "#FLG0102" (id 0) (at 54.61 56.515 0)
+      (effects (font (size 1.27 1.27)) hide)
+    )
+    (property "Value" "PWR_FLAG" (id 1) (at 54.61 53.34 0)
+      (effects (font (size 1.27 1.27)) hide)
+    )
+    (property "Footprint" "" (id 2) (at 54.61 58.42 0)
+      (effects (font (size 1.27 1.27)) hide)
+    )
+    (property "Datasheet" "~" (id 3) (at 54.61 58.42 0)
+      (effects (font (size 1.27 1.27)) hide)
+    )
+    (pin "1")
+  )
   (symbol (lib_id "Connector:TestPoint") (at 51.435 81.28 90) (unit 1)
     (in_bom no) (on_board yes)
@@
     (pin "1")
   )
+  (symbol (lib_id "power:PWR_FLAG") (at 54.61 50.8 0) (unit 1)
+    (in_bom yes) (on_board yes) (fields_autoplaced)
+    (property "Reference" "#FLG0101" (id 0) (at 54.61 48.895 0)
+      (effects (font (size 1.27 1.27)) hide)
+    )
+    (property "Value" "PWR_FLAG" (id 1) (at 54.61 45.72 0)
+      (effects (font (size 1.27 1.27)) hide)
+    )
+    (property "Footprint" "" (id 2) (at 54.61 50.8 0)
+      (effects (font (size 1.27 1.27)) hide)
+    )
+    (property "Datasheet" "~" (id 3) (at 54.61 50.8 0)
+      (effects (font (size 1.27 1.27)) hide)
+    )
+    (pin "1")
+  )
   (symbol (lib_id "power:GND") (at 60.325 81.28 90) (unit 1)
     (in_bom yes) (on_board yes) (fields_autoplaced)
@@
     )
   )
+  (symbol (lib_id "power:PWR_FLAG") (at 54.61 66.04 0) (unit 1)
+    (in_bom yes) (on_board yes) (fields_autoplaced)
+    (property "Reference" "#FLG0103" (id 0) (at 54.61 64.135 0)
+      (effects (font (size 1.27 1.27)) hide)
+    )
+    (property "Value" "PWR_FLAG" (id 1) (at 54.61 60.96 0)
+      (effects (font (size 1.27 1.27)) hide)
+    )
+    (property "Footprint" "" (id 2) (at 54.61 66.04 0)
+      (effects (font (size 1.27 1.27)) hide)
+    )
+    (property "Datasheet" "~" (id 3) (at 54.61 66.04 0)
+      (effects (font (size 1.27 1.27)) hide)
+    )
+    (pin "1")
+  )
   (symbol (lib_id "Mechanical:MountingHole") (at 156.845 46.355 0) (unit 1)

Commit message: Finished routing. Need to add logos
Parts:
- removed TP701: VIN, 0_various:TestPoint, symbol Connector:TestPoint
- removed TP706: GND, 0_various:TestPoint, symbol Connector:TestPoint
- renumbered TP702 to TP701, TP703 to TP702, TP704 to TP703, TP705 to TP704
Changed lines of the file:
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@@
     (comment 2 "Author: Vincent Nguyen")
   )
-  (junction (at 54.61 50.8) (diameter 0) (color 0 0 0 0)
-  )
   (junction (at 54.61 66.04) (diameter 0) (color 0 0 0 0)
   )
   (junction (at 54.61 58.42) (diameter 0) (color 0 0 0 0)
   )
-  (wire (pts (xy 51.435 88.9) (xy 60.325 88.9))
-    (stroke (width 0) (type default) (color 0 0 0 0))
-  )
   (polyline (pts (xy 14.605 14.605) (xy 14.605 132.715))
     (stroke (width 0) (type default) (color 0 0 0 0))
   )
-  (wire (pts (xy 54.61 50.8) (xy 60.325 50.8))
-    (stroke (width 0) (type default) (color 0 0 0 0))
-  )
   (polyline (pts (xy 90.17 14.605) (xy 194.31 14.605))
     (stroke (width 0) (type default) (color 0 0 0 0))
@@
   )
   (wire (pts (xy 54.61 66.04) (xy 60.325 66.04))
-    (stroke (width 0) (type default) (color 0 0 0 0))
-  )
-  (wire (pts (xy 51.435 50.8) (xy 54.61 50.8))
     (stroke (width 0) (type default) (color 0 0 0 0))
   )
@@
     )
   )
-  (global_label "VIN" (shape passive) (at 60.325 50.8 0) (fields_autoplaced)
-    (effects (font (size 1.27 1.27) bold) (justify left))
-    (property "Intersheet References" "${INTERSHEET_REFS}" (id 0) (at 65.9523 50.673 0)
-      (effects (font (size 1.27 1.27) bold) (justify left) hide)
-    )
-  )
   (global_label "VIO" (shape passive) (at 60.325 73.66 0) (fields_autoplaced)
     (effects (font (size 1.27 1.27) bold) (justify left))
@@
     )
   )
-  (symbol (lib_id "Connector:TestPoint") (at 51.435 50.8 90) (unit 1)
-    (in_bom no) (on_board yes)
-    (property "Reference" "TP701" (id 0) (at 38.735 50.8 90)
-      (effects (font (size 1.27 1.27)) (justify right))
-    )
-    (property "Value" "VIN" (id 1) (at 35.56 50.8 90)
-      (effects (font (size 1.27 1.27)) (justify left))
-    )
-    (property "Footprint" "0_various:TestPoint" (id 2) (at 51.435 45.72 0)
-      (effects (font (size 1.27 1.27)) hide)
-    )
-    (property "Datasheet" "~" (id 3) (at 51.435 45.72 0)
-      (effects (font (size 1.27 1.27)) hide)
-    )
-    (pin "1")
-  )
   (symbol (lib_id "Mechanical:MountingHole") (at 133.35 70.485 0) (unit 1)
     (in_bom no) (on_board yes) (fields_autoplaced)
@@
   (symbol (lib_id "Connector:TestPoint") (at 51.435 81.28 90) (unit 1)
     (in_bom no) (on_board yes)
-    (property "Reference" "TP705" (id 0) (at 38.735 81.28 90)
+    (property "Reference" "TP704" (id 0) (at 38.735 81.28 90)
       (effects (font (size 1.27 1.27)) (justify right))
     )
@@
     )
     (property "Datasheet" "~" (id 3) (at 51.435 76.2 0)
-      (effects (font (size 1.27 1.27)) hide)
-    )
-    (pin "1")
-  )
-  (symbol (lib_id "power:PWR_FLAG") (at 54.61 50.8 0) (unit 1)
-    (in_bom yes) (on_board yes) (fields_autoplaced)
-    (property "Reference" "#FLG0101" (id 0) (at 54.61 48.895 0)
-      (effects (font (size 1.27 1.27)) hide)
-    )
-    (property "Value" "PWR_FLAG" (id 1) (at 54.61 45.72 0)
-      (effects (font (size 1.27 1.27)) hide)
-    )
-    (property "Footprint" "" (id 2) (at 54.61 50.8 0)
-      (effects (font (size 1.27 1.27)) hide)
-    )
-    (property "Datasheet" "~" (id 3) (at 54.61 50.8 0)
       (effects (font (size 1.27 1.27)) hide)
     )
@@
   (symbol (lib_id "Connector:TestPoint") (at 51.435 58.42 90) (unit 1)
     (in_bom no) (on_board yes)
-    (property "Reference" "TP702" (id 0) (at 38.735 58.42 90)
+    (property "Reference" "TP701" (id 0) (at 38.735 58.42 90)
       (effects (font (size 1.27 1.27)) (justify right))
     )
@@
       (effects (font (size 1.27 1.27)) hide)
     )
-  )
-  (symbol (lib_id "Connector:TestPoint") (at 51.435 88.9 90) (unit 1)
-    (in_bom no) (on_board yes)
-    (property "Reference" "TP706" (id 0) (at 38.735 88.9 90)
-      (effects (font (size 1.27 1.27)) (justify right))
-    )
-    (property "Value" "GND" (id 1) (at 35.56 88.9 90)
-      (effects (font (size 1.27 1.27)) (justify left))
-    )
-    (property "Footprint" "0_various:TestPoint" (id 2) (at 51.435 83.82 0)
-      (effects (font (size 1.27 1.27)) hide)
-    )
-    (property "Datasheet" "~" (id 3) (at 51.435 83.82 0)
-      (effects (font (size 1.27 1.27)) hide)
-    )
-    (pin "1")
   )
   (symbol (lib_id "Mechanical:MountingHole") (at 156.845 62.865 0) (unit 1)
@@
   (symbol (lib_id "Connector:TestPoint") (at 51.435 73.66 90) (unit 1)
     (in_bom no) (on_board yes)
-    (property "Reference" "TP704" (id 0) (at 38.735 73.66 90)
+    (property "Reference" "TP703" (id 0) (at 38.735 73.66 90)
       (effects (font (size 1.27 1.27)) (justify right))
     )
@@
   (symbol (lib_id "Connector:TestPoint") (at 51.435 66.04 90) (unit 1)
     (in_bom no) (on_board yes)
-    (property "Reference" "TP703" (id 0) (at 38.735 66.04 90)
+    (property "Reference" "TP702" (id 0) (at 38.735 66.04 90)
       (effects (font (size 1.27 1.27)) (justify right))
     )
@@
       (effects (font (size 1.27 1.27)) hide)
     )
-    (pin "1")
-  )
-  (symbol (lib_id "power:GND") (at 60.325 88.9 90) (unit 1)
-    (in_bom yes) (on_board yes) (fields_autoplaced)
-    (property "Reference" "#PWR0702" (id 0) (at 66.675 88.9 0)
-      (effects (font (size 1.27 1.27)) hide)
-    )
-    (property "Value" "GND" (id 1) (at 64.135 88.8999 90)
-      (effects (font (size 1.27 1.27)) (justify right))
-    )
-    (property "Footprint" "" (id 2) (at 60.325 88.9 0)
-      (effects (font (size 1.27 1.27)) hide)
-    )
-    (property "Datasheet" "" (id 3) (at 60.325 88.9 0)
-      (effects (font (size 1.27 1.27)) hide)
-    )
