File: node_pcb/orion_pcb/USB_UART.kicad_sch (KiCad schematic)
At the start: 18 parts

Commit message: Power and ESP32 moved to daugtherboards
Parts:
- removed C?: 4.7uF, symbol Device:C_Small
- removed C?: 100nF, symbol Device:C_Small
- added C301, C302: 1uF, symbol Device:C_Small
- added U302: NCV8161ASN330T1G, Package_TO_SOT_SMD:SOT-23-5, symbol 0_regulator_linear:NCV8161ASN330T1G
- gave numbers to parts that had none: 16
Connections:
- net GND: now also C301.2, C302.2, U302.2 (GND)
- net VBUS_REV: now also C301.1, U302.1 (IN), U302.3 (EN); no longer C303.1, C304.1, U303.7 (VREGIN)
- net VIO: now also C303.1, C304.1, U303.7 (VREGIN), C302.1, U302.5 (OUT)
Other:
- note added: "We choose not to use the internal 3.3 V regulator of the CP2102 IC. This is because multiple people have reported a voltage of ~4 V at the output of that regulator instead of 3.3 V."
- company: (none) -> EPFL Xplore
- title: (none) -> USB to UART Bridge
- moved on the sheet: C303, C304, D301, F301, J301, Q301, R301, R302, R305, U301

Commit message: Added titles and plots
Other:
- note added: "USB to UART bridge"
- moved on the sheet: C301, C302, C303, C304, D301, D302, D303, D304, F301, J301, Q301, R301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

Commit message: Partial layout with max3232. To change to max3225
Parts:
- removed D304: ESDALC6V1W5, Package_TO_SOT_SMD:SOT-23-5, symbol 0_power_protection:ESDALC6V1W5
- C301, C302, C303, C304: footprint (none) -> Capacitor_SMD:C_0603_1608Metric
- R301, R302, R303, R304, R305: footprint (none) -> Resistor_SMD:R_0603_1608Metric
Connections:
- net U1TX_LED_CAT: now reaches D302.1 (K), R304.1
- net U1RX_LED_CAT: now reaches D303.1 (K), R305.2
- no-connect marks 15 -> 13
Other:
- moved on the sheet: D302, D303, R304, R305

Commit message: updated paths
Parts:
- J301: footprint Connector_USB:USB_Micro-B_Molex-105017-0001 -> 0_connectors:USB_Micro-B_Molex-105017-0001
- U302: Digikey ref (none) -> NCV8161ASN330T1GOSCT-ND; Manufacturer ref  (none) -> NCV8161ASN330T1G
- U303: Digikey ref (none) -> 1175-1628-ND; Manufacturer ref (none) -> 3220-10-0200-00
Changed lines of the file:
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@@
     (property "Reference" "J301" (id 0) (at 29.21 57.785 0))
     (property "Value" "USB_B_Micro" (id 1) (at 29.21 60.325 0))
-    (property "Footprint" "Connector_USB:USB_Micro-B_Molex-105017-0001" (id 2) (at 33.02 72.39 0)
+    (property "Footprint" "0_connectors:USB_Micro-B_Molex-105017-0001" (id 2) (at 33.02 72.39 0)
       (effects (font (size 1.27 1.27)) hide)
     )
@@
     )
     (property "Datasheet" "https://www.silabs.com/documents/public/data-sheets/cp2102n-datasheet.pdf" (id 3) (at 171.45 112.395 0)
+      (effects (font (size 1.27 1.27)) hide)
+    )
+    (property "Manufacturer ref" "3220-10-0200-00" (id 4) (at 171.45 113.665 0)
+      (effects (font (size 1.27 1.27)) hide)
+    )
+    (property "Digikey ref" "1175-1628-ND" (id 5) (at 171.45 113.665 0)
       (effects (font (size 1.27 1.27)) hide)
     )
@@
       (effects (font (size 1.27 1.27)) hide)
     )
+    (property "Manufacturer ref " "NCV8161ASN330T1G" (id 4) (at 150.495 68.58 0)
+      (effects (font (size 1.27 1.27)) hide)
+    )
+    (property "Digikey ref" "NCV8161ASN330T1GOSCT-ND" (id 5) (at 150.495 68.58 0)
+      (effects (font (size 1.27 1.27)) hide)
+    )

Commit message: ädded BOM
Parts:
- U302: Manufacturer ref (none) -> NCV8161ASN330T1G; Manufacturer ref  NCV8161ASN330T1G -> (none)
Changed lines of the file:
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@@
       (effects (font (size 1.27 1.27)) hide)
     )
-    (property "Manufacturer ref " "NCV8161ASN330T1G" (id 4) (at 150.495 68.58 0)
+    (property "Manufacturer ref" "NCV8161ASN330T1G" (id 4) (at 150.495 68.58 0)
       (effects (font (size 1.27 1.27)) hide)
     )

Commit message: Added test pads for usart1
Parts:
- added TP301: U1RX, TestPoint:TestPoint_Pad_D1.5mm, symbol Connector:TestPoint
- added TP302: U1TX, TestPoint:TestPoint_Pad_D1.5mm, symbol Connector:TestPoint
Connections:
- net USART1_RX: now also TP301.1
- net USART1_TX: now also TP302.1
Changed lines of the file:
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@@
   (junction (at 171.45 83.185) (diameter 0) (color 0 0 0 0)
   )
+  (junction (at 221.615 90.805) (diameter 0) (color 0 0 0 0)
+  )
   (junction (at 105.41 66.04) (diameter 0) (color 0 0 0 0)
   )
@@
   )
   (junction (at 135.89 66.04) (diameter 0) (color 0 0 0 0)
+  )
+  (junction (at 221.615 93.345) (diameter 0) (color 0 0 0 0)
   )
   (junction (at 161.29 66.04) (diameter 0) (color 0 0 0 0)
@@
     (stroke (width 0) (type default) (color 0 0 0 0))
   )
-  (wire (pts (xy 184.15 90.805) (xy 238.125 90.805))
+  (wire (pts (xy 184.15 90.805) (xy 221.615 90.805))
     (stroke (width 0) (type default) (color 0 0 0 0))
   )
@@
     (stroke (width 0) (type default) (color 0 0 0 0))
   )
+  (wire (pts (xy 221.615 93.345) (xy 238.125 93.345))
+    (stroke (width 0) (type default) (color 0 0 0 0))
+  )
   (wire (pts (xy 59.69 87.63) (xy 59.69 106.68))
     (stroke (width 0) (type default) (color 0 0 0 0))
@@
     (stroke (width 0) (type default) (color 0 0 0 0))
   )
-  (wire (pts (xy 184.15 93.345) (xy 238.125 93.345))
+  (wire (pts (xy 184.15 93.345) (xy 221.615 93.345))
     (stroke (width 0) (type default) (color 0 0 0 0))
   )
@@
   )
   (wire (pts (xy 184.785 66.04) (xy 171.45 66.04))
+    (stroke (width 0) (type default) (color 0 0 0 0))
+  )
+  (wire (pts (xy 221.615 90.805) (xy 238.125 90.805))
     (stroke (width 0) (type default) (color 0 0 0 0))
   )
@@
   (hierarchical_label "{USART1}" (shape bidirectional) (at 243.205 89.535 0)
     (effects (font (size 1.27 1.27)) (justify left))
+  )
+  (symbol (lib_id "Connector:TestPoint") (at 221.615 90.805 0) (unit 1)
+    (in_bom no) (on_board yes)
+    (property "Reference" "TP301" (id 0) (at 221.615 85.09 0))
+    (property "Value" "U1RX" (id 1) (at 221.615 82.55 0))
+    (property "Footprint" "TestPoint:TestPoint_Pad_D1.5mm" (id 2) (at 226.695 90.805 0)
+      (effects (font (size 1.27 1.27)) hide)
+    )
+    (property "Datasheet" "~" (id 3) (at 226.695 90.805 0)
+      (effects (font (size 1.27 1.27)) hide)
+    )
+    (pin "1")
   )
   (symbol (lib_id "Device:R_Small") (at 201.93 117.475 0) (unit 1)
@@
       (effects (font (size 1.27 1.27)) hide)
     )
+    (pin "1")
+  )
+  (symbol (lib_id "Connector:TestPoint") (at 221.615 93.345 180) (unit 1)
+    (in_bom no) (on_board yes)
+    (property "Reference" "TP302" (id 0) (at 221.615 99.06 0))
+    (property "Value" "U1TX" (id 1) (at 221.615 101.6 0))
+    (property "Footprint" "TestPoint:TestPoint_Pad_D1.5mm" (id 2) (at 216.535 93.345 0)
+      (effects (font (size 1.27 1.27)) hide)
+    )
+    (property "Datasheet" "~" (id 3) (at 216.535 93.345 0)
+      (effects (font (size 1.27 1.27)) hide)
+    )

Commit message: Updated uart
Changed lines of the file:
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@@
   (junction (at 221.615 90.805) (diameter 0) (color 0 0 0 0)
   )
+  (junction (at 173.99 66.04) (diameter 0) (color 0 0 0 0)
+  )
   (junction (at 105.41 66.04) (diameter 0) (color 0 0 0 0)
   )
+  (junction (at 173.99 83.185) (diameter 0) (color 0 0 0 0)
+  )
   (junction (at 138.43 66.04) (diameter 0) (color 0 0 0 0)
   )
@@
   )
   (junction (at 127.635 66.04) (diameter 0) (color 0 0 0 0)
-  )
-  (junction (at 171.45 66.04) (diameter 0) (color 0 0 0 0)
   )
   (no_connect (at 184.15 103.505))
@@
     (stroke (width 0) (type default) (color 0 0 0 0))
   )
+  (wire (pts (xy 161.29 66.04) (xy 173.99 66.04))
+    (stroke (width 0) (type default) (color 0 0 0 0))
+  )
   (wire (pts (xy 86.36 66.04) (xy 105.41 66.04))
     (stroke (width 0) (type default) (color 0 0 0 0))
@@
     (stroke (width 0) (type default) (color 0 0 0 0))
   )
-  (wire (pts (xy 171.45 83.185) (xy 171.45 66.04))
+  (wire (pts (xy 173.99 83.185) (xy 173.99 66.04))
     (stroke (width 0) (type default) (color 0 0 0 0))
   )
@@
     (stroke (width 0) (type default) (color 0 0 0 0))
   )
-  (wire (pts (xy 161.29 66.04) (xy 171.45 66.04))
-    (stroke (width 0) (type default) (color 0 0 0 0))
-  )
   (wire (pts (xy 152.4 128.905) (xy 158.75 128.905))
     (stroke (width 0) (type default) (color 0 0 0 0))
@@
     (stroke (width 0) (type default) (color 0 0 0 0))
   )
-  (wire (pts (xy 184.785 66.04) (xy 171.45 66.04))
-    (stroke (width 0) (type default) (color 0 0 0 0))
-  )
+  (wire (pts (xy 184.785 66.04) (xy 173.99 66.04))
+    (stroke (width 0) (type default) (color 0 0 0 0))
+  )
