File: node_pcb/orion_pcb/POWER_CONNECTORS.kicad_sch (KiCad schematic)
At the start: 6 parts, among them J401 Conn_02x05_Odd_Even, J402 Conn_01x02, J403 Conn_01x04, Q401 PJA3405

Commit message: Partial layout with max3232. To change to max3225
Parts:
- removed D401: SMBJ3V3-E3/5B, Diode_SMD:D_SMB, symbol 0_power_protection:SMBJ3V3-E3-5B
- removed J403: Conn_01x04, symbol Connector_Generic:Conn_01x04
- J401: value Conn_02x05_Odd_Even -> 02x05 2.54mm boxed header; footprint (none) -> 0_connectors:302-S101; Digikey ref (none) -> ED1543-ND; Manufacturer ref (none) -> 302-S101
- J402: value Conn_01x02 -> Terminal block 2.54 mm; footprint (none) -> TerminalBlock_Phoenix:TerminalBlock_Phoenix_MPT-0,5-2-2.54_1x02_P2.54mm_Horizontal; Digikey ref (none) -> 277-1273-ND; Manufacturer ref (none) -> 1725656
Connections:
- net 3V3_RAW: now reaches F401.2, J402.2 (Pin_2)
Other:
- note removed: "ESP32 Connector"
- moved on the sheet: F401

Commit message: updated paths
Connections:
- net 3V3_RAW: now also J402.1 (Pin_1); no longer J402.2 (Pin_2)
- net GND: now also J402.2 (Pin_2); no longer J402.1 (Pin_1)
Changed lines of the file:
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@@
     (pin "1")
   )
-  (symbol (lib_id "Connector_Generic:Conn_01x02") (at 68.58 43.18 0) (mirror x) (unit 1)
+  (symbol (lib_id "Connector_Generic:Conn_01x02") (at 68.58 40.64 0) (unit 1)
     (in_bom yes) (on_board yes)
-    (property "Reference" "J402" (id 0) (at 69.85 46.99 0)
+    (property "Reference" "J402" (id 0) (at 69.85 46.355 0)
       (effects (font (size 1.27 1.27)) (justify right))
     )
-    (property "Value" "Terminal block 2.54 mm" (id 1) (at 69.85 49.53 0)
+    (property "Value" "Terminal block 2.54 mm" (id 1) (at 69.85 48.26 0)
       (effects (font (size 1.27 1.27)) (justify right))
     )
-    (property "Footprint" "TerminalBlock_Phoenix:TerminalBlock_Phoenix_MPT-0,5-2-2.54_1x02_P2.54mm_Horizontal" (id 2) (at 68.58 43.18 0)
+    (property "Footprint" "TerminalBlock_Phoenix:TerminalBlock_Phoenix_MPT-0,5-2-2.54_1x02_P2.54mm_Horizontal" (id 2) (at 68.58 40.64 0)
       (effects (font (size 1.27 1.27)) hide)
     )
-    (property "Datasheet" "https://www.phoenixcontact.com/product/pdf/MTcyNTY1Ng?_realm=us&_locale=en-US&blocks=commercial-data%2Ctechnical-data%2Cdrawings%2Capprovals%2Cclassifications%2Cenvironmental-compliance-data%2Call-accessories" (id 3) (at 68.58 43.18 0)
+    (property "Datasheet" "https://www.phoenixcontact.com/product/pdf/MTcyNTY1Ng?_realm=us&_locale=en-US&blocks=commercial-data%2Ctechnical-data%2Cdrawings%2Capprovals%2Cclassifications%2Cenvironmental-compliance-data%2Call-accessories" (id 3) (at 68.58 40.64 0)
       (effects (font (size 1.27 1.27)) hide)
     )
-    (property "Manufacturer ref" "1725656" (id 5) (at 68.58 43.18 0)
+    (property "Manufacturer ref" "1725656" (id 5) (at 68.58 40.64 0)
       (effects (font (size 1.27 1.27)) hide)
     )
-    (property "Digikey ref" "277-1273-ND" (id 4) (at 68.58 43.18 0)
+    (property "Digikey ref" "277-1273-ND" (id 4) (at 68.58 40.64 0)
       (effects (font (size 1.27 1.27)) hide)
     )

Commit message: Added logos
Connections:
- net VIN is gone; now on net +5V: J401.7 (Pin_7), J401.8 (Pin_8)
- net +5V: no longer J401.5 (Pin_5), J401.6 (Pin_6)
- net GND: now also J401.5 (Pin_5), J401.6 (Pin_6)
Changed lines of the file:
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@@
     (comment 2 "Author: Vincent Nguyen")
   )
+  (junction (at 64.77 109.22) (diameter 0) (color 0 0 0 0)
+  )
   (junction (at 45.72 113.665) (diameter 0) (color 0 0 0 0)
+  )
+  (junction (at 45.72 109.22) (diameter 0) (color 0 0 0 0)
   )
   (no_connect (at 62.23 99.06))
@@
     (stroke (width 0) (type default) (color 0 0 0 0))
   )
-  (wire (pts (xy 32.385 97.155) (xy 32.385 101.6))
-    (stroke (width 0) (type default) (color 0 0 0 0))
-  )
   (polyline (pts (xy 194.945 64.77) (xy 194.945 14.605))
     (stroke (width 0) (type default) (color 0 0 0 0))
@@
     (stroke (width 0) (type default) (color 0 0 0 0))
   )
+  (wire (pts (xy 45.72 104.14) (xy 49.53 104.14))
+    (stroke (width 0) (type default) (color 0 0 0 0))
+  )
   (wire (pts (xy 19.685 106.68) (xy 49.53 106.68))
     (stroke (width 0) (type default) (color 0 0 0 0))
@@
     (stroke (width 0) (type default) (color 0 0 0 0))
   )
-  (wire (pts (xy 75.565 97.79) (xy 75.565 104.14))
-    (stroke (width 0) (type default) (color 0 0 0 0))
-  )
-  (wire (pts (xy 62.23 101.6) (xy 68.58 101.6))
+  (wire (pts (xy 75.565 95.25) (xy 75.565 101.6))
     (stroke (width 0) (type default) (color 0 0 0 0))
   )
@@
     (stroke (width 0) (type default) (color 0 0 0 0))
   )
+  (wire (pts (xy 64.77 104.14) (xy 62.23 104.14))
+    (stroke (width 0) (type default) (color 0 0 0 0))
+  )
   (wire (pts (xy 46.99 99.06) (xy 49.53 99.06))
     (stroke (width 0) (type default) (color 0 0 0 0))
@@
     (stroke (width 0) (type default) (color 0 0 0 0))
   )
-  (wire (pts (xy 75.565 104.14) (xy 62.23 104.14))
+  (wire (pts (xy 75.565 101.6) (xy 62.23 101.6))
     (stroke (width 0) (type default) (color 0 0 0 0))
   )
@@
     (stroke (width 0) (type default) (color 0 0 0 0))
   )
+  (wire (pts (xy 64.77 109.22) (xy 64.77 104.14))
+    (stroke (width 0) (type default) (color 0 0 0 0))
+  )
   (polyline (pts (xy 80.645 14.605) (xy 194.945 14.605))
     (stroke (width 0) (type default) (color 0 0 0 0))
@@
     (stroke (width 0) (type default) (color 0 0 0 0))
   )
-  (wire (pts (xy 68.58 97.79) (xy 68.58 101.6))
+  (wire (pts (xy 45.72 109.22) (xy 45.72 104.14))
     (stroke (width 0) (type default) (color 0 0 0 0))
   )
@@
     (stroke (width 0) (type default) (color 0 0 0 0))
   )
-  (wire (pts (xy 26.035 104.14) (xy 49.53 104.14))
-    (stroke (width 0) (type default) (color 0 0 0 0))
-  )
-  (wire (pts (xy 32.385 101.6) (xy 49.53 101.6))
+  (wire (pts (xy 26.035 101.6) (xy 49.53 101.6))
     (stroke (width 0) (type default) (color 0 0 0 0))
   )
@@
     (stroke (width 0) (type default) (color 0 0 0 0))
   )
-  (wire (pts (xy 26.035 97.155) (xy 26.035 104.14))
+  (wire (pts (xy 26.035 94.615) (xy 26.035 101.6))
     (stroke (width 0) (type default) (color 0 0 0 0))
   )
@@
     (effects (font (size 1.27 1.27)) (justify right bottom))
   )
-  (symbol (lib_id "power:+5V") (at 26.035 97.155 0) (unit 1)
-    (in_bom yes) (on_board yes) (fields_autoplaced)
-    (property "Reference" "#PWR0402" (id 0) (at 26.035 100.965 0)
-      (effects (font (size 1.27 1.27)) hide)
-    )
-    (property "Value" "+5V" (id 1) (at 26.035 92.075 0))
-    (property "Footprint" "" (id 2) (at 26.035 97.155 0)
-      (effects (font (size 1.27 1.27)) hide)
-    )
-    (property "Datasheet" "" (id 3) (at 26.035 97.155 0)
+  (symbol (lib_id "power:+5V") (at 26.035 94.615 0) (unit 1)
+    (in_bom yes) (on_board yes) (fields_autoplaced)
+    (property "Reference" "#PWR0402" (id 0) (at 26.035 98.425 0)
+      (effects (font (size 1.27 1.27)) hide)
+    )
+    (property "Value" "+5V" (id 1) (at 26.035 89.535 0))
+    (property "Footprint" "" (id 2) (at 26.035 94.615 0)
+      (effects (font (size 1.27 1.27)) hide)
+    )
+    (property "Datasheet" "" (id 3) (at 26.035 94.615 0)
       (effects (font (size 1.27 1.27)) hide)
     )
@@
     (pin "1")
   )
-  (symbol (lib_id "0_power_symbols:VIN") (at 32.385 97.155 0) (unit 1)
-    (in_bom no) (on_board no) (fields_autoplaced)
-    (property "Reference" "#PWR0403" (id 0) (at 36.195 97.79 0)
-      (effects (font (size 1.27 1.27)) hide)
-    )
-    (property "Value" "VIN" (id 1) (at 32.385 92.075 0))
-    (property "Footprint" "" (id 2) (at 32.385 97.155 0)
-      (effects (font (size 1.27 1.27)) hide)
-    )
-    (property "Datasheet" "" (id 3) (at 32.385 97.155 0)
-      (effects (font (size 1.27 1.27)) hide)
-    )
-    (pin "1")
-  )
   (symbol (lib_id "power:GND") (at 45.72 116.205 0) (unit 1)
     (in_bom yes) (on_board yes) (fields_autoplaced)
@@
     (pin "2")
     (pin "3")
-  )
-  (symbol (lib_id "0_power_symbols:VIN") (at 68.58 97.79 0) (unit 1)
-    (in_bom no) (on_board no) (fields_autoplaced)
-    (property "Reference" "#PWR0407" (id 0) (at 72.39 98.425 0)
-      (effects (font (size 1.27 1.27)) hide)
-    )
-    (property "Value" "VIN" (id 1) (at 68.58 92.71 0))
-    (property "Footprint" "" (id 2) (at 68.58 97.79 0)
-      (effects (font (size 1.27 1.27)) hide)
-    )
-    (property "Datasheet" "" (id 3) (at 68.58 97.79 0)
-      (effects (font (size 1.27 1.27)) hide)
-    )
-    (pin "1")
   )
   (symbol (lib_id "power:+3.3V") (at 85.725 40.64 0) (unit 1)
@@
   )
   (symbol (lib_id "power:+3.3V") (at 82.55 97.79 0) (unit 1)
-    (in_bom yes) (on_board yes) (fields_autoplaced)
+    (in_bom yes) (on_board yes)
     (property "Reference" "#PWR0409" (id 0) (at 82.55 101.6 0)
       (effects (font (size 1.27 1.27)) hide)
     )
-    (property "Value" "+3.3V" (id 1) (at 82.55 92.71 0))
+    (property "Value" "+3.3V" (id 1) (at 82.55 90.17 0))
     (property "Footprint" "" (id 2) (at 82.55 97.79 0)
       (effects (font (size 1.27 1.27)) hide)
@@
     (pin "1")
   )
-  (symbol (lib_id "power:+5V") (at 75.565 97.79 0) (unit 1)
-    (in_bom yes) (on_board yes) (fields_autoplaced)
-    (property "Reference" "#PWR0408" (id 0) (at 75.565 101.6 0)
-      (effects (font (size 1.27 1.27)) hide)
-    )
-    (property "Value" "+5V" (id 1) (at 75.565 92.71 0))
-    (property "Footprint" "" (id 2) (at 75.565 97.79 0)
-      (effects (font (size 1.27 1.27)) hide)
-    )
-    (property "Datasheet" "" (id 3) (at 75.565 97.79 0)
-      (effects (font (size 1.27 1.27)) hide)
-    )
+  (symbol (lib_id "power:+5V") (at 75.565 95.25 0) (unit 1)
+    (in_bom yes) (on_board yes) (fields_autoplaced)
+    (property "Reference" "#PWR0408" (id 0) (at 75.565 99.06 0)
+      (effects (font (size 1.27 1.27)) hide)
+    )
+    (property "Value" "+5V" (id 1) (at 75.565 90.17 0))
+    (property "Footprint" "" (id 2) (at 75.565 95.25 0)
+      (effects (font (size 1.27 1.27)) hide)
+    )
+    (property "Datasheet" "" (id 3) (at 75.565 95.25 0)
+      (effects (font (size 1.27 1.27)) hide)
+    )

Commit message: Updated values/bom
Parts:
- Q401: Digikey ref (none) -> 3757-PJA3405_R1_00001CT-ND; Manufacturer ref (none) -> PJA3405_R1_00001
Changed lines of the file:
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@@
     (pin "9")
+  )
+  (symbol (lib_id "0_transistor:PJA3405") (at 104.14 46.99 270) (unit 1)
+    (in_bom yes) (on_board yes) (fields_autoplaced)
+    (property "Reference" "Q401" (id 0) (at 104.14 53.34 90))
+    (property "Value" "PJA3405" (id 1) (at 104.14 55.88 90))
+    (property "Footprint" "Package_TO_SOT_SMD:SOT-23" (id 2) (at 104.14 48.895 0)
+      (effects (font (size 1.27 1.27)) hide)
+    )
+    (property "Datasheet" "https://www.panjit.com.tw/upload/datasheet/PJA3405.pdf" (id 3) (at 104.14 48.895 0)
+      (effects (font (size 1.27 1.27)) hide)
+    )
+    (property "Manufacturer ref" "PJA3405_R1_00001" (id 4) (at 104.14 46.99 90)
+      (effects (font (size 1.27 1.27)) hide)
+    )
+    (property "Digikey ref" "3757-PJA3405_R1_00001CT-ND" (id 5) (at 104.14 46.99 90)
+      (effects (font (size 1.27 1.27)) hide)
+    )
+    (pin "1")
+    (pin "2")
+    (pin "3")
   )
   (symbol (lib_id "power:+3.3V") (at 36.195 31.75 0) (unit 1)
@@
     (pin "1")
   )
-  (symbol (lib_id "0_transistor:PJA3405") (at 104.14 46.99 270) (unit 1)
-    (in_bom yes) (on_board yes) (fields_autoplaced)
-    (property "Reference" "Q401" (id 0) (at 104.14 53.34 90))
-    (property "Value" "PJA3405" (id 1) (at 104.14 55.88 90))
-    (property "Footprint" "Package_TO_SOT_SMD:SOT-23" (id 2) (at 104.14 48.895 0)
-      (effects (font (size 1.27 1.27)) hide)
-    )
-    (property "Datasheet" "https://www.panjit.com.tw/upload/datasheet/PJA3405.pdf" (id 3) (at 104.14 48.895 0)
-      (effects (font (size 1.27 1.27)) hide)
-    )
-    (pin "1")
-    (pin "2")
-    (pin "3")
-  )
   (symbol (lib_id "power:+3.3V") (at 85.725 40.64 0) (unit 1)

Commit message: Added orion rev2 (no teardrops/rounded traces)
Parts:
- removed F401: 0805L150SLYR, Fuse:Fuse_0805_2012Metric, symbol Device:Polyfuse_Small
- removed J402: Terminal block 2.54 mm, TerminalBlock_Phoenix:TerminalBlock_Phoenix_MPT-0,5-2-2.54_1x02_P2.54mm_Horizontal, symbol Connector_Generic:Conn_01x02
- removed Q401: PJA3405, Package_TO_SOT_SMD:SOT-23, symbol 0_transistor:PJA3405
- added JP401: BYPASS_3V3, 0_various:Jumper_wide, symbol Jumper:Jumper_2_Open
- added JP402: BYPASS_5V, 0_various:Jumper_wide, symbol Jumper:Jumper_2_Open
- added R401, R402: 100k, Resistor_SMD:R_0603_1608Metric, symbol Device:R_Small
- added R403: 10k, Resistor_SMD:R_0603_1608Metric, symbol Device:R_Small
- added U401, U402: TPS2116DRLR, 0_mux:TPS2116DRLR, symbol 0_mux:TPS2116DRLR
Connections:
- net +3.3V: now also JP401.2 (B), R403.2, U401.2 (VOUT), U401.7 (VOUT); no longer J401.3 (Pin_3), J401.4 (Pin_4)
- net +5V: now also JP402.2 (B), U402.2 (VOUT), U402.7 (VOUT); no longer J401.7 (Pin_7), J401.8 (Pin_8)
- net GND: now also R401.1, R402.1, U401.1 (GND), U402.1 (GND)
- net VIO: now also U401.6 (VIN2)
- new net +3.3V_EXT: J401.3 (Pin_3), J401.4 (Pin_4), JP401.1 (A), R401.2, U401.3 (VIN1), U401.4 (PR1), U401.5 (MODE)
- new net +5V_EXT: J401.7 (Pin_7), J401.8 (Pin_8), JP402.1 (A), R402.2, U402.3 (VIN1), U402.4 (PR1), U402.5 (MODE)
- new net 5V_STATUS: R403.1, U402.8 (ST)
- new net VBUS_REV: U402.6 (VIN2)
- no-connect marks 1 -> 2
Other:
- note added: "Switching converter connector"
- note removed: "Diode forward voltage VDS = 1.2 V (VSD = -1.2 V) 1) External power is not connected (PGOOD2 = 0 V) 1a) USB is connected (VIO = 3.3 V) Initially: VS = VIO - VDS = 3.3 V - 1.2 V = 2.1 V VGS = VG - VS = 0 V - 2.1 V = -2.1 V <= VGS(th) -> CLOSED Then: CLOSED -> VS = VD = VIO = 3.3 V VGS = VG - VS = 0 V - 3.3 V < VGS(th) -> stays CLOSED 1b) USB is disconnected (VIO = 0 V) No voltages, everything is at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"
- note removed: "Raw power input"
- note removed: "Voltage regulator connector"
