File: node_pcb/orion_pcb/NODE_TO_HATS.kicad_sch (KiCad schematic)
At the start: 1 part

Commit message: Power and ESP32 moved to daugtherboards
Parts:
- gave numbers to parts that had none: 1
Other:
- removed sheet Hat connector circuit
- added sheet Hat connector circuit3 (HAT_CONNECTOR.kicad_sch)
- note added: "10"
- note added: "11"
- note added: "12"
- note added: "9"
- company: (none) -> EPFL Xplore
- title: (none) -> Hat Connectors and Delocalized Connectors
Changed lines of the file:
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@@
 (kicad_sch (version 20211123) (generator eeschema)
   (paper "A5")
+  (title_block
+    (title "Hat Connectors and Delocalized Connectors")
+    (company "EPFL Xplore")
+    (comment 2 "Author: Vincent Nguyen")
+  )
   (junction (at 41.91 20.955) (diameter 0) (color 0 0 0 0)
   )
@@
   (wire (pts (xy 124.46 26.67) (xy 144.78 26.67))
     (stroke (width 0) (type default) (color 0 0 0 0))
+  )
+  (text "9" (at 85.09 54.61 180)
+    (effects (font (size 2.54 2.54) bold) (justify right bottom))
+  )
+  (text "12" (at 165.1 99.06 180)
+    (effects (font (size 2.54 2.54) bold) (justify right bottom))
+  )
+  (text "10" (at 165.1 53.975 180)
+    (effects (font (size 2.54 2.54) bold) (justify right bottom))
+  )
+  (text "11" (at 85.09 99.06 180)
+    (effects (font (size 2.54 2.54) bold) (justify right bottom))
   )
   (text "Due to lack of space,\nSPI4, I2C4 and TIM2 will\nonly be accessible with \ndelocalized connectors."
@@
   (symbol (lib_id "Connector_Generic:Conn_01x03") (at 62.865 119.38 0) (unit 1)
     (in_bom yes) (on_board yes) (fields_autoplaced)
-    (property "Reference" "J?" (id 0) (at 66.04 118.1099 0)
+    (property "Reference" "J801" (id 0) (at 66.04 118.1099 0)
       (effects (font (size 1.27 1.27)) (justify left))
     )
@@
     (stroke (width 0.1524) (type solid) (color 0 0 0 0))
     (fill (color 100 255 100 1.0000))
-    (property "Sheet name" "Hat connector circuit2" (id 0) (at 64.77 60.8834 0)
+    (property "Sheet name" "Hat connector circuit3" (id 0) (at 64.77 60.8834 0)
       (effects (font (size 1.27 1.27)) (justify left bottom))
     )
@@
     (stroke (width 0.1524) (type solid) (color 0 0 0 0))
     (fill (color 100 255 100 1.0000))
-    (property "Sheet name" "Hat connector circuit" (id 0) (at 64.77 16.4334 0)
+    (property "Sheet name" "Hat connector circuit1" (id 0) (at 64.77 16.4334 0)
       (effects (font (size 1.27 1.27)) (justify left bottom))
     )
@@
     (stroke (width 0.1524) (type solid) (color 0 0 0 0))
     (fill (color 100 255 100 1.0000))
-    (property "Sheet name" "Hat connector circuit1" (id 0) (at 144.78 15.7984 0)
+    (property "Sheet name" "Hat connector circuit2" (id 0) (at 144.78 15.7984 0)
       (effects (font (size 1.27 1.27)) (justify left bottom))
     )

Commit message: Added titles and plots
Other:
- note added: "Node to Hat connectors"
Changed lines of the file:
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@@
     (effects (font (size 1.27 1.27)) (justify left bottom))
+  )
+  (text "Node to Hat connectors" (at 13.335 17.145 0)
+    (effects (font (size 2.54 2.54) bold) (justify left bottom))
   )
   (label "I2C4_SCL" (at 137.795 76.835 180)

Commit message: Partial layout with max3232. To change to max3225
Parts:
- removed J801: 01x03 2.54 mm, Connector_PinHeader_2.54mm:PinHeader_1x03_P2.54mm_Vertical, symbol Connector_Generic:Conn_01x03
Other:
- removed sheet Hat connector delocalized
- note removed: "12"
- note removed: "Due to lack of space, SPI4, I2C4 and TIM2 will only be accessible with delocalized connectors."

Commit message: Replaced timer 3 with timer 8 (timer 8 is an advanced control timer, dead time might be useful for h-bridge)
Changed lines of the file:
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@@
     (effects (font (size 2.54 2.54) bold) (justify left bottom))
   )
-  (label "TIM3_CH2" (at 57.785 42.545 180)
+  (label "TIM8_CH2" (at 57.785 42.545 180)
     (effects (font (size 1.27 1.27)) (justify right bottom))
   )
@@
     (effects (font (size 1.27 1.27)) (justify right bottom))
   )
-  (label "TIM3_CH3" (at 57.785 45.085 180)
+  (label "TIM8_CH3" (at 57.785 45.085 180)
     (effects (font (size 1.27 1.27)) (justify right bottom))
   )
@@
     (effects (font (size 1.27 1.27)) (justify right bottom))
   )
-  (label "TIM3_CH1" (at 57.785 40.005 180)
+  (label "TIM8_CH1" (at 57.785 40.005 180)
     (effects (font (size 1.27 1.27)) (justify right bottom))
   )

Commit message: Broke out I2C4 instead of GPIOs on top left hat to support concurrent I2C sensors (easier for sensor fusion)
Changed lines of the file:
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@@
     (effects (font (size 1.27 1.27)) (justify right bottom))
   )
-  (label "PE3" (at 57.785 94.615 180)
+  (label "I2C4_SCL" (at 57.785 94.615 180)
     (effects (font (size 1.27 1.27)) (justify right bottom))
   )
@@
     (effects (font (size 1.27 1.27)) (justify right bottom))
   )
-  (label "PE2" (at 57.785 97.155 180)
+  (label "I2C4_SDA" (at 57.785 97.155 180)
     (effects (font (size 1.27 1.27)) (justify right bottom))
   )

Commit message: Added support for CAN and RS485 (hats should be designed for top right and bottom left)
Changed lines of the file:
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@@
     (effects (font (size 1.27 1.27)) (justify right bottom))
   )
-  (label "UART4_TX" (at 129.54 63.5 180)
+  (label "USART2_TX" (at 129.54 63.5 180)
     (effects (font (size 1.27 1.27)) (justify right bottom))
   )
@@
     (effects (font (size 1.27 1.27)) (justify right bottom))
   )
-  (label "TIM4_CH4" (at 129.54 60.96 180)
+  (label "USART2_RTS" (at 129.54 60.96 180)
     (effects (font (size 1.27 1.27)) (justify right bottom))
   )
@@
     (effects (font (size 1.27 1.27)) (justify right bottom))
   )
-  (label "TIM1_CH4" (at 50.165 66.04 180)
+  (label "FDCAN1_RX" (at 50.165 66.04 180)
     (effects (font (size 1.27 1.27)) (justify right bottom))
   )
@@
     (effects (font (size 1.27 1.27)) (justify right bottom))
   )
-  (label "TIM1_CH3" (at 50.165 63.5 180)
+  (label "FDCAN1_TX" (at 50.165 63.5 180)
     (effects (font (size 1.27 1.27)) (justify right bottom))
   )
@@
     (effects (font (size 1.27 1.27)) (justify right bottom))
   )
-  (label "UART4_RX" (at 129.54 66.04 180)
+  (label "USART2_RX" (at 129.54 66.04 180)
     (effects (font (size 1.27 1.27)) (justify right bottom))
   )

Commit message: Changed order of USART2 RX, TX, RTS pins on hat for easier routing of RS485 transceiver
Changed lines of the file:
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@@
     (effects (font (size 1.27 1.27)) (justify right bottom))
   )
-  (label "USART2_TX" (at 129.54 63.5 180)
+  (label "USART2_TX" (at 129.54 66.04 180)
     (effects (font (size 1.27 1.27)) (justify right bottom))
   )
@@
     (effects (font (size 1.27 1.27)) (justify right bottom))
   )
-  (label "USART2_RTS" (at 129.54 60.96 180)
+  (label "USART2_RTS" (at 129.54 63.5 180)
     (effects (font (size 1.27 1.27)) (justify right bottom))
   )
@@
     (effects (font (size 1.27 1.27)) (justify right bottom))
   )
-  (label "USART2_RX" (at 129.54 66.04 180)
+  (label "USART2_RX" (at 129.54 60.96 180)
     (effects (font (size 1.27 1.27)) (justify right bottom))
   )
