File: node_pcb/orion_pcb/FLASH.kicad_sch (KiCad schematic)
At the start: 2 parts, among them U601 W25Q128JVS

Commit message: Added titles and plots
Other:
- note added: "Quad-SPI external flash memory"
- moved on the sheet: C601, U601

Commit message: Partial layout with max3232. To change to max3225
Parts:
- C601: footprint (none) -> Capacitor_SMD:C_0603_1608Metric
Changed lines of the file:
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@@
       (effects (font (size 1.27 1.27)) (justify left))
     )
-    (property "Footprint" "" (id 2) (at 111.125 51.435 0)
+    (property "Footprint" "Capacitor_SMD:C_0603_1608Metric" (id 2) (at 111.125 51.435 0)
       (effects (font (size 1.27 1.27)) hide)
     )

Commit message: Added pullup resistor on qspi N_CS
Parts:
- added R601: 4k7, Resistor_SMD:R_0402_1005Metric, symbol Device:R_Small
Connections:
- net +3.3V: now also R601.1
- net QUADSPI_BK2_NCS: now also R601.2
Changed lines of the file:
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@@
     (comment 2 "Author: Vincent Nguyen")
   )
+  (junction (at 111.125 46.99) (diameter 0) (color 0 0 0 0)
+  )
+  (junction (at 97.155 67.945) (diameter 0) (color 0 0 0 0)
+  )
   (junction (at 122.555 46.99) (diameter 0) (color 0 0 0 0)
   )
-  (junction (at 62.865 68.58) (diameter 0) (color 0 0 0 0)
-  )
-  (bus_entry (at 65.405 77.47) (size -2.54 -2.54)
-    (stroke (width 0) (type default) (color 0 0 0 0))
-  )
-  (bus_entry (at 65.405 69.85) (size -2.54 -2.54)
-    (stroke (width 0) (type default) (color 0 0 0 0))
-  )
-  (bus_entry (at 65.405 72.39) (size -2.54 -2.54)
-    (stroke (width 0) (type default) (color 0 0 0 0))
-  )
-  (bus_entry (at 65.405 67.31) (size -2.54 -2.54)
-    (stroke (width 0) (type default) (color 0 0 0 0))
-  )
-  (bus_entry (at 65.405 64.77) (size -2.54 -2.54)
-    (stroke (width 0) (type default) (color 0 0 0 0))
-  )
-  (bus_entry (at 65.405 74.93) (size -2.54 -2.54)
-    (stroke (width 0) (type default) (color 0 0 0 0))
-  )
-  (wire (pts (xy 84.455 77.47) (xy 65.405 77.47))
+  (junction (at 38.1 68.58) (diameter 0) (color 0 0 0 0)
+  )
+  (bus_entry (at 40.64 77.47) (size -2.54 -2.54)
+    (stroke (width 0) (type default) (color 0 0 0 0))
+  )
+  (bus_entry (at 40.64 69.85) (size -2.54 -2.54)
+    (stroke (width 0) (type default) (color 0 0 0 0))
+  )
+  (bus_entry (at 40.64 72.39) (size -2.54 -2.54)
+    (stroke (width 0) (type default) (color 0 0 0 0))
+  )
+  (bus_entry (at 40.64 67.31) (size -2.54 -2.54)
+    (stroke (width 0) (type default) (color 0 0 0 0))
+  )
+  (bus_entry (at 40.64 64.77) (size -2.54 -2.54)
+    (stroke (width 0) (type default) (color 0 0 0 0))
+  )
+  (bus_entry (at 40.64 74.93) (size -2.54 -2.54)
+    (stroke (width 0) (type default) (color 0 0 0 0))
+  )
+  (wire (pts (xy 59.69 77.47) (xy 40.64 77.47))
     (stroke (width 0) (type default) (color 0 0 0 0))
   )
@@
     (stroke (width 0) (type default) (color 0 0 0 0))
   )
-  (bus (pts (xy 62.865 68.58) (xy 62.865 69.85))
-    (stroke (width 0) (type default) (color 0 0 0 0))
-  )
-  (bus (pts (xy 62.865 64.77) (xy 62.865 67.31))
-    (stroke (width 0) (type default) (color 0 0 0 0))
-  )
-  (wire (pts (xy 84.455 72.39) (xy 65.405 72.39))
+  (bus (pts (xy 38.1 68.58) (xy 38.1 69.85))
+    (stroke (width 0) (type default) (color 0 0 0 0))
+  )
+  (bus (pts (xy 38.1 64.77) (xy 38.1 67.31))
+    (stroke (width 0) (type default) (color 0 0 0 0))
+  )
+  (wire (pts (xy 59.69 72.39) (xy 40.64 72.39))
     (stroke (width 0) (type default) (color 0 0 0 0))
   )
@@
     (stroke (width 0) (type default) (color 0 0 0 0))
   )
-  (wire (pts (xy 84.455 67.31) (xy 65.405 67.31))
+  (wire (pts (xy 97.155 67.945) (xy 109.855 67.945))
+    (stroke (width 0) (type default) (color 0 0 0 0))
+  )
+  (wire (pts (xy 59.69 67.31) (xy 40.64 67.31))
     (stroke (width 0) (type default) (color 0 0 0 0))
   )
@@
     (stroke (width 0) (type default) (color 0 0 0 0))
   )
-  (wire (pts (xy 84.455 69.85) (xy 65.405 69.85))
-    (stroke (width 0) (type default) (color 0 0 0 0))
-  )
-  (bus (pts (xy 62.865 67.31) (xy 62.865 68.58))
-    (stroke (width 0) (type default) (color 0 0 0 0))
-  )
-  (wire (pts (xy 107.95 73.025) (xy 109.855 73.025))
-    (stroke (width 0) (type default) (color 0 0 0 0))
-  )
-  (wire (pts (xy 84.455 64.77) (xy 65.405 64.77))
+  (wire (pts (xy 59.69 69.85) (xy 40.64 69.85))
+    (stroke (width 0) (type default) (color 0 0 0 0))
+  )
+  (bus (pts (xy 38.1 67.31) (xy 38.1 68.58))
+    (stroke (width 0) (type default) (color 0 0 0 0))
+  )
+  (wire (pts (xy 86.995 73.025) (xy 109.855 73.025))
+    (stroke (width 0) (type default) (color 0 0 0 0))
+  )
+  (wire (pts (xy 59.69 64.77) (xy 40.64 64.77))
     (stroke (width 0) (type default) (color 0 0 0 0))
   )
@@
     (stroke (width 0) (type default) (color 0 0 0 0))
   )
-  (bus (pts (xy 62.865 62.23) (xy 62.865 64.77))
-    (stroke (width 0) (type default) (color 0 0 0 0))
-  )
-  (bus (pts (xy 62.865 69.85) (xy 62.865 72.39))
+  (bus (pts (xy 38.1 62.23) (xy 38.1 64.77))
+    (stroke (width 0) (type default) (color 0 0 0 0))
+  )
+  (bus (pts (xy 38.1 69.85) (xy 38.1 72.39))
     (stroke (width 0) (type default) (color 0 0 0 0))
   )
@@
     (stroke (width 0) (type default) (color 0 0 0 0))
   )
-  (bus (pts (xy 62.865 68.58) (xy 60.325 68.58))
-    (stroke (width 0) (type default) (color 0 0 0 0))
-  )
-  (wire (pts (xy 107.95 67.945) (xy 109.855 67.945))
-    (stroke (width 0) (type default) (color 0 0 0 0))
-  )
-  (bus (pts (xy 62.865 72.39) (xy 62.865 74.93))
+  (wire (pts (xy 97.155 53.975) (xy 97.155 67.945))
+    (stroke (width 0) (type default) (color 0 0 0 0))
+  )
+  (bus (pts (xy 38.1 68.58) (xy 35.56 68.58))
+    (stroke (width 0) (type default) (color 0 0 0 0))
+  )
+  (wire (pts (xy 86.995 67.945) (xy 97.155 67.945))
+    (stroke (width 0) (type default) (color 0 0 0 0))
+  )
+  (bus (pts (xy 38.1 72.39) (xy 38.1 74.93))
+    (stroke (width 0) (type default) (color 0 0 0 0))
+  )
+  (wire (pts (xy 97.155 46.99) (xy 111.125 46.99))
     (stroke (width 0) (type default) (color 0 0 0 0))
   )
@@
     (stroke (width 0) (type default) (color 0 0 0 0))
   )
+  (wire (pts (xy 97.155 46.99) (xy 97.155 48.895))
+    (stroke (width 0) (type default) (color 0 0 0 0))
+  )
   (wire (pts (xy 122.555 80.645) (xy 122.555 83.185))
     (stroke (width 0) (type default) (color 0 0 0 0))
   )
-  (wire (pts (xy 84.455 74.93) (xy 65.405 74.93))
+  (wire (pts (xy 59.69 74.93) (xy 40.64 74.93))
     (stroke (width 0) (type default) (color 0 0 0 0))
   )
@@
     (effects (font (size 1.27 1.27)) (justify left bottom))
   )
-  (label "QUADSPI_BK2_IO3" (at 84.455 77.47 180)
-    (effects (font (size 1.27 1.27)) (justify right bottom))
-  )
-  (label "QUADSPI_BK2_IO2" (at 84.455 74.93 180)
-    (effects (font (size 1.27 1.27)) (justify right bottom))
-  )
-  (label "QUADSPI_BK2_NCS" (at 84.455 67.31 180)
+  (label "QUADSPI_BK2_IO3" (at 59.69 77.47 180)
+    (effects (font (size 1.27 1.27)) (justify right bottom))
+  )
+  (label "QUADSPI_BK2_IO2" (at 59.69 74.93 180)
+    (effects (font (size 1.27 1.27)) (justify right bottom))
+  )
+  (label "QUADSPI_BK2_NCS" (at 59.69 67.31 180)
     (effects (font (size 1.27 1.27)) (justify right bottom))
   )
@@
     (effects (font (size 1.27 1.27)) (justify left bottom))
   )
-  (label "QUADSPI_CLK" (at 84.455 64.77 180)
-    (effects (font (size 1.27 1.27)) (justify right bottom))
-  )
-  (label "QUADSPI_BK2_IO0" (at 84.455 69.85 180)
-    (effects (font (size 1.27 1.27)) (justify right bottom))
-  )
-  (label "QUADSPI_CLK" (at 107.95 73.025 180)
-    (effects (font (size 1.27 1.27)) (justify right bottom))
-  )
-  (label "QUADSPI_BK2_IO1" (at 84.455 72.39 180)
-    (effects (font (size 1.27 1.27)) (justify right bottom))
-  )
-  (label "QUADSPI_BK2_NCS" (at 107.95 67.945 180)
+  (label "QUADSPI_CLK" (at 59.69 64.77 180)
+    (effects (font (size 1.27 1.27)) (justify right bottom))
+  )
+  (label "QUADSPI_BK2_IO0" (at 59.69 69.85 180)
+    (effects (font (size 1.27 1.27)) (justify right bottom))
+  )
+  (label "QUADSPI_CLK" (at 86.995 73.025 180)
+    (effects (font (size 1.27 1.27)) (justify right bottom))
+  )
+  (label "QUADSPI_BK2_IO1" (at 59.69 72.39 180)
+    (effects (font (size 1.27 1.27)) (justify right bottom))
+  )
+  (label "QUADSPI_BK2_NCS" (at 86.995 67.945 180)
     (effects (font (size 1.27 1.27)) (justify right bottom))
   )
@@
     (effects (font (size 1.27 1.27)) (justify left bottom))
   )
-  (hierarchical_label "{QUADSPI}" (shape bidirectional) (at 60.325 68.58 180)
+  (hierarchical_label "{QUADSPI}" (shape bidirectional) (at 35.56 68.58 180)
     (effects (font (size 1.27 1.27)) (justify right))
   )
@@
     (pin "1")
   )
+  (symbol (lib_id "Device:R_Small") (at 97.155 51.435 0) (unit 1)
+    (in_bom yes) (on_board yes) (fields_autoplaced)
+    (property "Reference" "R601" (id 0) (at 99.06 50.1649 0)
+      (effects (font (size 1.27 1.27)) (justify left))
+    )
+    (property "Value" "4k7" (id 1) (at 99.06 52.7049 0)
+      (effects (font (size 1.27 1.27)) (justify left))
+    )
+    (property "Footprint" "Resistor_SMD:R_0402_1005Metric" (id 2) (at 97.155 51.435 0)
+      (effects (font (size 1.27 1.27)) hide)
+    )
+    (property "Datasheet" "~" (id 3) (at 97.155 51.435 0)
+      (effects (font (size 1.27 1.27)) hide)
+    )
+    (pin "1")
+    (pin "2")
+  )
   (symbol (lib_id "power:GND") (at 122.555 83.185 0) (unit 1)

Commit message: Updated values/bom
Parts:
- U601: Digikey ref (none) -> W25Q128JVSIQCT-ND; Manufacturer ref (none) -> W25Q128JVSIQ TR
Changed lines of the file:
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@@
+      (effects (font (size 1.27 1.27)) hide)
+    )
+    (property "Manufacturer ref" "W25Q128JVSIQ TR" (id 4) (at 122.555 70.485 0)
+      (effects (font (size 1.27 1.27)) hide)
+    )
+    (property "Digikey ref" "W25Q128JVSIQCT-ND" (id 5) (at 122.555 70.485 0)
       (effects (font (size 1.27 1.27)) hide)
     )

Commit message: Updated BOMs and added ST-LINK adapter
Parts:
- removed U601: W25Q128JVS, Package_SO:SOIC-8_5.23x5.23mm_P1.27mm, symbol Memory_Flash:W25Q128JVS
- added U601: IS25LP128F, Package_SO:SOIC-8_5.23x5.23mm_P1.27mm, symbol 0_memory_flash:IS25LP128F
Connections:
- net +3.3V: now also U601.8 (VCC)
- net GND: now also U601.4 (GND)
- net QUADSPI_BK2_IO0: now also U601.5 (DI(IO0))
- net QUADSPI_BK2_IO1: now also U601.2 (DO(IO1))
- net QUADSPI_BK2_IO2: now also U601.3 (IO2)
- net QUADSPI_BK2_IO3: now also U601.7 (IO3)
- net QUADSPI_BK2_NCS: now also U601.1 (~{CS})
- net QUADSPI_CLK: now also U601.6 (CLK)
Changed lines of the file:
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@@
     (pin "1")
+  )
+  (symbol (lib_id "0_memory_flash:IS25LP128F") (at 122.555 70.485 0) (unit 1)
+    (in_bom yes) (on_board yes) (fields_autoplaced)
+    (property "Reference" "U601" (id 0) (at 124.5744 57.785 0)
+      (effects (font (size 1.27 1.27)) (justify left))
+    )
+    (property "Value" "IS25LP128F" (id 1) (at 124.5744 60.325 0)
+      (effects (font (size 1.27 1.27)) (justify left))
+    )
+    (property "Footprint" "Package_SO:SOIC-8_5.23x5.23mm_P1.27mm" (id 2) (at 122.555 70.485 0)
+      (effects (font (size 1.27 1.27)) hide)
+    )
+    (property "Datasheet" "https://www.mouser.ch/datasheet/2/198/25LP_WP128F-1146765.pdf" (id 3) (at 122.555 70.485 0)
+      (effects (font (size 1.27 1.27)) hide)
+    )
+    (property "Manufacturer ref" "IS25LP128F-JBLE" (id 4) (at 122.555 70.485 0)
+      (effects (font (size 1.27 1.27)) hide)
+    )
+    (property "Mouser ref" "870-IS25LP128F-JBLE" (id 5) (at 122.555 70.485 0)
+      (effects (font (size 1.27 1.27)) hide)
+    )
+    (pin "1")
+    (pin "2")
+    (pin "3")
+    (pin "4")
+    (pin "5")
+    (pin "6")
+    (pin "7")
+    (pin "8")
   )
   (symbol (lib_id "power:+3.3V") (at 122.555 45.085 0) (unit 1)
@@
     (pin "2")
   )
-  (symbol (lib_id "Memory_Flash:W25Q128JVS") (at 122.555 70.485 0) (unit 1)
-    (in_bom yes) (on_board yes) (fields_autoplaced)
-    (property "Reference" "U601" (id 0) (at 124.5744 57.15 0)
-      (effects (font (size 1.27 1.27)) (justify left))
-    )
-    (property "Value" "W25Q128JVS" (id 1) (at 124.5744 59.69 0)
-      (effects (font (size 1.27 1.27)) (justify left))
-    )
-    (property "Footprint" "Package_SO:SOIC-8_5.23x5.23mm_P1.27mm" (id 2) (at 122.555 70.485 0)
-      (effects (font (size 1.27 1.27)) hide)
-    )
-    (property "Datasheet" "http://www.winbond.com/resource-files/w25q128jv_dtr%20revc%2003272018%20plus.pdf" (id 3) (at 122.555 70.485 0)
-      (effects (font (size 1.27 1.27)) hide)
-    )
-    (property "Manufacturer ref" "W25Q128JVSIQ TR" (id 4) (at 122.555 70.485 0)
-      (effects (font (size 1.27 1.27)) hide)
-    )
-    (property "Digikey ref" "W25Q128JVSIQCT-ND" (id 5) (at 122.555 70.485 0)
-      (effects (font (size 1.27 1.27)) hide)
-    )
-    (pin "1")
-    (pin "2")
-    (pin "3")
-    (pin "4")
-    (pin "5")
-    (pin "6")
-    (pin "7")
-    (pin "8")
-  )
 )
