File: can_controller_interface/can_controller_board.kicad_pcb (KiCad board)
At the start: 2 copper layers, 56 parts, among them J1 Analog I/O (X8), J10 Micro_USB (X13), J2 LSHM-140-02.5-L-DV-A-N-K-TR, J3 CAN 1 (X11), J4 CAN 2 (X12), J5 Power_supply (X1), J6 Motor (X3), J7 Hall Sensor (X4), J8 Encoder (X5), J9 Sensor (X6), SW1 450301014042-ND, SW2 219-8LPS, U1 MAX15462BATA+T, U2 SRV05-4, U3 MAX1486CUB+

Commit message: Changed footprint for the motor choke inductors
Parts:
- L2: footprint Inductor_SMD:L_1210_3225Metric_Pad1.42x2.65mm_HandSolder -> Inductor_SMD:L_Wuerth_WE-PD-Typ-LS_Handsoldering
- moved L1 83.1 mm to (101.8, 140.0), turned to 180 degrees
- moved J9 54.2 mm to (137.5, 79.2)
- moved L3 53.9 mm to (77.7, 122.9)
- moved TP1 51.8 mm to (107.5, 140.0)
- moved Cf2 50.3 mm to (104.3, 121.9)
- moved R3 49.9 mm to (117.8, 115.4)
- moved D3 48.9 mm to (169.5, 78.4)
- moved R7 48.9 mm to (178.3, 75.8)
- moved U3 48.9 mm to (170.7, 74.3)
- moved R8 48.9 mm to (178.3, 78.3)
- moved C6 48.9 mm to (168.6, 86.4)
- moved C7 48.9 mm to (176.6, 73.2)
- moved C8 48.9 mm to (168.6, 81.4)
- moved R4 48.9 mm to (172.9, 81.4)
- moved R5 48.9 mm to (174.0, 77.8)
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Connections:
- R1 pad 2: GND -> Net-(R1-Pad2)
- R2 pad 1: GND -> Net-(R1-Pad2)
- U1 pad 5: GND -> Net-(R1-Pad2)

Commit message: tracing started for can
Parts:
- removed J9: Sensor (X6), can_proj_footprints:MOLEX_5031541090
- added C10: 220pF, Capacitor_SMD:C_0603_1608Metric_Pad1.08x0.95mm_HandSolder, F.Cu at (384.9, 131.2)
- added C11: 0.1uF, Capacitor_SMD:C_0603_1608Metric_Pad1.08x0.95mm_HandSolder, F.Cu at (377.0, 139.4)
- added C12: 1uF, Capacitor_SMD:C_0603_1608Metric_Pad1.08x0.95mm_HandSolder, F.Cu at (383.5, 111.0)
- added C13: 1uF, Capacitor_SMD:C_0603_1608Metric_Pad1.08x0.95mm_HandSolder, F.Cu at (352.9, 138.5)
- added C14: EEH-ZA1V680XP, can_proj_footprints:CAP_EEHZA1V680XP, F.Cu at (349.4, 128.9)
- added C15: 10uF, Capacitor_SMD:C_0603_1608Metric_Pad1.08x0.95mm_HandSolder, F.Cu at (357.3, 138.5)
- added C16: 0.1uF, Capacitor_SMD:C_0603_1608Metric_Pad1.08x0.95mm_HandSolder, F.Cu at (368.2, 127.9)
- added C17: 220pF, Capacitor_SMD:C_0603_1608Metric_Pad1.08x0.95mm_HandSolder, F.Cu at (384.0, 74.3)
- added C18: 220pF, Capacitor_SMD:C_0603_1608Metric_Pad1.08x0.95mm_HandSolder, F.Cu at (392.0, 61.1)
- added C19: 0.1uF, Capacitor_SMD:C_0603_1608Metric_Pad1.08x0.95mm_HandSolder, F.Cu at (384.0, 69.3)
- added C20: 1uF, Capacitor_SMD:C_0603_1608Metric_Pad1.08x0.95mm_HandSolder, F.Cu at (383.5, 51.5)
- added C21: 1uF, Capacitor_SMD:C_0603_1608Metric_Pad1.08x0.95mm_HandSolder, F.Cu at (352.9, 79.0)
- added C22: EEH-ZA1V680XP, can_proj_footprints:CAP_EEHZA1V680XP, F.Cu at (349.4, 69.4)
- added C23: 10uF, Capacitor_SMD:C_0603_1608Metric_Pad1.08x0.95mm_HandSolder, F.Cu at (357.3, 79.0)
- added C24: 0.1uF, Capacitor_SMD:C_0603_1608Metric_Pad1.08x0.95mm_HandSolder, F.Cu at (368.2, 68.4)
- added C25: 220pF, Capacitor_SMD:C_0603_1608Metric_Pad1.08x0.95mm_HandSolder, B.Cu at (128.9, 77.2)
- added C26: 220pF, Capacitor_SMD:C_0603_1608Metric_Pad1.08x0.95mm_HandSolder, B.Cu at (120.9, 64.0)
- added C27: 0.1uF, Capacitor_SMD:C_0603_1608Metric_Pad1.08x0.95mm_HandSolder, B.Cu at (128.9, 72.1)
- added C28: 1uF, Capacitor_SMD:C_0603_1608Metric_Pad1.08x0.95mm_HandSolder, B.Cu at (138.2, 46.5)
- added C29: 1uF, Capacitor_SMD:C_0603_1608Metric_Pad1.08x0.95mm_HandSolder, B.Cu at (99.5, 68.2)
- added C30: EEH-ZA1V680XP, can_proj_footprints:CAP_EEHZA1V680XP, F.Cu at (72.5, 177.5)
- added C31: 10uF, Capacitor_SMD:C_0603_1608Metric_Pad1.08x0.95mm_HandSolder, B.Cu at (103.9, 68.2)
- added C32: 0.1uF, Capacitor_SMD:C_0603_1608Metric_Pad1.08x0.95mm_HandSolder, B.Cu at (114.8, 57.7)
- added C9: 220pF, Capacitor_SMD:C_0603_1608Metric_Pad1.08x0.95mm_HandSolder, F.Cu at (377.0, 144.4)
- added Cf10: 220pF, Capacitor_SMD:C_0603_1608Metric_Pad1.08x0.95mm_HandSolder, B.Cu at (130.2, 38.0)
- added Cf11: 220pF, Capacitor_SMD:C_0603_1608Metric_Pad1.08x0.95mm_HandSolder, B.Cu at (138.2, 44.0)
- added Cf12: 220pF, Capacitor_SMD:C_0603_1608Metric_Pad1.08x0.95mm_HandSolder, B.Cu at (109.0, 62.3)
- added Cf4: 220pF, Capacitor_SMD:C_0603_1608Metric_Pad1.08x0.95mm_HandSolder, F.Cu at (135.5, 120.0)
- added Cf5: 220pF, Capacitor_SMD:C_0603_1608Metric_Pad1.08x0.95mm_HandSolder, F.Cu at (383.5, 108.4)
- added Cf6: 220pF, Capacitor_SMD:C_0603_1608Metric_Pad1.08x0.95mm_HandSolder, F.Cu at (362.4, 132.5)
- added Cf7: 220pF, Capacitor_SMD:C_0603_1608Metric_Pad1.08x0.95mm_HandSolder, F.Cu at (391.5, 43.0)
- added Cf8: 220pF, Capacitor_SMD:C_0603_1608Metric_Pad1.08x0.95mm_HandSolder, F.Cu at (383.5, 49.0)
- added Cf9: 220pF, Capacitor_SMD:C_0603_1608Metric_Pad1.08x0.95mm_HandSolder, F.Cu at (362.4, 73.0)
- added Cs10: 470pF, Capacitor_SMD:C_0603_1608Metric_Pad1.08x0.95mm_HandSolder, B.Cu at (144.3, 49.9)
- added Cs11: 470pF, Capacitor_SMD:C_0603_1608Metric_Pad1.08x0.95mm_HandSolder, B.Cu at (96.7, 71.4)
- added Cs12: 470pF, Capacitor_SMD:C_0603_1608Metric_Pad1.08x0.95mm_HandSolder, B.Cu at (140.0, 49.9)
- added Cs4: 470pF, Capacitor_SMD:C_0603_1608Metric_Pad1.08x0.95mm_HandSolder, F.Cu at (137.5, 120.0)
- added Cs5: 470pF, Capacitor_SMD:C_0603_1608Metric_Pad1.08x0.95mm_HandSolder, F.Cu at (350.1, 141.7)
- added Cs6: 470pF, Capacitor_SMD:C_0603_1608Metric_Pad1.08x0.95mm_HandSolder, F.Cu at (381.7, 114.4)
- added Cs7: 470pF, Capacitor_SMD:C_0603_1608Metric_Pad1.08x0.95mm_HandSolder, F.Cu at (377.3, 54.9)
- added Cs8: 470pF, Capacitor_SMD:C_0603_1608Metric_Pad1.08x0.95mm_HandSolder, F.Cu at (350.1, 82.2)
- added Cs9: 470pF, Capacitor_SMD:C_0603_1608Metric_Pad1.08x0.95mm_HandSolder, F.Cu at (381.7, 54.9)
- added D10: TPD4E1B06DCKR, can_proj_footprints:TVS_TPD4E1B06DCKR, B.Cu at (128.0, 69.1)
- added D11: SMF30A, Diode_SMD:D_SOD-123, F.Cu at (69.1, 135.5)
- added D12: SMF30A, Diode_SMD:D_SOD-123, F.Cu at (69.1, 128.0)
- added D4: TPD4E1B06DCKR, can_proj_footprints:TVS_TPD4E1B06DCKR, F.Cu at (377.9, 136.4)
- added D5: SMF30A, Diode_SMD:D_SOD-123, F.Cu at (327.4, 148.7)
- added D6: SMF30A, Diode_SMD:D_SOD-123, F.Cu at (333.2, 148.7)
- added D7: TPD4E1B06DCKR, can_proj_footprints:TVS_TPD4E1B06DCKR, F.Cu at (384.9, 66.2)
- added D8: SMF30A, Diode_SMD:D_SOD-123, F.Cu at (327.4, 89.2)
- added D9: SMF30A, Diode_SMD:D_SOD-123, F.Cu at (333.2, 89.2)
- added F2: 0157010, Fuse:Fuseholder_Littelfuse_Nano2_157x, F.Cu at (346.3, 137.8)
- added F3: 0157010, Fuse:Fuseholder_Littelfuse_Nano2_157x, F.Cu at (346.3, 78.3)
- added F4: 0157010, Fuse:Fuseholder_Littelfuse_Nano2_157x, F.Cu at (71.6, 120.5)
- added H10: MountingHole_Pad, MountingHole:MountingHole_2.2mm_M2_Pad_Via, F.Cu at (378.4, 110.2)
- added H11: MountingHole_Pad, MountingHole:MountingHole_2.2mm_M2_Pad_Via, F.Cu at (372.2, 112.3)
- added H12: MountingHole_Pad, MountingHole:MountingHole_2.2mm_M2_Pad_Via, F.Cu at (392.3, 98.3)
- added H13: MountingHole_Pad, MountingHole:MountingHole_2.2mm_M2_Pad_Via, F.Cu at (357.3, 74.8)
- added H14: MountingHole_Pad, MountingHole:MountingHole_2.2mm_M2_Pad_Via, F.Cu at (344.9, 83.9)
- added H15: MountingHole_Pad, MountingHole:MountingHole_2.2mm_M2_Pad_Via, F.Cu at (372.2, 58.8)
- added H16: MountingHole_Pad, MountingHole:MountingHole_2.2mm_M2_Pad_Via, F.Cu at (378.4, 50.7)
- added H17: MountingHole_Pad, MountingHole:MountingHole_2.2mm_M2_Pad_Via, F.Cu at (372.2, 52.9)
- added H18: MountingHole_Pad, MountingHole:MountingHole_2.2mm_M2_Pad_Via, F.Cu at (392.3, 38.8)
- added H19: MountingHole_Pad, MountingHole:MountingHole_2.2mm_M2_Pad_Via, F.Cu at (103.9, 64.0)
- added H20: MountingHole_Pad, MountingHole:MountingHole_2.2mm_M2_Pad_Via, F.Cu at (91.5, 73.2)
- added H21: MountingHole_Pad, MountingHole:MountingHole_2.2mm_M2_Pad_Via, F.Cu at (130.2, 54.5)
- added H22: MountingHole_Pad, MountingHole:MountingHole_2.2mm_M2_Pad_Via, F.Cu at (125.0, 39.9)
- added H23: MountingHole_Pad, MountingHole:MountingHole_2.2mm_M2_Pad_Via, F.Cu at (130.2, 48.5)
- added H24: MountingHole_Pad, MountingHole:MountingHole_2.2mm_M2_Pad_Via, F.Cu at (138.9, 28.1)
- added H7: MountingHole_Pad, MountingHole:MountingHole_2.2mm_M2_Pad_Via, F.Cu at (357.3, 134.2)
- added H8: MountingHole_Pad, MountingHole:MountingHole_2.2mm_M2_Pad_Via, F.Cu at (344.9, 143.4)
- added H9: MountingHole_Pad, MountingHole:MountingHole_2.2mm_M2_Pad_Via, F.Cu at (372.2, 118.3)
- added J11: LSHM-140-02.5-L-DV-A-N-K-TR, Connector_Samtec:Samtec_LSHM-140-xx.x-x-DV-N_2x40_P0.50mm_Vertical, B.Cu at (148.0, 137.5)
- added J13: Motor (X3), Connector_Molex:Molex_Mini-Fit_Jr_5566-04A2_2x02_P4.20mm_Vertical, F.Cu at (124.0, 131.3)
- added J14: Hall Sensor (X4), Connector_Molex:Molex_Micro-Fit_3.0_43045-1212_2x06_P3.00mm_Vertical, F.Cu at (303.3, 106.1)
- added J15: Encoder (X5), Connector_PinHeader_2.54mm:PinHeader_2x05_P2.54mm_Vertical_SMD, F.Cu at (362.8, 116.7)
- added J16: Sensor (X6), can_proj_footprints:MOLEX_5031541090, F.Cu at (335.7, 127.9)
- added J18: Analog I/O (X8), Connector_Molex:Molex_CLIK-Mate_502585-0770_1x07-1MP_P1.50mm_Horizontal, F.Cu at (347.3, 114.4)
- added J20: Micro_USB (X13), Connector_USB:USB_Micro-B_Molex-105133-0001, F.Cu at (361.1, 127.1)
- added J21: LSHM-140-02.5-L-DV-A-N-K-TR, Connector_Samtec:Samtec_LSHM-140-xx.x-x-DV-N_2x40_P0.50mm_Vertical, B.Cu at (148.0, 89.0)
- added J23: Motor (X3), Connector_Molex:Molex_Mini-Fit_Jr_5566-04A2_2x02_P4.20mm_Vertical, F.Cu at (145.6, 246.2)
- added J24: Hall Sensor (X4), Connector_Molex:Molex_Micro-Fit_3.0_43045-1212_2x06_P3.00mm_Vertical, F.Cu at (303.3, 46.6)
- added J25: Encoder (X5), Connector_PinHeader_2.54mm:PinHeader_2x05_P2.54mm_Vertical_SMD, F.Cu at (362.8, 57.3)
- added J26: Sensor (X6), can_proj_footprints:MOLEX_5031541090, F.Cu at (325.0, 70.0)
- added J28: Analog I/O (X8), Connector_Molex:Molex_CLIK-Mate_502585-0770_1x07-1MP_P1.50mm_Horizontal, F.Cu at (347.3, 54.9)
- added J30: Micro_USB (X13), Connector_USB:USB_Micro-B_Molex-105133-0001, F.Cu at (361.1, 67.6)
- added J31: LSHM-140-02.5-L-DV-A-N-K-TR, Connector_Samtec:Samtec_LSHM-140-xx.x-x-DV-N_2x40_P0.50mm_Vertical, B.Cu at (57.4, 143.0)
- added J33: Motor (X3), Connector_Molex:Molex_Mini-Fit_Jr_5566-04A2_2x02_P4.20mm_Vertical, F.Cu at (25.2, 137.1)
- added J34: Hall Sensor (X4), Connector_Molex:Molex_Micro-Fit_3.0_43045-1212_2x06_P3.00mm_Vertical, F.Cu at (33.8, 149.1)
- added J35: Encoder (X5), Connector_PinHeader_2.54mm:PinHeader_2x05_P2.54mm_Vertical_SMD, F.Cu at (109.4, 46.5)
- added J36: Sensor (X6), can_proj_footprints:MOLEX_5031541090, F.Cu at (82.7, 114.3)
- added J38: Analog I/O (X8), Connector_Molex:Molex_CLIK-Mate_502585-0770_1x07-1MP_P1.50mm_Horizontal, F.Cu at (94.0, 44.2)
- added J40: Micro_USB (X13), Connector_USB:USB_Micro-B_Molex-105133-0001, F.Cu at (74.0, 86.0)
- added L10: 15uH, Inductor_SMD:L_Wuerth_WE-PD-Typ-LS_Handsoldering, F.Cu at (366.1, 42.9)
- added L11: 15uH, Inductor_SMD:L_Wuerth_WE-PD-Typ-LS_Handsoldering, F.Cu at (347.6, 42.9)
- added L12: 47uH, can_proj_footprints:IND_LQH5BPH470MT0L, F.Cu at (321.0, 85.7)
- added L13: 15uH, Inductor_SMD:L_Wuerth_WE-PD-Typ-LS_Handsoldering, F.Cu at (44.0, 126.8)
- added L14: 15uH, Inductor_SMD:L_Wuerth_WE-PD-Typ-LS_Handsoldering, B.Cu at (44.0, 133.0)
- added L15: 15uH, Inductor_SMD:L_Wuerth_WE-PD-Typ-LS_Handsoldering, F.Cu at (44.0, 139.2)
- added L16: 47uH, can_proj_footprints:IND_LQH5BPH470MT0L, B.Cu at (68.0, 51.0)
- added L5: 15uH, Inductor_SMD:L_Wuerth_WE-PD-Typ-LS_Handsoldering, F.Cu at (145.5, 115.0)
- added L6: 15uH, Inductor_SMD:L_Wuerth_WE-PD-Typ-LS_Handsoldering, F.Cu at (166.3, 123.0)
- added L7: 15uH, Inductor_SMD:L_Wuerth_WE-PD-Typ-LS_Handsoldering, F.Cu at (347.6, 102.3)
- added L8: 47uH, can_proj_footprints:IND_LQH5BPH470MT0L, F.Cu at (321.0, 145.2)
- added L9: 15uH, Inductor_SMD:L_Wuerth_WE-PD-Typ-LS_Handsoldering, F.Cu at (308.2, 84.3)
- added R10: 150R, Resistor_SMD:R_0603_1608Metric_Pad0.98x0.95mm_HandSolder, F.Cu at (381.3, 139.4)
- added R11: 150R, Resistor_SMD:R_0603_1608Metric_Pad0.98x0.95mm_HandSolder, F.Cu at (382.3, 135.8)
- added R12: 20k, Resistor_SMD:R_0603_1608Metric_Pad0.98x0.95mm_HandSolder, F.Cu at (389.3, 131.2)
- added R13: 20k, Resistor_SMD:R_0603_1608Metric_Pad0.98x0.95mm_HandSolder, F.Cu at (386.7, 133.7)
- added R14: 22k, Resistor_SMD:R_0603_1608Metric_Pad0.98x0.95mm_HandSolder, F.Cu at (386.7, 136.3)
- added R15: 1k, Resistor_SMD:R_0603_1608Metric_Pad0.98x0.95mm_HandSolder, F.Cu at (377.0, 141.9)
- added R16: 0R, Resistor_SMD:R_0603_1608Metric_Pad0.98x0.95mm_HandSolder, F.Cu at (319.7, 149.8)
- added R17: 0R, Resistor_SMD:R_0603_1608Metric_Pad0.98x0.95mm_HandSolder, F.Cu at (368.2, 125.4)
- added R18: 120R, Resistor_SMD:R_0603_1608Metric_Pad0.98x0.95mm_HandSolder, F.Cu at (371.4, 122.5)
- added R19: 150R, Resistor_SMD:R_0603_1608Metric_Pad0.98x0.95mm_HandSolder, F.Cu at (388.4, 69.3)
- added R20: 150R, Resistor_SMD:R_0603_1608Metric_Pad0.98x0.95mm_HandSolder, F.Cu at (389.4, 65.7)
- added R21: 20k, Resistor_SMD:R_0603_1608Metric_Pad0.98x0.95mm_HandSolder, F.Cu at (396.4, 61.1)
- added R22: 20k, Resistor_SMD:R_0603_1608Metric_Pad0.98x0.95mm_HandSolder, F.Cu at (393.8, 63.6)
- added R23: 22k, Resistor_SMD:R_0603_1608Metric_Pad0.98x0.95mm_HandSolder, F.Cu at (393.8, 66.1)
- added R24: 1k, Resistor_SMD:R_0603_1608Metric_Pad0.98x0.95mm_HandSolder, F.Cu at (384.0, 71.8)
- added R25: 0R, Resistor_SMD:R_0603_1608Metric_Pad0.98x0.95mm_HandSolder, F.Cu at (319.7, 90.3)
- added R26: 0R, Resistor_SMD:R_0603_1608Metric_Pad0.98x0.95mm_HandSolder, F.Cu at (368.2, 65.9)
- added R27: 120R, Resistor_SMD:R_0603_1608Metric_Pad0.98x0.95mm_HandSolder, F.Cu at (371.4, 63.0)
- added R28: 150R, Resistor_SMD:R_0603_1608Metric_Pad0.98x0.95mm_HandSolder, B.Cu at (124.6, 72.1)
- added R29: 150R, Resistor_SMD:R_0603_1608Metric_Pad0.98x0.95mm_HandSolder, B.Cu at (123.5, 68.6)
- added R30: 20k, Resistor_SMD:R_0603_1608Metric_Pad0.98x0.95mm_HandSolder, B.Cu at (116.6, 64.0)
- added R31: 20k, Resistor_SMD:R_0603_1608Metric_Pad0.98x0.95mm_HandSolder, B.Cu at (119.2, 66.5)
- added R32: 22k, Resistor_SMD:R_0603_1608Metric_Pad0.98x0.95mm_HandSolder, B.Cu at (119.2, 69.0)
- added R33: 1k, Resistor_SMD:R_0603_1608Metric_Pad0.98x0.95mm_HandSolder, B.Cu at (128.9, 74.7)
- added R34: 0R, Resistor_SMD:R_0603_1608Metric_Pad0.98x0.95mm_HandSolder, B.Cu at (66.3, 79.5)
- added R35: 0R, Resistor_SMD:R_0603_1608Metric_Pad0.98x0.95mm_HandSolder, B.Cu at (114.8, 55.1)
- added R36: 120R, Resistor_SMD:R_0603_1608Metric_Pad0.98x0.95mm_HandSolder, B.Cu at (118.0, 52.3)
- added Rs10: 270R, Resistor_SMD:R_0603_1608Metric_Pad0.98x0.95mm_HandSolder, B.Cu at (90.0, 78.1)
- added Rs11: 270R, Resistor_SMD:R_0603_1608Metric_Pad0.98x0.95mm_HandSolder, B.Cu at (96.7, 74.0)
- added Rs12: 270R, Resistor_SMD:R_0603_1608Metric_Pad0.98x0.95mm_HandSolder, B.Cu at (144.3, 52.4)
- added Rs4: 270R, Resistor_SMD:R_0603_1608Metric_Pad0.98x0.95mm_HandSolder, F.Cu at (137.5, 123.5)
- added Rs5: 270R, Resistor_SMD:R_0603_1608Metric_Pad0.98x0.95mm_HandSolder, F.Cu at (350.1, 144.2)
- added Rs6: 270R, Resistor_SMD:R_0603_1608Metric_Pad0.98x0.95mm_HandSolder, F.Cu at (377.3, 116.9)
- added Rs7: 270R, Resistor_SMD:R_0603_1608Metric_Pad0.98x0.95mm_HandSolder, F.Cu at (343.4, 88.8)
- added Rs8: 270R, Resistor_SMD:R_0603_1608Metric_Pad0.98x0.95mm_HandSolder, F.Cu at (350.1, 84.7)
- added Rs9: 270R, Resistor_SMD:R_0603_1608Metric_Pad0.98x0.95mm_HandSolder, F.Cu at (377.3, 57.4)
- added SW3: 450301014042-ND, can_proj_footprints:450301014042, F.Cu at (350.4, 122.8)
- added SW4: 219-8LPS, can_proj_footprints:SW_219-8LPSTRF, F.Cu at (332.0, 107.0)
- added SW5: 450301014042-ND, can_proj_footprints:450301014042, F.Cu at (350.4, 63.3)
- added SW6: 219-8LPS, can_proj_footprints:SW_219-8LPSTRF, F.Cu at (332.0, 47.5)
- added SW7: 450301014042-ND, can_proj_footprints:450301014042, F.Cu at (97.0, 52.6)
- added SW8: 219-8LPS, can_proj_footprints:SW_219-8LPSTRF, F.Cu at (78.6, 36.8)
- added TP2: RESET_TP, TestPoint:TestPoint_Pad_D2.0mm, F.Cu at (397.3, 97.3)
- added TP3: RESET_TP, TestPoint:TestPoint_Pad_D2.0mm, F.Cu at (397.3, 37.9)
- added TP4: RESET_TP, TestPoint:TestPoint_Pad_D2.0mm, F.Cu at (143.9, 27.1)
- added U10: MAX1486CUB+, can_proj_footprints:SOP50P490X110-10N, B.Cu at (126.8, 65.0)
- added U11: MAX15462BATA+T, can_proj_footprints:SON50P200X200X80-8N, B.Cu at (69.9, 45.0)
- added U12: SRV05-4, Package_TO_SOT_SMD:SOT-23-6, B.Cu at (85.2, 79.0)
- added U4: MAX1486CUB+, can_proj_footprints:SOP50P490X110-10N, F.Cu at (379.1, 132.3)
- added U5: MAX15462BATA+T, can_proj_footprints:SON50P200X200X80-8N, F.Cu at (323.3, 115.3)
- added U6: SRV05-4, Package_TO_SOT_SMD:SOT-23-6, F.Cu at (338.6, 149.3)
- added U7: MAX1486CUB+, can_proj_footprints:SOP50P490X110-10N, F.Cu at (386.2, 62.2)
- added U8: MAX15462BATA+T, can_proj_footprints:SON50P200X200X80-8N, F.Cu at (323.3, 55.8)
- added U9: SRV05-4, Package_TO_SOT_SMD:SOT-23-6, F.Cu at (338.6, 89.8)
- C1, C2: value 1uF -> 220pF
- C3: value EEH-ZA1V680XP -> 0.1uF; footprint can_proj_footprints:CAP_EEHZA1V680XP -> Capacitor_SMD:C_0603_1608Metric_Pad1.08x0.95mm_HandSolder
- C4: value 10uF -> 1uF
- C5: value 0.1uF -> 1uF
- C6: value 220pF -> EEH-ZA1V680XP; footprint Capacitor_SMD:C_0603_1608Metric_Pad1.08x0.95mm_HandSolder -> can_proj_footprints:CAP_EEHZA1V680XP
- C7: value 220pF -> 10uF
- D1: value SMF30A -> TPD4E1B06DCKR; footprint Diode_SMD:D_SOD-123 -> can_proj_footprints:TVS_TPD4E1B06DCKR
- D3: value TPD4E1B06DCKR -> SMF30A; footprint can_proj_footprints:TVS_TPD4E1B06DCKR -> Diode_SMD:D_SOD-123
- H1, H2, H3, H4, H5, H6: value MountingHole -> MountingHole_Pad
- J1: value Analog I/O (X8) -> LSHM-140-02.5-L-DV-A-N-K-TR; footprint Connector_Molex:Molex_CLIK-Mate_502585-0770_1x07-1MP_P1.50mm_Horizontal -> Connector_Samtec:Samtec_LSHM-140-xx.x-x-DV-N_2x40_P0.50mm_Vertical; moved to B.Cu
- J10: footprint Connector_USB:USB_Micro-B_Molex-105017-0001 -> Connector_USB:USB_Micro-B_Molex-105133-0001
- J2: value LSHM-140-02.5-L-DV-A-N-K-TR -> Power_supply (X1); footprint Connector_Samtec:Samtec_LSHM-140-xx.x-x-DV-N_2x40_P0.50mm_Vertical -> Connector_Molex:Molex_Mini-Fit_Jr_5569-02A2_2x01_P4.20mm_Horizontal
- J3: value CAN 1 (X11) -> Motor (X3); footprint can_proj_footprints:MOLEX_5025840460 -> Connector_Molex:Molex_Mini-Fit_Jr_5566-04A2_2x02_P4.20mm_Vertical
- J4: value CAN 2 (X12) -> Hall Sensor (X4); footprint can_proj_footprints:MOLEX_5025840460 -> Connector_Molex:Molex_Micro-Fit_3.0_43045-1212_2x06_P3.00mm_Vertical
- J5: value Power_supply (X1) -> Encoder (X5); footprint Connector_Molex:Molex_Mini-Fit_Jr_5569-02A2_2x01_P4.20mm_Horizontal -> Connector_PinHeader_2.54mm:PinHeader_2x05_P2.54mm_Vertical_SMD
- J6: value Motor (X3) -> Sensor (X6); footprint Connector_Molex:Molex_Mini-Fit_Jr_5569-04A1_2x02_P4.20mm_Horizontal -> can_proj_footprints:MOLEX_5031541090
- J7: value Hall Sensor (X4) -> CAN 1 (X11); footprint Connector_Molex:Molex_Micro-Fit_3.0_43045-1212_2x06_P3.00mm_Vertical -> can_proj_footprints:MOLEX_5025840460
- J8: value Encoder (X5) -> Analog I/O (X8); footprint Connector_PinHeader_2.54mm:PinHeader_2x10_P2.54mm_Vertical_SMD -> Connector_Molex:Molex_CLIK-Mate_502585-0770_1x07-1MP_P1.50mm_Horizontal
- L1: value 47uH -> 15uH; footprint can_proj_footprints:IND_LQH5BPH470MT0L -> Inductor_SMD:L_Wuerth_WE-PD-Typ-LS_Handsoldering
- L3: footprint Inductor_SMD:L_1210_3225Metric_Pad1.42x2.65mm_HandSolder -> Inductor_SMD:L_Wuerth_WE-PD-Typ-LS_Handsoldering
- L4: value 15uH -> 47uH; footprint Inductor_SMD:L_1210_3225Metric_Pad1.42x2.65mm_HandSolder -> can_proj_footprints:IND_LQH5BPH470MT0L
- R1, R2: value 0R -> 150R
- R3: value 120R -> 20k
- R4: value 150R -> 20k
- R5: value 150R -> 22k
- R6: value 20k -> 1k
- R7: value 20k -> 0R
- R8: value 22k -> 0R
- R9: value 1k -> 120R
- U1: value MAX15462BATA+T -> MAX1486CUB+; footprint can_proj_footprints:SON50P200X200X80-8N -> can_proj_footprints:SOP50P490X110-10N
- U2: value SRV05-4 -> MAX15462BATA+T; footprint Package_TO_SOT_SMD:SOT-23-6 -> can_proj_footprints:SON50P200X200X80-8N
- U3: value MAX1486CUB+ -> SRV05-4; footprint can_proj_footprints:SOP50P490X110-10N -> Package_TO_SOT_SMD:SOT-23-6
- moved H6 297.6 mm to (394.6, 156.9)
- moved TP1 292.5 mm to (399.6, 156.0)
- moved C4 288.4 mm to (385.9, 169.6), turned to 0 degrees
- moved J8 288.0 mm to (349.6, 173.1)
- moved Cf2 285.2 mm to (385.9, 167.1)
- moved Cs3 284.8 mm to (384.0, 173.1)
- moved Cf1 280.2 mm to (393.8, 161.2)
- moved C2 279.3 mm to (369.8, 201.8), turned to 0 degrees
- moved SW1 278.4 mm to (352.7, 181.4)
- moved Cs1 275.7 mm to (379.6, 173.1)
- moved R1 274.3 mm to (366.2, 209.9)
- moved C1 272.2 mm to (361.8, 215.0), turned to 0 degrees
- moved H4 271.5 mm to (380.7, 168.8)
- moved R3 270.6 mm to (374.1, 201.8)
- moved R2 270.2 mm to (367.2, 206.4), turned to 0 degrees
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Connections:
- C1 pad 1: GND -> Net-(C1-Pad1)
- C1 pad 2: +Vcc -> GND
- C3 pad 1: Net-(C3-Pad1) -> /Connector layout13/Vaux
- C4 pad 1: VDD -> GND
- C4 pad 2: GND -> VCC
- C5 pad 1: VBus -> Net-(C5-Pad1)
- C7 pad 1: Net-(C7-Pad1) -> /Connector layout13/VDD
- C8 pad 1: Vaux -> /Connector layout13/VBus
- Cf1 pad 1: Motor + -> /Connector layout13/Motor+
- Cf2 pad 1: Motor - -> /Connector layout13/Motor-
- Cf3 pad 1: Motor 3 -> /Connector layout13/Motor3
- Cs1 pad 1: Motor + -> /Connector layout13/Motor+
- Cs2 pad 1: Motor - -> /Connector layout13/Motor-
- Cs3 pad 1: Motor 3 -> /Connector layout13/Motor3
- D1 pad 1: Net-(C3-Pad1) -> /Connector layout13/IN_Clock/HsDigOUT1\
- D2 pad 1: +Vcc -> Net-(C6-Pad1)
- D3 pad 1: IN_Clock/HsDigOUT1\ -> VCC
- F1 pad 1: +Vcc -> VCC
- F1 pad 2: Net-(C3-Pad1) -> Net-(C6-Pad1)
- H1 pad 1: (no net) -> GND
- H2 pad 1: (no net) -> GND
- H3 pad 1: (no net) -> GND
- H4 pad 1: (no net) -> GND
- H5 pad 1: (no net) -> GND
- H6 pad 1: (no net) -> GND
- J1 pad 1: AnIN1+ -> Net-(J1-Pad1)
- J1 pad 2: AnIN1- -> Net-(J1-Pad1)
- J1 pad 3: AnIN2+ -> Net-(J1-Pad1)
- J1 pad 4: AnIN2- -> Net-(J1-Pad1)
- J1 pad 5: AnOUT1 -> Net-(J1-Pad1)
- J1 pad 6: unconnected-(J1-Pad6) -> Net-(J1-Pad1)
- J1 pad 7: GND -> Net-(J1-Pad10)
- J10 pad 1: VBus -> /Connector layout13/VBus
- J10 pad 2: USB_D- -> /Connector layout13/USB_D-
- J10 pad 3: USB_D+ -> /Connector layout13/USB_D+
- J2 pad 1: Net-(J2-Pad1) -> GND
- J2 pad 2: Net-(J2-Pad1) -> VCC
- J3 pad 1: CAN high -> /Connector layout13/Motor+
- J3 pad 2: CAN low -> /Connector layout13/Motor-
- J3 pad 3: GND -> /Connector layout13/Motor3
- J4 pad 1: CAN high -> /Connector layout13/Hall Sensor 1
- J4 pad 2: CAN low -> /Connector layout13/Hall Sensor 2
- J4 pad 3: GND -> /Connector layout13/Hall Sensor 3
- J5 pad 1: GND -> unconnected-(J5-Pad1)
- J5 pad 2: +Vcc -> /Connector layout13/Vsensor
- J6 pad 1: Motor + -> unconnected-(J6-Pad1)
- J6 pad 2: Motor - -> unconnected-(J6-Pad2)
- J6 pad 3: Motor 3 -> unconnected-(J6-Pad3)
- J6 pad 4: GND -> unconnected-(J6-Pad4)
- J7 pad 1: Hall Sensor 1 -> CAN high
- J7 pad 2: Hall Sensor 2 -> CAN low
- J7 pad 3: Hall Sensor 3 -> GND
- J8 pad 1: unconnected-(J8-Pad1) -> /Connector layout13/AnIN1+
- J8 pad 2: Vsensor -> /Connector layout13/AnIN1-
- J8 pad 3: GND -> /Connector layout13/AnIN2+
- J8 pad 4: unconnected-(J8-Pad4) -> /Connector layout13/AnIN2-
- J8 pad 5: Channel_A\ -> /Connector layout13/AnOUT1
- J8 pad 6: Channel_A -> unconnected-(J8-Pad6)
- J8 pad 7: Channel_B\ -> GND
- L1 pad 1: Net-(L1-Pad1) -> Net-(J1-Pad1)
- L1 pad 2: VDD -> /Connector layout13/Motor+
- L2 pad 1: Net-(J2-Pad1) -> Net-(J1-Pad10)
- L2 pad 2: Motor + -> /Connector layout13/Motor-
- L3 pad 1: Net-(J2-Pad10) -> Net-(J1-Pad13)
- L3 pad 2: Motor - -> /Connector layout13/Motor3
- L4 pad 1: Net-(J2-Pad13) -> Net-(L4-Pad1)
- L4 pad 2: Motor 3 -> /Connector layout13/VDD
- R1 pad 1: +Vcc -> /Connector layout13/IN_Data
- R1 pad 2: Net-(R1-Pad2) -> Net-(C1-Pad1)
- R2 pad 1: Net-(R1-Pad2) -> /Connector layout13/IN_Data\
- R2 pad 2: GND -> Net-(C2-Pad1)
- R3 pad 1: Net-(R3-Pad1) -> Net-(C2-Pad1)
- R3 pad 2: CAN low -> /Connector layout13/Vaux
- R4 pad 1: IN_Data -> GND
- R4 pad 2: Net-(C6-Pad1) -> Net-(C2-Pad1)
- R5 pad 1: IN_Data\ -> GND
- R5 pad 2: Net-(C7-Pad1) -> Net-(C1-Pad1)
- R6 pad 1: Net-(C7-Pad1) -> Net-(R6-Pad1)
- R6 pad 2: Vaux -> /Connector layout13/Data/HsDigIN4
- R7 pad 1: GND -> VCC
- R7 pad 2: Net-(C7-Pad1) -> GND
- R8 pad 2: Net-(C6-Pad1) -> GND
- R9 pad 2: Data/HsDigIN4 -> CAN low
- SW1 pad 1: Vsensor -> /Connector layout13/Vsensor
- SW1 pad 2: Vaux -> /Connector layout13/Vaux
- SW1 pad 3: VDD -> /Connector layout13/VDD
- SW2 pad 1: ID 1 -> /Connector layout13/ID 1
- SW2 pad 10: Net-(R3-Pad1) -> Net-(R9-Pad1)
- SW2 pad 2: ID 2 -> /Connector layout13/ID 2
- SW2 pad 3: ID 3 -> /Connector layout13/ID 3
- SW2 pad 4: ID 4 -> /Connector layout13/ID 4
- SW2 pad 5: ID 5 -> /Connector layout13/ID 5
- SW2 pad 6: Auto bit rate -> /Connector layout13/Auto bit rate
- U1 pad 1: +Vcc -> Net-(R6-Pad1)
- U1 pad 2: +Vcc -> GND
- U1 pad 3: Net-(C2-Pad1) -> /Connector layout13/Vaux
- U1 pad 4: VDD -> /Connector layout13/Clock/HsDigOUT1
- U1 pad 5: Net-(R1-Pad2) -> GND
- U1 pad 6: Net-(TP1-Pad1) -> Net-(C2-Pad1)
- U1 pad 7: GND -> /Connector layout13/IN_Clock/HsDigOUT1
- U1 pad 8: Net-(L1-Pad1) -> /Connector layout13/IN_Clock/HsDigOUT1\
- U2 pad 1: USB_D+ -> VCC
- U2 pad 2: GND -> VCC
- U2 pad 3: USB_D+ -> Net-(C5-Pad1)
- U2 pad 4: USB_D- -> /Connector layout13/VDD
- U2 pad 5: VBus -> GND
- U2 pad 6: USB_D- -> Net-(TP1-Pad1)
- U3 pad 1: Net-(R9-Pad1) -> /Connector layout13/USB_D+
- U3 pad 3: Vaux -> /Connector layout13/USB_D+
- U3 pad 4: Clock/HsDigOUT1 -> /Connector layout13/USB_D-
- U3 pad 5: GND -> /Connector layout13/VBus
- U3 pad 6: Net-(C7-Pad1) -> /Connector layout13/USB_D-
Other:
- copper layers 2 -> 4
