File: hats/voltmeter/voltmeter.kicad_pcb (KiCad board)
At the start: 2 copper layers, 30.7 x 33.1 mm, 23 parts, among them J1 XT30PW-M, J2 JST_Picoblade_I2C, J3 Hat_connector_hole, U1 TPS7A2030PDBVR, U2 OPA2336, U3 ADS1113IDGS

Commit message: Updated steps
Parts:
- added kibuzzard-638A3310: G***, kibuzzard-638A3310, F.Cu at (140.6, 101.3)
- added kibuzzard-638A335E: G***, kibuzzard-638A335E, F.Cu at (140.6, 99.6)
