File: hats/PWMBoard.kicad_sch (KiCad schematic)
At the start: 12 parts, among them IC1 CD40109B-Q1, J1 Hat_connector_hole, J2 Ext, J3 S1, J4 S2, J5 S3, J6 S4

Commit message: Updated localization files
Parts:
- added J7: Conn_01x06, Connector_JST:JST_GH_BM06B-GHS-TBT_1x06-1MP_P1.25mm_Vertical, symbol Connector_Generic:Conn_01x06
- J2: value Ext -> (none); footprint Connector_AMASS:AMASS_XT30U-M_1x02_P5.0mm_Vertical -> (none)
Connections:
- net +3.3V: now also J7.1 (Pin_1)
- net +5V: now also J1.15 (5V)
- net GND: now also J7.6 (Pin_6)
- net GPIO_2: now reaches IC1.6 (B), J1.10 (GPIO_2)
- net GPIO_2: now also J7.4 (Pin_4)
- net GPIO_3: now reaches IC1.10 (C), J1.11 (GPIO_3)
- net GPIO_3: now also J7.3 (Pin_3)
- net GPIO_4: now reaches IC1.14 (D), J1.12 (GPIO_4)
- net GPIO_4: now also J7.2 (Pin_2)
- net GPIO_1: now reaches IC1.3 (A), J1.9 (GPIO_1)
- net GPIO_1: now also J7.5 (Pin_5)
Changed lines of the file:
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@@
   (junction (at 151.13 116.84) (diameter 0) (color 0 0 0 0)
   )
+  (junction (at 72.39 69.85) (diameter 0) (color 0 0 0 0)
+  )
   (junction (at 205.74 95.25) (diameter 0) (color 0 0 0 0)
   )
@@
   (junction (at 161.29 116.84) (diameter 0) (color 0 0 0 0)
   )
+  (junction (at 236.22 69.85) (diameter 0) (color 0 0 0 0)
+  )
+  (junction (at 139.7 116.84) (diameter 0) (color 0 0 0 0)
+  )
+  (junction (at 199.39 67.31) (diameter 0) (color 0 0 0 0)
+  )
+  (junction (at 232.41 97.79) (diameter 0) (color 0 0 0 0)
+  )
+  (junction (at 199.39 92.71) (diameter 0) (color 0 0 0 0)
+  )
+  (junction (at 236.22 95.25) (diameter 0) (color 0 0 0 0)
+  )
+  (junction (at 232.41 85.09) (diameter 0) (color 0 0 0 0)
+  )
+  (junction (at 232.41 110.49) (diameter 0) (color 0 0 0 0)
+  )
+  (junction (at 139.7 92.71) (diameter 0) (color 0 0 0 0)
+  )
+  (junction (at 214.63 116.84) (diameter 0) (color 0 0 0 0)
+  )
   (junction (at 214.63 92.71) (diameter 0) (color 0 0 0 0)
   )
-  (junction (at 236.22 69.85) (diameter 0) (color 0 0 0 0)
-  )
-  (junction (at 139.7 116.84) (diameter 0) (color 0 0 0 0)
-  )
-  (junction (at 199.39 67.31) (diameter 0) (color 0 0 0 0)
-  )
-  (junction (at 232.41 97.79) (diameter 0) (color 0 0 0 0)
-  )
-  (junction (at 199.39 92.71) (diameter 0) (color 0 0 0 0)
-  )
-  (junction (at 236.22 95.25) (diameter 0) (color 0 0 0 0)
-  )
-  (junction (at 232.41 85.09) (diameter 0) (color 0 0 0 0)
-  )
-  (junction (at 232.41 110.49) (diameter 0) (color 0 0 0 0)
-  )
-  (junction (at 139.7 92.71) (diameter 0) (color 0 0 0 0)
-  )
-  (junction (at 214.63 116.84) (diameter 0) (color 0 0 0 0)
-  )
   (wire (pts (xy 68.58 102.87) (xy 161.29 102.87))
     (stroke (width 0) (type default) (color 0 0 0 0))
   )
-  (wire (pts (xy 68.58 69.85) (xy 80.01 69.85))
+  (wire (pts (xy 68.58 69.85) (xy 72.39 69.85))
+    (stroke (width 0) (type default) (color 0 0 0 0))
+  )
+  (wire (pts (xy 72.39 69.85) (xy 80.01 69.85))
     (stroke (width 0) (type default) (color 0 0 0 0))
   )
@@
     (stroke (width 0) (type default) (color 0 0 0 0))
   )
-  (wire (pts (xy 214.63 86.36) (xy 214.63 92.71))
+  (wire (pts (xy 68.58 67.31) (xy 72.39 67.31))
     (stroke (width 0) (type default) (color 0 0 0 0))
   )
@@
     (stroke (width 0) (type default) (color 0 0 0 0))
   )
+  (wire (pts (xy 180.34 139.7) (xy 180.34 140.97))
+    (stroke (width 0) (type default) (color 0 0 0 0))
+  )
   (wire (pts (xy 199.39 54.61) (xy 199.39 67.31))
     (stroke (width 0) (type default) (color 0 0 0 0))
@@
     (stroke (width 0) (type default) (color 0 0 0 0))
   )
+  (wire (pts (xy 184.15 139.7) (xy 180.34 139.7))
+    (stroke (width 0) (type default) (color 0 0 0 0))
+  )
   (wire (pts (xy 245.11 69.85) (xy 236.22 69.85))
     (stroke (width 0) (type default) (color 0 0 0 0))
@@
     (stroke (width 0) (type default) (color 0 0 0 0))
   )
+  (wire (pts (xy 180.34 127) (xy 184.15 127))
+    (stroke (width 0) (type default) (color 0 0 0 0))
+  )
   (wire (pts (xy 245.11 95.25) (xy 236.22 95.25))
     (stroke (width 0) (type default) (color 0 0 0 0))
@@
     (stroke (width 0) (type default) (color 0 0 0 0))
   )
+  (wire (pts (xy 72.39 67.31) (xy 72.39 69.85))
+    (stroke (width 0) (type default) (color 0 0 0 0))
+  )
+  (wire (pts (xy 214.63 80.01) (xy 214.63 92.71))
+    (stroke (width 0) (type default) (color 0 0 0 0))
+  )
   (wire (pts (xy 143.51 78.74) (xy 151.13 78.74))
+    (stroke (width 0) (type default) (color 0 0 0 0))
+  )
+  (wire (pts (xy 180.34 125.73) (xy 180.34 127))
     (stroke (width 0) (type default) (color 0 0 0 0))
   )
@@
   (text "Power flags" (at 39.37 160.02 0)
     (effects (font (size 3 3) (thickness 0.254) bold) (justify left bottom))
+  )
+  (label "GPIO_4" (at 73.66 105.41 0)
+    (effects (font (size 1.27 1.27)) (justify left bottom))
+  )
+  (label "GPIO_1" (at 73.66 97.79 0)
+    (effects (font (size 1.27 1.27)) (justify left bottom))
+  )
+  (label "GPIO_3" (at 184.15 132.08 180)
+    (effects (font (size 1.27 1.27)) (justify right bottom))
+  )
+  (label "GPIO_2" (at 73.66 100.33 0)
+    (effects (font (size 1.27 1.27)) (justify left bottom))
+  )
+  (label "GPIO_1" (at 184.15 137.16 180)
+    (effects (font (size 1.27 1.27)) (justify right bottom))
+  )
+  (label "GPIO_3" (at 73.66 102.87 0)
+    (effects (font (size 1.27 1.27)) (justify left bottom))
+  )
+  (label "GPIO_4" (at 184.15 129.54 180)
+    (effects (font (size 1.27 1.27)) (justify right bottom))
+  )
+  (label "GPIO_2" (at 184.15 134.62 180)
+    (effects (font (size 1.27 1.27)) (justify right bottom))
+  )
+  (symbol (lib_id "power:GND") (at 180.34 140.97 0) (unit 1)
+    (in_bom yes) (on_board yes) (fields_autoplaced)
+    (property "Reference" "#PWR0117" (id 0) (at 180.34 147.32 0)
+      (effects (font (size 1.27 1.27)) hide)
+    )
+    (property "Value" "GND" (id 1) (at 180.34 146.05 0))
+    (property "Footprint" "" (id 2) (at 180.34 140.97 0)
+      (effects (font (size 1.27 1.27)) hide)
+    )
+    (property "Datasheet" "" (id 3) (at 180.34 140.97 0)
+      (effects (font (size 1.27 1.27)) hide)
+    )
+    (pin "1")
   )
   (symbol (lib_id "power:+3.3V") (at 101.6 55.88 0) (unit 1)
@@
     (pin "2")
   )
+  (symbol (lib_id "power:+3.3V") (at 180.34 125.73 0) (unit 1)
+    (in_bom yes) (on_board yes) (fields_autoplaced)
+    (property "Reference" "#PWR0116" (id 0) (at 180.34 129.54 0)
+      (effects (font (size 1.27 1.27)) hide)
+    )
+    (property "Value" "+3.3V" (id 1) (at 180.34 120.65 0))
+    (property "Footprint" "" (id 2) (at 180.34 125.73 0)
+      (effects (font (size 1.27 1.27)) hide)
+    )
+    (property "Datasheet" "" (id 3) (at 180.34 125.73 0)
+      (effects (font (size 1.27 1.27)) hide)
+    )
+    (pin "1")
+  )
   (symbol (lib_id "power:PWR_FLAG") (at 62.23 180.34 0) (mirror x) (unit 1)
     (in_bom yes) (on_board yes)
@@
   (symbol (lib_id "0_connectors:Hat_connector_hole") (at 59.69 93.98 0) (mirror y) (unit 1)
     (in_bom yes) (on_board yes) (fields_autoplaced)
-    (property "Reference" "J1" (id 0) (at 60.0075 54.61 0))
-    (property "Value" "Hat_connector_hole" (id 1) (at 60.0075 57.15 0))
+    (property "Reference" "J1" (id 0) (at 59.3725 54.61 0))
+    (property "Value" "Hat_connector_hole" (id 1) (at 59.3725 57.15 0))
     (property "Footprint" "0_connectors:Hat_connector_hole" (id 2) (at 59.69 93.98 0)
       (effects (font (size 1.27 1.27)) hide)
@@
       (effects (font (size 1.27 1.27)) (justify left))
     )
-    (property "Value" "Ext" (id 1) (at 137.16 39.3699 0)
-      (effects (font (size 1.27 1.27)) (justify left))
-    )
-    (property "Footprint" "Connector_AMASS:AMASS_XT30U-M_1x02_P5.0mm_Vertical" (id 2) (at 134.62 36.83 0)
+    (property "Value" "" (id 1) (at 137.16 39.3699 0)
+      (effects (font (size 1.27 1.27)) (justify left))
+    )
+    (property "Footprint" "" (id 2) (at 134.62 36.83 0)
       (effects (font (size 1.27 1.27)) hide)
     )
@@
     (pin "1")
   )
-  (symbol (lib_id "power:VCC") (at 214.63 86.36 0) (unit 1)
-    (in_bom yes) (on_board yes) (fields_autoplaced)
-    (property "Reference" "#PWR?" (id 0) (at 214.63 90.17 0)
-      (effects (font (size 1.27 1.27)) hide)
-    )
-    (property "Value" "VCC" (id 1) (at 214.63 81.28 0))
-    (property "Footprint" "" (id 2) (at 214.63 86.36 0)
-      (effects (font (size 1.27 1.27)) hide)
-    )
-    (property "Datasheet" "" (id 3) (at 214.63 86.36 0)
-      (effects (font (size 1.27 1.27)) hide)
-    )
-    (pin "1")
+  (symbol (lib_id "power:VCC") (at 214.63 80.01 0) (unit 1)
+    (in_bom yes) (on_board yes) (fields_autoplaced)
+    (property "Reference" "#PWR0115" (id 0) (at 214.63 83.82 0)
+      (effects (font (size 1.27 1.27)) hide)
+    )
+    (property "Value" "VCC" (id 1) (at 214.63 74.93 0))
+    (property "Footprint" "" (id 2) (at 214.63 80.01 0)
+      (effects (font (size 1.27 1.27)) hide)
+    )
+    (property "Datasheet" "" (id 3) (at 214.63 80.01 0)
+      (effects (font (size 1.27 1.27)) hide)
+    )
+    (pin "1")
+  )
+  (symbol (lib_id "Connector_Generic:Conn_01x06") (at 189.23 132.08 0) (unit 1)
+    (in_bom yes) (on_board yes) (fields_autoplaced)
+    (property "Reference" "J7" (id 0) (at 191.262 132.5153 0)
+      (effects (font (size 1.27 1.27)) (justify left))
+    )
+    (property "Value" "Conn_01x06" (id 1) (at 191.262 135.0522 0)
+      (effects (font (size 1.27 1.27)) (justify left))
+    )
+    (property "Footprint" "Connector_JST:JST_GH_BM06B-GHS-TBT_1x06-1MP_P1.25mm_Vertical" (id 2) (at 189.23 132.08 0)
+      (effects (font (size 1.27 1.27)) hide)
+    )
+    (property "Datasheet" "~" (id 3) (at 189.23 132.08 0)
+      (effects (font (size 1.27 1.27)) hide)
+    )
+    (pin "1")
+    (pin "2")
+    (pin "3")
+    (pin "4")
+    (pin "5")
+    (pin "6")
   )
   (symbol (lib_id "Analog_Switch:CD40109BQNSRQ1") (at 161.29 92.71 0) (unit 1)
@@
       (reference "#PWR0114") (unit 1) (value "GND") (footprint "")
     )
-    (path "/cd3851c8-43a7-44ba-a57d-7da51bf4d405"
-      (reference "#PWR?") (unit 1) (value "VCC") (footprint "")
+    (path "/d5e98c55-90e8-47a8-9457-9bda841c82e4"
+      (reference "#PWR0115") (unit 1) (value "VCC") (footprint "")
+    )
+    (path "/6bd8e7f4-065e-421a-abdc-08a78a0a5e6c"
+      (reference "#PWR0116") (unit 1) (value "+3.3V") (footprint "")
+    )
+    (path "/0832e915-358a-4a3e-8521-d901d2675a6c"
+      (reference "#PWR0117") (unit 1) (value "GND") (footprint "")
     )
     (path "/7858b86b-45c4-4f4f-9a4e-2c52d3ba3cc0"
@@
       (reference "J6") (unit 1) (value "S4") (footprint "Connector_Molex:Molex_Micro-Fit_3.0_43650-0315_1x03_P3.00mm_Vertical")
     )
+    (path "/d77dd3e5-b28f-47be-9806-596bc283d3f9"
+      (reference "J7") (unit 1) (value "Conn_01x06") (footprint "Connector_JST:JST_GH_BM06B-GHS-TBT_1x06-1MP_P1.25mm_Vertical")
+    )
     (path "/271775ec-ef4b-4d33-b4da-941adbf57d07"
