File: nav_controller_interface_v2/nav_controller_interface_v2.kicad_sch (KiCad schematic)
At the start: 0 parts

Commit message: Added v2 of nav interface board
Other:
- sheet Driving inteface ports: added {CAN}; removed none

Commit message: Added schematic for can controller interface v2
Other:
- added sheet Logos (logos.kicad_sch)
- note added: "1 Overview"
- note added: "2"
- note added: "3"
- note added: "4"
- note added: "5"
- note added: "7"
- note added: "Logos"
- note added: "Mechanical"
- note added: "Power/CAN"
- company: (none) -> EPFL Xplore
- title: (none) -> Steering/Driving CAN Controller Interfaces Overview
