File: nav_controller_interface_v2/nav_controller_interface_v2.kicad_pcb (KiCad board)
At the start: 4 copper layers, 150 x 100 mm, 68 parts, among them J201 EPOS4 Micro 24/5 CAN Terminal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, J202 Motor (X3) - Molex Mini-Fit J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, J203 Hall Sensor (X4) - Molex Micr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, J204 Encoder (X5) - Pin headers 2.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, J205 Sensor (X6) - Molex CLIK-Mate, J206 USB_B_Micro, J301 02x23 Socket header (SSM-123-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, J302 02x16 Socket header (SSM-116-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, J303 Motor (X3) - Molex Mini-Fit J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, J304 Hall Sensor (X4) - Molex Micr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, J305 Encoder (X5) - Pin headers 2.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, J306 Sensor (X6) - Molex CLIK-Mate, J401 Power supply (X1) - XT60, J402 Power supply (X1) - XT60, J403 CAN 1 (X11) - Molex CLIK-Mate, J404 CAN2 (X12) - Molex CLIK-Mate, SW201 218-8LPST, SW202 SW_SPDT, SW301 218-8LPST, U201 MAX15462BATA+T, U601 ISL8490E

Commit message: fixed position
Parts:
- moved C301 0.86 mm to (192.9, 91.3)
- moved J204 0.45 mm to (94.2, 131.7)
Changed lines of the file:
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@@
   )
   (footprint "0_connectors:SAMTEC-HTST-105-01-X-DV" (layer "F.Cu")
-    (at 93.8 131.65 -90)
+    (at 94.25 131.65 -90)
     (descr "translated Allegro footprint")
     (property "Distributor" "Mouser")
@@
   )
   (footprint "Capacitor_SMD:CP_Elec_16x17.5" (layer "F.Cu")
-    (at 192.9 92.1575 90)
+    (at 192.9 91.3 90)
     (descr "SMD capacitor, aluminum electrolytic, Vishay 1616, 16.0x17.5mm, http://www.vishay.com/docs/28395/150crz.pdf")
     (tags "capacitor electrolytic")
@@
   (segment (start 187.805 64.1) (end 192.05 68.345) (width 0.2) (layer "F.Cu") (net 26))
   (segment (start 167 58.1) (end 173 64.1) (width 0.2) (layer "F.Cu") (net 26))
-  (segment (start 97.038 131.65) (end 100.45 131.65) (width 0.2) (layer "F.Cu") (net 34))
   (segment (start 100.45 131.65) (end 101.15 130.95) (width 0.2) (layer "F.Cu") (net 34))
+  (segment (start 97.488 131.65) (end 100.45 131.65) (width 0.2) (layer "F.Cu") (net 34))
   (segment (start 107.1 121.3) (end 139.3 121.3) (width 0.2) (layer "F.Cu") (net 34))
   (segment (start 101.15 127.25) (end 107.1 121.3) (width 0.2) (layer "F.Cu") (net 34))
@@
   (segment (start 101.75 131.35) (end 101.75 127.65) (width 0.2) (layer "F.Cu") (net 36))
   (segment (start 101.75 127.65) (end 107.4 122) (width 0.2) (layer "F.Cu") (net 36))
+  (segment (start 91.88 132.9) (end 94.5 132.9) (width 0.2) (layer "F.Cu") (net 36))
   (segment (start 100.2 132.9) (end 101.75 131.35) (width 0.2) (layer "F.Cu") (net 36))
+  (segment (start 90.63 131.65) (end 91.88 132.9) (width 0.2) (layer "F.Cu") (net 36))
   (segment (start 107.4 122) (end 139.6 122) (width 0.2) (layer "F.Cu") (net 36))
-  (segment (start 90.18 131.65) (end 91.43 132.9) (width 0.2) (layer "F.Cu") (net 36))
+  (segment (start 94.5 132.9) (end 100.2 132.9) (width 0.2) (layer "F.Cu") (net 36))
   (segment (start 141.25 120.35) (end 141.25 115.8) (width 0.2) (layer "F.Cu") (net 36))
   (segment (start 139.6 122) (end 141.25 120.35) (width 0.2) (layer "F.Cu") (net 36))
-  (segment (start 91.43 132.9) (end 100.2 132.9) (width 0.2) (layer "F.Cu") (net 36))
   (segment (start 102.3 128.2) (end 107.8 122.7) (width 0.2) (layer "F.Cu") (net 38))
+  (segment (start 97.488 134.19) (end 100.01 134.19) (width 0.2) (layer "F.Cu") (net 38))
+  (segment (start 100.01 134.19) (end 102.3 131.9) (width 0.2) (layer "F.Cu") (net 38))
   (segment (start 102.3 131.9) (end 102.3 128.2) (width 0.2) (layer "F.Cu") (net 38))
   (segment (start 107.8 122.7) (end 139.9 122.7) (width 0.2) (layer "F.Cu") (net 38))
-  (segment (start 97.038 134.19) (end 100.01 134.19) (width 0.2) (layer "F.Cu") (net 38))
-  (segment (start 100.01 134.19) (end 102.3 131.9) (width 0.2) (layer "F.Cu") (net 38))
   (segment (start 141.75 120.85) (end 141.75 115.8) (width 0.2) (layer "F.Cu") (net 38))
   (segment (start 139.9 122.7) (end 141.75 120.85) (width 0.2) (layer "F.Cu") (net 38))
   (segment (start 100 135.4) (end 102.9 132.5) (width 0.2) (layer "F.Cu") (net 39))
+  (segment (start 90.63 134.19) (end 91.84 135.4) (width 0.2) (layer "F.Cu") (net 39))
   (segment (start 142.25 121.25) (end 142.25 115.8) (width 0.2) (layer "F.Cu") (net 39))
   (segment (start 102.9 128.5) (end 108.1 123.3) (width 0.2) (layer "F.Cu") (net 39))
   (segment (start 108.1 123.3) (end 140.2 123.3) (width 0.2) (layer "F.Cu") (net 39))
-  (segment (start 91.39 135.4) (end 100 135.4) (width 0.2) (layer "F.Cu") (net 39))
+  (segment (start 91.84 135.4) (end 93.4 135.4) (width 0.2) (layer "F.Cu") (net 39))
+  (segment (start 93.4 135.4) (end 100 135.4) (width 0.2) (layer "F.Cu") (net 39))
   (segment (start 102.9 132.5) (end 102.9 128.5) (width 0.2) (layer "F.Cu") (net 39))
   (segment (start 140.2 123.3) (end 142.25 121.25) (width 0.2) (layer "F.Cu") (net 39))
-  (segment (start 90.18 134.19) (end 91.39 135.4) (width 0.2) (layer "F.Cu") (net 39))
-  (segment (start 99.67 136.73) (end 103.5 132.9) (width 0.2) (layer "F.Cu") (net 41))
-  (segment (start 97.038 136.73) (end 99.67 136.73) (width 0.2) (layer "F.Cu") (net 41))
-  (segment (start 140.5 124) (end 142.75 121.75) (width 0.2) (layer "F.Cu") (net 41))
-  (segment (start 108.2 124) (end 140.5 124) (width 0.2) (layer "F.Cu") (net 41))
-  (segment (start 142.75 121.75) (end 142.75 115.8) (width 0.2) (layer "F.Cu") (net 41))
-  (segment (start 103.5 132.9) (end 103.5 128.7) (width 0.2) (layer "F.Cu") (net 41))
-  (segment (start 103.5 128.7) (end 108.2 124) (width 0.2) (layer "F.Cu") (net 41))
+  (segment (start 142.75 115.8) (end 142.75 121.75) (width 0.2) (layer "F.Cu") (net 41))
+  (segment (start 142.75 121.75) (end 140.5 124) (width 0.2) (layer "F.Cu") (net 41))
+  (segment (start 103.5 128.7) (end 103.5 133.5) (width 0.2) (layer "F.Cu") (net 41))
+  (segment (start 140.5 124) (end 108.2 124) (width 0.2) (layer "F.Cu") (net 41))
+  (segment (start 100.27 136.73) (end 97.488 136.73) (width 0.2) (layer "F.Cu") (net 41))
+  (segment (start 103.5 133.5) (end 100.27 136.73) (width 0.2) (layer "F.Cu") (net 41))
+  (segment (start 108.2 124) (end 103.5 128.7) (width 0.2) (layer "F.Cu") (net 41))
+  (segment (start 100.5 138) (end 104 134.5) (width 0.2) (layer "F.Cu") (net 43))
+  (segment (start 108.5 124.6) (end 140.9 124.6) (width 0.2) (layer "F.Cu") (net 43))
+  (segment (start 104 134.5) (end 104 129.1) (width 0.2) (layer "F.Cu") (net 43))
   (segment (start 104 129.1) (end 108.5 124.6) (width 0.2) (layer "F.Cu") (net 43))
-  (segment (start 102.2 135.8) (end 102.2 135.7) (width 0.2) (layer "F.Cu") (net 43))
-  (segment (start 102.2 135.7) (end 104 133.9) (width 0.2) (layer "F.Cu") (net 43))
-  (segment (start 140.9 124.6) (end 143.25 122.25) (width 0.2) (layer "F.Cu") (net 43))
   (segment (start 143.25 122.25) (end 143.25 115.8) (width 0.2) (layer "F.Cu") (net 43))
-  (segment (start 90.18 136.73) (end 91.45 138) (width 0.2) (layer "F.Cu") (net 43))
-  (segment (start 108.5 124.6) (end 140.9 124.6) (width 0.2) (layer "F.Cu") (net 43))
-  (segment (start 104 133.9) (end 104 129.1) (width 0.2) (layer "F.Cu") (net 43))
-  (segment (start 100 138) (end 102.2 135.8) (width 0.2) (layer "F.Cu") (net 43))
-  (segment (start 91.45 138) (end 100 138) (width 0.2) (layer "F.Cu") (net 43))
+  (segment (start 140.9 124.6) (end 143.25 122.25) (width 0.2) (layer "F.Cu") (net 43))
+  (segment (start 91.9 138) (end 100.5 138) (width 0.2) (layer "F.Cu") (net 43))
+  (segment (start 90.63 136.73) (end 91.9 138) (width 0.2) (layer "F.Cu") (net 43))
   (segment (start 132.68 51.68) (end 131 50) (width 0.2) (layer "F.Cu") (net 66))
   (segment (start 131 50) (end 115.77 50) (width 0.2) (layer "F.Cu") (net 66))

Commit message: Updated Nav can board Mk2
Parts:
- added G***: LOGO, LOGO, B.Cu at (154.9, 65.3)
- added G***: LOGO, LOGO, B.Cu at (198.8, 121.9)
- added G***: LOGO, LOGO, B.Cu at (122.9, 65.3)
- added G***: LOGO, LOGO, B.Cu at (183.1, 65.3)
- added G***: LOGO, LOGO, B.Cu at (211.1, 64.3)
- added G***: LOGO, LOGO, B.Cu at (91.2, 64.8)
- added kibuzzard-6421C441: G***, kibuzzard-6421C441, F.Cu at (217.4, 120.7)
- added kibuzzard-6421C441: G***, kibuzzard-6421C441, F.Cu at (82.5, 120.4)
- added kibuzzard-6421C452: G***, kibuzzard-6421C452, F.Cu at (88.4, 77.2)
- added kibuzzard-6421C45D: G***, kibuzzard-6421C45D, F.Cu at (100.8, 79.5)
- added kibuzzard-6421C46C: G***, kibuzzard-6421C46C, F.Cu at (101.3, 111.0)
- added kibuzzard-6421C47E: G***, kibuzzard-6421C47E, F.Cu at (211.8, 79.0)
- added kibuzzard-6421C548: G***, kibuzzard-6421C548, F.Cu at (86.1, 131.6)
- added kibuzzard-6421C577: G***, kibuzzard-6421C577, F.Cu at (102.4, 56.9)
- added kibuzzard-6421C5BF: G***, kibuzzard-6421C5BF, F.Cu at (120.1, 53.8)
- added kibuzzard-6421C5E9: G***, kibuzzard-6421C5E9, F.Cu at (108.2, 127.3)
- added kibuzzard-6421CB63: G***, kibuzzard-6421CB63, F.Cu at (157.0, 136.1)
- added kibuzzard-6421CC2C: G***, kibuzzard-6421CC2C, F.Cu at (110.7, 91.7)
- added kibuzzard-6421CC3B: G***, kibuzzard-6421CC3B, F.Cu at (110.7, 112.5)
- SW202: value SW_SPDT -> 450301014042
- moved D202 74.3 mm to (213.3, 98.3), turned to 180 degrees
- moved D201 66.7 mm to (213.4, 101.6), turned to 180 degrees
- moved D301 57.9 mm to (206.2, 101.6)
- moved D302 55.2 mm to (211.1, 91.2), turned to -90 degrees
- moved J404 16.2 mm to (217.5, 113.0)
- moved F201 15.6 mm to (217.9, 92.3), turned to -90 degrees
- moved R201 14.1 mm to (190.6, 132.4), turned to -90 degrees
- moved JP201 10.3 mm to (166.5, 132.1)
- moved J401 10.1 mm to (82.7, 81.8)
- moved C204 9.56 mm to (164.4, 134.9), turned to 0 degrees
- moved C203 9.13 mm to (171.1, 133.4), turned to 90 degrees
- moved J403 8.74 mm to (82.0, 112.9)
- moved L201 7.17 mm to (165.8, 139.7), turned to 180 degrees
- moved R301 5.52 mm to (198.1, 67.3), turned to -90 degrees
- moved C503 5.46 mm to (212.1, 141.3), turned to 180 degrees
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Connections:
- D203 pad 2: /Steering interface/USB_D- -> /Steering interface/USB_D+
- D203 pad 3: /Steering interface/USB_D+ -> /Steering interface/USB_D-
- J301 pad 17: /Driving inteface/STO-IN1+ -> Vaux2
- J301 pad 18: /Driving inteface/STO-IN1- -> GND
- J301 pad 19: /Driving inteface/STO-IN2+ -> Vaux2
- J301 pad 20: /Driving inteface/STO-IN2- -> GND
Routing:
- net /Driving inteface/CANL: track 0.00 -> 303.8 mm, vias 0 -> 8
- net /Driving inteface/CANH: track 0.00 -> 296.0 mm, vias 0 -> 4
- net VCC: track 0.00 -> 104.1 mm, vias 0 -> 139
- net Vsensor: track 0.00 -> 103.4 mm, vias 0 -> 4
- net /Steering interface/Hall Sensor 3: track 0.00 -> 70.2 mm, vias 0 -> 1
- net /Steering interface/Hall Sensor 2: track 0.00 -> 63.5 mm, vias 0 -> 1
- net /Steering interface/Hall Sensor 1: track 0.00 -> 56.6 mm, vias 0 -> 1
- net /Steering interface/CAN ID 4: track 0.00 -> 54.6 mm, vias 0 -> 2
- net /Steering interface/CAN ID 3: track 0.00 -> 54.1 mm, vias 0 -> 2
- net /Steering interface/CAN ID 2: track 0.00 -> 53.1 mm, vias 0 -> 2
- net /Steering interface/CAN ID 1: track 0.00 -> 46.3 mm, vias 0 -> 2
- net /Steering interface/CAN ID 5: track 0.00 -> 45.1 mm
- net /Steering interface/Auto bit rate: track 0.00 -> 44.9 mm
- net Vaux: track 0.00 -> 37.2 mm, vias 0 -> 11
- net GND: track 0.00 -> 32.7 mm, vias 10 -> 668
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- added copper zone on B.Cu, net /Driving inteface/M1/+M
- added copper zone on B.Cu, net /Driving inteface/M2/-M
- added copper zone on B.Cu, net /Driving inteface/M3
- added copper zone on F.Cu, net /Steering interface/LX
- added copper zone on B.Cu, net /Steering interface/M1/+M
- added copper zone on B.Cu, net /Steering interface/M2/-M
- added copper zone on B.Cu, net /Steering interface/M3
- added copper zone on F.Cu, net /Steering interface/MAX_VCC
- added copper zone on B.Cu, net /Steering interface/VCC_FUSED
- added copper zone on B.Cu, net GND
- added copper zone on In1.Cu, net GND
- added copper zone on In2.Cu, net GND
- added copper zone on F.Cu, net Net-(C501-Pad1)
- added copper zone on F.Cu, net Net-(C502-Pad1)
- added copper zone on F.Cu, net Net-(C503-Pad1)
- added copper zone on F.Cu, net Net-(C504-Pad1)
- added copper zone on B.Cu, net VCC
- added copper zone on B.Cu, net VDD
- added copper zone on F.Cu, net VDD
- added copper zone on B.Cu, net Vaux
- added copper zone on F.Cu, net Vaux
Other:
- outline, holes or cut-outs redrawn
- board text added: "AUTOBITRATE"
- board text added: "CAN TERM"
- board text added: "CANID 1"
- board text added: "CANID 2"
- board text added: "CANID 3"
- board text added: "CANID 4"
- board text added: "CANID 5"

Commit message: Updated Nav can board Mk2
Routing:
- net VCC: vias 139 -> 153
- net GND: vias 668 -> 695

Commit message: Nav board now bullet riddled
Routing:
- net /Driving inteface/CANH: track 296.0 -> 346.9 mm, vias 4 -> 7
- net /Driving inteface/CANL: track 303.8 -> 353.6 mm, vias 8 -> 10
- net /Steering interface/DSP_TxD: track 20.9 -> 3.70 mm, vias 2 -> 0
- net /Steering interface/CAN ID 2: track 53.1 -> 46.6 mm, vias 2 -> 4
- net /Steering interface/CAN ID 3: track 54.1 -> 48.5 mm, vias 2 -> 4
- net /Steering interface/CAN ID 4: track 54.6 -> 49.1 mm
- net /Steering interface/CAN ID 1: track 46.3 -> 43.6 mm, vias 2 -> 4
- net GND: track 32.7 -> 31.2 mm, vias 695 -> 870
- net /Steering interface/Clock/HsDigOUT1_A55: track 29.4 -> 30.2 mm
- net VCC: vias 153 -> 218
- net /Steering interface/M3: vias 46 -> 24
- net /Steering interface/M2/-M: vias 23 -> 13
- net /Steering interface/M1/+M: vias 38 -> 21
- net /Driving inteface/M3: vias 73 -> 38
- net /Driving inteface/M2/-M: vias 60 -> 30
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
Commit message: Updatede nav_controller_interface_v2
Routing:
- net /Driving inteface/CANL: track 353.6 -> 316.4 mm
- net GND: track 31.2 -> 26.8 mm, vias 870 -> 883
- net /Driving inteface/CANH: track 346.9 -> 344.5 mm, vias 7 -> 6
- net /Steering interface/CAN ID 2: track 46.6 -> 45.6 mm
- net /Steering interface/Hall Sensor 3: track 70.2 -> 71.1 mm
Other:
- board text added: "EPFL Xplore"
- board text added: "Made by Yassine Bakkali, Vincent Nguyen"
- board text added: "Rev 2.0"

Commit message: Corrected CANL line not connected to switch for Driving
Routing:
- net /Driving inteface/CANL: track 316.4 -> 355.4 mm
- net /Driving inteface/CANH: track 344.5 -> 343.7 mm
- net VCC: vias 218 -> 190
- net GND: vias 883 -> 829
