File: nav_controller_interface_v2/power_can_connectors.kicad_sch (KiCad schematic)
At the start: 4 parts

Commit message: Added v2 of nav interface board
Parts:
- gave numbers to parts that had none: 4
Changed lines of the file:
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@@
   (symbol (lib_id "power:GND") (at 125.095 52.705 0) (unit 1)
     (in_bom yes) (on_board yes) (fields_autoplaced)
-    (property "Reference" "#PWR?" (id 0) (at 125.095 59.055 0)
+    (property "Reference" "#PWR0405" (id 0) (at 125.095 59.055 0)
       (effects (font (size 1.27 1.27)) hide)
     )
@@
   (symbol (lib_id "power:GND") (at 62.865 51.435 0) (unit 1)
     (in_bom yes) (on_board yes) (fields_autoplaced)
-    (property "Reference" "#PWR?" (id 0) (at 62.865 57.785 0)
+    (property "Reference" "#PWR0402" (id 0) (at 62.865 57.785 0)
       (effects (font (size 1.27 1.27)) hide)
     )
@@
   (symbol (lib_id "power:GND") (at 62.865 83.185 0) (unit 1)
     (in_bom yes) (on_board yes) (fields_autoplaced)
-    (property "Reference" "#PWR?" (id 0) (at 62.865 89.535 0)
+    (property "Reference" "#PWR0404" (id 0) (at 62.865 89.535 0)
       (effects (font (size 1.27 1.27)) hide)
     )
@@
   (symbol (lib_id "power:VCC") (at 62.865 37.465 0) (unit 1)
     (in_bom yes) (on_board yes) (fields_autoplaced)
-    (property "Reference" "#PWR?" (id 0) (at 62.865 41.275 0)
+    (property "Reference" "#PWR0401" (id 0) (at 62.865 41.275 0)
       (effects (font (size 1.27 1.27)) hide)
     )
@@
   (symbol (lib_id "power:VCC") (at 62.865 69.215 0) (unit 1)
     (in_bom yes) (on_board yes) (fields_autoplaced)
-    (property "Reference" "#PWR?" (id 0) (at 62.865 73.025 0)
+    (property "Reference" "#PWR0403" (id 0) (at 62.865 73.025 0)
       (effects (font (size 1.27 1.27)) hide)
     )
@@
   (symbol (lib_id "Connector_Generic:Conn_01x04") (at 139.065 42.545 0) (unit 1)
     (in_bom yes) (on_board yes) (fields_autoplaced)
-    (property "Reference" "J?" (id 0) (at 141.605 42.5449 0)
+    (property "Reference" "J403" (id 0) (at 141.605 42.5449 0)
       (effects (font (size 1.27 1.27)) (justify left))
     )
@@
   (symbol (lib_id "Connector_Generic:Conn_01x02") (at 74.295 75.565 0) (unit 1)
     (in_bom yes) (on_board yes) (fields_autoplaced)
-    (property "Reference" "J?" (id 0) (at 76.835 75.5649 0)
+    (property "Reference" "J402" (id 0) (at 76.835 75.5649 0)
       (effects (font (size 1.27 1.27)) (justify left))
     )
@@
   (symbol (lib_id "Connector_Generic:Conn_01x04") (at 139.065 74.93 0) (unit 1)
     (in_bom yes) (on_board yes) (fields_autoplaced)
-    (property "Reference" "J?" (id 0) (at 141.605 74.9299 0)
+    (property "Reference" "J404" (id 0) (at 141.605 74.9299 0)
       (effects (font (size 1.27 1.27)) (justify left))
     )
@@
   (symbol (lib_id "Connector_Generic:Conn_01x02") (at 74.295 43.815 0) (unit 1)
     (in_bom yes) (on_board yes) (fields_autoplaced)
-    (property "Reference" "J?" (id 0) (at 76.835 43.8149 0)
+    (property "Reference" "J401" (id 0) (at 76.835 43.8149 0)
       (effects (font (size 1.27 1.27)) (justify left))
     )
@@
   (symbol (lib_id "power:GND") (at 125.095 85.09 0) (unit 1)
     (in_bom yes) (on_board yes) (fields_autoplaced)
-    (property "Reference" "#PWR?" (id 0) (at 125.095 91.44 0)
+    (property "Reference" "#PWR0406" (id 0) (at 125.095 91.44 0)
       (effects (font (size 1.27 1.27)) hide)
     )

Commit message: Added schematic for can controller interface v2
Parts:
- J401, J402: Distributor (none) -> TME; Distributor ref (none) -> XT60UPB-M; Manufacturer ref (none) -> XT60UPB-M
- J403, J404: Distributor (none) -> Mouser; Distributor ref (none) -> 538-502584-0460; Manufacturer ref (none) -> 502584-0460
Connections:
- net GND: now also J401.1 (Pin_1), J402.1 (Pin_1); no longer J401.2 (Pin_2), J402.2 (Pin_2)
- net VCC: now also J401.2 (Pin_2), J402.2 (Pin_2); no longer J401.1 (Pin_1), J402.1 (Pin_1)
Other:
- note added: "Back to overview"

Commit message: Changed placement of CAN connectors
Connections:
- net CANH: now also J403.2 (Pin_2), J404.2 (Pin_2); no longer J403.1 (Pin_1), J404.1 (Pin_1)
- net CANL: now also J403.1 (Pin_1), J404.1 (Pin_1); no longer J403.2 (Pin_2), J404.2 (Pin_2)
Changed lines of the file:
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@@
+    (stroke (width 0) (type default))
+  )
+  (wire (pts (xy 125.095 72.39) (xy 133.985 72.39))
     (stroke (width 0) (type default))
   )
@@
     (stroke (width 0) (type default))
   )
-  (bus (pts (xy 122.555 69.85) (xy 122.555 69.215))
+  (wire (pts (xy 125.095 74.93) (xy 133.985 74.93))
     (stroke (width 0) (type default))
   )
-  (wire (pts (xy 125.095 74.93) (xy 133.985 74.93))
+  (bus (pts (xy 122.555 69.85) (xy 122.555 69.215))
     (stroke (width 0) (type default))
   )
@@
     (stroke (width 0) (type default))
   )
-  (wire (pts (xy 125.095 72.39) (xy 133.985 72.39))
-    (stroke (width 0) (type default))
-  )
   (wire (pts (xy 125.095 42.545) (xy 133.985 42.545))
     (stroke (width 0) (type default))
@@
     (effects (font (size 2.85 2.85) (thickness 0.6) bold italic) (justify right bottom) (href "#1"))
   )
-  (label "CANL" (at 133.985 74.93 180) (fields_autoplaced)
+  (label "CANL" (at 133.985 72.39 180) (fields_autoplaced)
     (effects (font (size 1.27 1.27)) (justify right bottom))
   )
@@
     (effects (font (size 1.27 1.27)) (justify right bottom))
   )
-  (label "CANH" (at 133.985 40.005 180) (fields_autoplaced)
+  (label "CANL" (at 133.985 40.005 180) (fields_autoplaced)
     (effects (font (size 1.27 1.27)) (justify right bottom))
   )
-  (label "CANL" (at 133.985 42.545 180) (fields_autoplaced)
+  (label "CANH" (at 133.985 42.545 180) (fields_autoplaced)
     (effects (font (size 1.27 1.27)) (justify right bottom))
   )
-  (label "CANH" (at 133.985 72.39 180) (fields_autoplaced)
+  (label "CANH" (at 133.985 74.93 180) (fields_autoplaced)
     (effects (font (size 1.27 1.27)) (justify right bottom))
   )

Commit message: finished routing
Connections:
- net CANH: now also J403.1 (Pin_1), J404.1 (Pin_1); no longer J403.2 (Pin_2), J404.2 (Pin_2)
- net CANL: now also J403.2 (Pin_2), J404.2 (Pin_2); no longer J403.1 (Pin_1), J404.1 (Pin_1)
Changed lines of the file:
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@@
     (effects (font (size 2.85 2.85) (thickness 0.6) bold italic) (justify right bottom) (href "#1"))
   )
-  (label "CANL" (at 133.985 72.39 180) (fields_autoplaced)
+  (label "CANL" (at 133.985 74.93 180) (fields_autoplaced)
     (effects (font (size 1.27 1.27)) (justify right bottom))
   )
@@
     (effects (font (size 1.27 1.27)) (justify right bottom))
   )
-  (label "CANL" (at 133.985 40.005 180) (fields_autoplaced)
+  (label "CANL" (at 133.985 42.545 180) (fields_autoplaced)
     (effects (font (size 1.27 1.27)) (justify right bottom))
   )
-  (label "CANH" (at 133.985 42.545 180) (fields_autoplaced)
+  (label "CANH" (at 133.985 40.005 180) (fields_autoplaced)
     (effects (font (size 1.27 1.27)) (justify right bottom))
   )
-  (label "CANH" (at 133.985 74.93 180) (fields_autoplaced)
+  (label "CANH" (at 133.985 72.39 180) (fields_autoplaced)
     (effects (font (size 1.27 1.27)) (justify right bottom))
   )
