File: nav_controller_interface_v2/steering_interface.kicad_sch (KiCad schematic)
At the start: 22 parts

Commit message: Added v2 of nav interface board
Parts:
- removed U?: SRV05-4, Package_TO_SOT_SMD:SOT-23-6, symbol Power_Protection:SRV05-4
- added D203: PRTR5V0U2X, Package_TO_SOT_SMD:SOT-143, symbol Power_Protection:PRTR5V0U2X
- C201: renamed from C?; Distributor (none) -> Mouser; Distributor ref (none) -> 667-EEH-ZA1V680XP; Manufacturer ref (none) -> EEH-ZA1V680XP
- C202: renamed from C?; Distributor (none) -> Mouser; Distributor ref (none) -> 581-06035C105KAT2A; Manufacturer ref (none) -> 06035C105KAT2A
- C203: renamed from C?; Distributor (none) -> Mouser; Distributor ref (none) -> 80-C0603C105K9R; Manufacturer ref (none) -> C0603C105K9RACTU
- C204: renamed from C?; Distributor (none) -> Mouser; Distributor ref (none) -> 187-CL31B106KQHNFNE; Manufacturer ref (none) -> CL31B106KQHNFNE
- D201, D202: renamed from D?; Distributor (none) -> Mouser; Distributor ref (none) -> 637-SMF30A; Manufacturer ref (none) -> SMF30A
- F201: renamed from F?; value 0157010.DR -> 0157010; Distributor (none) -> Mouser; Distributor ref (none) -> 576-0157010.DR; Manufacturer ref (none) -> 0157010.DR
- J201: renamed from J?; Distributor (none) -> Mouser; Distributor ref (none) -> 200-LSHM1402.5LDVANK; Manufacturer ref (none) -> LSHM-140-02.5-L-DV-A-N-K-TR
- J202: renamed from J?; Distributor (none) -> Mouser; Distributor ref (none) -> 538-39-28-1043; Manufacturer ref (none) -> 39-28-1043
- J203: renamed from J?; footprint (none) -> 0_connectors:MOLEX_43045-0624; Distributor (none) -> Mouser; Distributor ref (none) -> 538-43045-0624; Manufacturer ref (none) -> 43045-0624
- gave numbers to parts that had none: 11
Connections:
- net +VC is gone; now on an unnamed net: D202.1 (K), J201.26 (Pin_26)
- net GND: now also D203.1 (GND)
- net USB_D+: now also D203.3 (I/O2)
- net USB_D-: now also D203.2 (I/O1)
- net VBUS: now also D203.4 (VCC)
Other:
- note added: "Connectors"
- note added: "Logic"
- note added: "Power"
- note added: "RS422 transceiver (SSI absolute encoder)"
- note added: "https://www.maxongroup.com/medias/sys_master/root/8839867334686/EPOS4-Micro-24-5-CAN-Hardware-Reference-En.pdf"
- note removed: "RS422 transceiver for SSI encoder"
- moved on the sheet: H201, H202, J202, J203, J204, J205, J206, R201, SW201

Commit message: Added schematic for can controller interface v2
Parts:
- removed U201: MAX15462BATA+T, nav_fp:SON50P200X200X80-8N, symbol custom_lib:MAX15462BATA+T
- added G201: ~, 0_maxon_controllers:Micro_24_5_CAN, symbol 0_graphic:EPOS4_Micro_24/5_CAN
- added U201: MAX15462BATA+T, 0_regulator:MAX15462BATA, symbol 0_regulator:MAX15462
- C202, C203: footprint Capacitor_SMD:C_0603_1608Metric_Pad1.08x0.95mm_HandSolder -> Capacitor_SMD:C_0603_1608Metric
- F201: footprint Fuse:Fuseholder_Littelfuse_Nano2_157x -> 0_fuse:Fuseholder_Littelfuse_Nano2_157x
- H201, H202: footprint MountingHole:MountingHole_2.2mm_M2_Pad_Via -> MountingHole:MountingHole_2.2mm_M2_Pad; Distributor (none) -> Mouser; Distributor ref (none) -> 710-9774045243R; Manufacturer ref (none) -> 9774045243R; now in the parts list
- J201: footprint Connector_Samtec:Samtec_LSHM-140-xx.x-x-DV-N_2x40_P0.50mm_Vertical -> 0_connectors:Samtec_LSHM-140-xx.x-x-DV-N_2x40_P0.50mm_Vertical
- J202: footprint Connector_Molex:Molex_Mini-Fit_Jr_5566-04A_2x02_P4.20mm_Vertical -> 0_connectors:Molex_Mini-Fit_Jr_5566-04A_2x02_P4.20mm_Vertical
- J204: footprint Connector_PinHeader_2.54mm:PinHeader_2x05_P2.54mm_Vertical_SMD -> 0_connectors:SAMTEC-HTST-105-01-X-DV; Distributor (none) -> Mouser; Distributor ref (none) -> 200-HTSS10501TDV; Manufacturer ref (none) -> HTSS-105-01-T-DVHTSS-105-01-T-DV
- J205: footprint (none) -> 0_connectors:MOLEX_5031541090; Distributor (none) -> Mouser; Distributor ref (none) -> 538-503154-1090; Manufacturer ref (none) -> 503154-1090
- J206: footprint Connector_USB:USB_Micro-B_Molex-105133-0001 -> 0_connectors:USB_Micro-B_Molex-105133-0001; Distributor (none) -> Mouser; Distributor ref (none) -> 538-105133-0001; Manufacturer ref (none) -> 105133-0001
- JP201: footprint (none) -> Jumper:SolderJumper-2_P1.3mm_Open_RoundedPad1.0x1.5mm; now left out of the parts list
- L201: value Coilcraft LPS4018-473ML (47uH) -> LQH5BPH470MT0L (47uH); footprint Inductor_SMD:L_Coilcraft_LPS4018 -> 0_inductors:LQH5BPB100MT0L; Distributor (none) -> Mouser; Distributor ref (none) -> 81-LQH5BPH470MT0L; Manufacturer ref (none) -> LQH5BPH470MT0L
- R201: Distributor (none) -> Mouser; Distributor ref (none) -> 71-CRCW0603120RFKEAH; Manufacturer ref (none) -> CRCW0603120RFKEAHP
- SW201: footprint (none) -> 0_switch:2188LPST; Distributor (none) -> Mouser; Distributor ref (none) -> 774-2188LPST; Manufacturer ref (none) -> 218-8LPST
- SW202: value SW_SPDT -> 450301014042; footprint (none) -> 0_switch:450301014042; Distributor (none) -> Mouser; Distributor ref (none) -> 710-450301014042; Manufacturer ref (none) -> 450301014042
Connections:
- net GND: now also U201.7 (GND)
- net VCC: now also U201.1 (VIN), U201.2 (EN/UVLO); no longer D201.1 (K)
- net VDD: now also U201.4 (FB/Vout)
- net MAX_VCC: now reaches C203.1
- net MAX_VCC: now also U201.3 (VCC)
- net MODE: now reaches JP201.2 (B)
- net MODE: now also U201.5 (MODE)
- net LX: now reaches L201.1
- net LX: now also U201.8 (LX)
- net VCC_FUSED: now reaches C201.1, D202.1 (K), F201.2, J201.19 (Pin_19), J201.20 (Pin_20), J201.21 (Pin_21), J201.22 (Pin_22), J201.23 (Pin_23), J201.24 (Pin_24), J201.26 (Pin_26)
- net VCC_FUSED: now also D201.1 (K)
- net ID 1 renamed CAN ID 1
- net ID 2 renamed CAN ID 2
- net ID 3 renamed CAN ID 3
- net ID 4 renamed CAN ID 4
- net ID 5 renamed CAN ID 5
- net ID 6 renamed CAN ID 6
- no-connect marks 13 -> 27
Other:
- note added: "6"
- note added: "Back to overview"
- note added: "Datasheet"
- note added: "Standoffs"
- note removed: "Mounting holes"
- note removed: "https://www.maxongroup.com/medias/sys_master/root/8839867334686/EPOS4-Micro-24-5-CAN-Hardware-Reference-En.pdf"
- company: (none) -> EPFL Xplore
- title: (none) -> Steering controller interface (EPOS4 Micro 24/5 CAN)
- moved on the sheet: D201, F201, L201

Commit message: Updated Nav can board Mk2
Connections:
- net USB_D+: now also D203.2 (I/O1); no longer D203.3 (I/O2)
- net USB_D-: now also D203.3 (I/O2); no longer D203.2 (I/O1)
Changed lines of the file:
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@@
   (junction (at 284.48 137.795) (diameter 0) (color 0 0 0 0)
   )
-  (junction (at 314.96 46.355) (diameter 0) (color 0 0 0 0)
+  (junction (at 314.96 43.815) (diameter 0) (color 0 0 0 0)
+  )
+  (junction (at 346.71 46.355) (diameter 0) (color 0 0 0 0)
   )
   (junction (at 135.255 90.17) (diameter 0) (color 0 0 0 0)
@@
   )
   (junction (at 83.82 102.87) (diameter 0) (color 0 0 0 0)
-  )
-  (junction (at 346.71 43.815) (diameter 0) (color 0 0 0 0)
   )
   (junction (at 90.17 80.01) (diameter 0) (color 0 0 0 0)
@@
     (stroke (width 0) (type default))
   )
-  (wire (pts (xy 314.96 46.355) (xy 314.96 67.945))
-    (stroke (width 0) (type default))
-  )
   (wire (pts (xy 105.41 125.73) (xy 128.27 125.73))
     (stroke (width 0) (type default))
@@
     (stroke (width 0) (type default))
   )
+  (wire (pts (xy 346.71 46.355) (xy 346.71 67.945))
+    (stroke (width 0) (type default))
+  )
   (wire (pts (xy 342.9 212.09) (xy 342.9 205.74))
     (stroke (width 0) (type default))
@@
     (stroke (width 0) (type default))
   )
-  (wire (pts (xy 346.71 43.815) (xy 358.14 43.815))
-    (stroke (width 0) (type default))
-  )
   (wire (pts (xy 105.41 118.11) (xy 128.27 118.11))
     (stroke (width 0) (type default))
@@
     (stroke (width 0) (type default))
   )
+  (wire (pts (xy 314.96 43.815) (xy 358.14 43.815))
+    (stroke (width 0) (type default))
+  )
   (wire (pts (xy 170.18 151.765) (xy 170.18 137.795))
     (stroke (width 0) (type default))
@@
     (stroke (width 0) (type default))
   )
-  (wire (pts (xy 314.96 46.355) (xy 358.14 46.355))
+  (wire (pts (xy 306.07 46.355) (xy 346.71 46.355))
     (stroke (width 0) (type default))
   )
@@
     (stroke (width 0) (type default))
   )
+  (wire (pts (xy 346.71 46.355) (xy 358.14 46.355))
+    (stroke (width 0) (type default))
+  )
   (wire (pts (xy 90.17 49.53) (xy 92.71 49.53))
     (stroke (width 0) (type default))
@@
     (stroke (width 0) (type default))
   )
-  (wire (pts (xy 306.07 46.355) (xy 314.96 46.355))
-    (stroke (width 0) (type default))
-  )
   (wire (pts (xy 83.82 105.41) (xy 83.82 107.95))
     (stroke (width 0) (type default))
@@
     (stroke (width 0) (type default))
   )
-  (wire (pts (xy 306.07 43.815) (xy 346.71 43.815))
+  (wire (pts (xy 306.07 43.815) (xy 314.96 43.815))
     (stroke (width 0) (type default))
   )
@@
     (stroke (width 0) (type default))
   )
-  (wire (pts (xy 346.71 43.815) (xy 346.71 67.945))
-    (stroke (width 0) (type default))
-  )
   (polyline (pts (xy 243.84 104.14) (xy 404.495 104.14))
     (stroke (width 0) (type default))
@@
     (stroke (width 0) (type default))
   )
+  (wire (pts (xy 314.96 43.815) (xy 314.96 67.945))
+    (stroke (width 0) (type default))
+  )

Commit message: finished routing
Connections:
- net CANH: now also SW201.10; no longer R201.1
- net CANL: now also R201.1; no longer SW201.10
- net DSP_TxD: no longer J201.77 (Pin_77)
- new net DSP_RxD: J201.77 (Pin_77)
Changed lines of the file:
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@@
     (effects (font (size 1.27 1.27)) (justify left bottom))
   )
-  (label "CANL" (at 285.75 146.685 0) (fields_autoplaced)
-    (effects (font (size 1.27 1.27)) (justify left bottom))
+  (label "CANL" (at 256.54 146.685 180) (fields_autoplaced)
+    (effects (font (size 1.27 1.27)) (justify right bottom))
   )
   (label "Channel A" (at 73.66 118.11 0) (fields_autoplaced)
@@
     (effects (font (size 1.27 1.27)) (justify right bottom))
   )
-  (label "CANH" (at 256.54 146.685 180) (fields_autoplaced)
-    (effects (font (size 1.27 1.27)) (justify right bottom))
+  (label "CANH" (at 285.75 146.685 0) (fields_autoplaced)
+    (effects (font (size 1.27 1.27)) (justify left bottom))
   )
   (label "SHIELD" (at 195.58 97.155 0) (fields_autoplaced)
@@
     (effects (font (size 1.27 1.27)) (justify right bottom))
   )
-  (label "DSP_TxD" (at 105.41 41.91 0) (fields_autoplaced)
+  (label "DSP_RxD" (at 105.41 41.91 0) (fields_autoplaced)
     (effects (font (size 1.27 1.27)) (justify left bottom))
   )
