File: node_pcb/orion_can/MCU.kicad_sch (KiCad schematic)
At the start: 53 parts, among them J201 SWD_02x05_1.27mm, J202 Conn_Picoblade_JST_DEBUG, SW201 CL-SB-12C-02, SW202 MJTP1140ATR, U201 STM32H750VBT6, Y201 ABM10W-48.0000MHZ-8-D7G-T3, Y202 ECS-.327-7-12-C-TR9 (32.768 K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

Commit message: Changed layout of canorion
Connections:
- net +3.3V: no longer C201.1, C202.1, C204.1, C205.1, C206.1, C208.1, C210.1, C212.1, FB201.2, R1.1, R2.1, R208.1, R209.1, R212.1, R213.1, R214.1, R215.1, U201.100 (VDD), U201.11 (VDD), U201.27 (VDD), U201.50 (VDD), U201.6 (VBAT), U201.75 (VDD)
- net PE2 renamed PR1_CTRL
- new net VMCU: C201.1, C202.1, C204.1, C205.1, C206.1, C208.1, C210.1, C212.1, FB201.2, R1.1, R2.1, R208.1, R209.1, R212.1, R213.1, R214.1, R215.1, U201.100 (VDD), U201.11 (VDD), U201.27 (VDD), U201.50 (VDD), U201.6 (VBAT), U201.75 (VDD)
- no-connect marks 22 -> 19
