File: hats/RS485_interface/RS485_interface/RS485_interface.kicad_sch (KiCad schematic)
At the start: 13 parts, among them J1 Hat_connector_hole, J2 Conn_01x04, J3 Conn_01x04, U1 MAX485E

Commit message: RS485 transceiver 2
Parts:
- removed U1: MAX485E, Package_SO:SOIC-8_3.9x4.9mm_P1.27mm, symbol Interface_UART:MAX485E
- added C3: 0.1uF, Capacitor_SMD:C_0603_1608Metric_Pad1.08x0.95mm_HandSolder, symbol Device:C_Small
- added C4: 1uF, Capacitor_SMD:C_0603_1608Metric_Pad1.08x0.95mm_HandSolder, symbol Device:C_Small
- added D1: SM5819PL, Diode_SMD:D_SOD-123F, symbol Device:D_Small
- added L1: 10uH, footprint.ugly:IND_CDRH3D11HPNP-100NC_SUM, symbol Device:L_Small
- added R8: 5.1k, Resistor_SMD:R_0603_1608Metric_Pad0.98x0.95mm_HandSolder, symbol Device:R_Small
- added R9: 92.82k, Resistor_SMD:R_0603_1608Metric_Pad0.98x0.95mm_HandSolder, symbol Device:R_Small
- added U2: AP3012, Package_TO_SOT_SMD:SOT-23-5, symbol Regulator_Switching:AP3012
- added U3: MAX3486, Package_SO:SOIC-8_3.9x4.9mm_P1.27mm, symbol Interface_UART:MAX3486
- J2, J3: footprint 0_connectors:PicoBlade-JST-GH-1x04_1.25mm_Vertical -> Connector_JST:JST_PH_B4B-PH-SM4-TB_1x04-1MP_P2.00mm_Vertical
Connections:
- net +3V3: now also U3.8 (VCC)
- net +5V: now also C3.1, L1.1, U2.4 (~{SHDN}), U2.5 (IN); no longer J2.1 (Pin_1), J3.1 (Pin_1)
- net GND: now also C3.2, C4.2, R8.2, U2.2 (GND), U3.5 (GND)
- net RS485-: now reaches J2.2 (Pin_2), J3.2 (Pin_2), R5.2, R7.1
- net RS485-: now also U3.7 (B)
- net RS485+: now reaches J2.3 (Pin_3), J3.3 (Pin_3), R6.1, R7.2
- net RS485+: now also U3.6 (A)
- net at J1.13 (GPIO_5), R2.2: now also U3.2 (~{RE})
- net at J1.12 (GPIO_4), R1.2: now also U3.1 (RO)
- net at J1.14 (GPIO_6), R4.2: now also U3.4 (DI)
- net at J1.11 (GPIO_3), R3.2: now also U3.3 (DE)
- new net: R8.1, R9.2, U2.3 (FB)
- new net: D1.2 (A), L1.2, U2.1 (SW)
- new net +24V: C4.1, D1.1 (K), J2.1 (Pin_1), J3.1 (Pin_1), R9.1
Other:
- note added: "It's just a phase"
- company: (none) -> EPFL Xplore
- title: (none) -> RS485 interface board
- moved on the sheet: C1, C2, J1, J2, J3, R1, R2, R3, R4, R5, R6, R7

Commit message: small changes
Other:
- note added: "Come, come and put that disgusting mission patch here. I dare you"
Changed lines of the file:
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@@
     (date "2023-07-14")
     (company "EPFL Xplore")
-    (comment 3 "Author : Your mom")
+    (comment 3 "Author : Yassine Bakkali")
   )
   (junction (at 153.67 37.465) (diameter 0) (color 0 0 0 0)
@@
     (effects (font (size 1.27 1.27)) (justify left bottom))
   )
+  (text "Come, come and put that disgusting \nmission patch here. I dare you"
+    (at 219.075 177.165 0)
+    (effects (font (size 2.27 2.27) (thickness 0.454) bold) (justify left bottom))
+  )
   (label "RS485+" (at 67.945 149.225 0) (fields_autoplaced)
