File: hats/Yassine_Leds/Yassine_Leds.kicad_sch (KiCad schematic)
At the start: 57 parts, among them IC1 74LVCH1T45GW,125, J1 Hat_connector_hole, J2 JST_XH_01x03, J3 USB_C_Receptacle_USB2.0, J4 XT-30, SW2 KMR731NG LFS, SW3 KMR731NG LFS, U1 RP2040, U2 W25Q128JVS, U4 TPS2116DRLR, U5 MIC5504-3.3YM5, U6 TPS2121RUXR, U7 USBLC6-2P6, Y1 RH100-12.000-18-2020-EXT-TR

Commit message: Advanced on the proper led board
Parts:
- removed D1: D_Schottky_Small_Filled, symbol Device:D_Schottky_Small_Filled
- removed IC1: 74LVCH1T45GW,125, Package_TO_SOT_SMD:SOT-363_SC-70-6_Handsoldering, symbol 0_level_shifter:74LVCH1T45GW,125
- removed J2: JST_XH_01x03, Connector_JST:JST_XH_B3B-XH-AM_1x03_P2.50mm_Vertical, symbol Connector_Generic:Conn_01x03
- added C25, C26: 0.1uF, Capacitor_SMD:C_0402_1005Metric_Pad0.74x0.62mm_HandSolder, symbol Device:C_Small
- added J5: Conn_01x04, Connector_JST:JST_XH_B4B-XH-AM_1x04_P2.50mm_Vertical, symbol Connector_Generic:Conn_01x04
- added R19: 10k, Resistor_SMD:R_0402_1005Metric_Pad0.72x0.64mm_HandSolder, symbol Device:R_Small
- added U3: TXB0102DCT, Package_SO:TSSOP-8_3x3mm_P0.65mm, symbol Logic_LevelTranslator:TXB0102DCT
Connections:
- net +3V3: now also C25.2, R19.2, U3.3 (VCCA)
- net +5V: now also C26.2, J5.1 (Pin_1), U3.7 (VCCB)
- net GND: now also C25.1, C26.1, J5.4 (Pin_4), U3.2 (GND)
- net I2C0_SCL: now also U1.41 (GPIO29_ADC3); no longer U1.3 (GPIO1)
- net I2C0_SDA: now also U1.40 (GPIO28_ADC2); no longer U1.2 (GPIO0)
- net LED_DATA: now also J5.2 (Pin_2), U3.8 (B1)
- net RP_GPIO12: now also U1.17 (GPIO14); no longer U1.15 (GPIO12)
- net RP_GPIO13: now reaches U1.18 (GPIO15)
- net SPI1_RX: now reaches U1.36 (GPIO24)
- net SPI1_RX: now also J1.4 (SPI_MOSI)
- net SPI1_~{CS}: now reaches U1.37 (GPIO25)
- net SPI1_~{CS}: now also J1.6 (SPI_CS)
- net SPI1_SCK: now reaches U1.38 (GPIO26_ADC0)
- net SPI1_SCK: now also J1.3 (SPI_SCK)
- net SPI1_TX: now reaches U1.39 (GPIO27_ADC1)
- net SPI1_TX: now also J1.5 (SPI_MISO)
- net SPI0_RX: no longer names the net of U1.6 (GPIO4)
- net SPI0_RX: no longer J1.4 (SPI_MOSI)
- net SPI0_SCK: no longer names the net of U1.4 (GPIO2)
- net SPI0_SCK: no longer J1.3 (SPI_SCK)
- net SPI0_TX: no longer names the net of U1.5 (GPIO3)
- net SPI0_TX: no longer J1.5 (SPI_MISO)
- net SPI0_~{CS}: no longer names the net of U1.7 (GPIO5)
- net SPI0_~{CS}: no longer J1.6 (SPI_CS)
- new net: R19.1, U3.6 (OE)
- new net LED_CLK: J5.3 (Pin_3)
- new net LED_CLOCK: U3.1 (B2)
- new net RP_GPIO14: U3.5 (A1)
- new net RP_GPIO15: U3.4 (A2)
Other:
- moved on the sheet: C19, C20, R9, U1, Y1

Commit message: Led ready for prototyping, awaiting clean up of schematic for austists and cringe redditors appreciation
Parts:
- J5: footprint Connector_JST:JST_XH_B4B-XH-AM_1x04_P2.50mm_Vertical -> Connector_JST:JST_XH_B4B-XH-A_1x04_P2.50mm_Vertical
Connections:
- net LED_CLOCK is gone; now on net LED_DATA: U3.1 (B2)
- net RP_GPIO12 is gone; now on net RP_GPIO14: U1.17 (GPIO14)
- net RP_GPIO13 is gone; now on net RP_GPIO15: U1.18 (GPIO15)
- net +5V: now also U6.1_1 (OUT), U6.8_1 (OUT)
- net +5V_EXT: now also J4.2 (Pin_2), U6.2_1 (IN2); no longer J4.1 (Pin_1)
- net +5V_MCU: now also U6.7_1 (IN1)
- net GND: now also J4.1 (Pin_1), U2.9 (EP); no longer J4.2 (Pin_2)
- net LED_CLK: now also U3.8 (B1)
- net LED_DATA: no longer U3.8 (B1)
- net MCU_GPIO1: no longer J1.9 (GPIO_1)
- net MCU_GPIO2: no longer J1.10 (GPIO_2)
- net MCU_GPIO3: no longer names the net of J1.11 (GPIO_3)
- net MCU_GPIO3: no longer U1.11 (GPIO8)
- net MCU_GPIO4: no longer names the net of J1.12 (GPIO_4)
- net MCU_GPIO4: no longer U1.12 (GPIO9)
- net MCU_GPIO5: no longer names the net of J1.13 (GPIO_5)
- net MCU_GPIO5: no longer U1.13 (GPIO10)
- net MCU_GPIO6: no longer names the net of J1.14 (GPIO_6)
- net MCU_GPIO6: no longer U1.14 (GPIO11)
- no-connect marks 22 -> 32
Other:
- moved on the sheet: C19, C20, J4, J5, R9, U1, Y1
