File: nav_controller_interface/nav_controller_interface_v3/nav_lower_controller/RS422_interface.kicad_sch (KiCad schematic)
At the start: 10 parts, among them U1 ISL8490E

Commit message: Nav board completed
Other:
- note removed: "Note: Vaux = 5VDC"
Changed lines of the file:
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@@
     (stroke (width 0) (type default))
-  )
-  (text "Note: Vaux = 5VDC" (at 138.43 25.4 0)
-    (effects (font (size 1.27 1.27)) (justify left bottom))
   )
   (text "Note: see 4-68 for reference circuit" (at 135.89 77.47 0)
@@
       (effects (font (size 1.27 1.27)) hide)
     )
-    (property "Value" "Vaux" (at 68.58 33.02 0)
+    (property "Value" "Vsensor" (at 68.58 33.02 0)
       (effects (font (size 1.27 1.27)))
     )
@@
       (effects (font (size 1.27 1.27)) hide)
     )
-    (property "Value" "Vaux" (at 133.35 24.765 0)
+    (property "Value" "Vsensor" (at 133.35 25.4 0)
       (effects (font (size 1.27 1.27)))
     )
