File: hats/voltmeter_Alexandre_Eliot/voltmeter_Alexandre_Eliot.kicad_pcb (KiCad board)
At the start: 2 copper layers, 30.7 x 33.1 mm, 18 parts, among them J1 Hat_connector, J2 5025850670, Q1 PJA3404, SW1 CL-SB-12C-01, U1 LT3960JMSE#PBF

Commit message: Voltmeter with changes
Parts:
- C3, C4: moved to B.Cu
- moved C4 2.61 mm to (149.3, 95.7), turned to 180 degrees
- moved C3 2.55 mm to (156.9, 95.0), turned to 0 degrees
- moved R7 1.06 mm to (151.0, 97.8)
- moved D2 0.94 mm to (152.1, 101.3)
- moved R6 0.68 mm to (153.2, 97.8)
- moved R2 0.53 mm to (155.1, 97.3)
- moved D1 0.52 mm to (156.2, 100.8)
- moved R5 0.49 mm to (157.2, 97.3)
Routing:
- net /TERM_MID_SCL: track 2.48 -> 8.77 mm, vias 0 -> 2
- net /TERM_MID_SDA: track 2.59 -> 7.99 mm, vias 0 -> 2
- net +3V3: track 50.9 -> 47.6 mm
- net Net-(Q1-D): track 16.2 -> 18.3 mm
- net GND: track 22.6 -> 24.0 mm, vias 44 -> 62
- net /CANSCL+: track 14.8 -> 13.9 mm
- net /CANSDA+: track 14.5 -> 13.8 mm
- net /CANSDA-: track 14.7 -> 14.1 mm

Commit message: redid routing high speed lines, removed MOSFET.
Parts:
- removed Q1: PJA3404, Package_TO_SOT_SMD:SOT-23
- C3, C4: moved to F.Cu
- moved C4 1.88 mm to (151.1, 96.3), turned to 90 degrees
- moved R7 1.23 mm to (149.8, 97.6)
- moved D2 1.06 mm to (151.1, 101.1)
- moved R6 0.86 mm to (152.4, 97.6)
- moved C3 0.82 mm to (156.1, 95.2), turned to 90 degrees
- moved R5 0.51 mm to (156.9, 97.7)
- moved R2 0.49 mm to (155.3, 97.7)
- moved D1 0.35 mm to (156.1, 101.1)
- moved R1 0.20 mm to (159.7, 89.6)
Connections:
- R1 pad 2: Net-(Q1-D) -> /MODE
- SW1 pad 3: Net-(Q1-D) -> /MODE
Routing:
- net /MODE: track 4.23 -> 22.9 mm
- net Net-(Q1-D): track 18.3 -> 0.00 mm
- net /TERM_MID_SCL: track 8.77 -> 2.71 mm, vias 2 -> 0
- net /TERM_MID_SDA: track 7.99 -> 2.57 mm, vias 2 -> 0
- net /CANSDA-: track 14.1 -> 15.7 mm
- net GND: track 24.0 -> 22.7 mm, vias 62 -> 72
- net /CANSCL+: track 13.9 -> 14.7 mm
- net /CANSDA+: track 13.8 -> 14.6 mm
- net /CANSCL-: track 14.3 -> 14.9 mm

Commit message: updated power trace
Routing:
- net +3V3: track 47.6 -> 42.9 mm, vias 1 -> 0
- added copper zone on F.Cu, net +3V3
Changed lines of the file:
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@@
     (property "Sheetname" "")
     (attr through_hole)
-    (fp_text reference "J1" (at 0 -0.5 unlocked) (layer "F.SilkS")
+    (fp_text reference "J1" (at 0.840357 -0.880356 unlocked) (layer "F.SilkS") hide
         (effects (font (size 1 1) (thickness 0.15)))
     )
@@
     (effects (font (size 1 1) (thickness 0.2) bold) (justify left bottom))
   )
+  (segment (start 153.584643 86.982856) (end 153.584643 89.145356) (width 0.3) (layer "F.Cu") (net 1))
+  (segment (start 145.083213 96.808213) (end 145.265356 96.626069) (width 0.3) (layer "F.Cu") (net 1))
   (segment (start 153.61 84.444999) (end 153.61 85.357499) (width 0.3) (layer "F.Cu") (net 1))
-  (segment (start 145.409643 100.620356) (end 144.059643 100.620356) (width 0.3) (layer "F.Cu") (net 1))
   (segment (start 153.864643 84.190356) (end 156.210356 84.190356) (width 0.3) (layer "F.Cu") (net 1))
-  (segment (start 153.584643 86.982856) (end 153.597143 86.970356) (width 0.3) (layer "F.Cu") (net 1))
   (segment (start 154.584643 87.957856) (end 153.597143 86.970356) (width 0.3) (layer "F.Cu") (net 1))
+  (segment (start 153.584643 89.870356) (end 153.304999 90.15) (width 0.15) (layer "F.Cu") (net 1))
   (segment (start 144.059643 100.620356) (end 144.059643 98.095356) (width 0.3) (layer "F.Cu") (net 1))
   (segment (start 145.265356 96.626069) (end 145.265356 96.614644) (width 0.3) (layer "F.Cu") (net 1))
+  (segment (start 144.059643 97.831782) (end 145.083213 96.808213) (width 0.3) (layer "F.Cu") (net 1))
+  (segment (start 153.304999 90.15) (end 151.741426 90.15) (width 0.15) (layer "F.Cu") (net 1))
   (segment (start 159.65 87.63) (end 159.65 88.8) (width 0.3) (layer "F.Cu") (net 1))
-  (segment (start 153.584643 89.145356) (end 153.584643 86.982856) (width 0.3) (layer "F.Cu") (net 1))
   (segment (start 156.210356 84.190356) (end 159.65 87.63) (width 0.3) (layer "F.Cu") (net 1))
-  (segment (start 149.934643 105.145356) (end 145.409643 100.620356) (width 0.3) (layer "F.Cu") (net 1))
+  (segment (start 146 101.25) (end 145.370356 100.620356) (width 0.3) (layer "F.Cu") (net 1))
+  (segment (start 145.083213 96.808213) (end 151.516426 90.375) (width 0.3) (layer "F.Cu") (net 1))
+  (segment (start 145.370356 100.620356) (end 144.059643 100.620356) (width 0.3) (layer "F.Cu") (net 1))
+  (segment (start 146.039287 101.25) (end 146 101.25) (width 0.3) (layer "F.Cu") (net 1))
+  (segment (start 149.934643 105.145356) (end 146.039287 101.25) (width 0.3) (layer "F.Cu") (net 1))
   (segment (start 153.864643 84.190356) (end 153.452143 83.777857) (width 0.3) (layer "F.Cu") (net 1))
   (segment (start 145.265356 96.614644) (end 145.27 96.61) (width 0.3) (layer "F.Cu") (net 1))
@@
   (segment (start 153.61 85.357499) (end 153.597143 85.370356) (width 0.3) (layer "F.Cu") (net 1))
   (segment (start 154.584643 89.145356) (end 154.584643 87.957856) (width 0.3) (layer "F.Cu") (net 1))
+  (segment (start 153.597143 86.970356) (end 153.584643 86.982856) (width 0.3) (layer "F.Cu") (net 1))
   (segment (start 152.514643 82.840356) (end 153.864643 84.190356) (width 0.3) (layer "F.Cu") (net 1))
   (segment (start 153.864643 84.190356) (end 153.61 84.444999) (width 0.3) (layer "F.Cu") (net 1))
-  (segment (start 144.059643 97.831782) (end 145.265356 96.626069) (width 0.3) (layer "F.Cu") (net 1))
-  (via (at 145.27 96.61) (size 0.7) (drill 0.3) (layers "F.Cu" "B.Cu") (net 1))
-  (segment (start 152.514643 89.365357) (end 152.514643 82.840356) (width 0.3) (layer "B.Cu") (net 1))
-  (segment (start 145.27 96.61) (end 152.514643 89.365357) (width 0.3) (layer "B.Cu") (net 1))
+  (segment (start 153.584643 89.145356) (end 153.584643 89.870356) (width 0.15) (layer "F.Cu") (net 1))
+  (segment (start 151.741426 90.15) (end 151.516426 90.375) (width 0.15) (layer "F.Cu") (net 1))
   (segment (start 155.184643 91.295356) (end 156.119643 92.230356) (width 0.2) (layer "F.Cu") (net 2))
   (segment (start 155.322143 86.970356) (end 155.322143 87.672856) (width 0.2) (layer "F.Cu") (net 2))
@@
   (segment (start 154.084643 89.870356) (end 154.394643 90.180356) (width 0.15) (layer "F.Cu") (net 25))
   (segment (start 155.144643 90.205356) (end 158.709643 93.770356) (width 0.2) (layer "F.Cu") (net 25))
+  (zone (net 1) (net_name "+3V3") (layer "F.Cu") (hatch edge 0.5)
+    (priority 1)
+    (connect_pads (clearance 0.5))
+    (min_thickness 0.25) (filled_areas_thickness no)
+    (fill yes (thermal_gap 0.5) (thermal_bridge_width 0.5))
+    (polygon
+      (pts
+        (xy 151.45 90.25)
+        (xy 151.625 90.075)
+        (xy 152.1 90.075)
+        (xy 152.1 90.225)
+        (xy 152.075 90.225)
+        (xy 151.85 90.25)
+        (xy 151.55 90.55)
+        (xy 151.525 90.55)
+        (xy 151.3375 90.3625)
+        (xy 151.45 90.25)
+      )
+    )
+  )
   (zone (net 2) (net_name "GND") (layers "F&B.Cu") (hatch edge 0.5)
     (connect_pads (clearance 0.5))
