File: hats/jetson_hat/HatV5.kicad_pcb (KiCad board)
At the start: 4 copper layers, 62 x 31.5 mm, 31 parts, among them J1 CLIK-Mate 502584, J2 CLIK-Mate 502584, J3 CLIK-Mate 502584, J4 CLIK-Mate 502584, J5 02x20 2.54 mm Female Socket, J6 24 Pin Header, U1 TCAN1051HGVDRBRQ1, U2 PESD2CANFD27V-TR, U3 TCAN1051HGVDRBRQ1, U4 PESD2CANFD27V-TR

Commit message: Minor routing ajustment and silkscreen error correction
Routing:
- net +3V3: track 153.9 -> 155.5 mm
Changed lines of the file:
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@@
 			(at -1.27 2.77 90)
 			(layer "F.SilkS")
+			(hide yes)
 			(effects
 				(font
@@
 	)
 	(via
-		(at 163.9824 95.6194)
+		(at 164.4824 96.1194)
 		(size 0.8)
 		(drill 0.4)
@@
 	)
 	(via
-		(at 164.9824 94.6194)
+		(at 165.4824 95.1194)
 		(size 0.8)
 		(drill 0.4)
@@
 	)
 	(segment
-		(start 165.9824 91.3394)
-		(end 163.7224 89.0794)
-		(width 1)
-		(layer "B.Cu")
-		(net 5)
-	)
-	(segment
 		(start 144.193778 101.274822)
 		(end 143.177778 102.290822)
@@
 	)
 	(segment
+		(start 165.9824 92.6194)
+		(end 165.9824 89.6194)
+		(width 1)
+		(layer "B.Cu")
+		(net 5)
+	)
+	(segment
 		(start 148.6824 98.288029)
 		(end 148.6824 98.885829)
@@
 	)
 	(segment
+		(start 165.4424 89.0794)
+		(end 163.7224 89.0794)
+		(width 1)
+		(layer "B.Cu")
+		(net 5)
+	)
+	(segment
 		(start 148.6824 98.885829)
 		(end 146.293407 101.274822)
@@
 	)
 	(segment
+		(start 161.9824 95.1194)
+		(end 163.4824 95.1194)
+		(width 1)
+		(layer "B.Cu")
+		(net 5)
+	)
+	(segment
 		(start 118.440778 97.210822)
 		(end 118.440778 96.194822)
@@
 	)
 	(segment
+		(start 165.9824 89.6194)
+		(end 165.4424 89.0794)
+		(width 1)
+		(layer "B.Cu")
+		(net 5)
+	)
+	(segment
 		(start 167.4824 101.775897)
 		(end 167.4824 105.1194)
@@
 	)
 	(segment
-		(start 165.9824 91.551432)
-		(end 165.9824 91.3394)
-		(width 1)
-		(layer "B.Cu")
-		(net 5)
-	)
-	(segment
-		(start 161.9824 95.1194)
-		(end 162.414432 95.1194)
+		(start 163.4824 95.1194)
+		(end 165.9824 92.6194)
 		(width 1)
 		(layer "B.Cu")
@@
 		(layer "B.Cu")
 		(net 5)
-	)
-	(segment
-		(start 162.414432 95.1194)
-		(end 165.9824 91.551432)
-		(width 1)
-		(layer "B.Cu")
-		(net 5)

Commit message: impedance checked and traces spaced out
Routing:
- net /SPI1_MOSI: track 70.8 -> 76.9 mm
- net /SPI1_MISO: track 69.0 -> 73.1 mm
- net /SPI1_CS0: track 51.7 -> 55.6 mm
- net /SPI1_SCK: track 63.5 -> 66.7 mm
- net /UART1_TX: track 56.4 -> 59.1 mm
- net /UART1_RX: track 62.5 -> 65.1 mm
- net /CAN0_DOUT: track 30.1 -> 32.5 mm
- net /SPI1_CS1: track 51.3 -> 53.6 mm
- net /CAN BUS 0/CH0-: track 45.5 -> 43.4 mm
- net /CAN BUS 0/CH0+: track 44.7 -> 42.7 mm
- net /GPIO27_PWM2: track 72.9 -> 74.7 mm
- net /CAN0_DIN: track 29.3 -> 31.0 mm
- net /PWM01: track 65.9 -> 67.3 mm
- net /I2C_GP2_DAT: track 77.9 -> 76.8 mm
- net /I2C_GP5_DAT: track 64.4 -> 65.5 mm
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- added copper zone on B.Cu, net GND
- added copper zone on F.Cu, net GND

Commit message: Moved a hole 2 mm so its cleaner and plotted the gerbers/drill files
Parts:
- moved H1 1.10 mm to (116.6, 111.1)
Routing:
- net +3V3: track 155.5 -> 163.4 mm
- net /SPI1_CS1: track 53.6 -> 55.5 mm
- net /SPI1_CS0: track 55.6 -> 56.4 mm
