File: terminal_block/terminal_block/Version V3/terminal_block.kicad_sch (KiCad schematic)
At the start: 42 parts, among them J1 XT60F, J10 XT60F, J11 XT60F, J12 XT60F, J13 XT60F, J14 XT60F, J15 XT60F, J16 XT60F, J17 XT60F, J18 XT60F, J19 XT60F, J2 XT60F, J20 XT60F, J21 XT60F, J22 XT60F, J23 XT60F, J24 XT60F, J25 XT60F, J26 XT60F, J27 XT60M, J28 XT60F, J29 XT60M, J3 XT60F, J30 XT60F, J31 XT60F, J32 XT60M, J33 XT60M, J34 XT30F, J35 XT30F, J36 XT30F, J37 XT30F, J38 XT60M, J4 XT60F, J41 XT30F, J42 XT30F, J43 XT30F, J45 XT30F, J5 XT60F, J6 XT60F, J7 XT60F, J8 XT60F, J9 XT60F

Commit message: terminal block routing finished, some checks tomorrow and its done
Parts:
- added J39, J40, J44, J46, J47, J48: XT30F, Connector_AMASS:AMASS_XT30UPB-M_1x02_P5.0mm_Vertical, symbol Connector_Generic:Conn_01x02
- J10, J15, J18, J23, J9: footprint Connector_AMASS:AMASS_XT60PW-F_1x02_P7.20mm_Horizontal -> Connector_AMASS:AMASS_XT60-F_1x02_P7.20mm_Vertical
- J27, J29, J32: value XT60M -> XT60F; footprint Connector_AMASS:AMASS_XT60PW-M_1x02_P7.20mm_Horizontal -> Connector_AMASS:AMASS_XT60-F_1x02_P7.20mm_Vertical
- J33: value XT60M -> XT30F; footprint Connector_AMASS:AMASS_XT60PW-M_1x02_P7.20mm_Horizontal -> Connector_AMASS:AMASS_XT30UPB-F_1x02_P5.0mm_Vertical
- J38: value XT60M -> XT30F; footprint Connector_AMASS:AMASS_XT60PW-M_1x02_P7.20mm_Horizontal -> Connector_AMASS:AMASS_XT30UPB-M_1x02_P5.0mm_Vertical
Connections:
- net +12V: now also J27.2 (Pin_2), J32.2 (Pin_2); no longer J15.2 (Pin_2), J33.2 (Pin_2)
- net +15V: now also J15.2 (Pin_2); no longer J32.2 (Pin_2)
- net +24V: now also J9.2 (Pin_2); no longer J29.2 (Pin_2)
- net +5V: now also J33.2 (Pin_2), J39.2 (Pin_2), J40.2 (Pin_2), J44.2 (Pin_2), J46.2 (Pin_2), J47.2 (Pin_2), J48.2 (Pin_2); no longer J23.2 (Pin_2)
- net +BATT: now also J23.2 (Pin_2), J29.2 (Pin_2); no longer J27.2 (Pin_2), J9.2 (Pin_2)
- net GND: now also J39.1 (Pin_1), J40.1 (Pin_1), J44.1 (Pin_1), J46.1 (Pin_1), J47.1 (Pin_1), J48.1 (Pin_1)
Other:
- note removed: "Extension Connectors"
- moved on the sheet: J37, J45
