File: hats/neopixel_Eliot/neopixel_eliot_hat.kicad_sch (KiCad schematic)
At the start: 51 parts, among them J1 B3B-XH-A(LF)(SN), J2 Hat_connector, J3 Conn_01x07, J4 USB_C_Receptacle_USB2.0, Q1 NPN, Q2 NPN, SW201 CL-SB-12C-01, U1 ESP32-PICO-D4, U2 AMS1117, U3 CP2102N-Axx-xQFN28, U301 SRV05-4A

Commit message: Neopixel v2
Parts:
- removed C3: 0.1uF, Capacitor_SMD:C_0603_1608Metric, symbol Device:C
- removed C4: 4.7uF, Capacitor_SMD:C_0603_1608Metric, symbol Device:C
- removed Q1, Q2: NPN, 2N3904:TO92127P495H495-3, symbol Simulation_SPICE:NPN
- removed R19: 10k, Resistor_SMD:R_0402_1005Metric, symbol Device:R
- removed U3: CP2102N-Axx-xQFN28, Package_DFN_QFN:QFN-28-1EP_5x5mm_P0.5mm_EP3.35x3.35mm, symbol Interface_USB:CP2102N-Axx-xQFN28
- added C301, C302: 1uF, Capacitor_SMD:C_0402_1005Metric, symbol Device:C_Small
- added C303: 100nF, Capacitor_SMD:C_0402_1005Metric, symbol Device:C_Small
- added C304: 4.7uF, Capacitor_SMD:C_0402_1005Metric, symbol Device:C_Small
- added D2: RED, LED_SMD:LED_0603_1608Metric, symbol Device:LED
- added Q1, Q2: SS8050-G, SS8050-G:TRANS_SS8050-G, symbol SS8050-G:SS8050-G
- added R12: 2K(1%), Resistor_SMD:R_0603_1608Metric_Pad0.98x0.95mm_HandSolder, symbol Device:R_Small
- added R20: 10k, Resistor_SMD:R_0402_1005Metric, symbol Device:R
- added R22: 1k, Resistor_SMD:R_0402_1005Metric, symbol Device:R
- added R3: 499R, Resistor_SMD:R_0603_1608Metric, symbol Device:R
- added TP1: Test_LED, TestPoint:TestPoint_Pad_D1.0mm, symbol Connector:TestPoint
- added TP2: Test_VIO, TestPoint:TestPoint_Pad_D1.0mm, symbol Connector:TestPoint
- added TP3: Test_RXD, TestPoint:TestPoint_Pad_D1.0mm, symbol Connector:TestPoint
- added TP4: Test_TXD, TestPoint:TestPoint_Pad_D1.0mm, symbol Connector:TestPoint
- added TP5: Test_VBUS, TestPoint:TestPoint_Pad_D1.0mm, symbol Connector:TestPoint
- added TP6: Test_EN, TestPoint:TestPoint_Pad_D1.0mm, symbol Connector:TestPoint
- added TP7: Test_DTR, TestPoint:TestPoint_Pad_D1.0mm, symbol Connector:TestPoint
- added TP8: Test_RTS, TestPoint:TestPoint_Pad_D1.0mm, symbol Connector:TestPoint
- added TP9: Test_IO0, TestPoint:TestPoint_Pad_D1.0mm, symbol Connector:TestPoint
- added U302: NCV8161ASN330T1G, Package_TO_SOT_SMD:SOT-23-5, symbol 0_regulator_linear:NCV8161ASN330T1G
- added U303: CP2102N-A02-GQFN24, Package_DFN_QFN:QFN-24-1EP_4x4mm_P0.5mm_EP2.6x2.6mm_ThermalVias, symbol 0_interface_uart:CP2102N-A02-GQFN24
- C7: value 1uF -> 0.1uF
- R2: now fitted; now in the parts list
- R4, SW201: now not fitted; now left out of the parts list
- renumbered C12 to C14, C13 to C15, D2 to D3, R11 to R13, R13 to R14, R14 to R15
Connections:
- net +3V3: now also C302.1, C303.1, C304.1, R12.2, R22.1, TP2.1, U302.5 (OUT), U303.5 (VIO), U303.6 (VDD), U303.7 (VREGIN)
- net +5V_MCU: now also C301.1, TP5.1, U302.1 (IN), U302.3 (EN)
- net D+: now also U303.3 (D+)
- net D-: now also U303.4 (D-)
- net DTR: now also Q2.2, TP7.1, U303.23 (~{DTR})
- net EN: now also Q1.3, TP6.1
- net GND: now also C301.2, C302.2, C303.2, C304.2, D2.1 (K), R20.2, U302.2 (GND), U303.2 (GND), U303.25 (GND)
- net GPIO0: now also Q2.3, TP9.1
- net RTS: now also Q1.2, TP8.1, U303.19 (~{RTS})
- net U0RXD: now also TP3.1, U303.21 (TXD)
- net U0TXD: now also R3.2, TP4.1, U303.20 (RXD); no longer U1.41 (U0TXD/IO1)
- net at C3.1, R1.2, R2.1: now also U303.8 (VBUS)
- net VBUS_USB: now reaches F1.1, J4.A4 (VBUS), J4.A9 (VBUS), J4.B4 (VBUS), J4.B9 (VBUS)
- net at R2.2: now also Q1.1
- net at R2.2: now also Q2.1
- net IO27 renamed SIGNAL_LED
- net SIGNAL_LED: now also TP1.1; no longer U1.16 (IO27)
- new net: R3.1, U1.41 (U0TXD/IO1)
- new net: D2.2 (A), R12.1
- new net: R20.1, U303.15 (~{SUSPEND})
- new net: R22.2, U303.9 (~{RST})
- new net SINGAL_LED: U1.16 (IO27)
- no-connect marks 41 -> 34
Other:
- note added: "499R resistor to suppress 80MHz harmonics"
- note added: "Found complaints regarding the internal regulator of the CP2102 with multiple complaints of 4v instead of 3v3 output."
- note added: "I_hold of 3A I_trip of 5A"
- note added: "Output 1A"
- note removed: "Here two potential options are present: Two switches for EN and GPIO - EN and GPIO0 high = run code from internal flash, else reboot autoprogram with NPN - who knows, maybe it'll work on the first try for once. Stability concerns with this. Switches are a backup option to replace the autoprogram if it doesn't work. Would just have switches to rest/reboot board."
- note removed: "Q1 and Q2 need to be L8050QLT1G"
- moved on the sheet: C14, C3, F1, J1, J4, R1, R14, R15, R2, U301

Commit message: neopixel update pour Farouk
Parts:
- removed C301, C302: 1uF, Capacitor_SMD:C_0402_1005Metric, symbol Device:C_Small
- removed D1: ESDA6V1-5SC6, Package_TO_SOT_SMD:SOT-23-6, symbol Power_Protection:ESDA6V1-5SC6
- removed D3: ORANGE, LED_SMD:LED_0603_1608Metric, symbol Device:LED
- removed F1: 2920L300, KiCad:2920L030DR, symbol 2920L300:2920L300
- removed J3: Conn_01x07, Connector_PinHeader_1.00mm:PinHeader_1x07_P1.00mm_Vertical, symbol Connector_Generic:Conn_01x07
- removed J4: USB_C_Receptacle_USB2.0, Connector_USB:USB_C_Receptacle_GCT_USB4105-xx-A_16P_TopMnt_Horizontal, symbol Connector:USB_C_Receptacle_USB2.0
- removed LV1: SN74LVC1T45, SN74LVC1T45:SN74LVC1T45_DRL, symbol SN74LVC1T45:SN74LVC1T45
- removed R13: 2K(1%), Resistor_SMD:R_0603_1608Metric_Pad0.98x0.95mm_HandSolder, symbol Device:R_Small
- removed R14, R15: 5.1k, Resistor_SMD:R_0603_1608Metric_Pad0.98x0.95mm_HandSolder, symbol Device:R_Small
- removed R205: 22R, Resistor_SMD:R_0402_1005Metric, symbol Device:R_Small
- removed R4 (x2): 10k, Resistor_SMD:R_0402_1005Metric, symbol Device:R
- removed SW201 (x2): CL-SB-12C-01, Button_Switch_SMD:SW_DIP_SPSTx01_Slide_Copal_CVS-01xB_W5.9mm_P1mm, symbol Switch:SW_SPDT
- removed TP5: Test_VBUS, TestPoint:TestPoint_Pad_D1.0mm, symbol Connector:TestPoint
- removed U302: NCV8161ASN330T1G, Package_TO_SOT_SMD:SOT-23-5, symbol 0_regulator_linear:NCV8161ASN330T1G
- added D204: ESDALC6V1W5, 0_various:SOT323-5L, symbol 0_power_protection:ESDALC6V1W5
- added D301: SMF5.0CA-TP, Diode_SMD:D_SOD-123, symbol 0_power_protection:SMF5.0CA
- added F301: 0805L075SLYR, Fuse:Fuse_0805_2012Metric, symbol Device:Polyfuse_Small
- added J202: Conn_Picoblade_JST_DEBUG, 0_connectors:PicoBlade-JST-GH-1x06_1.25mm_Horizontal, symbol Connector_Generic:Conn_01x06
- added J301: USB_B_Micro, 0_connectors:USB_Micro-B_Molex-105017-0001, symbol 0_connectors:USB_B_Micro
- added LV1: SN74LVC1T45DCKT, SN74LVC1T45DCKT:SOP65P210X110-6N, symbol SN74LVC1T45DCKT:SN74LVC1T45DCKT
- added Q301: PJA3405, Package_TO_SOT_SMD:SOT-23, symbol 0_transistor:PJA3405
- TP2: value Test_VIO -> Test_VBUS
Connections:
- net SINGAL_LED is gone; now on net SIGNAL_LED: U1.16 (IO27)
- net +3V3: now also J202.1 (Pin_1), LV1.1 (VCCA); no longer TP2.1
- net +5V_MCU: now also LV1.6 (VCCB); no longer R1.1, U301.5 (VP)
- net D+: now also J301.3 (D+)
- net D-: now also J301.2 (D-)
- net GND: now also D204.2 (GND), D301.1 (A1), J202.6 (Pin_6), J301.5 (GND), J301.6 (Shield), LV1.2 (GND), Q301.1 (G)
- net SIGNAL_LED: now also LV1.3 (A)
- net at R207.1: now also D204.3 (IO2), J202.3 (Pin_3)
- net DIR_LED: now reaches R2.2
- net DIR_LED: now also LV1.5 (DIR)
- net I2C_SCL: now reaches J2.7 (I2C_SCL), R3.2, U1.39 (IO22)
- net I2C_SDA: now reaches J2.8 (I2C_SDA), R3.2, U1.42 (IO21)
- net at R3.2: now also LV1.4 (B)
- net base_Q2: now reaches Q2.1, R2.2
- net at R206.1: now also D204.1 (IO1), J202.2 (Pin_2)
- net at R204.1: now also D204.5 (IO4), J202.4 (Pin_4)
- net at R204.1: now also D204.4 (IO3), J202.5 (Pin_5)
- net VBUS: now reaches C3.1, R1.2, R2.1, U303.8 (VBUS)
- net RSTb: now reaches R22.2, U303.9 (~{RST})
- net base_Q1: now reaches Q1.1, R2.2
- new net: F301.1, J301.1 (VBUS)
- new net VBUS_FUSE: D301.2 (A2), F301.2, Q301.3 (D)
- new net VBUS_REV: Q301.2 (S), R1.1, TP2.1, U301.5 (VP)
Other:
- note added: "USB Micro & USB-UART"
- note removed: "Found complaints regarding the internal regulator of the CP2102 with multiple complaints of 4v instead of 3v3 output."
- note removed: "I_hold of 3A I_trip of 5A"
- note removed: "USB Type-C 5V & USB-UART"
- moved on the sheet: C3, C303, C304, Q1, Q2, R1, R2, R20, R22, R3, TP6, TP7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

Commit message: completed v2 Neopixel with gerbers and drill files
Parts:
- TP1: value Test_LED -> LED_Sig
- TP2: value Test_VBUS -> VBUS_REV
- TP3: value Test_RXD -> RXD
- TP4: value Test_TXD -> TXD
- TP6: value Test_EN -> EN
- TP7: value Test_DTR -> DTR
- TP8: value Test_RTS -> RTS
- TP9: value Test_IO0 -> IO0
Connections:
- net U0TXD: now also R3.1, U1.41 (U0TXD/IO1); no longer R3.2, TP4.1, U303.20 (RXD)
- net VBUS: now also F301.1, J301.1 (VBUS); no longer C3.1, R1.2, R2.1, U303.8 (VBUS)
- net JTMS_SIG: now reaches J202.3 (Pin_3), R207.1
- net JTMS_SIG: now also D204.1 (IO1); no longer D204.3 (IO2)
- net SPI_CS: now reaches J2.6 (SPI_CS), U1.34 (IO5)
- net SPI_SCK: now reaches J2.3 (SPI_SCK), U1.35 (IO18)
- net SPI_MISO: now reaches J2.5 (SPI_MISO), U1.36 (IO23)
- net SPI_MOSI: now reaches J2.4 (SPI_MOSI), U1.38 (IO19)
- net JTCK_SIG: now reaches J202.2 (Pin_2), R206.1
- net JTCK_SIG: now also D204.3 (IO2); no longer D204.1 (IO1)
- net JTD0_SIG: now reaches J202.4 (Pin_4), R204.1
- net JTD0_SIG: now also D204.4 (IO3); no longer D204.5 (IO4)
- net JTDI_SIG: now reaches J202.5 (Pin_5), R204.1
- net JTDI_SIG: now also D204.5 (IO4); no longer D204.4 (IO3)
- net SUSPENDb: now reaches R20.1, U303.15 (~{SUSPEND})
- net JTCK renamed JTCK_MCU
- net JTDI renamed JTDI_MCU
- net JTDO renamed JTDO_MCU
- net JTMS renamed JTMS_MCU
- new net U0TXD_R: R3.2, TP4.1, U303.20 (RXD)
- new net VBUS_USB: C3.1, R1.2, R2.1, U303.8 (VBUS)
Other:
- moved on the sheet: R20, R3

Commit message: Neopixel v2.1
Parts:
- added C17, C18: 0.1uF, Capacitor_SMD:C_0603_1608Metric_Pad1.08x0.95mm_HandSolder, symbol Device:C_Small
- added C303: 0.1uF, Capacitor_SMD:C_0603_1608Metric, symbol Device:C_Small
- added C304: 4.7uF, Capacitor_SMD:C_0603_1608Metric, symbol Device:C_Small
- C303: value 100nF -> 0.1uF
- C6: value 10uF -> 0.1uF
- TP1, TP2, TP3, TP4, TP6, TP7, TP8, TP9: footprint TestPoint:TestPoint_Pad_D1.0mm -> 0_various:TestPoint
Connections:
- net +3V3: now also C17.1, C18.1
- net +5V_MCU: now also C303.1, C304.1
- net GND: now also C17.2, C18.2, C303.2, C304.2
- net JTCK_SIG: now also D204.5 (IO4); no longer D204.3 (IO2)
- net JTD0_SIG: now also D204.3 (IO2); no longer D204.4 (IO3)
- net JTDI_SIG: now also D204.1 (IO1); no longer D204.5 (IO4)
- net JTMS_SIG: now also D204.4 (IO3); no longer D204.1 (IO1)
- net VBUS: now also D301.2 (A2), Q301.3 (D); no longer F301.1
- net VBUS_REV: now also F301.2; no longer Q301.2 (S)
- removed net VBUS_FUSE: D301.2 (A2), F301.2, Q301.3 (D)
- new net: F301.1, Q301.2 (S)
Other:
- moved on the sheet: D301, Q301

Commit message: Neopixel v2.2 with BOM and Gerber/Drill files
Parts:
- removed C17, C18, C5, C6, C7: 0.1uF, Capacitor_SMD:C_0603_1608Metric_Pad1.08x0.95mm_HandSolder, symbol Device:C_Small
- removed C2: 0.1uF, Capacitor_SMD:C_0603_1608Metric, symbol Device:C
- removed C303: 0.1uF, Capacitor_SMD:C_0603_1608Metric, symbol Device:C_Small
- removed C304: 4.7uF, Capacitor_SMD:C_0603_1608Metric, symbol Device:C_Small
- added C1: 4.7uF, Capacitor_SMD:C_0603_1608Metric, symbol Device:C
- added C2 (x5): 0.1uF, Capacitor_SMD:C_0603_1608Metric, symbol Device:C_Small
- added C2 (x2): 0.1uF, Capacitor_SMD:C_0603_1608Metric, symbol Device:C
- C1: link (none) -> https://eu.mouser.com/ProductDetail/Samsung-Electro-Mechani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
- C14: footprint Capacitor_SMD:C_0603_1608Metric_Pad1.08x0.95mm_HandSolder -> Capacitor_SMD:C_0603_1608Metric; Distributor (none) -> Mouser; link (none) -> https://eu.mouser.com/ProductDetail/Murata-Electronics/GRM1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
- C15: footprint Capacitor_SMD:C_0603_1608Metric_Pad1.08x0.95mm_HandSolder -> Capacitor_SMD:C_0805_2012Metric; Distributor (none) -> Mouser; link (none) -> https://eu.mouser.com/ProductDetail/Samsung-Electro-Mechani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
- C2: link (none) -> https://eu.mouser.com/ProductDetail/TAIYO-YUDEN/TMK107B7104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
- C3: Distributor ref TMK107B7104KAHT -> MBAST168AB7105KTNA01; Manufacturer ref 963-TMK107B7104KAHT -> 963-BAST168AB7105KT; link (none) -> https://eu.mouser.com/ProductDetail/TAIYO-YUDEN/MBAST168AB7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
- C303: Distributor (none) -> Mouser; link (none) -> https://eu.mouser.com/ProductDetail/TAIYO-YUDEN/UMK105B7104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
- C304: Distributor (none) -> Mouser; link (none) -> https://eu.mouser.com/ProductDetail/Samsung-Electro-Mechani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
- D2: Distributor (none) -> Mouser; link (none) -> https://eu.mouser.com/ProductDetail/ams-OSRAM/LS-L296-N2Q1-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
- D204: Digikey ref 497-7231-1-ND -> (none); Distributor (none) -> Mouser; link (none) -> https://eu.mouser.com/ProductDetail/STMicroelectronics/ESDA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
- D301: Distributor (none) -> Mouser; link (none) -> https://eu.mouser.com/ProductDetail/Micro-Commercial-Compon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
- F301: link (none) -> https://eu.mouser.com/ProductDetail/Littelfuse/0805L075SLYR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
- J1, J202: Distributor (none) -> Digikey; link (none) -> https://www.digikey.com/en/products/detail/jst-sales-americ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
- J301: Distributor (none) -> Digikey; link (none) -> https://www.digikey.com/en/products/detail/molex/1050170001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
- LV1: Distributor (none) -> Mouser; link (none) -> https://www.mouser.ch/ProductDetail/Texas-Instruments/SN74L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
- Q1, Q2: Distributor (none) -> Digikey; link (none) -> https://www.digikey.com/en/products/detail/comchip-technolo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
- Q301: link (none) -> https://www.digikey.com/en/products/detail/panjit-internati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
- R1: link (none) -> https://www.mouser.ch/ProductDetail/Panasonic/ERA-3ARB2212V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
- R12: footprint Resistor_SMD:R_0603_1608Metric_Pad0.98x0.95mm_HandSolder -> Resistor_SMD:R_0603_1608Metric; Distributor (none) -> Mouser; link (none) -> https://www.mouser.ch/ProductDetail/Panasonic/ERA-3AED202V?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
- R2: footprint Resistor_SMD:R_0603_1608Metric_Pad0.98x0.95mm_HandSolder -> Resistor_SMD:R_0603_1608Metric; Distributor (none) -> Mouser; link (none) -> https://www.mouser.ch/ProductDetail/Vishay-Dale/CRCW060310K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
- R2, R3: link (none) -> https://www.mouser.ch/ProductDetail/Vishay-Dale/CRCW060310K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
- R2: link (none) -> https://www.mouser.ch/ProductDetail/Panasonic/ERA-3AEB47R5V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
- R20: Distributor (none) -> Mouser; link (none) -> https://www.mouser.ch/ProductDetail/Panasonic/ERJ-S02D1002X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
- R204, R206, R207: Distributor (none) -> Digikey; link (none) -> https://www.digikey.com/en/products/detail/te-connectivity-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
- R22: link (none) -> https://www.mouser.ch/ProductDetail/Panasonic/ERA-2ARC102X?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
- R3: link (none) -> https://www.mouser.ch/ProductDetail/Panasonic/ERA-3AED4990V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
- R3: link (none) -> https://www.mouser.ch/ProductDetail/Panasonic/ERA-3APB222V?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
- R3: footprint Resistor_SMD:R_0603_1608Metric_Pad0.98x0.95mm_HandSolder -> Resistor_SMD:R_0603_1608Metric; Distributor (none) -> Mouser; link (none) -> https://www.mouser.ch/ProductDetail/Panasonic/ERA-3AED101V?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
- U1: link (none) -> https://www.digikey.com/en/products/detail/espressif-system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
- U2: link (none) -> https://www.digikey.ch/en/products/detail/evvo/AMS1117-3-3/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
- U301: link (none) -> https://www.digikey.ch/en/products/detail/smc-diode-solutio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
- U303: link (none) -> https://www.digikey.ch/en/products/detail/silicon-labs/CP21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
Connections:
- net +3V3: now also C2.1, C2.1, C2.1, C2.2, C2.2
- net +5V_MCU: now also C1.1, C2.1
- net EN: now also C2.1
- net GND: now also C1.2, C2.1, C2.1, C2.2, C2.2, C2.2, C2.2, C2.2

Commit message: Updated bom
Parts:
- D301: link https://eu.mouser.com/ProductDetail/Micro-Commercial-Compon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 -> https://www.digikey.ch/en/products/detail/micro-commercial-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
- F301: link https://eu.mouser.com/ProductDetail/Littelfuse/0805L075SLYR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 -> https://www.digikey.ch/en/products/detail/littelfuse-inc/08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
- R12: value 2K(1%) -> 50R; link https://www.mouser.ch/ProductDetail/Panasonic/ERA-3AED202V?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 -> https://www.mouser.ch/ProductDetail/Vishay-Draloric/TNPU060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
Changed lines of the file:
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@@
       (effects (font (size 1.27 1.27)) hide)
     )
-    (property "link" "https://eu.mouser.com/ProductDetail/Littelfuse/0805L075SLYR?qs=C%2F0tY%2F%2FqZe89Ht%2FbgKOotQ%3D%3D" (at 90.17 203.3524 0)
+    (property "link" "https://www.digikey.ch/en/products/detail/littelfuse-inc/0805L075SLYR/2764997" (at 90.17 203.3524 0)
       (effects (font (size 1.27 1.27)) hide)
     )
@@
       (effects (font (size 1.27 1.27)) hide)
     )
-    (property "link" "https://eu.mouser.com/ProductDetail/Micro-Commercial-Components-MCC/SMF5.0CA-TP?qs=y6ZabgHbY%252Bx5chrSGzaXjw%3D%3D" (at 42.7482 221.1324 0)
+    (property "link" "https://www.digikey.ch/en/products/detail/micro-commercial-co/SMF5-0CA-TP/7320159" (at 42.7482 221.1324 0)
       (effects (font (size 1.27 1.27)) hide)
     )
@@
       (effects (font (size 1.27 1.27)))
     )
-    (property "Value" "2K(1%)" (at 359.2322 210.1088 0)
+    (property "Value" "50R" (at 357.9622 209.9564 0)
       (effects (font (size 1.27 1.27)))
     )
@@
       (effects (font (size 1.27 1.27)) hide)
     )
-    (property "link" "https://www.mouser.ch/ProductDetail/Panasonic/ERA-3AED202V?qs=sGAEpiMZZMtlubZbdhIBINnjttWTECnXPYH118Z5ZyA%3D" (at 354.1522 209.4738 0)
-      (effects (font (size 1.27 1.27)) hide)
-    )
+    (property "link" "https://www.mouser.ch/ProductDetail/Vishay-Draloric/TNPU060350R0BZEN00?qs=t7xnP681wgWwtWlrkwxO6w%3D%3D" (at 354.1522 209.4738 0)
+      (effects (font (size 1.27 1.27)) hide)
+    )

Commit message: start of revision, changed the i2c to UART and usb micro to usb c
Parts:
- removed J301: USB_B_Micro, 0_connectors:USB_Micro-B_Molex-105017-0001, symbol 0_connectors:USB_B_Micro
- removed R3 (x2): 2k2, Resistor_SMD:R_0603_1608Metric, symbol Device:R
- added J3: USB_C_Receptacle, Connector_USB:USB_C_Receptacle_Molex_105450-0101, symbol Connector:USB_C_Receptacle
- added R4, R5: 5.1k, symbol Device:R
Connections:
- net D+: now also J3.A6 (D+), J3.B6 (D+)
- net D-: now also J3.A7 (D-), J3.B7 (D-)
- net GND: now also J3.A1 (GND), J3.A12 (GND), J3.B1 (GND), J3.B12 (GND), J3.S1 (SHIELD), R4.2, R5.2
- net MCU_GPIO1: no longer J2.9 (GPIO_1)
- net MCU_GPIO2: no longer J2.10 (GPIO_2)
- net MCU_GPIO3: no longer J2.11 (GPIO_3)
- net MCU_GPIO4: no longer J2.12 (GPIO_4)
- net VBUS: now also J3.A4 (VBUS), J3.A9 (VBUS), J3.B4 (VBUS), J3.B9 (VBUS)
- net I2C_SCL: no longer names the net of U1.39 (IO22)
- net I2C_SCL: no longer J2.7 (I2C_SCL)
- net I2C_SDA: no longer names the net of U1.42 (IO21)
- net I2C_SDA: no longer J2.8 (I2C_SDA)
- new net: J3.A5 (CC1), R4.1
- new net: J3.B5 (CC2), R5.1
- no-connect marks 34 -> 48
Other:
- note added: "Note to self: swap routing in pcb layout"
- note added: "Replace by USB-c and pull down to ground (see link)"
- note added: "USB C & USB-UART"
- note removed: "USB Micro & USB-UART"
- moved on the sheet: C3, D301, F301, Q301, R1, R2, TP2, U301

Commit message: added power MUX and made space for e fuse
Parts:
- removed F301: 0805L075SLYR, Fuse:Fuse_0805_2012Metric, symbol Device:Polyfuse_Small
- added IC1: TPS2116DRLR, SOTFL50P160X60-8N, symbol SamacSys_Parts:TPS2116DRLR
Connections:
- net +5V_MCU: now also IC1.3 (VIN1), IC1.4 (PR1), IC1.5 (MODE); no longer C15.1, U2.3 (VI)
- net GND: now also IC1.1 (GND)
- net VBUS_REV: now also IC1.6 (VIN2)
- new net Vout_MUX: C15.1, IC1.2 (VOUT_1), U2.3 (VI)
- no-connect marks 48 -> 50
Other:
- note added: "add efuse <"
- note added: "power mux"
- moved on the sheet: C3, C303, C304, Q1, Q2, R1, R2, R20, R22, TP2, TP6, TP7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
