File: Power/ElonMux/ElonMux.kicad_pcb (KiCad board)
At the start: 6 copper layers, 0 parts

Commit message: Rough layout
Parts:
- added C1001: 100n X7R 50V, Capacitor_SMD:C_0402_1005Metric, F.Cu at (162.8, 54.5)
- added C1002: 100n X7R 50V, Capacitor_SMD:C_0402_1005Metric, F.Cu at (209.1, 61.8)
- added C1003: 100n X7R 50V, Capacitor_SMD:C_0402_1005Metric, F.Cu at (204.1, 61.8)
- added C401: 1u X7R 50V, Capacitor_SMD:C_0603_1608Metric, F.Cu at (192.0, 54.0)
- added C402: 100n X7R 50V, Capacitor_SMD:C_0402_1005Metric, F.Cu at (193.5, 54.5)
- added C403: 10u X7R 50V, Capacitor_SMD:C_1206_3216Metric, F.Cu at (187.4, 70.8)
- added C404: 1u X7R 50V, Capacitor_SMD:C_0603_1608Metric, F.Cu at (188.2, 68.8)
- added C405: 100n X7R 50V, Capacitor_SMD:C_0402_1005Metric, F.Cu at (188.7, 67.5)
- added C406: 100n X7R 50V, Capacitor_SMD:C_0402_1005Metric, F.Cu at (188.7, 64.5)
- added C407: 100n X7R 50V, Capacitor_SMD:C_0402_1005Metric, F.Cu at (196.0, 59.8)
- added C408: 100n X7R 50V, Capacitor_SMD:C_0402_1005Metric, F.Cu at (186.2, 58.0)
- added C409: 10p X7R 25V, Capacitor_SMD:C_0402_1005Metric, F.Cu at (186.2, 60.9)
- added C410: 10p X7R 25V, Capacitor_SMD:C_0402_1005Metric, F.Cu at (182.5, 57.0)
- added C411: 1u X7R 50V, Capacitor_SMD:C_0603_1608Metric, F.Cu at (184.8, 63.2)
- added C412: 10n X7R 50V, Capacitor_SMD:C_0402_1005Metric, F.Cu at (186.2, 62.9)
- added C413: 100n X7R 50V, Capacitor_SMD:C_0402_1005Metric, F.Cu at (196.5, 72.8)
- added C601: 1u X7R 50V, Capacitor_SMD:C_0603_1608Metric, F.Cu at (202.5, 87.5)
- added C602: 1u X7R 50V, Capacitor_SMD:C_0603_1608Metric, F.Cu at (206.8, 88.2)
- added C603: 4u7 X7R 50V, Capacitor_SMD:C_0805_2012Metric, F.Cu at (199.8, 89.0)
- added C604: 100n X7R 50V, Capacitor_SMD:C_0402_1005Metric, F.Cu at (198.5, 92.0)
- added C605: 10p X7R 25V, Capacitor_SMD:C_0603_1608Metric, F.Cu at (206.8, 86.5)
- added C606: 22u X5R 50V, Capacitor_SMD:C_0603_1608Metric, F.Cu at (206.8, 83.0)
- added C607: 22u X5R 50V, Capacitor_SMD:C_0603_1608Metric, F.Cu at (203.2, 82.8)
- added C608: 4u7 X7R 50V, Capacitor_SMD:C_0805_2012Metric, F.Cu at (210.0, 89.8)
- added C609: 100n X7R 50V, Capacitor_SMD:C_0402_1005Metric, F.Cu at (200.0, 92.5)
- added C610: 4u7 X7R 50V, Capacitor_SMD:C_0805_2012Metric, F.Cu at (202.2, 95.5)
- added C701: 100n X7R 50V, Capacitor_SMD:C_0402_1005Metric, F.Cu at (135.8, 77.2)
- added C702: 27u 63V, Capacitor_SMD:CP_Elec_8x6.7, F.Cu at (148.2, 114.2)
- added C703: 27u 63V, Capacitor_SMD:CP_Elec_8x6.7, F.Cu at (139.2, 114.2)
- added C704: 27u 63V, Capacitor_SMD:CP_Elec_8x6.7, F.Cu at (130.2, 114.2)
- added C705: 10u X7R 50V, Capacitor_SMD:C_1206_3216Metric, F.Cu at (124.0, 114.0)
- added C706: 10u X7R 50V, Capacitor_SMD:C_1206_3216Metric, F.Cu at (145.3, 82.2)
- added C707: 10u X7R 50V, Capacitor_SMD:C_1206_3216Metric, F.Cu at (137.2, 89.2)
- added C708: 10u X7R 50V, Capacitor_SMD:C_1206_3216Metric, F.Cu at (137.2, 82.1)
- added C709: 10u X7R 50V, Capacitor_SMD:C_1206_3216Metric, F.Cu at (137.2, 84.5)
- added C710: 10u X7R 50V, Capacitor_SMD:C_1206_3216Metric, F.Cu at (137.2, 86.9)
- added C711: 27u 63V, Capacitor_SMD:CP_Elec_8x6.7, F.Cu at (139.5, 72.2)
- added C712: 100n X7R 50V, Capacitor_SMD:C_0402_1005Metric, F.Cu at (129.2, 106.8)
- added C713: 100n X7R 50V, Capacitor_SMD:C_0402_1005Metric, F.Cu at (145.2, 104.2)
- added C714: 100n X7R 50V, Capacitor_SMD:C_0402_1005Metric, F.Cu at (145.7, 102.0)
- added C715: 100n X7R 50V, Capacitor_SMD:C_0402_1005Metric, F.Cu at (142.8, 97.5)
- added C716: 10n X7R 50V, Capacitor_SMD:C_0402_1005Metric, F.Cu at (141.0, 106.5)
- added C717: 100n X7R 50V, Capacitor_SMD:C_0402_1005Metric, F.Cu at (140.2, 97.5)
- added C718: 100n X7R 50V, Capacitor_SMD:C_0402_1005Metric, F.Cu at (138.2, 97.5)
- added C719: 22u X5R 50V, Capacitor_SMD:C_0603_1608Metric, F.Cu at (135.8, 98.5)
- added C720: 22u X5R 50V, Capacitor_SMD:C_0603_1608Metric, F.Cu at (142.2, 107.0)
- added C721: 220p X7R 50V, Capacitor_SMD:C_0402_1005Metric, F.Cu at (140.0, 106.5)
- added C722: 22u X5R 50V, Capacitor_SMD:C_0603_1608Metric, F.Cu at (135.7, 100.0)
- added C801: 100n X7R 50V, Capacitor_SMD:C_0402_1005Metric, F.Cu at (172.7, 68.5)
- added C802: 100n X7R 50V, Capacitor_SMD:C_0402_1005Metric, F.Cu at (171.8, 86.2)
- added C803: 100n X7R 50V, Capacitor_SMD:C_0402_1005Metric, F.Cu at (173.5, 88.8)
- added C804: 100n X7R 50V, Capacitor_SMD:C_0402_1005Metric, F.Cu at (171.8, 76.8)
- added C805: 100n X7R 50V, Capacitor_SMD:C_0402_1005Metric, F.Cu at (136.2, 60.8)
- added C806: 100n X7R 50V, Capacitor_SMD:C_0402_1005Metric, F.Cu at (161.8, 93.2)
- added C807: 100n X7R 50V, Capacitor_SMD:C_0402_1005Metric, F.Cu at (168.5, 84.8)
- added C808: 1u X7R 50V, Capacitor_SMD:C_0603_1608Metric, F.Cu at (169.0, 86.2)
- added C809: 1u X7R 50V, Capacitor_SMD:C_0603_1608Metric, F.Cu at (165.2, 89.0)
- added C810: 1u X7R 50V, Capacitor_SMD:C_0603_1608Metric, F.Cu at (162.5, 76.2)
- added C811: 1u X7R 50V, Capacitor_SMD:C_0603_1608Metric, F.Cu at (162.5, 78.0)
- added C901: 100n X7R 50V, Capacitor_SMD:C_0402_1005Metric, F.Cu at (175.2, 64.5)
- added D1001: D5V0P4UR6SO-7, Charge_Manager_FP:D5V0P4UR6SO-7 SOT95P285X140-6N, F.Cu at (171.6, 62.5)
- added D1002: PRTR5V0U2X, Package_TO_SOT_SMD:SOT-143, F.Cu at (206.6, 61.3)
- added D501: SMBJ30CA, Charge_Manager_FP:DIOM5436X244N, F.Cu at (172.2, 112.5)
- added D502: SMBJ30CA, Charge_Manager_FP:DIOM5436X244N, F.Cu at (144.5, 78.8)
- added D503: SMBJ30CA, Charge_Manager_FP:DIOM5436X244N, F.Cu at (139.5, 61.2)
- added D504: SMBJ30CA, Charge_Manager_FP:DIOM5436X244N, F.Cu at (198.2, 99.8)
- added D801: VBT3045C-E3_8W, Charge_Manager_FP:V30DL45BPM3I, F.Cu at (156.8, 88.0)
- added D802: PMEG4030ER,115, Diode_SMD:Nexperia_CFP3_SOD-123W, F.Cu at (175.2, 87.3)
- added D803: PMEG4030ER,115, Diode_SMD:Nexperia_CFP3_SOD-123W, F.Cu at (172.0, 79.8)
- added IC601: LTC3126IUFD#PBF, Charge_Manager_FP:LTC3126EUFD, F.Cu at (204.2, 91.8)
- added IC801: LTC7000EMSE#PBF, Charge_Manager_FP:LTC7000EMSE#PBF, F.Cu at (169.5, 89.5)
- added IC802: LTC7000EMSE#PBF, Charge_Manager_FP:LTC7000EMSE#PBF, F.Cu at (167.3, 77.8)
- added IC803: TPS3701DDCR, Charge_Manager_FP:TPS3701DDCR, F.Cu at (165.5, 83.5)
- added J1001: FTSH-107-01-F-DV-K, Charge_Manager_FP:FTSH-107-XX-YYY-DV-K, F.Cu at (168.0, 54.5)
- added J1002: USB4105-GF-A, Charge_Manager_FP:GCT_USB4105-GF-A, F.Cu at (206.5, 52.8)
- added J1003: PPTC042LFBN-RC, Connector_PinSocket_2.54mm:PinSocket_2x04_P2.54mm_Vertical, F.Cu at (174.9, 52.0)
- added J501: XT60PW-M, Charge_Manager_FP:AMASS_XT60PW-M_1x02_P7.20mm_Horizontal, F.Cu at (165.1, 104.8)
- added J502: XT60PW-M, Charge_Manager_FP:AMASS_XT60PW-M_1x02_P7.20mm_Horizontal, F.Cu at (132.2, 83.2)
- added J503: XT60PW-M, Charge_Manager_FP:AMASS_XT60PW-M_1x02_P7.20mm_Horizontal, F.Cu at (132.2, 62.9)
- added J504: XT60PW-M, Charge_Manager_FP:AMASS_XT60PW-M_1x02_P7.20mm_Horizontal, F.Cu at (200.3, 104.8)
- added L401: 2n (0.1n), Inductor_SMD:L_0402_1005Metric, F.Cu at (189.2, 66.0)
- added L601: 4u7, Inductor_SMD:L_0805_2012Metric, F.Cu at (204.2, 87.2)
- added L701: 1u, Charge_Manager_FP:74439323010, F.Cu at (139.8, 94.0)
- added LED1101: YELLOW, LED_SMD:LED_1206_3216Metric, F.Cu at (199.8, 52.8)
- added LED601: RED, LED_SMD:LED_1206_3216Metric, F.Cu at (200.0, 84.8)
- added LED701: RED, LED_SMD:LED_1206_3216Metric, F.Cu at (125.2, 69.5)
- added LED801: RED, LED_SMD:LED_1206_3216Metric, F.Cu at (183.0, 116.2)
- added LED802: RED, LED_SMD:LED_1206_3216Metric, F.Cu at (206.8, 116.2)
- added NT801: NetTie_TS, NetTie:NetTie-2_SMD_Pad0.5mm, F.Cu at (181.0, 92.8)
- added NT901: NetTie_CSA, NetTie:NetTie-2_SMD_Pad0.5mm, F.Cu at (174.0, 66.2)
- added NT902: NetTie_CSA, NetTie:NetTie-2_SMD_Pad0.5mm, F.Cu at (173.0, 66.0)
- added Q1101: PMV90ENER, Package_TO_SOT_SMD:SOT-23-3, F.Cu at (196.8, 52.5)
- added Q701: CSD18540Q5B, Package_TO_SOT_SMD:TDSON-8-1, F.Cu at (126.2, 98.1)
- added Q702: CSD18540Q5B, Package_TO_SOT_SMD:TDSON-8-1, F.Cu at (142.4, 87.0)
- added Q703: CSD18540Q5B, Package_TO_SOT_SMD:TDSON-8-1, F.Cu at (129.5, 90.9)
- added Q704: CSD18540Q5B, Package_TO_SOT_SMD:TDSON-8-1, F.Cu at (146.4, 93.8)
- added Q801: CSD18540Q5B, Package_TO_SOT_SMD:TDSON-8-1, F.Cu at (179.3, 104.4)
- added Q802: CSD18540Q5B, Package_TO_SOT_SMD:TDSON-8-1, F.Cu at (185.7, 104.4)
- added Q803: CSD18540Q5B, Package_TO_SOT_SMD:TDSON-8-1, F.Cu at (179.3, 81.3)
- added Q804: CSD18540Q5B, Package_TO_SOT_SMD:TDSON-8-1, F.Cu at (185.6, 81.3)
- added R1001: 10k 1%, Resistor_SMD:R_0402_1005Metric, F.Cu at (166.9, 59.1)
- added R1002: 10k 1%, Resistor_SMD:R_0402_1005Metric, F.Cu at (166.9, 60.2)
- added R1003: 10k 1%, Resistor_SMD:R_0402_1005Metric, F.Cu at (167.0, 61.4)
- added R1004: 10k 1%, Resistor_SMD:R_0402_1005Metric, F.Cu at (166.9, 62.5)
- added R1005: 27R 1%, Resistor_SMD:R_0402_1005Metric, F.Cu at (173.3, 59.6)
- added R1006: 27R 1%, Resistor_SMD:R_0402_1005Metric, F.Cu at (172.2, 59.6)
- added R1007: 27R 1%, Resistor_SMD:R_0402_1005Metric, F.Cu at (170.8, 59.6)
- added R1008: 27R 1%, Resistor_SMD:R_0402_1005Metric, F.Cu at (169.6, 59.6)
- added R1009: 5k1 1%, Resistor_SMD:R_0402_1005Metric, F.Cu at (209.1, 59.8)
- added R1010: 5k1 1%, Resistor_SMD:R_0402_1005Metric, F.Cu at (204.1, 59.8)
- added R1011: 27R 1%, Resistor_SMD:R_0402_1005Metric, F.Cu at (197.8, 58.8)
- added R1012: 27R 1%, Resistor_SMD:R_0402_1005Metric, F.Cu at (197.8, 57.8)
- added R1101: 56R 1% 0.5W, Resistor_SMD:R_0805_2012Metric_Pad1.20x1.40mm_HandSolder, F.Cu at (198.5, 56.0)
- added R1102: 100R 1% 0.2W, Resistor_SMD:R_0402_1005Metric, F.Cu at (196.0, 56.5)
- added R1103: 100k 1%, Resistor_SMD:R_0402_1005Metric, F.Cu at (194.8, 55.8)
- added R401: 10k 1%, Resistor_SMD:R_0402_1005Metric, F.Cu at (191.3, 66.8)
- added R402: 10k 1%, Resistor_SMD:R_0402_1005Metric, F.Cu at (191.7, 65.8)
- added R403: 10k 1%, Resistor_SMD:R_0402_1005Metric, F.Cu at (192.0, 64.8)
- added R404: 10k 1%, Resistor_SMD:R_0402_1005Metric, F.Cu at (190.5, 54.0)
- added R405: 10k 1%, Resistor_SMD:R_0402_1005Metric, F.Cu at (189.5, 54.0)
- added R406: 10k 1%, Resistor_SMD:R_0402_1005Metric, F.Cu at (197.2, 60.8)
- added R407: 10k 1%, Resistor_SMD:R_0402_1005Metric, F.Cu at (189.2, 72.5)
- added R408: 10k 1%, Resistor_SMD:R_0402_1005Metric, F.Cu at (196.5, 71.5)
- added R601: 56R 1% 0.5W, Resistor_SMD:R_0805_2012Metric_Pad1.20x1.40mm_HandSolder, F.Cu at (203.2, 84.5)
- added R602: 10k 1%, Resistor_SMD:R_0402_1005Metric, F.Cu at (203.8, 78.3)
- added R603: 10k 1%, Resistor_SMD:R_0402_1005Metric, F.Cu at (203.8, 79.6)
- added R604: 10k 1%, Resistor_SMD:R_0402_1005Metric, F.Cu at (203.8, 81.0)
- added R605: 10k 1%, Resistor_SMD:R_0402_1005Metric, F.Cu at (203.8, 77.1)
- added R606: 909k 1%, Resistor_SMD:R_0805_2012Metric_Pad1.20x1.40mm_HandSolder, F.Cu at (207.0, 84.8)
- added R607: 301k 1%, Resistor_SMD:R_0805_2012Metric_Pad1.20x1.40mm_HandSolder, F.Cu at (210.0, 93.8)
- added R608: 44k2 1%, Resistor_SMD:R_0402_1005Metric, F.Cu at (208.5, 91.8)
- added R701: 7m 1% 1W, Resistor_SMD:R_0805_2012Metric_Pad1.20x1.40mm_HandSolder, F.Cu at (135.5, 79.0)
- added R702: 3R 1%, Resistor_SMD:R_0603_1608Metric, F.Cu at (129.7, 101.8)
- added R703: 3R 1%, Resistor_SMD:R_0603_1608Metric, F.Cu at (146.9, 89.8)
- added R704: 130k 1%, Resistor_SMD:R_0402_1005Metric, F.Cu at (146.2, 84.2)
- added R705: 75k 1%, Resistor_SMD:R_0402_1005Metric, F.Cu at (127.0, 108.0)
- added R706: 130k 1%, Resistor_SMD:R_0402_1005Metric, F.Cu at (127.0, 105.5)
- added R707: 1k 1% 2W, Resistor_SMD:R_2010_5025Metric, F.Cu at (131.0, 69.5)
- added R708: 0R 1%, Resistor_SMD:R_0603_1608Metric, F.Cu at (129.7, 103.5)
- added R709: 0R 1%, Resistor_SMD:R_0603_1608Metric, F.Cu at (146.9, 88.0)
- added R710: 10k 1%, Resistor_SMD:R_0402_1005Metric, F.Cu at (129.2, 108.0)
- added R711: 5k6 1%, Resistor_SMD:R_0402_1005Metric, F.Cu at (129.2, 105.5)
- added R712: 1m 1% 2W, Resistor_SMD:R_1206_3216Metric_Pad1.30x1.75mm_HandSolder, F.Cu at (133.8, 95.2)
- added R713: 5k6 1%, Resistor_SMD:R_0402_1005Metric, F.Cu at (146.2, 85.8)
- added R714: 3R 1%, Resistor_SMD:R_0603_1608Metric, F.Cu at (125.0, 93.7)
- added R715: 3R 1%, Resistor_SMD:R_0603_1608Metric, F.Cu at (151.5, 98.3)
- added R716: 0R 1%, Resistor_SMD:R_0603_1608Metric, F.Cu at (123.2, 93.7)
- added R717: 0R 1%, Resistor_SMD:R_0603_1608Metric, F.Cu at (149.8, 98.3)
- added R718: 10R 1%, Resistor_SMD:R_0402_1005Metric, F.Cu at (146.8, 103.8)
- added R719: 10R 1%, Resistor_SMD:R_0402_1005Metric, F.Cu at (146.8, 104.8)
- added R720: 44k2 1%, Resistor_SMD:R_0402_1005Metric, F.Cu at (136.2, 104.0)
- added R721: 10k 1%, Resistor_SMD:R_0402_1005Metric, F.Cu at (140.5, 108.0)
- added R722: 20k5 1%, Resistor_SMD:R_0402_1005Metric, F.Cu at (136.2, 103.0)
- added R723: 56k 1%, Resistor_SMD:R_0402_1005Metric, F.Cu at (139.0, 106.5)
- added R801: 0R 1%, Resistor_SMD:R_0603_1608Metric, F.Cu at (175.8, 91.5)
- added R802: 100R 1% 0.2W, Resistor_SMD:R_0402_1005Metric, F.Cu at (183.0, 112.8)
- added R803: 1k 1% 2W, Resistor_SMD:R_2010_5025Metric, F.Cu at (186.5, 115.2)
- added R804: 3R 1%, Resistor_SMD:R_0603_1608Metric, F.Cu at (173.8, 91.5)
- added R805: 1m 1% 2W, Resistor_SMD:R_1206_3216Metric_Pad1.30x1.75mm_HandSolder, F.Cu at (167.0, 98.5)
- added R806: 1m 1% 2W, Resistor_SMD:R_1206_3216Metric_Pad1.30x1.75mm_HandSolder, F.Cu at (172.8, 70.2)
- added R807: 3R 1%, Resistor_SMD:R_0603_1608Metric, F.Cu at (170.5, 83.8)
- added R808: 1k 1% 2W, Resistor_SMD:R_2010_5025Metric, F.Cu at (206.8, 109.4)
- added R809: 0R 1%, Resistor_SMD:R_0603_1608Metric, F.Cu at (172.0, 83.8)
- added R810: 240k 1%, Resistor_SMD:R_0805_2012Metric_Pad1.20x1.40mm_HandSolder, F.Cu at (163.5, 93.0)
- added R811: 20k5 1%, Resistor_SMD:R_0402_1005Metric, F.Cu at (165.8, 86.5)
- added R812: 20k5 1%, Resistor_SMD:R_0402_1005Metric, F.Cu at (165.0, 80.8)
- added R813: 100R 1% 0.2W, Resistor_SMD:R_0402_1005Metric, F.Cu at (173.5, 86.8)
- added R814: 100R 1% 0.2W, Resistor_SMD:R_0402_1005Metric, F.Cu at (171.8, 75.5)
- added R815: 100R 1% 0.2W, Resistor_SMD:R_0402_1005Metric, F.Cu at (163.2, 90.0)
- added R816: 10k 1%, Resistor_SMD:R_0402_1005Metric, F.Cu at (163.2, 87.8)
- added R817: 10k 1%, Resistor_SMD:R_0402_1005Metric, F.Cu at (165.2, 91.5)
- added R818: 10k 1%, Resistor_SMD:R_0402_1005Metric, F.Cu at (163.2, 81.2)
- added R819: 100k 1%, Resistor_SMD:R_0402_1005Metric, F.Cu at (171.2, 92.5)
- added R820: 100k 1%, Resistor_SMD:R_0402_1005Metric, F.Cu at (169.0, 80.8)
- added S401: B3U-1100P-B, Charge_Manager_FP:B3U1100PB, F.Cu at (192.8, 72.2)
- added S402: B3U-1100P-B, Charge_Manager_FP:B3U1100PB, F.Cu at (200.2, 72.2)
- added TP1001: VIN2, TestPoint:TestPoint_Pad_D1.0mm, F.Cu at (210.0, 65.0)
- added TP1002: GND, TestPoint:TestPoint_Pad_D1.0mm, F.Cu at (217.5, 45.5)
- added TP401: MTCK, TestPoint:TestPoint_Pad_D1.0mm, F.Cu at (228.8, 44.6)
- added TP402: MTDO, TestPoint:TestPoint_Pad_D1.0mm, F.Cu at (228.8, 47.6)
- added TP403: MTDI, TestPoint:TestPoint_Pad_D1.0mm, F.Cu at (228.8, 50.7)
- added TP404: MTMS, TestPoint:TestPoint_Pad_D1.0mm, F.Cu at (228.8, 53.8)
- added TP405: SPI_NCS, TestPoint:TestPoint_Pad_D1.0mm, F.Cu at (228.8, 56.8)
- added TP406: SPI_MOSI, TestPoint:TestPoint_Pad_D1.0mm, F.Cu at (215.4, 47.9)
- added TP407: SPI_MISO, TestPoint:TestPoint_Pad_D1.0mm, F.Cu at (231.8, 44.6)
- added TP408: SPI_CLK, TestPoint:TestPoint_Pad_D1.0mm, F.Cu at (231.8, 47.6)
- added TP409: SCL, TestPoint:TestPoint_Pad_D1.0mm, F.Cu at (231.8, 50.7)
- added TP410: SDA, TestPoint:TestPoint_Pad_D1.0mm, F.Cu at (231.8, 53.8)
- added TP411: CHARGER_STATUS, TestPoint:TestPoint_Pad_D1.0mm, F.Cu at (231.8, 56.8)
- added TP412: LED_DBG, TestPoint:TestPoint_Pad_D1.0mm, F.Cu at (218.4, 47.9)
- added TP413: PRIORITY, TestPoint:TestPoint_Pad_D1.0mm, F.Cu at (234.8, 44.6)
- added TP414: VALID1, TestPoint:TestPoint_Pad_D1.0mm, F.Cu at (234.8, 47.6)
- added TP415: VALID2, TestPoint:TestPoint_Pad_D1.0mm, F.Cu at (234.8, 50.7)
- added TP416: PGOOD, TestPoint:TestPoint_Pad_D1.0mm, F.Cu at (234.8, 53.8)
- added TP417: FAULT1, TestPoint:TestPoint_Pad_D1.0mm, F.Cu at (234.8, 56.8)
- added TP418: FAULT2, TestPoint:TestPoint_Pad_D1.0mm, F.Cu at (221.5, 47.9)
- added TP419: IMON1, TestPoint:TestPoint_Pad_D1.0mm, F.Cu at (237.9, 44.6)
- added TP420: IMON2, TestPoint:TestPoint_Pad_D1.0mm, F.Cu at (237.9, 47.6)
- added TP421: GND, TestPoint:TestPoint_Pad_D1.0mm, F.Cu at (237.9, 50.7)
- added TP422: GND, TestPoint:TestPoint_Pad_D1.0mm, F.Cu at (237.9, 53.8)
- added TP601: +VOUT, TestPoint:TestPoint_Pad_D1.0mm, F.Cu at (218.7, 53.6)
- added TP602: +VBUS, TestPoint:TestPoint_Pad_D1.0mm, F.Cu at (215.8, 52.6)
- added TP603: VIN2, TestPoint:TestPoint_Pad_D1.0mm, F.Cu at (216.6, 55.6)
- added TP604: GND, TestPoint:TestPoint_Pad_D1.0mm, F.Cu at (220.7, 51.9)
- added TP605: GND, TestPoint:TestPoint_Pad_D1.0mm, F.Cu at (220.7, 54.9)
- added TP701: +VCHARGE, TestPoint:TestPoint_Pad_D1.0mm, F.Cu at (162.7, 128.7)
- added TP702: +VSUPPLY, TestPoint:TestPoint_Pad_D1.0mm, F.Cu at (162.7, 131.7)
- added TP703: HO1, TestPoint:TestPoint_Pad_D1.0mm, F.Cu at (162.7, 134.8)
- added TP704: HO2, TestPoint:TestPoint_Pad_D1.0mm, F.Cu at (162.7, 137.8)
- added TP705: LO1, TestPoint:TestPoint_Pad_D1.0mm, F.Cu at (162.7, 140.8)
- added TP706: LO2, TestPoint:TestPoint_Pad_D1.0mm, F.Cu at (165.8, 128.7)
- added TP707: SW1, TestPoint:TestPoint_Pad_D1.0mm, F.Cu at (165.8, 131.7)
- added TP708: SW2, TestPoint:TestPoint_Pad_D1.0mm, F.Cu at (165.8, 134.8)
- added TP709: GND, TestPoint:TestPoint_Pad_D1.0mm, F.Cu at (165.8, 137.8)
- added TP710: GND, TestPoint:TestPoint_Pad_D1.0mm, F.Cu at (165.8, 140.8)
- added TP801: OUTA, TestPoint:TestPoint_Pad_D1.0mm, F.Cu at (166.8, 92.5)
- added TP802: TGDN1, TestPoint:TestPoint_Pad_D1.0mm, F.Cu at (177.2, 93.8)
- added TP803: OUTB, TestPoint:TestPoint_Pad_D1.0mm, F.Cu at (163.2, 79.5)
- added TP804: TGDN2, TestPoint:TestPoint_Pad_D1.0mm, F.Cu at (173.5, 84.2)
- added TP805: INX, TestPoint:TestPoint_Pad_D1.0mm, F.Cu at (163.0, 85.8)
- added TP806: VCC1, TestPoint:TestPoint_Pad_D1.0mm, F.Cu at (169.0, 92.5)
- added TP807: VCC2, TestPoint:TestPoint_Pad_D1.0mm, F.Cu at (163.8, 73.5)
- added TP808: +VCHARGE, TestPoint:TestPoint_Pad_D1.0mm, F.Cu at (176.0, 111.0)
- added TP809: GND, TestPoint:TestPoint_Pad_D1.0mm, F.Cu at (180.1, 114.1)
- added TP810: +VSUPPLY, TestPoint:TestPoint_Pad_D1.0mm, F.Cu at (136.5, 55.8)
- added TP811: GND, TestPoint:TestPoint_Pad_D1.0mm, F.Cu at (203.5, 100.0)
- added TP812: VDD, TestPoint:TestPoint_Pad_D1.0mm, F.Cu at (163.0, 83.2)
- added U401: ESP32-S3FN8, Package_DFN_QFN:QFN-56-1EP_7x7mm_P0.4mm_EP4x4mm, F.Cu at (191.2, 59.8)
- added U701: LM51772RHAR, Charge_Manager_FP:LM51772RHAR, F.Cu at (141.0, 101.8)
- added U901: INA239AQDGSRQ1, Charge_Manager_FP:INA239AQDGSRQ1, F.Cu at (179.0, 65.5)
- added Y401: ECS-400-10-33B-CKM-TR, Charge_Manager_FP:XTAL_ECS-400-10-33B-CKM-TR, F.Cu at (183.8, 59.7)
- added kibuzzard-67141537: G***, kibuzzard-67141537, F.Cu at (209.2, 111.2)
- added kibuzzard-67161F44: G***, kibuzzard-67161F44, F.Cu at (180.1, 114.1)
Routing:
- net /Project Architecture/Power - Power Path/GATE2: track 0.00 -> 20.9 mm
- net /Project Architecture/Power - Power Path/GATE1: track 0.00 -> 20.0 mm
- net /Project Architecture/Power - Generation/FB: track 0.00 -> 10.9 mm, vias 0 -> 2
- net /Project Architecture/Power - Power Path/SOURCE1: track 0.00 -> 10.0 mm
- net /Project Architecture/Power - Power Path/TGDN2: track 0.00 -> 5.78 mm
- net /Project Architecture/Power - Generation/+VOUT: track 0.00 -> 5.69 mm
- net /Project Architecture/Power - Power Path/TS: track 0.00 -> 5.44 mm
- net /Project Architecture/Power - Power Path/TGDN1: track 0.00 -> 4.71 mm
- net Net-(IC601-ENA): track 0.00 -> 3.71 mm
- net Net-(IC601-BST1): track 0.00 -> 3.67 mm
- net Net-(LED801-A): track 0.00 -> 3.54 mm
- net /Project Architecture/Power - Generation/SW1_3V3: track 0.00 -> 3.50 mm
- net Net-(LED802-A): track 0.00 -> 3.14 mm
- net Net-(R802-Pad2): track 0.00 -> 3.07 mm
- net Net-(LED601-A): track 0.00 -> 2.76 mm
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- added copper zone on F.Cu, net +3V3
- added copper zone on F.Cu, net +VBAT
- added copper zone on F.Cu, net +VCHARGE
- added copper zone on F.Cu, net +VSUPPLY
- added copper zone on F.Cu, net /Project Architecture/Power - Charger/SW1
- added copper zone on F.Cu, net /Project Architecture/Power - Charger/SW2
- added copper zone on F.Cu, net /Project Architecture/Power - Charger/shunt_bridge-
- added copper zone on F.Cu, net /Project Architecture/Power - Generation/+VOUT
- added copper zone on F.Cu, net /Project Architecture/Power - Power Path/SOURCE1
- added copper zone on F.Cu, net GND
Other:
- board outline added: 95 x 70 mm
- copper layers 6 -> 4
