File: Power/ElonMux/Misc - Mounting Holes.kicad_sch (KiCad schematic)
At the start: 12 parts

Commit message: Implemented more fede recommandations
Parts:
- added C1201, C1202, C1203: 1n X7R 1kV, Capacitor_SMD:C_0603_1608Metric, symbol Device:C_Small
Connections:
- net GND: now also C1201.2, C1202.2, C1203.2
- net at H1203.1, R1203.1: now also C1203.1
- net at H1202.1, R1202.1: now also C1202.1
- net at H1201.1, R1201.1: now also C1201.1
Other:
- moved on the sheet: H1201

Commit message: Preliminary Submission
Parts:
- added C1204: 1n X7R 1kV, Capacitor_SMD:C_0603_1608Metric, symbol Device:C_Small
- added H1204: M3 (3.2mm), MountingHole:MountingHole_3.2mm_M3_Pad_Via, symbol Mechanical:MountingHole_Pad
- added R1204: 0R 1%, Resistor_SMD:R_0603_1608Metric, symbol Device:R
Connections:
- net GND: now also C1204.2, R1204.2
- new net: C1204.1, H1204.1, R1204.1
Other:
- moved on the sheet: C1201, C1202, C1203, H1201, H1202, H1203, R1201, R1202, R1203

Commit message: Removed some weird rooting angles, and fixed capa for reset button
Other:
- title: Misc - Mouting Holes -> Misc - Mouting Holes & Fiducials
Changed lines of the file:
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@@
 	(paper "A4")
 	(title_block
-		(title "Misc - Mouting Holes")
+		(title "Misc - Mouting Holes & Fiducials")
 		(date "Last Modified Date")
 		(rev "${REVISION}")
@@
 	(text_box "[${#}] ${TITLE}"
 		(exclude_from_sim no)
-		(at 96.52 15.24 0)
-		(size 107.315 12.7)
+		(at 10.16 15.24 0)
+		(size 276.86 12.7)
 		(stroke
 			(width -0.0001)

Commit message: Added MODE, U0TX, U0RX, sourced from Mouser
Parts:
- C1201, C1202, C1203, C1204: Manufacturer Part Number C0603V102KDRAC7867 -> C0603C102MDRAC7081; Supplier Digikey -> Mouser Electronics; Supplier Part Number 399-12306-1-ND -> 80-C0603C102MDRAC

Commit message: Final version with Buck-Boost
Other:
- moved on the sheet: C1201, C1202, C1203, C1204, H1201, H1202, H1203, H1204, R1201, R1202, R1203, R1204

Commit message: More corrections and adjustments
Connections:
- net HOLE1: now reaches C1201.1, H1201.1, R1201.1
- net HOLE3: now reaches C1203.1, H1203.1, R1203.1
- net HOLE4: now reaches C1204.1, H1204.1, R1204.1
- net HOLE2: now reaches C1202.1, H1202.1, R1202.1
Changed lines of the file:
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@@
+		)
+	)
+	(label "HOLE3"
+		(at 151.13 91.44 0)
+		(fields_autoplaced yes)
+		(effects
+			(font
+				(size 1.27 1.27)
+			)
+			(justify left bottom)
+		)
+	)
+	(label "HOLE4"
+		(at 179.07 91.44 0)
+		(fields_autoplaced yes)
+		(effects
+			(font
+				(size 1.27 1.27)
+			)
+			(justify left bottom)
+		)
+	)
+	(label "HOLE2"
+		(at 121.92 91.44 0)
+		(fields_autoplaced yes)
+		(effects
+			(font
+				(size 1.27 1.27)
+			)
+			(justify left bottom)
+		)
+	)
+	(label "HOLE1"
+		(at 92.71 91.44 0)
+		(fields_autoplaced yes)
+		(effects
+			(font
+				(size 1.27 1.27)
+			)
+			(justify left bottom)
 		)
 	)

Commit message: Re-rooted charger area for reduced EMI and added 24V FAN soldering holes
Parts:
- removed C1202: 1n X7R 1kV, Capacitor_SMD:C_0603_1608Metric, symbol Device:C_Small
- removed R1202: 0R 1%, Resistor_SMD:R_0603_1608Metric, symbol Device:R
- renumbered C1203 to C1202, C1204 to C1203, R1203 to R1202, R1204 to R1203
Connections:
- net HOLE2 is gone; now on net GND: H1202.1

Commit message: Changed inductors footprints, cleaned copper fills areas, improved silkscreen
Parts:
- removed FM1204, FM1205, FM1206: Fiducial, Charge_Manager_FP:Fiducial_1mm_Mask2mm, symbol Mechanical:Fiducial
Changed lines of the file:
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@@
-		)
-	)
-	(text_box "Back"
-		(exclude_from_sim no)
-		(at 215.265 95.25 0)
-		(size 31.115 9.525)
-		(stroke
-			(width -0.0001)
-			(type default)
-		)
-		(fill
-			(type none)
-		)
-		(effects
-			(font
-				(face "Times New Roman")
-				(size 2.54 2.54)
-				(thickness 0.508)
-				(bold yes)
-				(color 0 0 0 1)
-			)
-			(justify bottom)
 		)
 	)
@@
 	(label "HOLE3"
 		(at 151.13 91.44 0)
-		(fields_autoplaced yes)
 		(effects
 			(font
@@
 	(label "HOLE4"
 		(at 179.07 91.44 0)
-		(fields_autoplaced yes)
 		(effects
 			(font
@@
 	(label "HOLE2"
 		(at 121.92 91.44 0)
-		(fields_autoplaced yes)
 		(effects
 			(font
@@
 	(label "HOLE1"
 		(at 92.71 91.44 0)
-		(fields_autoplaced yes)
 		(effects
 			(font
@@
 			)
 			(justify left bottom)
-		)
-	)
-	(symbol
-		(lib_id "Mechanical:Fiducial")
-		(at 231.14 110.49 0)
-		(unit 1)
-		(exclude_from_sim no)
-		(in_bom no)
-		(on_board yes)
-		(dnp no)
-		(property "Reference" "FM1205"
-			(at 231.14 106.68 0)
-			(effects
-				(font
-					(size 1.27 1.27)
-				)
-			)
-		)
-		(property "Value" "Fiducial"
-			(at 233.68 111.76 0)
-			(effects
-				(font
-					(size 1.27 1.27)
-				)
-				(justify left)
-				(hide yes)
-			)
-		)
-		(property "Footprint" "Charge_Manager_FP:Fiducial_1mm_Mask2mm"
-			(at 231.14 110.49 0)
-			(effects
-				(font
-					(size 1.27 1.27)
-				)
-				(hide yes)
-			)
-		)
-		(property "Datasheet" "~"
-			(at 231.14 110.49 0)
-			(effects
-				(font
-					(size 1.27 1.27)
-				)
-				(hide yes)
-			)
-		)
-		(property "Description" ""
-			(at 231.14 110.49 0)
-			(effects
-				(font
-					(size 1.27 1.27)
-				)
-				(hide yes)
-			)
-		)
-		(instances
-			(project "ElonMux"
-				(path "/0650c7a8-acba-429c-9f8e-eec0baf0bc1c/fede4c36-00cc-4d3d-b71c-5243ba232202/e246552c-c235-46f6-8325-624faa438117"
-					(reference "FM1205")
-					(unit 1)
-				)
-			)
 		)
 	)
@@
 	)
 	(symbol
-		(lib_id "Mechanical:Fiducial")
-		(at 221.615 110.49 0)
-		(unit 1)
-		(exclude_from_sim no)
-		(in_bom no)
-		(on_board yes)
-		(dnp no)
-		(property "Reference" "FM1204"
-			(at 221.615 106.68 0)
-			(effects
-				(font
-					(size 1.27 1.27)
-				)
-			)
-		)
-		(property "Value" "Fiducial"
-			(at 224.155 111.76 0)
-			(effects
-				(font
-					(size 1.27 1.27)
-				)
-				(justify left)
-				(hide yes)
-			)
-		)
-		(property "Footprint" "Charge_Manager_FP:Fiducial_1mm_Mask2mm"
-			(at 221.615 110.49 0)
-			(effects
-				(font
-					(size 1.27 1.27)
-				)
-				(hide yes)
-			)
-		)
-		(property "Datasheet" "~"
-			(at 221.615 110.49 0)
-			(effects
-				(font
-					(size 1.27 1.27)
-				)
-				(hide yes)
-			)
-		)
-		(property "Description" ""
-			(at 221.615 110.49 0)
-			(effects
-				(font
-					(size 1.27 1.27)
-				)
-				(hide yes)
-			)
-		)
-		(instances
-			(project "ElonMux"
-				(path "/0650c7a8-acba-429c-9f8e-eec0baf0bc1c/fede4c36-00cc-4d3d-b71c-5243ba232202/e246552c-c235-46f6-8325-624faa438117"
-					(reference "FM1204")
-					(unit 1)
-				)
-			)
-		)
-	)
-	(symbol
 		(lib_id "Device:C_Small")
 		(at 172.72 96.52 0)
@@
 					(unit 1)
 				)
-			)
-		)
-	)
-	(symbol
-		(lib_id "Mechanical:Fiducial")
-		(at 240.03 110.49 0)
-		(unit 1)
-		(exclude_from_sim no)
-		(in_bom no)
-		(on_board yes)
-		(dnp no)
-		(property "Reference" "FM1206"
-			(at 240.03 106.68 0)
-			(effects
-				(font
-					(size 1.27 1.27)
-				)
-			)
-		)
-		(property "Value" "Fiducial"
-			(at 242.57 111.76 0)
-			(effects
-				(font
-					(size 1.27 1.27)
-				)
-				(justify left)
-				(hide yes)
-			)
-		)
-		(property "Footprint" "Charge_Manager_FP:Fiducial_1mm_Mask2mm"
-			(at 240.03 110.49 0)
-			(effects
-				(font
-					(size 1.27 1.27)
-				)
-				(hide yes)
-			)
-		)
-		(property "Datasheet" "~"
-			(at 240.03 110.49 0)
-			(effects
-				(font
-					(size 1.27 1.27)
-				)
-				(hide yes)
-			)
-		)
-		(property "Description" ""
-			(at 240.03 110.49 0)
-			(effects
-				(font
-					(size 1.27 1.27)
-				)
-				(hide yes)
-			)
-		)
-		(instances
-			(project "ElonMux"
-				(path "/0650c7a8-acba-429c-9f8e-eec0baf0bc1c/fede4c36-00cc-4d3d-b71c-5243ba232202/e246552c-c235-46f6-8325-624faa438117"
-					(reference "FM1206")
-					(unit 1)
-				)
