File: Power/ElonMux/User - LED Indicators.kicad_sch (KiCad schematic)
At the start: 5 parts, among them Q1101 PMV90ENER

Commit message: Almost done with schematics
Parts:
- LED1101: footprint LEDC1608X60N -> LED_SMD:LED_1206_3216Metric
- Q1101: footprint 0_package_SOT_TO_SMD:SOT-23-3 -> Package_TO_SOT_SMD:SOT-23-3
- R1101: footprint (none) -> Resistor_SMD:R_0805_2012Metric_Pad1.20x1.40mm_HandSolder; Manufacturer (none) -> KOA Speer; Manufacturer Part Number (none) -> SG73P2ATTD56R0F; Supplier (none) -> Mouser Electronics; Supplier Part Number (none) -> 660-SG73P2ATTD56R0F
- R1102: footprint (none) -> Resistor_SMD:R_0402_1005Metric; Manufacturer (none) -> Vishay / Dale; Manufacturer Part Number (none) -> CRCW0402100RFKEDHP; Supplier (none) -> Mouser Electronics; Supplier Part Number (none) -> 71-CRCW0402100RFKEDH
- R1103: footprint (none) -> Resistor_SMD:R_0402_1005Metric; Manufacturer (none) -> Panasonic; Manufacturer Part Number (none) -> ERJ-PA2F1003X; Supplier (none) -> Mouser Electronics; Supplier Part Number (none) -> 667-ERJ-PA2F1003X
Changed lines of the file:
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@@
 			)
 		)
-		(property "Footprint" "0_package_SOT_TO_SMD:SOT-23-3"
+		(property "Footprint" "Package_TO_SOT_SMD:SOT-23-3"
 			(at 177.8 88.9 0)
 			(effects
@@
 			)
 		)
-		(property "Footprint" ""
+		(property "Footprint" "Resistor_SMD:R_0402_1005Metric"
 			(at 160.02 99.822 90)
 			(effects
@@
 			)
 		)
-		(property "Datasheet" "~"
+		(property "Datasheet" "https://www.vishay.com/docs/20043/crcwhpe3.pdf"
 			(at 160.02 101.6 0)
 			(effects
@@
 			)
 		)
-		(property "Manufacturer Part Number" ""
+		(property "Manufacturer Part Number" "CRCW0402100RFKEDHP"
 			(at 160.02 101.6 0)
 			(effects
@@
 			)
 		)
-		(property "Supplier" ""
+		(property "Supplier" "Mouser Electronics"
+			(at 160.02 101.6 0)
+			(effects
+				(font
+					(size 1.27 1.27)
+				)
+				(hide yes)
+			)
+		)
+		(property "Manufacturer" "Vishay / Dale"
+			(at 160.02 101.6 0)
+			(effects
+				(font
+					(size 1.27 1.27)
+				)
+				(hide yes)
+			)
+		)
+		(property "Supplier Part Number" "71-CRCW0402100RFKEDH"
 			(at 160.02 101.6 0)
 			(effects
@@
 			)
 		)
-		(property "Footprint" ""
+		(property "Footprint" "Resistor_SMD:R_0805_2012Metric_Pad1.20x1.40mm_HandSolder"
 			(at 173.482 74.93 90)
 			(effects
@@
 			)
 		)
-		(property "Datasheet" "~"
+		(property "Datasheet" "https://www.koaspeer.com/pdfs/SG73P.pdf"
 			(at 175.26 74.93 0)
 			(effects
@@
 			)
 		)
-		(property "Manufacturer Part Number" ""
+		(property "Manufacturer Part Number" "SG73P2ATTD56R0F"
 			(at 175.26 74.93 0)
 			(effects
@@
 			)
 		)
-		(property "Supplier" ""
+		(property "Supplier" "Mouser Electronics"
+			(at 175.26 74.93 0)
+			(effects
+				(font
+					(size 1.27 1.27)
+				)
+				(hide yes)
+			)
+		)
+		(property "Manufacturer" "KOA Speer"
+			(at 175.26 74.93 0)
+			(effects
+				(font
+					(size 1.27 1.27)
+				)
+				(hide yes)
+			)
+		)
+		(property "Supplier Part Number" "660-SG73P2ATTD56R0F"
 			(at 175.26 74.93 0)
 			(effects
@@
 			)
 		)
-		(property "Footprint" ""
+		(property "Footprint" "Resistor_SMD:R_0402_1005Metric"
 			(at 151.892 107.95 90)
 			(effects
@@
 			)
 		)
-		(property "Datasheet" "~"
+		(property "Datasheet" "https://www.mouser.ch/datasheet/2/315/AOA0000C331-1141874.pdf"
 			(at 153.67 107.95 0)
 			(effects
@@
 			)
 		)
-		(property "Manufacturer Part Number" ""
+		(property "Manufacturer Part Number" "ERJ-PA2F1003X"
 			(at 153.67 107.95 0)
 			(effects
@@
 			)
 		)
-		(property "Supplier" ""
+		(property "Supplier" "Mouser Electronics"
+			(at 153.67 107.95 0)
+			(effects
+				(font
+					(size 1.27 1.27)
+				)
+				(hide yes)
+			)
+		)
+		(property "Manufacturer" "Panasonic"
+			(at 153.67 107.95 0)
+			(effects
+				(font
+					(size 1.27 1.27)
+				)
+				(hide yes)
+			)
+		)
+		(property "Supplier Part Number" "667-ERJ-PA2F1003X"
 			(at 153.67 107.95 0)
 			(effects
@@
 			)
 		)
-		(property "Footprint" "LEDC1608X60N"
+		(property "Footprint" "LED_SMD:LED_1206_3216Metric"
 			(at 268.91 74.93 0)
 			(effects
@@
 			)
 		)
-		(property "Datasheet" "https://componentsearchengine.com/Datasheets/1/SM1206GC.pdf"
+		(property "Datasheet" "https://s3-us-west-2.amazonaws.com/catsy.557/Dialight_CBI_data_599-1206_Apr2018.pdf"
 			(at 368.91 74.93 0)
 			(effects

Commit message: Ready for layout review
Connections:
- net LED_D0: now reaches Q1101.1 (G), R1102.1
- net LED_D1: now reaches LED1101.1 (K), Q1101.3 (D)
- net LED_D2: now reaches LED1101.2 (A), R1101.2
Changed lines of the file:
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@@
+		)
+	)
+	(label "LED_D0"
+		(at 166.37 101.6 270)
+		(fields_autoplaced yes)
+		(effects
+			(font
+				(face "Arial")
+				(size 1.27 1.27)
+			)
+			(justify right bottom)
+		)
+	)
+	(label "LED_D1"
+		(at 175.26 96.52 0)
+		(fields_autoplaced yes)
+		(effects
+			(font
+				(face "Arial")
+				(size 1.27 1.27)
+			)
+			(justify left bottom)
 		)
 	)
 	(label "LED_DBG"
 		(at 133.35 101.6 0)
+		(fields_autoplaced yes)
+		(effects
+			(font
+				(face "Arial")
+				(size 1.27 1.27)
+			)
+			(justify left bottom)
+		)
+	)
+	(label "LED_D2"
+		(at 175.26 81.28 0)
 		(fields_autoplaced yes)
 		(effects
@@
 		)
 		(instances
-			(project "Charge Manager"
+			(project ""
 				(path "/0650c7a8-acba-429c-9f8e-eec0baf0bc1c/fede4c36-00cc-4d3d-b71c-5243ba232202/95e919be-32f9-400a-bc42-ccd9343a00dc"
 					(reference "Q1101")
@@
 		)
 		(instances
-			(project "Charge Manager"
+			(project ""
 				(path "/0650c7a8-acba-429c-9f8e-eec0baf0bc1c/fede4c36-00cc-4d3d-b71c-5243ba232202/95e919be-32f9-400a-bc42-ccd9343a00dc"
 					(reference "R1102")
@@
 		)
 		(instances
-			(project "Charge Manager"
+			(project ""
 				(path "/0650c7a8-acba-429c-9f8e-eec0baf0bc1c/fede4c36-00cc-4d3d-b71c-5243ba232202/95e919be-32f9-400a-bc42-ccd9343a00dc"
 					(reference "#PWR01101")
@@
 		)
 		(instances
-			(project "Charge Manager"
+			(project ""
 				(path "/0650c7a8-acba-429c-9f8e-eec0baf0bc1c/fede4c36-00cc-4d3d-b71c-5243ba232202/95e919be-32f9-400a-bc42-ccd9343a00dc"
 					(reference "R1101")
@@
 		)
 		(instances
-			(project "Charge Manager"
+			(project ""
 				(path "/0650c7a8-acba-429c-9f8e-eec0baf0bc1c/fede4c36-00cc-4d3d-b71c-5243ba232202/95e919be-32f9-400a-bc42-ccd9343a00dc"
 					(reference "#PWR01102")
@@
 		)
 		(instances
-			(project "Charge Manager"
+			(project ""
 				(path "/0650c7a8-acba-429c-9f8e-eec0baf0bc1c/fede4c36-00cc-4d3d-b71c-5243ba232202/95e919be-32f9-400a-bc42-ccd9343a00dc"
 					(reference "R1103")

Commit message: Merged ElonMux v1.0
Parts:
- R1101: value 56R 1% 0.5W -> 56R 1% 0.1W; footprint Resistor_SMD:R_0805_2012Metric_Pad1.20x1.40mm_HandSolder -> Resistor_SMD:R_0402_1005Metric; Manufacturer KOA Speer -> Panasonic; Manufacturer Part Number SG73P2ATTD56R0F -> ERJ-2RKF56R0X; Supplier Part Number 660-SG73P2ATTD56R0F -> 667-ERJ-2RKF56R0X
- R1103: Manufacturer Part Number ERJ-PA2F1003X -> ERJ-2RKF1003X; Supplier Part Number 667-ERJ-PA2F1003X -> 667-ERJ-2RKF1003X
