File: hats/new_imu_hat/Xplore ERC IMU HAT.kicad_sch (KiCad schematic)
At the start: 20 parts, among them J1 Hat_connector_hole, J2 5025850670, J3 BM04B-GHS-TBT, J4 BM04B-GHS-TBT, U1 LT3960JMSE-PBF

Commit message: Minor corrections
Layout needed some corrections
Parts:
- removed J2: 5025850670, IMU Library:CON_5025850670, symbol 502585-0670:5025850670
- removed J4: BM04B-GHS-TBT, IMU Library:CONN_BM04B-GHS-TBT_JST, symbol BM04B:BM04B-GHS-TBT
- removed JP1: SolderJumper_2_Open, symbol Jumper:SolderJumper_2_Open
- added J4: BM07B-GHS-TBTLFSNN, CONN_BM07B_JST, symbol BM07B-GHS-TBT:BM07B-GHS-TBTLFSNN
- added J5: 5025850470, CON_5025850470, symbol 502585470:5025850470
- added J6: 5025850570, CON_5025850570, symbol 502585570:5025850570
- added SW1: SW_DIP_x01, symbol Switch:SW_DIP_x01
- C1: value 1uF -> 2.2uF
- C4: value 2.2uF -> 1uF
- R6, R7: value 10k -> 4k7
Connections:
- net CANSCL+: now also J5.2
- net CANSCL-: now also J5.3
- net CANSDA+: now also J5.4
- net CANSDA-: now also J5.5
- net GND: now also U1.3 (GND), J4.7, J5.6, J6.7
- net INT1: now also J1.9 (GPIO_1), J4.2, J6.2; no longer J1.10 (GPIO_2)
- net INT3: now also J1.11 (GPIO_3), J4.4, J6.4; no longer J1.9 (GPIO_1)
- net at U1.7 (EN/MODE): now also SW1.2
- net INT4: now reaches J1.12 (GPIO_4)
- net INT4: now also J4.5, J6.5
- net +5V: now reaches J1.15 (5V)
- net +5V: now also C1.1, C4.1, R5.1, R6.1, R7.1, U1.6 (VIN), U1.8 (VCC), J5.1
- net at R5.2: now also SW1.1
- removed net +3V3: C1.1, C4.1, J1.2 (3.3V), J3.1, R5.1, R6.1, R7.1, U1.6 (VIN), U1.8 (VCC)
- new net +3.3V: J1.2 (3.3V), J3.1, J4.1, J6.1
- new net INT2: J1.10 (GPIO_2), J4.3, J6.3
- new net MAG_INT: J4.6, J6.6
- no-connect marks 10 -> 7
Other:
- note added: "CAN and INT/GPIO Headers"
- note added: "Switch should be turned on for Master Mode"
- note removed: "CAN and INT/GPIO Header"
- moved on the sheet: J1, J3

Commit message: IMU v3 review Ismail
Parts:
- renumbered C4 to C1, C1 to C2, C2 to C3, C3 to C4, J4 to J1, J5 to J2, J1 to J4, J6 to J5, R5 to R2, R2 to R3, R3 to R4, R7 to R5, R4 to R7
Connections:
- net +5V: now also J4.16 (5V), R2.2; no longer C2.1, R2.1, R5.1, R6.1, U1.8 (VCC)
- net SCL: now also R5.1; no longer R5.2
- net SDA: now also R6.1; no longer R6.2
- net at SW1.1: now also R2.1; no longer R2.2
- net +3.3V renamed +3v3
- net +3v3: now also C2.1, R5.2, R6.2, U1.8 (VCC)
- no-connect marks 7 -> 6
Other:
- note added: "Orion has I2C pullups, will need to make sure they aren't soldered on Orion so we use these ones"
- moved on the sheet: C1, C2, R2, R5, R6, SW1

Commit message: Updated new imu schematics and started layout and routing
Parts:
- removed J1: BM07B-GHS-TBTLFSNN, CONN_BM07B_JST, symbol BM07B-GHS-TBT:BM07B-GHS-TBTLFSNN
- removed J5: 5025850570, CON_5025850570, symbol 502585570:5025850570
- added J1: BM08B-GHS-TBT, footprints:CONN_BM08B-GHS-TBT_JST, symbol BM08B_GHS_TBT:BM08B-GHS-TBT
- added J5: 5025850470, footprints:CON_5025850470, symbol 502585470:5025850470
- C1, C2: footprint (none) -> Capacitor_SMD:C_0504_1310Metric
- CR1, CR2: footprint IMU Library:SOT23_PESD2_NEX -> footprints:SOT23_PESD2_NEX
- G1: footprint 0_graphic:Xplore_Logo_X_only_10mm -> footprints:Xplore_Logo_X_only_10mm
- J2: footprint CON_5025850470 -> footprints:CON_5025850470
- J3: footprint IMU Library:CONN_BM04B-GHS-TBT_JST -> footprints:CONN_BM04B-GHS-TBT_JST
- J4: footprint 0_connectors:Hat_connector_hole -> footprints:Hat_connector_hole
- R2, R5, R6: footprint (none) -> Resistor_SMD:R_0201_0603Metric
- SW1: footprint (none) -> Button_Switch_SMD:SW_DIP_SPSTx01_Slide_6.7x4.1mm_W6.73mm_P2.54mm_LowProfile_JPin
- U1: footprint IMU Library:LT3960 -> footprints:LT3960
Connections:
- net +3v3: now also J1.1
- net GND: now also J1.8
- net INT1: now also J1.2, J5.1
- net INT2: now also J1.3, J5.2
- net INT3: now also J1.4, J5.3
- net INT4: now also J1.5, J5.4
- net MAG_INT: now also J4.13 (GPIO_5), J1.6, J5.5
- net DRDY: now reaches J4.14 (GPIO_6)
- net DRDY: now also J1.7, J5.6
- no-connect marks 6 -> 4
Other:
- note added: "Additional connectors (Delocalizing)"
- note added: "BM08B might appear redundant because 502585470 has same labels but it is used to bring the interrupt signals to the IMU while this one delocalizes them if needed"
- note removed: "Additional connectors"
- moved on the sheet: J3

Commit message: First edition of the IMU routing done, waiting for reviews
Parts:
- G1: footprint footprints:Xplore_Logo_X_only_10mm -> footprints:Xplore_Logo_X_only_5mm
Changed lines of the file:
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@@
 			)
 		)
-		(property "Footprint" "footprints:Xplore_Logo_X_only_10mm"
+		(property "Footprint" "footprints:Xplore_Logo_X_only_5mm"
 			(at 247.65 149.86 0)
 			(effects

Commit message: IMU v2 after review, IMU is done HAT still isn't done and is WIP
Parts:
- removed J2, J5: 5025850470, footprints:CON_5025850470, symbol 502585470:5025850470
- added CR3, CR4, CR5, CR6: CDSOD323-T05C, footprints:DIODE_CDSOD323-T05C_BRN, symbol CDSOD323_T05C:CDSOD323-T05C
- added D1, D2, D3, D4, D5, D6, D7: PESD5V0S1UL_315, footprints:DIO_PESD5V0S1UL_315, symbol PESD5V0S1UL_315:PESD5V0S1UL_315
- added H1, H2, H3, H4: M2, MountingHole:MountingHole_2.2mm_M2, symbol Mechanical:MountingHole
- added J2: 5025850570, footprints:CON_5025850570, symbol 5025850570:5025850570
- added J5: 5025850670, footprints:CON_5025850670, symbol 502585670:5025850670
Connections:
- net +5V: now also D1.K
- net CANSCL+: now also CR5.1
- net CANSCL-: now also R3.1, CR6.1; no longer R3.2
- net CANSDA+: now also R4.2, CR3.1; no longer R4.1
- net CANSDA-: now also CR4.1
- net DRDY: now also D7.K
- net GND: now also J2.6, J2.7, J5.7, J5.8
- net INT1: now also D2.K
- net INT2: now also D3.K
- net INT3: now also D4.K
- net INT4: now also D5.K
- net MAG_INT: now also D6.K
- net at C3.1, R1.2: now also R3.2; no longer R3.1
- net at C4.1, R7.1: now also R4.1; no longer R4.2
- new net: D7.A, J5.6
- new net: D4.A, J5.3
- new net: CR5.2, J2.4
- new net: D5.A, J5.4
- new net: D3.A, J5.2
- new net: D2.A, J5.1
- new net: D6.A, J5.5
- new net: CR4.2, J2.2
- new net: CR3.2, J2.1
- new net: D1.A, J2.3
- new net: CR6.2, J2.5
Other:
- note added: "Mounting"
- moved on the sheet: R3, R4

Commit message: IMU v4.1, fixed diode selection
Parts:
- removed CR3, CR4, CR5, CR6: CDSOD323-T05C, footprints:DIODE_CDSOD323-T05C_BRN, symbol CDSOD323_T05C:CDSOD323-T05C
- removed D7: PESD5V0S1UL_315, footprints:DIO_PESD5V0S1UL_315, symbol PESD5V0S1UL_315:PESD5V0S1UL_315
- removed J2: 5025850570, footprints:CON_5025850570, symbol 5025850570:5025850570
- removed J5: 5025850670, footprints:CON_5025850670, symbol 502585670:5025850670
- added J2: 5025850670, footprints:CON_5025850670, symbol 502585670:5025850670
- added J5: 5025850570, footprints:CON_5025850570, symbol 5025850570:5025850570
- added U2: D5V0H1B2LP-7B, footprints:D5V0H1B2LP_7B, symbol D5V0H1B2LP_7B:D5V0H1B2LP-7B
- added U3: TPD4E05U06DQAR, footprints:TPD4E05U06DQAR, symbol TPD4E05U06DQAR:TPD4E05U06DQAR
Connections:
- net +5V: now also U2.1; no longer D1.K
- net CANSCL+: now also U3.4 (D2+)
- net CANSCL-: now also U3.5 (D2-)
- net CANSDA+: now also U3.1 (D1+)
- net CANSDA-: now also U3.2 (D1-)
- net DRDY: now also D6.K
- net GND: now also J2.7, J2.8, J5.6, J5.7, U3.3 (GND), U3.8 (GND)
- net INT1: now also D1.K; no longer D2.K
- net INT2: now also D2.K; no longer D3.K
- net INT3: now also D3.K; no longer D4.K
- net INT4: now also D4.K; no longer D5.K
- net MAG_INT: now also D5.K; no longer D6.K
- net at D4.A: now also J2.4
- net at D5.A: now also J2.5
- net at D3.A: now also J2.3
- net at D2.A: now also J2.2
- net at D6.A: now also J2.6
- net at D1.A: now also J2.1
- new net: J5.1, U3.10 (NC)
- new net: J5.2, U3.9 (NC)
- new net: J5.4, U3.7 (NC)
- new net: J5.5, U3.6 (NC)
- new net 5v_in: J5.3, U2.2
Other:
- moved on the sheet: H1, H2, H3, H4, J4

Commit message: IMU Layout and routing fixes
Parts:
- removed J5: 5025850570, footprints:CON_5025850570, symbol 5025850570:5025850570
- removed U3: TPD4E05U06DQAR, footprints:TPD4E05U06DQAR, symbol TPD4E05U06DQAR:TPD4E05U06DQAR
- added J5: 5025850670, footprints:CON_5025850670, symbol 502585670:5025850670
- C1, C2: footprint Capacitor_SMD:C_0504_1310Metric -> Capacitor_SMD:C_0402_1005Metric
Connections:
- net 5v_in: now also J5.3
- net CANSCL+: now also J5.4
- net CANSCL-: now also J5.5
- net CANSDA+: now also J5.2
- net CANSDA-: now also J5.1
- net GND: now also J5.6, J5.7, J5.8
Other:
- moved on the sheet: U2

Commit message: IMU tweaks
Parts:
- added C5: 100nF, Capacitor_SMD:C_0402_1005Metric, symbol Device:C
Connections:
- net +5V: now also J5.3, C5.2
- net DRDY: now also J2.6
- net GND: now also D1.A, D2.A, D3.A, D4.A, D5.A, D6.A, U2.2, C5.1
- net INT1: now also J2.1
- net INT2: now also J2.2
- net INT3: now also J2.3
- net INT4: now also J2.4
- net MAG_INT: now also J2.5
- removed net 5v_in: J5.3, U2.2
Other:
- moved on the sheet: J5
