File: Power/GEOX/rev1/SMPS_Motherboard/connectors_communication.kicad_sch (KiCad schematic)
At the start: 99 parts, among them IC1101 LAN9252_ML, IC1102 M24C16-RMN6P, J1102 Nano-Fit 1x03, J1103 Nano-Fit 1x03, J1104 Nano-Fit 1x03, J1105 Nano-Fit 1x03, J1107 RJ45_Wuerth_74980111211, J1108 RJ45_Wuerth_74980111211, J1109 PTH 01x03 2.54mm, J1110 PTH 01x03 2.54mm, SW1101 CAS-220TA, SW1103 CAS-220TA, U1101 TCAN1051HGVDRBRQ1, U1102 TCAN1051HGVDRBRQ1, Y1101 7M-25.000MAAJ-T

Commit message: Nothing to declare
Parts:
- renumbered C403 to C1109, C403 to C1110, C403 to C1111, C403 to C1112, C403 to C1113, C403 to C1114, C403 to C1115, C403 to C1116, C403 to C1117, C403 to C1118, C403 to C1119, C403 to C1120, C403 to C1121, C403 to C1122, C403 to C1123, C403 to C1124, C403 to C1125, C403 to C1126, C403 to C1127, C403 to C1128
