File: Power/GEOX/rev1/SMPS_Motherboard/mcu_power.kicad_sch.kicad_sch (KiCad schematic)
At the start: 32 parts, among them J402 Conn_Picoblade_JST_DEBUG, J403 USB4105-GF-A, U401 STM32G483RET6, Y401 ABM8W-48.0000MHZ-4-D1X-T3

Commit message: Nothing to declare
Parts:
- Y401: value ABM8W-48.0000MHZ-4-D1X-T3 -> ABM8W-48.0000MHZ-4-D1X-T3
- renumbered R1103 to R407, R1103 to R408
