File: Power/GEOX/rev2/SMPS_legged_robot_module/connector_debug.kicad_sch (KiCad schematic)
At the start: 7 parts, among them J2 98414-G06-12ULF, U1 24LC025-I/ST

Commit message: Secret
Parts:
- renumbered C1 to C601, J2 to J601, R1 to R601, R2 to R602, R3 to R603, R4 to R604, U1 to U601
Other:
- company: (none) -> ${COMPANY}
- title: (none) -> Connector - Debug
- moved on the sheet: C601, R603, R604, U601

Commit message: Nothing to declare
Other:
- moved on the sheet: C601, J601, R601, R602, R603, R604, U601
