File: Power/GEOX/rev2/SMPS_legged_robot_module/mechanical holes.kicad_sch (KiCad schematic)
At the start: 8 parts

Commit message: Secret
Parts:
- renumbered FM701 to FM1101, FM704 to FM1102, FM702 to FM1103, FM705 to FM1104, FM706 to FM1105, FM703 to FM1106, H801 to H1101, H802 to H1102
Other:
- company: (none) -> ${COMPANY}
- title: (none) -> Mechanical Holes
Changed lines of the file:
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@@
 	(generator_version "8.0")
 	(paper "A5")
+	(title_block
+		(title "Mechanical Holes")
+		(date "Last Modified Date")
+		(rev "${REVISION}")
+		(company "${COMPANY}")
+	)
 	(no_connect
 		(at 69.215 67.31)
@@
 		)
 	)
-	(text_box "[9] Mechanical Holes"
+	(text_box "[${#}] ${TITLE}"
 		(exclude_from_sim no)
 		(at 12.7 14.605 0)
@@
 		(on_board yes)
 		(dnp no)
-		(property "Reference" "FM704"
+		(property "Reference" "FM1102"
 			(at 137.16 74.93 0)
 			(effects
@@
 			(project "SMPS_legged_robot_module"
 				(path "/0650c7a8-acba-429c-9f8e-eec0baf0bc1c/fede4c36-00cc-4d3d-b71c-5243ba232202/1dbdd458-9c8a-4b0b-ac5b-dcf9040035b1"
-					(reference "FM704")
+					(reference "FM1102")
 					(unit 1)
 				)
@@
 		(dnp no)
 		(fields_autoplaced yes)
-		(property "Reference" "H801"
+		(property "Reference" "H1101"
 			(at 71.755 62.23 0)
 			(effects
@@
 			(project "SMPS_legged_robot_module"
 				(path "/0650c7a8-acba-429c-9f8e-eec0baf0bc1c/fede4c36-00cc-4d3d-b71c-5243ba232202/1dbdd458-9c8a-4b0b-ac5b-dcf9040035b1"
-					(reference "H801")
+					(reference "H1101")
 					(unit 1)
 				)
@@
 		(on_board yes)
 		(dnp no)
-		(property "Reference" "FM702"
+		(property "Reference" "FM1103"
 			(at 146.685 59.69 0)
 			(effects
@@
 			(project "SMPS_legged_robot_module"
 				(path "/0650c7a8-acba-429c-9f8e-eec0baf0bc1c/fede4c36-00cc-4d3d-b71c-5243ba232202/1dbdd458-9c8a-4b0b-ac5b-dcf9040035b1"
-					(reference "FM702")
+					(reference "FM1103")
 					(unit 1)
 				)
@@
 		(on_board yes)
 		(dnp no)
-		(property "Reference" "FM701"
+		(property "Reference" "FM1101"
 			(at 137.16 59.69 0)
 			(effects
@@
 			(project "SMPS_legged_robot_module"
 				(path "/0650c7a8-acba-429c-9f8e-eec0baf0bc1c/fede4c36-00cc-4d3d-b71c-5243ba232202/1dbdd458-9c8a-4b0b-ac5b-dcf9040035b1"
-					(reference "FM701")
+					(reference "FM1101")
 					(unit 1)
 				)
@@
 		(dnp no)
 		(fields_autoplaced yes)
-		(property "Reference" "H802"
+		(property "Reference" "H1102"
 			(at 98.425 62.23 0)
 			(effects
@@
 			(project "SMPS_legged_robot_module"
 				(path "/0650c7a8-acba-429c-9f8e-eec0baf0bc1c/fede4c36-00cc-4d3d-b71c-5243ba232202/1dbdd458-9c8a-4b0b-ac5b-dcf9040035b1"
-					(reference "H802")
+					(reference "H1102")
 					(unit 1)
 				)
@@
 		(on_board yes)
 		(dnp no)
-		(property "Reference" "FM706"
+		(property "Reference" "FM1105"
 			(at 155.575 74.93 0)
 			(effects
@@
 			(project "SMPS_legged_robot_module"
 				(path "/0650c7a8-acba-429c-9f8e-eec0baf0bc1c/fede4c36-00cc-4d3d-b71c-5243ba232202/1dbdd458-9c8a-4b0b-ac5b-dcf9040035b1"
-					(reference "FM706")
+					(reference "FM1105")
 					(unit 1)
 				)
@@
 		(on_board yes)
 		(dnp no)
-		(property "Reference" "FM703"
+		(property "Reference" "FM1106"
 			(at 156.21 59.69 0)
 			(effects
@@
 			(project "SMPS_legged_robot_module"
 				(path "/0650c7a8-acba-429c-9f8e-eec0baf0bc1c/fede4c36-00cc-4d3d-b71c-5243ba232202/1dbdd458-9c8a-4b0b-ac5b-dcf9040035b1"
-					(reference "FM703")
+					(reference "FM1106")
 					(unit 1)
 				)
@@
 		(on_board yes)
 		(dnp no)
-		(property "Reference" "FM705"
+		(property "Reference" "FM1104"
 			(at 146.685 74.93 0)
 			(effects
@@
 			(project "SMPS_legged_robot_module"
 				(path "/0650c7a8-acba-429c-9f8e-eec0baf0bc1c/fede4c36-00cc-4d3d-b71c-5243ba232202/1dbdd458-9c8a-4b0b-ac5b-dcf9040035b1"
-					(reference "FM705")
-					(unit 1)
-				)
+					(reference "FM1104")
+					(unit 1)
+				)

Commit message: Nothing to declare
Other:
- moved on the sheet: FM1101, FM1102, FM1103, FM1104, FM1105, FM1106, H1101, H1102
