File: Power/GEOX/rev2/SMPS_legged_robot_module/power_generation.kicad_sch (KiCad schematic)
At the start: 8 parts, among them U2 LMR16006YDDCR

Commit message: Secret
Parts:
- renumbered C4 to C901, C2 to C902, C3 to C903, L1 to L901, R7 to R901, R5 to R902, R6 to R903, U2 to U901
Other:
- company: (none) -> ${COMPANY}
- title: (none) -> Power - Local Generation
Changed lines of the file:
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@@
 	(generator_version "8.0")
 	(paper "A5")
+	(title_block
+		(title "Power - Local Generation")
+		(date "Last Modified Date")
+		(rev "${REVISION}")
+		(company "${COMPANY}")
+	)
 	(junction
 		(at 133.35 71.12)
@@
 		)
 	)
-	(text_box "[] Power - Local Generation"
+	(text_box "[${#}] ${TITLE}"
 		(exclude_from_sim no)
 		(at 12.446 13.97 0)
@@
 		(dnp no)
 		(fields_autoplaced yes)
-		(property "Reference" "U2"
+		(property "Reference" "U901"
 			(at 97.79 49.53 0)
 			(effects
@@
 			(project ""
 				(path "/0650c7a8-acba-429c-9f8e-eec0baf0bc1c/fede4c36-00cc-4d3d-b71c-5243ba232202/e473a05a-7df5-4923-9156-fad3374dd463"
-					(reference "U2")
+					(reference "U901")
 					(unit 1)
 				)
@@
 		(dnp no)
 		(fields_autoplaced yes)
-		(property "Reference" "R5"
+		(property "Reference" "R902"
 			(at 135.89 64.7699 0)
 			(effects
@@
 			(project ""
 				(path "/0650c7a8-acba-429c-9f8e-eec0baf0bc1c/fede4c36-00cc-4d3d-b71c-5243ba232202/e473a05a-7df5-4923-9156-fad3374dd463"
-					(reference "R5")
+					(reference "R902")
 					(unit 1)
 				)
@@
 		(dnp no)
 		(fields_autoplaced yes)
-		(property "Reference" "R6"
+		(property "Reference" "R903"
 			(at 135.89 74.9299 0)
 			(effects
@@
 			(project "SMPS_legged_robot_module"
 				(path "/0650c7a8-acba-429c-9f8e-eec0baf0bc1c/fede4c36-00cc-4d3d-b71c-5243ba232202/e473a05a-7df5-4923-9156-fad3374dd463"
-					(reference "R6")
+					(reference "R903")
 					(unit 1)
 				)
@@
 		(dnp no)
 		(fields_autoplaced yes)
-		(property "Reference" "L1"
+		(property "Reference" "L901"
 			(at 125.73 57.15 90)
 			(effects
@@
 			(project ""
 				(path "/0650c7a8-acba-429c-9f8e-eec0baf0bc1c/fede4c36-00cc-4d3d-b71c-5243ba232202/e473a05a-7df5-4923-9156-fad3374dd463"
-					(reference "L1")
+					(reference "L901")
 					(unit 1)
 				)
@@
 		(on_board yes)
 		(dnp no)
-		(fields_autoplaced yes)
-		(property "Reference" "R7"
-			(at 78.74 57.15 90)
+		(property "Reference" "R901"
+			(at 78.74 59.944 90)
 			(effects
 				(font
@@
 		)
 		(property "Value" "100k"
-			(at 78.74 59.69 90)
+			(at 78.994 64.77 90)
 			(effects
 				(font
@@
 			(project "SMPS_legged_robot_module"
 				(path "/0650c7a8-acba-429c-9f8e-eec0baf0bc1c/fede4c36-00cc-4d3d-b71c-5243ba232202/e473a05a-7df5-4923-9156-fad3374dd463"
-					(reference "R7")
+					(reference "R901")
 					(unit 1)
 				)
@@
 		(dnp no)
 		(fields_autoplaced yes)
-		(property "Reference" "#PWR08"
+		(property "Reference" "#PWR0901"
 			(at 64.77 87.63 0)
 			(effects
@@
 			(project "SMPS_legged_robot_module"
 				(path "/0650c7a8-acba-429c-9f8e-eec0baf0bc1c/fede4c36-00cc-4d3d-b71c-5243ba232202/e473a05a-7df5-4923-9156-fad3374dd463"
-					(reference "#PWR08")
+					(reference "#PWR0901")
 					(unit 1)
 				)
@@
 		(dnp no)
 		(fields_autoplaced yes)
-		(property "Reference" "C3"
+		(property "Reference" "C903"
 			(at 156.21 69.8499 0)
 			(effects
@@
 			(project ""
 				(path "/0650c7a8-acba-429c-9f8e-eec0baf0bc1c/fede4c36-00cc-4d3d-b71c-5243ba232202/e473a05a-7df5-4923-9156-fad3374dd463"
-					(reference "C3")
+					(reference "C903")
 					(unit 1)
 				)
@@
 		(on_board yes)
 		(dnp no)
-		(property "Reference" "C4"
+		(property "Reference" "C901"
 			(at 60.96 68.5799 0)
 			(effects
@@
 			(project "SMPS_legged_robot_module"
 				(path "/0650c7a8-acba-429c-9f8e-eec0baf0bc1c/fede4c36-00cc-4d3d-b71c-5243ba232202/e473a05a-7df5-4923-9156-fad3374dd463"
-					(reference "C4")
+					(reference "C901")
 					(unit 1)
 				)
@@
 		(dnp no)
 		(fields_autoplaced yes)
-		(property "Reference" "C2"
+		(property "Reference" "C902"
 			(at 114.3063 50.8 90)
 			(effects
@@
 			(project ""
 				(path "/0650c7a8-acba-429c-9f8e-eec0baf0bc1c/fede4c36-00cc-4d3d-b71c-5243ba232202/e473a05a-7df5-4923-9156-fad3374dd463"
-					(reference "C2")
+					(reference "C902")
 					(unit 1)
 				)

Commit message: Nothing to declare
Other:
- moved on the sheet: C901, C902, C903, L901, R901, R902, R903, U901
